Commit message: Simulator update:
warning: starting from this update, simulator is compatible only with xacro for ROS Jade and newer. Support for Ubuntu 14.04 and ROS Indigo

 - update inertia parameters for the upper-body
 - update collision and visualization models
 - add choice of the end-effector through parameter
 - start joint_state publisher for gazebo from the main launch file
 - launch robot_state_publisher from a main launch file
 - remove pelvis link (and therefore inertia parameters) for pelvis when only upper-body elements are generated
 -

File: centauro/centauro_urdf/parameters.xacro (robot description, xacro)
@@ -19,5 +19,5 @@
 <xacro:property name="Pelvis_zz" value=" 1.369479 "/>
 <xacro:property name="Pelvis_xy" value=" 0.000000 "/>
-<xacro:property name="Pelvis_xz" value=" -0.233584 "/>
+<xacro:property name="Pelvis_xz" value=" 0.000000 "/>
 <xacro:property name="Pelvis_yz" value=" 0.000000 "/>
 <!-- Mass -->
@@ -63,107 +63,107 @@
 <xacro:property name="Leg_3_mass" value=" 3.500000 "/>
 <!-- Center of Mass -->
-<xacro:property name="Torso_2_x" value=" 0.000000 "/>
-<xacro:property name="Torso_2_y" value=" 0.000000 "/>
-<xacro:property name="Torso_2_z" value=" 0.183333 "/>
+<xacro:property name="Torso_2_x" value=" 0.0047281261 "/>
+<xacro:property name="Torso_2_y" value=" 0.00038307386 "/>
+<xacro:property name="Torso_2_z" value=" 0.14972892 "/>
 <!-- Inertia -->
-<xacro:property name="Torso_2_xx" value=" 0.094335 "/>
-<xacro:property name="Torso_2_yy" value=" 0.029946 "/>
-<xacro:property name="Torso_2_zz" value=" 0.068486 "/>
-<xacro:property name="Torso_2_xy" value=" 0.000085 "/>
-<xacro:property name="Torso_2_xz" value=" -0.000031 "/>
-<xacro:property name="Torso_2_yz" value=" 0.000017 "/>
+<xacro:property name="Torso_2_xx" value=" 0.063643392 "/>
+<xacro:property name="Torso_2_yy" value=" 0.02680235 "/>
+<xacro:property name="Torso_2_zz" value=" 0.04743015 "/>
+<xacro:property name="Torso_2_xy" value=" 0.00008939 "/>
+<xacro:property name="Torso_2_xz" value=" -0.00086873 "/>
+<xacro:property name="Torso_2_yz" value=" -0.00004657 "/>
 <!-- Mass -->
-<xacro:property name="Torso_2_mass" value=" 3.000000 "/>
+<xacro:property name="Torso_2_mass" value=" 4.5494226000 "/>
 <!-- Center of Mass -->
-<xacro:property name="Shoulder_1_x" value=" 0.000000 "/>
-<xacro:property name="Shoulder_1_y" value=" 0.064706 "/>
-<xacro:property name="Shoulder_1_z" value=" 0.000000 "/>
+<xacro:property name="Shoulder_1_x" value=" -0.0031005886 "/>
+<xacro:property name="Shoulder_1_y" value=" -0.0403245840 "/>
+<xacro:property name="Shoulder_1_z" value=" 0.0074519370 "/>
 <!-- Inertia -->
-<xacro:property name="Shoulder_1_xx" value=" 0.002332 "/>
-<xacro:property name="Shoulder_1_yy" value=" 0.001345 "/>
-<xacro:property name="Shoulder_1_zz" value=" 0.002332 "/>
-<xacro:property name="Shoulder_1_xy" value=" 0.000000 "/>
-<xacro:property name="Shoulder_1_xz" value=" 0.000000 "/>
-<xacro:property name="Shoulder_1_yz" value=" -0.000000 "/>
+<xacro:property name="Shoulder_1_xx" value=" 0.0032318636"/>
+<xacro:property name="Shoulder_1_yy" value=" 0.0027571800 "/>
+<xacro:property name="Shoulder_1_zz" value=" 0.0042750470 "/>
+<xacro:property name="Shoulder_1_xy" value=" -0.0000424587 "/>
+<xacro:property name="Shoulder_1_xz" value=" 0.0000491626 "/>
+<xacro:property name="Shoulder_1_yz" value=" 0.0002387056 "/>
 <!-- Mass -->
-<xacro:property name="Shoulder_1_mass" value=" 1.700000 "/>
+<xacro:property name="Shoulder_1_mass" value=" 1.5583338000 "/>
 <!-- Center of Mass -->
-<xacro:property name="Shoulder_2_x" value=" 0.000000 "/>
-<xacro:property name="Shoulder_2_y" value=" 0.000000 "/>
-<xacro:property name="Shoulder_2_z" value=" -0.125000 "/>
+<xacro:property name="Shoulder_2_x" value=" 0.05105435 "/>
+<xacro:property name="Shoulder_2_y" value=" -0.00011109 "/>
+<xacro:property name="Shoulder_2_z" value=" -0.07643596 "/>
 <!-- Inertia -->
-<xacro:property name="Shoulder_2_xx" value=" 0.005879 "/>
-<xacro:property name="Shoulder_2_yy" value=" 0.005879 "/>
-<xacro:property name="Shoulder_2_zz" value=" 0.001525 "/>
-<xacro:property name="Shoulder_2_xy" value=" 0.000000 "/>
-<xacro:property name="Shoulder_2_xz" value=" 0.000000 "/>
-<xacro:property name="Shoulder_2_yz" value=" 0.000000 "/>
+<xacro:property name="Shoulder_2_xx" value=" 0.01029558 "/>
+<xacro:property name="Shoulder_2_yy" value=" 0.01178018 "/>
+<xacro:property name="Shoulder_2_zz" value=" 0.00386123 "/>
+<xacro:property name="Shoulder_2_xy" value=" -0.00002846 "/>
+<xacro:property name="Shoulder_2_xz" value=" 0.00365670 "/>
+<xacro:property name="Shoulder_2_yz" value=" -0.00002088 "/>
 <!-- Mass -->
-<xacro:property name="Shoulder_2_mass" value=" 2.000000 "/>
+<xacro:property name="Shoulder_2_mass" value=" 1.5150610 "/>
 <!-- Center of Mass -->
-<xacro:property name="Shoulder_3_x" value=" 0.000000 "/>
-<xacro:property name="Shoulder_3_y" value=" 0.000000 "/>
-<xacro:property name="Shoulder_3_z" value=" -0.093750 "/>
+<xacro:property name="Shoulder_3_x" value=" 0.01207624 "/>
+<xacro:property name="Shoulder_3_y" value=" -0.00322013 "/>
+<xacro:property name="Shoulder_3_z" value=" -0.03427312 "/>
 <!-- Inertia -->
-<xacro:property name="Shoulder_3_xx" value=" 0.003989 "/>
-<xacro:property name="Shoulder_3_yy" value=" 0.003884 "/>
-<xacro:property name="Shoulder_3_zz" value=" 0.001629 "/>
-<xacro:property name="Shoulder_3_xy" value=" 0.000000 "/>
-<xacro:property name="Shoulder_3_xz" value=" 0.000000 "/>
-<xacro:property name="Shoulder_3_yz" value=" -0.000000 "/>
+<xacro:property name="Shoulder_3_xx" value=" 0.00469819 "/>
+<xacro:property name="Shoulder_3_yy" value=" 0.00501755 "/>
+<xacro:property name="Shoulder_3_zz" value=" 0.00310954 "/>
+<xacro:property name="Shoulder_3_xy" value=" 0.00026547 "/>
+<xacro:property name="Shoulder_3_xz" value=" 0.00077706 "/>
+<xacro:property name="Shoulder_3_yz" value=" -0.00029679 "/>
 <!-- Mass -->
-<xacro:property name="Shoulder_3_mass" value=" 2.000000 "/>
+<xacro:property name="Shoulder_3_mass" value=" 1.5088101 "/>
 <!-- Center of Mass -->
-<xacro:property name="Elbow_1_x" value=" 0.000000 "/>
-<xacro:property name="Elbow_1_y" value=" 0.000000 "/>
-<xacro:property name="Elbow_1_z" value=" -0.090000 "/>
+<xacro:property name="Elbow_1_x" value=" 0.0101475520 "/>
+<xacro:property name="Elbow_1_y" value=" 0.0299285370 "/>
+<xacro:property name="Elbow_1_z" value=" -0.032528288  "/>
 <!-- Inertia -->
-<xacro:property name="Elbow_1_xx" value=" 0.002589 "/>
-<xacro:property name="Elbow_1_yy" value=" 0.002589 "/>
-<xacro:property name="Elbow_1_zz" value=" 0.001105 "/>
-<xacro:property name="Elbow_1_xy" value=" 0.000000 "/>
-<xacro:property name="Elbow_1_xz" value=" 0.000000 "/>
-<xacro:property name="Elbow_1_yz" value=" 0.000000 "/>
+<xacro:property name="Elbow_1_xx" value=" 0.0026493567 "/>
+<xacro:property name="Elbow_1_yy" value=" 0.0023470955 "/>
+<xacro:property name="Elbow_1_zz" value=" 0.0012213063 "/>
+<xacro:property name="Elbow_1_xy" value=" -0.0000051632 "/>
+<xacro:property name="Elbow_1_xz" value=" 0.0001292309 "/>
+<xacro:property name="Elbow_1_yz" value=" 0.0007895755 "/>
 <!-- Mass -->
-<xacro:property name="Elbow_1_mass" value=" 1.300000 "/>
+<xacro:property name="Elbow_1_mass" value=" 0.9629732900 "/>
 <!-- Center of Mass -->
-<xacro:property name="Elbow_2_x" value=" 0.000000 "/>
-<xacro:property name="Elbow_2_y" value=" 0.000000 "/>
-<xacro:property name="Elbow_2_z" value=" -0.067857 "/>
+<xacro:property name="Wrist_1_x" value=" -0.0001574443 "/>
+<xacro:property name="Wrist_1_y" value=" -0.0041320907 "/>
+<xacro:property name="Wrist_1_z" value=" -0.1075661400 "/>
 <!-- Inertia -->
-<xacro:property name="Elbow_2_xx" value=" 0.002073 "/>
-<xacro:property name="Elbow_2_yy" value=" 0.001969 "/>
-<xacro:property name="Elbow_2_zz" value=" 0.001269 "/>
-<xacro:property name="Elbow_2_xy" value=" 0.000000 "/>
-<xacro:property name="Elbow_2_xz" value=" 0.000000 "/>
-<xacro:property name="Elbow_2_yz" value=" -0.000000 "/>
+<xacro:property name="Wrist_1_xx" value=" 0.0064160453 "/>
+<xacro:property name="Wrist_1_yy" value=" 0.0062016367 "/>
+<xacro:property name="Wrist_1_zz" value=" 0.0017091658 "/>
+<xacro:property name="Wrist_1_xy" value=" -0.0000196382 "/>
+<xacro:property name="Wrist_1_xz" value=" 0.0000249912 "/>
+<xacro:property name="Wrist_1_yz" value=" 0.0001987903 "/>
 <!-- Mass -->
-<xacro:property name="Elbow_2_mass" value=" 1.400000 "/>
+<xacro:property name="Wrist_1_mass" value=" 1.4703698000 "/>
 <!-- Center of Mass -->
-<xacro:property name="Wrist_1_x" value=" 0.000000 "/>
-<xacro:property name="Wrist_1_y" value=" 0.000000 "/>
-<xacro:property name="Wrist_1_z" value=" -0.094545 "/>
+<xacro:property name="Wrist_2_x" value=" 0.0000323645 "/>
+<xacro:property name="Wrist_2_y" value=" 0.0359472370 "/>
+<xacro:property name="Wrist_2_z" value=" -0.0808780610 "/>
 <!-- Inertia -->
-<xacro:property name="Wrist_1_xx" value=" 0.002301 "/>
-<xacro:property name="Wrist_1_yy" value=" 0.002301 "/>
-<xacro:property name="Wrist_1_zz" value=" 0.000985 "/>
-<xacro:property name="Wrist_1_xy" value=" 0.000000 "/>
-<xacro:property name="Wrist_1_xz" value=" 0.000000 "/>
-<xacro:property name="Wrist_1_yz" value=" 0.000000 "/>
+<xacro:property name="Wrist_2_xx" value=" 0.0036896582 "/>
+<xacro:property name="Wrist_2_yy" value=" 0.0034146283 "/>
+<xacro:property name="Wrist_2_zz" value=" 0.0010790183 "/>
+<xacro:property name="Wrist_2_xy" value=" -0.0000263667 "/>
+<xacro:property name="Wrist_2_xz" value=" 0.0000014005 "/>
+<xacro:property name="Wrist_2_yz" value=" 0.0008268103 "/>
 <!-- Mass -->
-<xacro:property name="Wrist_1_mass" value=" 1.100000 "/>
+<xacro:property name="Wrist_2_mass" value=" 0.9469386800 "/>
 <!-- Center of Mass -->
-<xacro:property name="Hand_x" value=" 0.000000 "/>
-<xacro:property name="Hand_y" value=" 0.000000 "/>
-<xacro:property name="Hand_z" value=" -0.075000 "/>
+<xacro:property name="Wrist_3_x" value=" 0.0000246596 "/>
+<xacro:property name="Wrist_3_y" value=" 0.0001467705 "/>
+<xacro:property name="Wrist_3_z" value=" -0.0052993013 "/>
 <!-- Inertia -->
-<xacro:property name="Hand_xx" value=" 0.001303 "/>
-<xacro:property name="Hand_yy" value=" 0.001303 "/>
-<xacro:property name="Hand_zz" value=" 0.001020 "/>
-<xacro:property name="Hand_xy" value=" 0.000000 "/>
-<xacro:property name="Hand_xz" value=" 0.000000 "/>
-<xacro:property name="Hand_yz" value=" 0.000000 "/>
+<xacro:property name="Wrist_3_xx" value=" 0.0004360175 "/>
+<xacro:property name="Wrist_3_yy" value=" 0.0004299166 "/>
+<xacro:property name="Wrist_3_zz" value=" 0.0004522224 "/>
+<xacro:property name="Wrist_3_xy" value=" -0.0000001397 "/>
+<xacro:property name="Wrist_3_xz" value=" -0.0000001382 "/>
+<xacro:property name="Wrist_3_yz" value=" 0.0000014752 "/>
 <!-- Mass -->
-<xacro:property name="Hand_mass" value=" 1.700000 "/>
+<xacro:property name="Wrist_3_mass" value=" 0.5598103600 "/>
 <!-- Center of Mass -->
 <xacro:property name="Wheel_x" value=" 0.000000 "/>
@@ -172,5 +172,5 @@
 <!-- Inertia -->
 <xacro:property name="Wheel_xx" value=" 0.005417 "/>
-<xacro:property name="Wheel_yy" value=" 0.010000 "/>
+<xacro:property name="Wheel_yy" value=" 0.01000 "/>
 <xacro:property name="Wheel_zz" value=" 0.005417 "/>
 <xacro:property name="Wheel_xy" value=" 0.000000 "/>

File: centauro/centauro_urdf/urdf/centauro.urdf.xacro (robot description, xacro)
@@ -1,14 +1,4 @@
 <?xml version="1.0"?>
 <robot xmlns:xacro="http://www.ros.org/wiki/xacro" name="centauro">
-<!-- config --> <!--
-<xacro:property name="ARMS" value="true"/>
-<xacro:property name="TORSO" value="true" />
-<xacro:property name="ARM_ACTUATORS" value="true"/>
-<xacro:property name="LEGS" value="true"/>
-<xacro:property name="LEG_ACTUATORS" value="true"/>
-<xacro:property name="TORSO_ACTUATORS" value="true"/>
-<xacro:property name="WHEELS" value="true"/>
-<xacro:property name="WHEELS_ACTUATORS" value="true"/>-->
-<!-- /config -->
 <!-- constants -->
 <xacro:property name="PI" value="3.14159265359"/>
@@ -16,90 +6,66 @@
 <!-- /constants -->
 <!-- other files -->
-<xacro:include filename="$(find centauro_gazebo)/urdf/centauro.gazebo"/>
+<xacro:include filename="$(find centauro)/centauro_urdf/urdf/config.xacro"/>
+ <xacro:if value="${GAZEBO}">
+  <xacro:include filename="$(find centauro_gazebo)/urdf/centauro.gazebo"/>
+</xacro:if>
 <xacro:include filename="$(find centauro)/centauro_urdf/parameters.xacro"/>
 <xacro:include filename="$(find centauro)/centauro_urdf/materials.xacro"/>
-<xacro:include filename="$(find centauro)/centauro_urdf/urdf/models/models.xacro"/>
-<xacro:if	value="$(arg LEGS)">
+<xacro:include filename="$(find centauro)/centauro_urdf/urdf/models/model.xacro"/>
+<xacro:include filename="$(find centauro)/centauro_urdf/urdf/centauro_actuators.urdf.xacro" />
+<xacro:if value="${LEGS}">
   <xacro:include filename="$(find centauro)/centauro_urdf/urdf/centauro_leg.urdf.xacro"/>
 </xacro:if>
-<xacro:if	value="$(arg ARMS)">
+<xacro:if value="${arm}">
   <xacro:include filename="$(find centauro)/centauro_urdf/urdf/centauro_arm.urdf.xacro"/>
-</xacro:if>
-<xacro:if	value="$(arg ARM_SENSORS)">
-  <xacro:include filename="$(find centauro)/centauro_urdf/urdf/sensors/force_torque_plugin.urdf.xacro"/>
 </xacro:if>
 <!-- /other files -->
 <!-- reference -->
 <link name="world"/>
-<xacro:unless	value="$(arg ONE_ARM)">
-<link name="pelvis">
-	<inertial>
-		<origin xyz="${Pelvis_x} ${Pelvis_y} ${Pelvis_z}"/>	<!-- TODO -->
-		<mass value="${Pelvis_mass}"/> <!-- org: 25 -->
-		<inertia ixx="${Pelvis_xx}" ixy="${Pelvis_xy}" ixz="${Pelvis_xz}" iyy="${Pelvis_yy}" iyz="${Pelvis_yz}" izz="${Pelvis_zz}"/>  <!-- TODO -->
-	</inertial>
-<xacro:if value="$(arg LEGS)">
+<xacro:if value="${pelvis}">
+   <link name="pelvis">
+      <inertial>
+         <origin xyz="${Pelvis_x} ${Pelvis_y} ${Pelvis_z}"/>
+         <mass value="${Pelvis_mass}"/>
+         <inertia ixx="${Pelvis_xx}" ixy="${Pelvis_xy}" ixz="${Pelvis_xz}" iyy="${Pelvis_yy}" iyz="${Pelvis_yz}" izz="${Pelvis_zz}"/>
+      </inertial>
       <visual>
-         <xacro:insert_block name="v_pelvis" />
+         <xacro:visual_model.pelvis />
          <material name="grey"/>
       </visual>
       <collision>
-         <xacro:insert_block name="c_pelvis" />
+         <xacro:collision_model.pelvis />
          <material name="grey"/>
       </collision>
+   </link>
+   <joint name="reference" type="${reference}">
+      <origin xyz="0 0 0.85"/>
+      <parent link="world"/>
+      <child link="pelvis"/>
+   </joint>
 </xacro:if>
-</link>
 <!-- /reference  -->
-<xacro:unless	value="$(arg ONE_ARM)">
-<xacro:if	value="$(arg STATIC)">
-	<joint name="reference" type="fixed">
-		<origin xyz="0 0 0.85"/>
-		<parent link="world"/>
-		<child link="pelvis"/>
-	</joint>
+<!-- torso -->
+<xacro:if value="${torso}">
+   <xacro:include filename="$(find centauro)/centauro_urdf/urdf/centauro_torso.urdf.xacro"/>
 </xacro:if>
-<xacro:unless value="$(arg STATIC)">
-	<xacro:unless	value="$(arg LEGS)">
-		<joint name="reference" type="fixed">
-			<origin xyz="0 0 0.85"/>
-			<parent link="world"/>
-			<child link="pelvis"/>
-		</joint>
-	</xacro:unless>
-	<xacro:if	value="$(arg LEGS)">
-		<xacro:unless	value="$(arg LEG_ACTUATORS)">
-			<joint name="reference" type="fixed">
-				<origin xyz="0 0 0.85"/>
-				<parent link="world"/>
-				<child link="pelvis"/>
-			</joint>
-		</xacro:unless>
-		<xacro:if	value="$(arg LEG_ACTUATORS)">
-			<joint name="reference" type="floating">
-				<origin xyz="0 0 0.85"/>
-				<parent link="world"/>
-				<child link="pelvis"/>
-			</joint>
-		</xacro:if>
-	</xacro:if>
-</xacro:unless>
-</xacro:unless>
-<!-- torso -->
-<xacro:if	value="$(arg TORSO)">
-<xacro:include filename="$(find centauro)/centauro_urdf/urdf/centauro_torso.urdf.xacro"/>
+<!-- /torso -->
 <!-- arms -->
-<xacro:if	value="$(arg ARMS)">
-<xacro:centauro_arm arm_num="1"  rot="1">
-	<origin xyz="0.04576 0.169137 0.190626" rpy="0.0 0 -0.5236026689864071" />
-</xacro:centauro_arm>
-<xacro:centauro_arm arm_num="2" rot="-1">
-	<origin xyz="0.0457475 -0.169137 0.190626" rpy="0.0 0 0.5236026689864071" />
-</xacro:centauro_arm>
+<xacro:if value="${arms == 'true'}">
+   <xacro:centauro_arm arm_num="1"  rot="1"  parent="torso_2">
+      <origin xyz="0.04576 0.169137 0.190626" rpy="0.0 0 -0.5236026689864071"/>
+   </xacro:centauro_arm>
+   <xacro:centauro_arm arm_num="2" rot="-1"  parent="torso_2">
+      <origin xyz="0.0457475 -0.169137 0.190626" rpy="0.0 0 0.5236026689864071" />
+   </xacro:centauro_arm>
+</xacro:if>
+<xacro:if value="${arm == 'true' and arms == 'false'}">
+        <xacro:centauro_arm arm_num="1"  rot="1" parent="world">
+           <origin xyz="${0.04576 + 0.3} ${0.169137} ${1.1+0.190626}" rpy="0.0 0 -0.5236026689864071"/>
+        </xacro:centauro_arm>
 </xacro:if>
 <!-- /arms -->
-</xacro:if>
-<!-- /torso -->
 <!-- legs -->
-<xacro:if	value="$(arg LEGS)">
+<xacro:if value="${legs}">
 <xacro:centauro_leg leg_num="1" origin_x="1" origin_y="1">
 </xacro:centauro_leg>
@@ -111,16 +77,4 @@
 </xacro:centauro_leg>
 </xacro:if>
-</xacro:unless>
-<xacro:if	value="$(arg ONE_ARM)">
-	<joint name="reference" type="fixed">
-		<origin xyz="0.3 0 1.1"/>
-		<parent link="world"/>
-		<child link="torso_2"/>
-	</joint>
-	<xacro:include filename="$(find centauro)/centauro_urdf/urdf/centauro_torso.urdf.xacro"/>
-<xacro:centauro_arm arm_num="1"  rot="1">
-	<origin xyz="0.04576 0.169137 0.190626" rpy="0.0 0 -0.5236026689864071" />
-</xacro:centauro_arm>
-</xacro:if>
 <!-- /legs -->
 </robot>
