Commit message: Simulator update:
warning: starting from this update, simulator is compatible only with xacro for ROS Jade and newer. Support for Ubuntu 14.04 and ROS Indigo

 - update inertia parameters for the upper-body
 - update collision and visualization models
 - add choice of the end-effector through parameter
 - start joint_state publisher for gazebo from the main launch file
 - launch robot_state_publisher from a main launch file
 - remove pelvis link (and therefore inertia parameters) for pelvis when only upper-body elements are generated
 -

File: centauro/centauro_urdf/urdf/centauro_arm.urdf.xacro (robot description, xacro)
@@ -1,22 +1,21 @@
 <robot xmlns:xacro="http://www.ros.org/wiki/xacro">
-<xacro:include filename="$(find centauro)/centauro_urdf/urdf/centauro_actuators.urdf.xacro" />
 <xacro:property name="cos_m10" value="0.984807753012208"/>
 <xacro:property name="sin_m10" value="-0.17364817766693033"/>
 <!-- macro arms -->
-<xacro:macro name="centauro_arm" params="arm_num rot *origin">
+<xacro:macro name="centauro_arm" params="arm_num rot parent *origin">
 <!-- LINKS -->
 <!-- shoulder yaw-roll-->
    <link name="arm${arm_num}_1">
       <inertial>
-         <origin xyz="${Shoulder_1_x} ${rot*Shoulder_1_y} ${Shoulder_1_z}"/>
-         <mass value="${Shoulder_1_mass}"/> <!-- OK: 1.7 -->
-         <inertia ixx="${Shoulder_1_xx}" ixy="${Shoulder_1_xy}" ixz="${Shoulder_1_xz}" iyy="${Shoulder_1_yy}" iyz="${Shoulder_1_yz}" izz="${Shoulder_1_zz}"/>
-      </inertial>
-      <visual>
-         <xacro:insert_block name="v_arm1" />
-         <material name="blue"/>
-      </visual>
-      <collision>
-         <xacro:insert_block name="c_arm1" />
+         <origin xyz="${Shoulder_1_x} ${-rot*Shoulder_1_y} ${Shoulder_1_z}"/>
+         <mass value="${Shoulder_1_mass}"/>
+         <inertia ixx="${Shoulder_1_xx}" ixy="${-rot*Shoulder_1_xy}" ixz="${Shoulder_1_xz}" iyy="${Shoulder_1_yy}" iyz="${-rot*Shoulder_1_yz}" izz="${Shoulder_1_zz}"/>
+      </inertial>
+      <visual>
+         <xacro:visual_model.arm1 />
+         <material name="blue"/>
+      </visual>
+      <collision>
+         <xacro:collision_model.arm1 />
          <material name="blue"/>
       </collision>
@@ -26,14 +25,14 @@
    <link name="arm${arm_num}_2">
       <inertial>
-         <origin xyz="${Shoulder_2_x} ${rot*Shoulder_2_y} ${Shoulder_2_z}"/>
-         <mass value="${Shoulder_2_mass}"/> <!-- OK: 2 -->
-         <inertia ixx="${Shoulder_2_xx}" ixy="${Shoulder_2_xy}" ixz="${Shoulder_2_xz}" iyy="${Shoulder_2_yy}" iyz="${Shoulder_2_yz}" izz="${Shoulder_2_zz}"/>
-      </inertial>
-      <visual>
-         <xacro:insert_block name="v_arm2" />
-         <material name="grey"/>
-      </visual>
-      <collision>
-         <xacro:insert_block name="c_arm2" />
+         <origin xyz="${Shoulder_2_x} ${-rot*Shoulder_2_y} ${Shoulder_2_z}"/>
+         <mass value="${Shoulder_2_mass}"/>
+         <inertia ixx="${Shoulder_2_xx}" ixy="${-rot*Shoulder_2_xy}" ixz="${Shoulder_2_xz}" iyy="${Shoulder_2_yy}" iyz="${-rot*Shoulder_2_yz}" izz="${Shoulder_2_zz}"/>
+      </inertial>
+      <visual>
+         <xacro:visual_model.arm2 />
+         <material name="grey"/>
+      </visual>
+      <collision>
+         <xacro:collision_model.arm2 />
          <material name="grey"/>
       </collision>
@@ -43,14 +42,14 @@
    <link name="arm${arm_num}_3">
       <inertial>
-         <origin xyz="${Shoulder_3_x} ${rot*Shoulder_3_y} ${Shoulder_3_z}"/>
-         <mass value="${Shoulder_3_mass}"/> <!-- OK: 2 -->
-         <inertia ixx="${Shoulder_3_xx}" ixy="${Shoulder_3_xy}" ixz="${Shoulder_3_xz}" iyy="${Shoulder_3_yy}" iyz="${Shoulder_3_yz}" izz="${Shoulder_3_zz}"/> <!-- TODO -->
-      </inertial>
-      <visual>
-         <xacro:insert_block name="v_arm3" />
-         <material name="blue"/>
-      </visual>
-      <collision>
-         <xacro:insert_block name="c_arm3" />
+         <origin xyz="${Shoulder_3_x} ${-rot*Shoulder_3_y} ${Shoulder_3_z}"/>
+         <mass value="${Shoulder_3_mass}"/>
+         <inertia ixx="${Shoulder_3_xx}" ixy="${-rot*Shoulder_3_xy}" ixz="${Shoulder_3_xz}" iyy="${Shoulder_3_yy}" iyz="${-rot*Shoulder_3_yz}" izz="${Shoulder_3_zz}"/>
+</inertial>
+      <visual>
+         <xacro:visual_model.arm3 />
+         <material name="blue"/>
+      </visual>
+      <collision>
+         <xacro:collision_model.arm3 />
          <material name="blue"/>
       </collision>
@@ -60,14 +59,14 @@
    <link name="arm${arm_num}_4">
       <inertial>
-         <origin xyz="${Elbow_1_x} ${rot*Elbow_1_y} ${Elbow_1_z}"/>
-         <mass value="${Elbow_1_mass}"/> <!-- OK: 1.3 -->
-         <inertia ixx="${Elbow_1_xx}" ixy="${Elbow_1_xy}" ixz="${Elbow_1_xz}" iyy="${Elbow_1_yy}" iyz="${Elbow_1_yz}" izz="${Elbow_1_zz}"/>
-      </inertial>
-      <visual>
-         <xacro:insert_block name="v_arm4" />
-         <material name="grey"/>
-      </visual>
-      <collision>
-         <xacro:insert_block name="c_arm4" />
+         <origin xyz="${Elbow_1_x} ${-rot*Elbow_1_y} ${Elbow_1_z}"/>
+         <mass value="${Elbow_1_mass}"/>
+         <inertia ixx="${Elbow_1_xx}" ixy="${-rot*Elbow_1_xy}" ixz="${Elbow_1_xz}" iyy="${Elbow_1_yy}" iyz="${-rot*Elbow_1_yz}" izz="${Elbow_1_zz}"/>
+</inertial>
+      <visual>
+         <xacro:visual_model.arm4 />
+         <material name="grey"/>
+      </visual>
+      <collision>
+         <xacro:collision_model.arm4 />
          <material name="grey"/>
       </collision>
@@ -77,14 +76,14 @@
    <link name="arm${arm_num}_5">
       <inertial>
-         <origin xyz="${Elbow_2_x} ${Elbow_2_y} ${Elbow_2_z}"/>
-         <mass value="${Elbow_2_mass}"/> <!-- OK: 1.4 -->
-         <inertia ixx="${Elbow_2_xx}" ixy="${Elbow_2_xy}" ixz="${Elbow_2_xz}" iyy="${Elbow_2_yy}" iyz="${Elbow_2_yz}" izz="${Elbow_2_zz}"/>
-      </inertial>
-      <visual>
-         <xacro:insert_block name="v_arm5" />
-         <material name="blue"/>
-      </visual>
-      <collision>
-         <xacro:insert_block name="c_arm5" />
+         <origin xyz="${Wrist_1_x} ${-rot*Wrist_1_y} ${Wrist_1_z}"/>
+         <mass value="${Wrist_1_mass}"/>
+         <inertia ixx="${Wrist_1_xx}" ixy="${-rot*Wrist_1_xy}" ixz="${Wrist_1_xz}" iyy="${Wrist_1_yy}" iyz="${-rot*Wrist_1_yz}" izz="${Wrist_1_zz}"/>
+</inertial>
+      <visual>
+         <xacro:visual_model.arm5 />
+         <material name="blue"/>
+      </visual>
+      <collision>
+         <xacro:collision_model.arm5 />
          <material name="blue"/>
       </collision>
@@ -94,40 +93,38 @@
    <link name="arm${arm_num}_6">
       <inertial>
-         <origin xyz="${Wrist_1_x} ${Wrist_1_y} ${Wrist_1_z}"/>
-         <mass value="${Wrist_1_mass}"/> <!-- OK: 1.1 -->
-         <inertia ixx="${Wrist_1_xx}" ixy="${Wrist_1_xy}" ixz="${Wrist_1_xz}" iyy="${Wrist_1_yy}" iyz="${Wrist_1_yz}" izz="${Wrist_1_zz}"/>
-      </inertial>
-      <visual>
-         <xacro:insert_block name="v_arm6" />
-         <material name="grey"/>
-      </visual>
-      <collision>
-         <xacro:insert_block name="c_arm6" />
+         <origin xyz="${Wrist_2_x} ${-rot*Wrist_2_y} ${Wrist_2_z}"/>
+         <mass value="${Wrist_2_mass}"/>
+         <inertia ixx="${Wrist_2_xx}" ixy="${-rot*Wrist_2_xy}" ixz="${Wrist_2_xz}" iyy="${Wrist_2_yy}" iyz="${-rot*Wrist_2_yz}" izz="${Wrist_2_zz}"/>
+</inertial>
+      <visual>
+         <xacro:visual_model.arm6 />
+         <material name="grey"/>
+      </visual>
+      <collision>
+         <xacro:collision_model.arm6 />
          <material name="grey"/>
       </collision>
    </link>
 <!-- /wrist yaw-pitch -->
-<!-- hand -->
-   <xacro:unless value="$(arg HANDS)">
-      <link name="arm${arm_num}_7">
-         <inertial>
-            <origin xyz="${Hand_x} ${Hand_y} ${Hand_z}"/>
-            <mass value="${Hand_mass}"/> <!-- OK: 1.7 -->
-            <inertia ixx="${Hand_xx}" ixy="${Hand_xy}" ixz="${Hand_xz}" iyy="${Hand_yy}" iyz="${Hand_yz}" izz="${Hand_zz}"/>
-         </inertial>
-         <visual>
-            <xacro:insert_block name="v_arm7" />
-            <material name="blue"/>
-         </visual>
-         <collision>
-            <xacro:insert_block name="c_arm7" />
-            <material name="blue"/>
-         </collision>
-      </link>
-   </xacro:unless>
+   <link name="arm${arm_num}_7">
+      <inertial>
+         <origin xyz="${Wrist_3_x} ${-rot*Wrist_3_y} ${Wrist_3_z}"/>
+         <mass value="${Wrist_3_mass}"/>
+         <inertia ixx="${Wrist_3_xx}" ixy="${-rot*Wrist_3_xy}" ixz="${Wrist_3_xz}" iyy="${Wrist_3_yy}" iyz="${-rot*Wrist_3_yz}" izz="${Wrist_3_zz}"/>
+      </inertial>
+      <visual>
+         <xacro:visual_model.arm7 />
+         <material name="blue"/>
+      </visual>
+      <collision>
+         <xacro:collision_model.arm7 />
+         <material name="blue"/>
+      </collision>
+   </link>
+<!-- mass -->
 <!--   <link name="mass${arm_num}_body">
       <inertial>
          <origin xyz="0 0 0"/> -->
-<!--         <mass value="10"/> --><!-- OK: 1.7 -->
+<!--         <mass value="10"/> -->
 <!--         <inertia ixx="0.001" ixy="0.00" ixz="0.00" iyy="0.001" iyz="0.00" izz="0.001"/>
       </inertial>
@@ -140,18 +137,18 @@
       </visual>
    </link> -->
-<!-- /hand -->
+<!-- /mass -->
 <!-- /LINKS -->
 <!-- JOINTS -->
 <!-- shoulder yaw -->
    <joint name="j_arm${arm_num}_1" type="revolute">
-      <parent link="torso_2"/>
+      <parent link="${parent}"/>
       <child link="arm${arm_num}_1"/>
       <xacro:insert_block name="origin"/>
       <axis xyz="0 ${rot*cos_m10} ${-sin_m10}"/>
       <xacro:unless value="${rot-1}" >
-         <limit lower="-3.403" upper="1.658" effort="350" velocity="6.5"/>
+         <limit lower="-3.403" upper="1.658" effort="1770" velocity="6.5"/>
       </xacro:unless>
       <xacro:unless value="${rot+1}" >
-         <limit lower="-1.658" upper="3.403" effort="350" velocity="6.5"/>
+         <limit lower="-1.658" upper="3.403" effort="1770" velocity="6.5"/>
       </xacro:unless>
    </joint>
@@ -164,8 +161,8 @@
       <axis xyz="-1 0 0"/>
       <xacro:unless value="${rot+1}" >
-         <limit lower="0" upper="3.49" effort="350" velocity="6.5"/> <!-- TODO -->
+         <limit lower="0" upper="3.49" effort="1770" velocity="6.5"/>
       </xacro:unless>
       <xacro:unless value="${rot-1}" >
-         <limit lower="-3.49" upper="0" effort="350" velocity="6.5"/> <!-- TODO -->
+         <limit lower="-3.49" upper="0" effort="1770" velocity="6.5"/>
       </xacro:unless>
    </joint>
@@ -177,5 +174,5 @@
       <origin xyz="0.09115 0 -0.21915"/>
       <axis xyz="0 0 -1"/>
-      <limit lower="-2.618" upper="2.618" effort="350" velocity="6.5"/> <!-- TODO -->
+      <limit lower="-2.618" upper="2.618" effort="1770" velocity="6.5"/>
    </joint>
 <!-- /shoulder pitch -->
@@ -187,8 +184,8 @@
       <axis xyz="0 ${rot} 0"/>
       <xacro:unless value="${rot-1}" >
-         <limit lower="-2.530" upper="0.349" effort="350" velocity="6.5"/> <!-- TODO -->
+         <limit lower="-2.530" upper="0.349" effort="1770" velocity="6.5"/>
       </xacro:unless>
       <xacro:unless value="${rot+1}" >
-         <limit lower="-0.349" upper="2.530" effort="350" velocity="6.5"/> <!-- TODO -->
+         <limit lower="-0.349" upper="2.530" effort="1770" velocity="6.5"/>
       </xacro:unless>
    </joint>
@@ -200,5 +197,5 @@
       <origin xyz="-0.015 ${-rot*0.05615} -0.061"/>
       <axis xyz="0 0 -1"/>
-      <limit lower="-2.618" upper="2.618" effort="350" velocity="6.5"/> <!-- TODO -->
+      <limit lower="-2.618" upper="2.618" effort="950" velocity="6.5"/>
    </joint>
 <!-- /elbow pitch-->
@@ -209,5 +206,5 @@
       <origin xyz="0 ${rot*0.049} -0.180"/>
       <axis xyz="0 ${rot} 0"/>
-      <limit lower="-1.570" upper="1.570" effort="350" velocity="6.5"/> <!-- TODO -->
+      <limit lower="-1.570" upper="1.570" effort="950" velocity="6.5"/>
    </joint>
 <!-- /wrist yaw-->
@@ -218,9 +215,10 @@
       <origin xyz="0 ${-rot*0.049} -0.169"/>
       <axis xyz="0 0 -1"/>
-      <limit lower="-2.618" upper="2.618" effort="350" velocity="6.5"/> <!-- TODO -->
+      <limit lower="-2.618" upper="2.618" effort="400" velocity="6.5"/>
    </joint>
 <!-- wrist pitch-->
+<!-- force-troque sensor -->
 <!-- actuators -->
-   <xacro:if value="$(arg ARM_ACTUATORS)">
+   <xacro:if value="${arm_actuators}">
       <xacro:position_actuator joint="j_arm${arm_num}_1" />
       <xacro:position_actuator joint="j_arm${arm_num}_2" />
@@ -233,7 +231,13 @@
 <!-- /actuators -->
 <!-- end-effector -->
-   <xacro:if value="$(arg HANDS)">
-      <xacro:include filename="$(find centauro)/centauro_urdf/urdf/centauro_hand.urdf.xacro" />
-   </xacro:if>
+<xacro:if value="${END_EFFECTOR == 'soft_hand'}" >
+  <xacro:include filename="$(find centauro)/centauro_urdf/urdf/centauro_hand.urdf.xacro" />
+</xacro:if>
+<xacro:if value="${END_EFFECTOR == 'stick'}" >
+  <xacro:include filename="$(find centauro)/centauro_urdf/urdf/centauro_stick.urdf.xacro" />
+</xacro:if>
+<xacro:if value="${END_EFFECTOR != 'stick' and END_EFFECTOR != 'soft_hand' }" >
+  <xacro:include filename="$(find centauro)/centauro_urdf/urdf/centauro_no_end_effector.urdf.xacro" />
+</xacro:if>
 <!-- /end-effector -->
 </xacro:macro>

File: centauro/centauro_urdf/urdf/centauro_hand.urdf.xacro (robot description, xacro)
@@ -2,70 +2,29 @@
 <robot xmlns:xacro="http://www.ros.org/wiki/xacro">
 <!-- links -->
-   <link name="arm${arm_num}_7">
+   <link name="arm${arm_num}_8">
       <inertial>
-         <origin xyz="${Hand_x} ${Hand_y} ${Hand_z}"/> <!-- TODO these are not correct values -->
-         <mass value="${Hand_mass}"/> <!-- TODO these are not correct values -->
-         <inertia ixx="${Hand_xx}" ixy="${Hand_xy}" ixz="${Hand_xz}" iyy="${Hand_yy}" iyz="${Hand_yz}" izz="${Hand_zz}"/> <!-- TODO these are not correct values -->
+         <origin xyz="0 0 0.10" rpy="0 0 0"/>
+         <mass value="0.3"/>
+         <inertia ixx="0.00024500"  ixy="0"  ixz="0" iyy="0.00024500" iyz="0" izz="0.00024500" />
       </inertial>
       <visual>
-        <!-- TODO: there is no available information about this link visual element -->
+         <xacro:visual_model.soft_hand />
+         <material name="grey"/>
       </visual>
       <collision>
-      <!-- TODO: there is no available information about this link collsiion element -->
+         <xacro:collision_model.soft_hand />
       </collision>
    </link>
-   <link name="arm${arm_num}_8">
-      <inertial>
-         <origin xyz="0 0 0" rpy="0 0 0"/>
-         <mass value="0.3"/>
-         <inertia ixx="0.001"  ixy="0"  ixz="0" iyy="0.001" iyz="0" izz="0.001" />
-      </inertial>
-      <visual>
-         <origin xyz="0 0 0" rpy="0 0 0" />
-         <geometry>
-            <box size="0.07 0.07 0.07" />
-         </geometry>
-         <material name="Cyan">
-            <color rgba="0 1.0 1.0 1.0"/>
-         </material>
-      </visual>
-<!--      <collision>
-         <origin xyz="0 0 0" rpy="0 0 0"/>
-         <geometry>
-            <box size="0.07 0.07 0.07" />
-         </geometry>
-      </collision> -->
-   </link>
 <!-- /links -->
-<!-- joints -->
    <joint name="j_arm${arm_num}_8" type="revolute">
-      <parent link="ft_arm${arm_num}_7"/>
+      <parent link="arm${arm_num}_7"/>
       <child link="arm${arm_num}_8"/>
-      <origin xyz="0 0 -0.015" rpy="0 ${PI} ${-PI/2}"/>
+      <origin xyz="0 0 -0.0405" rpy="0 ${PI} ${-PI/2}"/>
       <axis xyz="1 0 0" />
-      <limit velocity="4.0" effort="5" lower="0.0" upper="1.57075" />
-      <dynamics friction="0" damping="3.0"/>
-   </joint>
+      <limit velocity="6.5" effort="400" lower="0.0" upper="1.57075" />
+   </joint> -->
 <!-- /joints -->
 <!-- actuators -->
    <xacro:position_actuator joint="j_arm${arm_num}_8" />
 <!-- /actuators -->
-<!-- sensors -->
-<!--   <xacro:if value="$(arg ARM_SENSORS)"> -->
-      <link name="ft_arm${arm_num}_7">
-         <inertial>
-            <origin xyz="0 0 0" rpy="0 0 0"/>
-            <mass value="0.3"/>
-            <inertia ixx="0.001"  ixy="0"  ixz="0" iyy="0.001" iyz="0" izz="0.001" />
-         </inertial>
-      </link>
-      <joint name="ft_j_arm${arm_num}_7" type="fixed">
-         <parent link="arm${arm_num}_7"/>
-         <child link="ft_arm${arm_num}_7"/>
-         <origin xyz="0 0 -0.0255" rpy="0 0 0"/>
-         <axis xyz="1 0 0" />
-      </joint>
-      <xacro:force-torque_sensor joint="ft_j_arm${arm_num}_7" robot="centauro" />
- <!--  </xacro:if> -->
-<!-- /sensors -->
 </robot>

File: centauro/centauro_urdf/urdf/centauro_leg.urdf.xacro (robot description, xacro)
@@ -140,5 +140,5 @@
 </link>-->
 <!-- wheels -->
-<xacro:if	value="$(arg WHEELS)">
+<xacro:if	value="${wheels}">
 	<!-- links -->
 	<link name="wheel_hip_${leg_num}">
@@ -162,4 +162,18 @@
 		</collision>
 	</link>
+	<link name="wheel_hip_reference_${leg_num}">
+		<inertial>
+			<origin xyz="0 0 0"/>	<!-- TODO -->
+			<mass value="${0.01}"/>  <!-- org: 3.5, foot un modeled-->
+			<inertia ixx="${0.01/12*(0.01*0.01+0.01*0.01)}" ixy="0" ixz="0" iyy="${0.01/12*(wheel_radius*wheel_radius+0.01*0.01)}" iyz="0" izz="${0.01/12*(wheel_radius*wheel_radius+0.01*0.01)}"/>
+		</inertial>
+		<visual>
+			<origin xyz="0 0 0" rpy="0 0 0" />
+			<geometry>
+				<box size="${wheel_radius} 0.01 0.01"/>
+			</geometry>
+			<material name="blue"/>
+		</visual>
+	</link>
 	<link name="wheel_knee_${leg_num}">
 		<inertial>
@@ -181,4 +195,18 @@
 			</geometry>
 		</collision>
+	</link>
+	<link name="wheel_knee_reference_${leg_num}">
+		<inertial>
+			<origin xyz="0 0 0"/>	<!-- TODO -->
+			<mass value="${0.01}"/>  <!-- org: 3.5, foot un modeled-->
+			<inertia ixx="${0.01/12*(0.01*0.01+0.01*0.01)}" ixy="0" ixz="0" iyy="${0.01/12*(wheel_radius*wheel_radius+0.01*0.01)}" iyz="0" izz="${0.01/12*(wheel_radius*wheel_radius+0.01*0.01)}"/>
+		</inertial>
+		<visual>
+			<origin xyz="0 0 0" rpy="0 0 0" />
+			<geometry>
+				<box size="${wheel_radius} 0.01 0.01"/>
+			</geometry>
+			<material name="blue"/>
+		</visual>
 	</link>
 	<!-- /links -->
@@ -190,4 +218,9 @@
 		<axis xyz="0 ${origin_x*origin_y} 0"/>
 	</joint>
+	<joint name="j_wheel_hip_reeferece_${leg_num}" type="fixed">
+		<origin xyz="0 ${origin_y*(wheel_length+0.005)} 0"/>
+		<parent link="wheel_hip_${leg_num}"/>
+		<child link="wheel_hip_reference_${leg_num}"/>
+	</joint>
 	<joint name="j_wheel_knee_${leg_num}" type="continuous">
 		<parent link="knee_${leg_num}"/>
@@ -196,7 +229,12 @@
 		<axis xyz="0 ${origin_x*origin_y} 0"/>
 	</joint>
+	<joint name="j_wheel_knee_reeferece_${leg_num}" type="fixed">
+		<origin xyz="0 ${origin_y*(wheel_length+0.005)} 0"/>
+		<parent link="wheel_knee_${leg_num}"/>
+		<child link="wheel_knee_reference_${leg_num}"/>
+	</joint>
 	<!-- /joints -->
 	<!-- actuators -->
-<xacro:if	value="$(arg WHEELS_ACTUATORS)">
+<xacro:if	value="${wheels_actuators}">
 	<xacro:position_actuator joint="j_wheel_hip_${leg_num}" />
 	<xacro:position_actuator joint="j_wheel_knee_${leg_num}" />
@@ -210,5 +248,5 @@
 	<origin xyz="${origin_x*0.30} ${origin_y*0.15} 0" rpy="0 0 ${PI/2}"/>
 	<axis xyz="0 0 ${-origin_y}"/>
-	<limit lower="-2.09" upper="2.09" effort="350" velocity="6.5"/> <!-- TODO -->
+        <limit lower="-2.09" upper="2.09" effort="1770" velocity="6.5"/> <!-- TODO -->
 </joint>
 <joint name="hip_pitch_${leg_num}" type="revolute">
@@ -217,5 +255,5 @@
 	<origin xyz="0 0 -0.2"/>
 	<axis xyz="0 ${-origin_y} 0"/>
-	<limit lower="-3.14" upper="3.14" effort="350" velocity="6.5"/> <!-- TODO -->
+        <limit lower="-3.14" upper="3.14" effort="3300" velocity="6.5"/> <!-- TODO -->
 </joint>
 <joint name="knee_pitch_${leg_num}" type="revolute">
@@ -224,5 +262,5 @@
 	<origin xyz="0 0 -0.35"/>
 	<axis xyz="0 ${-origin_y} 0"/>
-	<limit  lower="-3.14" upper="3.14" effort="35000" velocity="600.5"/> <!-- TODO -->
+        <limit  lower="-3.14" upper="3.14" effort="3300" velocity="600.5"/> <!-- TODO -->
 </joint>
 <!--
@@ -234,5 +272,5 @@
 -->
 <!-- actuators -->
-<xacro:if	value="$(arg LEG_ACTUATORS)">
+<xacro:if	value="${leg_actuators}">
 	<xacro:position_actuator joint="hip_yaw_${leg_num}" />
 	<xacro:position_actuator joint="hip_pitch_${leg_num}" />

File: centauro/centauro_urdf/urdf/centauro_torso.urdf.xacro (robot description, xacro)
@@ -6,13 +6,12 @@
 		<origin xyz="${Torso_2_x} ${Torso_2_y} ${Torso_2_z}"/>
 		<mass value="${Torso_2_mass}"/> <!-- mass  7: torso_1 (2) + torso_2 (5), head un_modelled -->
-		<inertia ixx="${Torso_2_xx}" ixy="${Torso_2_xy}" ixz="${Torso_2_xz}" iyy="${Torso_2_yy}" iyz="${Torso_2_yz}" izz="${Torso_2_zz}"/>
-		<!-- <inertia ixx="0.01" ixy="0.01" ixz="0.01" iyy="0.01" iyz="0.01" izz="0.01"/> -->
-	</inertial>
+                <inertia ixx="${Torso_2_xx}" ixy="${Torso_2_xy}" ixz="${Torso_2_xz}" iyy="${Torso_2_yy}" iyz="${Torso_2_yz}" izz="${Torso_2_zz}"/>
+        </inertial>
 	<visual>
- 		<xacro:insert_block name="v_torso" />
+                <xacro:visual_model.torso />
 		<material name="grey"/>
 	</visual>
 	<collision>
- 		<xacro:insert_block name="c_torso" />
+                <xacro:collision_model.torso />
 		<material name="grey"/>
 	</collision>
@@ -20,18 +19,22 @@
 <!-- /torso links -->
 <!-- torso joints -->
-<xacro:unless	value="$(arg ONE_ARM)">
 <joint name="torso_yaw" type="revolute">
-	<parent link="pelvis"/>
-	<child link="torso_2"/>
-	<origin xyz="0.30 0 0.1"/>
-	<axis xyz="0 0 1"/>
-	<limit lower="-2.618" upper="2.618" effort="350" velocity="6.5"/> <!-- TODO -->
+   <xacro:if value="${pelvis}">
+      <parent link="pelvis"/>
+      <origin xyz="0.30 0 0.1"/>
+   </xacro:if>
+   <xacro:unless value="${pelvis}">
+      <parent link="world"/>
+      <origin xyz="0.30 0 ${0.1 + 0.85}"/>
+   </xacro:unless>
+   <child link="torso_2"/>
+   <axis xyz="0 0 1"/>
+   <limit lower="-2.618" upper="2.618" effort="1770" velocity="6.5"/> <!-- TODO -->
 </joint>
 <!-- /torso joints -->
-<xacro:if	value="$(arg TORSO_ACTUATORS)">
+<xacro:if	value="${torso_actuators}">
 <!-- torso actuators -->
 <xacro:position_actuator joint="torso_yaw" />
 <!-- /torso actuators -->
 </xacro:if>
-</xacro:unless>
 </robot>
