Commit message: Arturo's work for the walking video for PHOLUS visit.

File: centauro/centauro_urdf/urdf/centauro_torso.urdf.xacro (robot description, xacro)
@@ -55,3 +55,39 @@
 <!-- /torso actuators -->
 </xacro:if>
+<link name="camera_link">
+      <pose>0.05 0.05 0.05 0 0 0</pose>
+      <inertial>
+        <mass value="0.0"/> <!-- mass  7: torso_1 (2) + torso_2 (5), head un_modelled -->
+        <inertia ixx="0.0" ixy="0.0" ixz="0.0" iyy="0.0" iyz="0.0" izz="0.0"/>
+      </inertial>
+      <visual name="visual">
+        <geometry>
+          <box>
+            <size>0.1 0.1 0.1</size>
+          </box>
+        </geometry>
+      </visual>
+<!--      <sensor name="camera" type="camera">
+        <camera>
+          <horizontal_fov>1.047</horizontal_fov>
+          <image>
+            <width>1280</width>
+            <height>720</height>
+          </image>
+          <clip>
+            <near>0.1</near>
+            <far>100</far>
+          </clip>
+        </camera>
+        <always_on>1</always_on>
+        <update_rate>30</update_rate>
+        <visualize>true</visualize>
+      </sensor>-->
+</link>
+<joint name="camera_joint" type="fixed">
+    <parent link="torso_2"/>
+    <child link="camera_link"/>
+<!--     <axis xyz="3 3 0"/> -->
+    <origin xyz="0 -2 -0.3" rpy="0 0 1.57"/>
+</joint>
 </robot>
