Commit message: change centauro to have 14 joints

File: centauro/centauro_urdf/urdf/centauro_floating_arm0.urdf (robot description, URDF)
Before this commit: robot centauro, 22 links, 21 joints
Links:
- added link load, mass 20; collision box size=0.1 0.2 0.4; visual box size=0.1 0.2 0.4
Joints:
- added joint load_joint: type fixed, parent base_link, child load, origin xyz=0.04 0.0 0.4 rpy=0 0 0
- joint floating_base: type fixed -> floating

File: centauro/centauro_urdf/urdf/centauro_narrow_feet.urdf.xacro (robot description, xacro)
@@ -5,6 +5,6 @@
         <visual>
             <geometry>
-                <box size="0.3 0.1 0.02"/>
-                <!--box size="0.3 0.04 0.3"/-->
+                <box size="0.4 0.02 0.1"/>
+                <!--box size="0.3 0.1 0.02"/-->
                 <!--cylinder length="0.3" radius="0.02"/-->
             </geometry>
@@ -12,6 +12,6 @@
         <collision>
             <geometry>
-                <box size="0.3 0.1 0.02"/>
-                <!--box size="0.3 0.04 0.3"/-->
+                <box size="0.4 0.02 0.1"/>
+                <!--box size="0.3 0.1 0.02"/-->
                 <!--cylinder length="0.3" radius="0.02"/-->
             </geometry>
