Commit message: add some damping to arm joints

File: centauro/centauro_urdf/urdf/centauro_narrow_feet.urdf.xacro (robot description, xacro)
@@ -6,5 +6,5 @@
             <geometry>
                 <!--box size="0.4 0.02 0.1"/-->
-                <box size="0.3 0.1 0.02"/>
+                <box size="0.4 0.06 0.02"/>
                 <!--cylinder length="0.3" radius="0.02"/-->
             </geometry>
@@ -13,5 +13,5 @@
             <geometry>
                 <!--box size="0.4 0.02 0.1"/-->
-                <box size="0.3 0.1 0.02"/>
+                <box size="0.4 0.06 0.02"/>
                 <!--cylinder length="0.3" radius="0.02"/-->
             </geometry>
@@ -43,5 +43,5 @@
             <parent link="arm${arm_num}_7"/>
             <child link="arm${arm_num}_8"/>
-            <origin xyz="0 0 -0.05" rpy="0 0 0"/>
+            <origin xyz="0 0 -0.08" rpy="0 0 0"/>
         </joint>
 </robot>

Commit message: make feet shorter and simulation time step smaller

File: centauro/centauro_urdf/urdf/centauro_narrow_feet.urdf.xacro (robot description, xacro)
@@ -6,5 +6,5 @@
             <geometry>
                 <!--box size="0.4 0.02 0.1"/-->
-                <box size="0.4 0.03 0.03"/>
+                <box size="0.3 0.03 0.03"/>
                 <!--cylinder length="0.3" radius="0.02"/-->
             </geometry>
@@ -13,5 +13,5 @@
             <geometry>
                 <!--box size="0.4 0.02 0.1"/-->
-                <box size="0.4 0.03 0.03"/>
+                <box size="0.3 0.03 0.03"/>
                 <!--cylinder length="0.3" radius="0.02"/-->
             </geometry>
@@ -28,5 +28,5 @@
             <parent link="arm${arm_num}_7"/>
             <child link="arm${arm_num}_8"/>
-            <origin xyz="0 0 -0.05" rpy="0 0 0.5"/>
+            <origin xyz="0.0 0 -0.05" rpy="0 0 0.5"/>
         </joint>
     </xacro:if>
@@ -35,5 +35,5 @@
             <parent link="arm${arm_num}_7"/>
             <child link="arm${arm_num}_8"/>
-            <origin xyz="0 0 -0.05" rpy="0 0 -0.5"/>
+            <origin xyz="0.0 0 -0.05" rpy="0 0 -0.5"/>
         </joint>
     </xacro:if>
