Commit message: j_armX_8 joint changed to revolute in order to avoid issue with FT

File: centauro/centauro_urdf/urdf/centauro_stick.urdf.xacro (robot description, xacro)
@@ -19,5 +19,5 @@
 <!-- /links -->
 <!-- joints -->
-   <joint name="j_arm${arm_num}_8" type="fixed">
+   <joint name="j_arm${arm_num}_8" type="revolute">
       <parent link="arm${arm_num}_7"/>
       <child link="arm${arm_num}_8"/>
