Commit message: fixing FT issue to be compatible with XBotCore.

File: centauro/centauro_urdf/urdf/centauro_no_end_effector.urdf.xacro (robot description, xacro)
@@ -4,5 +4,5 @@
    <link name="arm${arm_num}_8"/>
 <!-- /links -->
-   <joint name="j_arm${arm_num}_8" type="revolute">
+   <joint name="j_arm${arm_num}_8" type="fixed">
       <parent link="arm${arm_num}_7"/>
       <child link="arm${arm_num}_8"/>

File: centauro/centauro_urdf/urdf/centauro_stick.urdf.xacro (robot description, xacro)
@@ -2,5 +2,5 @@
 <robot xmlns:xacro="http://www.ros.org/wiki/xacro">
 <!-- links -->
-   <link name="arm${arm_num}_8">
+   <link name="ft_arm${arm_num}">
       <inertial>
          <origin xyz="${Stick_x} ${Stick_y} ${Stick_z}" rpy="0 0 0"/>
@@ -19,7 +19,7 @@
 <!-- /links -->
 <!-- joints -->
-   <joint name="j_arm${arm_num}_8" type="revolute">
+   <joint name="j_ft_arm${arm_num}" type="revolute">
       <parent link="arm${arm_num}_7"/>
-      <child link="arm${arm_num}_8"/>
+      <child link="ft_arm${arm_num}"/>
       <origin xyz="${End_effector_Ox} ${End_effector_Oy} ${End_effector_Oz}" rpy="${End_effector_roll} ${End_effector_pitch} ${End_effector_yaw}"/>
       <axis xyz="1 0 0" />

File: centauro_gazebo/sensors/xbotcore/ft_sensor/load/arms.xacro (robot description, xacro)
@@ -2,7 +2,7 @@
 <robot  xmlns:xacro="http://www.ros.org/wiki/xacro">
 <xacro:include filename="$(find centauro)/centauro_urdf/urdf/config.xacro"/>
-  <xacro:force-torque_sensor joint="j_arm1_8" robot="centauro" ft_name="left_arm_ft" pose="0 0 0 0 0 0"/>
+  <xacro:force-torque_sensor joint="j_ft_arm1" robot="centauro" ft_name="ft_arm1" pose="0 0 0 0 0 0"/>
   <xacro:if value="${arms}">
-    <xacro:force-torque_sensor joint="j_arm2_8" robot="centauro" ft_name="right_arm_ft" pose="0 0 0 0 0 0"/>
+    <xacro:force-torque_sensor joint="j_ft_arm2" robot="centauro" ft_name="ft_arm2" pose="0 0 0 0 0 0"/>
   </xacro:if>
 </robot>
