Commit message: urdf bugfix

File: centauro/centauro_urdf/urdf/centauro_eef.urdf.xacro (robot description, xacro)
@@ -11,5 +11,5 @@
 </xacro:macro>
 <!-- leg eef links -->
-<xacro:macro name="leg_eef" params="prefix parent">
+<xacro:macro name="leg_eef" params="prefix parent *origin">
 		<link name="${prefix}_eef_link" />
 		<joint name="${prefix}_eef_joint" type="fixed">
