Commit message: try to modify urdf

File: centauro/centauro_urdf/urdf/centauro_config.urdf (robot description, URDF)
Before this commit: robot centauro, 53 links, 52 joints
Links:
- removed link camera_central
- removed link camera_left
- removed link camera_right
- removed link kinect
- removed link kinect2_rgb_optical_frame
- removed link velodyne_mount
- added link foot_fl, mass 0; visual box size=0.01 0.01 0.01
- added link foot_fr, mass 0; visual box size=0.01 0.01 0.01
- added link foot_hl, mass 0; visual box size=0.01 0.01 0.01
- added link foot_hr, mass 0; visual box size=0.01 0.01 0.01
- added link ft_arm1, mass 0.15; collision mesh filename=package://centauro/centauro_urdf/meshes/link9.stl scale=0.001 0.001 -0.001; visual mesh filename=package://centauro/centauro_urdf/meshes/link9.stl scale=0.001 0.001 -0.001
- added link ft_arm2, mass 0.15; collision mesh filename=package://centauro/centauro_urdf/meshes/link9.stl scale=0.001 0.001 -0.001; visual mesh filename=package://centauro/centauro_urdf/meshes/link9.stl scale=0.001 0.001 -0.001
- link ankle1_1: geometry collision mesh filename=package://centauro/centauro_urdf/meshes/convex_hull/ankle-p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 scale=0.001 0.001 0.001; visual mesh filename=package://centauro/centauro_urdf/meshes/ankle-pitch.stl scale=0.001 0.001 0.001
- link ankle1_2: geometry collision mesh filename=package://centauro/centauro_urdf/meshes/convex_hull/ankle-p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 scale=0.001 0.001 0.001; visual mesh filename=package://centauro/centauro_urdf/meshes/ankle-pitch.stl scale=0.001 0.001 0.001
- link ankle1_3: geometry collision mesh filename=package://centauro/centauro_urdf/meshes/convex_hull/ankle-p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 scale=0.001 0.001 0.001; visual mesh filename=package://centauro/centauro_urdf/meshes/ankle-pitch.stl scale=0.001 0.001 0.001
- link ankle1_4: geometry collision mesh filename=package://centauro/centauro_urdf/meshes/convex_hull/ankle-p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 scale=0.001 0.001 0.001; visual mesh filename=package://centauro/centauro_urdf/meshes/ankle-pitch.stl scale=0.001 0.001 0.001
- link ankle2_1: geometry collision mesh filename=package://centauro/centauro_urdf/meshes/convex_hull/ankle-y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 scale=0.001 0.001 0.001; visual mesh filename=package://centauro/centauro_urdf/meshes/ankle-yaw.stl scale=0.001 0.001 0.001
- link ankle2_2: geometry collision mesh filename=package://centauro/centauro_urdf/meshes/convex_hull/ankle-y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 scale=0.001 0.001 0.001; visual mesh filename=package://centauro/centauro_urdf/meshes/ankle-yaw.stl scale=0.001 0.001 0.001
- link ankle2_3: geometry collision mesh filename=package://centauro/centauro_urdf/meshes/convex_hull/ankle-y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 scale=0.001 0.001 0.001; visual mesh filename=package://centauro/centauro_urdf/meshes/ankle-yaw.stl scale=0.001 0.001 0.001
- link ankle2_4: geometry collision mesh filename=package://centauro/centauro_urdf/meshes/convex_hull/ankle-y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 scale=0.001 0.001 0.001; visual mesh filename=package://centauro/centauro_urdf/meshes/ankle-yaw.stl scale=0.001 0.001 0.001
- link arm1_1: geometry collision mesh filename=package://centauro/centauro_urdf/meshes/convex_hull/link2.s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 scale=0.001 -0.001 0.001; visual mesh filename=package://centauro/centauro_urdf/meshes/link2.stl scale=0.001 -0.001 0.001
- link arm1_2: geometry collision mesh filename=package://centauro/centauro_urdf/meshes/convex_hull/link3.s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 scale=0.001 -0.001 0.001; visual mesh filename=package://centauro/centauro_urdf/meshes/link3.stl scale=0.001 -0.001 0.001
- link arm1_3: geometry collision mesh filename=package://centauro/centauro_urdf/meshes/convex_hull/link4.s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 scale=0.001 -0.001 0.001; visual mesh filename=package://centauro/centauro_urdf/meshes/link4.stl scale=0.001 -0.001 0.001
- link arm1_4: geometry collision mesh filename=package://centauro/centauro_urdf/meshes/convex_hull/link5.s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 scale=0.001 -0.001 0.001; visual mesh filename=package://centauro/centauro_urdf/meshes/link5.stl scale=0.001 -0.001 0.001
- link arm1_5: geometry collision mesh filename=package://centauro/centauro_urdf/meshes/convex_hull/link6.s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 scale=0.001 -0.001 0.001; visual mesh filename=package://centauro/centauro_urdf/meshes/link6.stl scale=0.001 -0.001 0.001
- link arm1_6: geometry collision mesh filename=package://centauro/centauro_urdf/meshes/convex_hull/link7.s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 scale=0.001 -0.001 0.001; visual mesh filename=package://centauro/centauro_urdf/meshes/link7.stl scale=0.001 -0.001 0.001
- link arm1_7: geometry collision mesh filename=package://centauro/centauro_urdf/meshes/convex_hull/link8.s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 scale=0.001 -0.001 0.001; visual mesh filename=package://centauro/centauro_urdf/meshes/link8.stl scale=0.001 -0.001 0.001
- link arm1_8: mass 1.8366865 -> 0.15; geometry collision mesh filename=package://centauro/centauro_urdf/meshes/convex_hull/link9.s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 scale=0.001 -0.001 -0.001; visual mesh filename=package://centauro/centauro_urdf/meshes/link9.stl scale=0.001 -0.001 -0.001
- link arm2_1: geometry collision mesh filename=package://centauro/centauro_urdf/meshes/convex_hull/link2.s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 scale=0.001 0.001 0.001; visual mesh filename=package://centauro/centauro_urdf/meshes/link2.stl scale=0.001 0.001 0.001
- link arm2_2: geometry collision mesh filename=package://centauro/centauro_urdf/meshes/convex_hull/link3.s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 scale=0.001 0.001 0.001; visual mesh filename=package://centauro/centauro_urdf/meshes/link3.stl scale=0.001 0.001 0.001
- link arm2_3: geometry collision mesh filename=package://centauro/centauro_urdf/meshes/convex_hull/link4.s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 scale=0.001 0.001 0.001; visual mesh filename=package://centauro/centauro_urdf/meshes/link4.stl scale=0.001 0.001 0.001
- link arm2_4: geometry collision mesh filename=package://centauro/centauro_urdf/meshes/convex_hull/link5.s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 scale=0.001 0.001 0.001; visual mesh filename=package://centauro/centauro_urdf/meshes/link5.stl scale=0.001 0.001 0.001
- link arm2_5: geometry collision mesh filename=package://centauro/centauro_urdf/meshes/convex_hull/link6.s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 scale=0.001 0.001 0.001; visual mesh filename=package://centauro/centauro_urdf/meshes/link6.stl scale=0.001 0.001 0.001
- link arm2_6: geometry collision mesh filename=package://centauro/centauro_urdf/meshes/convex_hull/link7.s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 scale=0.001 0.001 0.001; visual mesh filename=package://centauro/centauro_urdf/meshes/link7.stl scale=0.001 0.001 0.001
- link arm2_7: geometry collision mesh filename=package://centauro/centauro_urdf/meshes/convex_hull/link8.s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 scale=0.001 0.001 0.001; visual mesh filename=package://centauro/centauro_urdf/meshes/link8.stl scale=0.001 0.001 0.001
- link arm2_8: mass 1.8366865 -> 0.15; geometry collision mesh filename=package://centauro/centauro_urdf/meshes/convex_hull/link9.s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 scale=0.001 0.001 -0.001; visual mesh filename=package://centauro/centauro_urdf/meshes/link9.stl scale=0.001 0.001 -0.001
- link hip1_1: geometry collision mesh filename=package://centauro/centauro_urdf/meshes/convex_hull/hip-yaw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 scale=0.001 0.001 0.001; visual mesh filename=package://centauro/centauro_urdf/meshes/hip-yaw.stl scale=0.001 0.001 0.001
- link hip1_2: geometry collision mesh filename=package://centauro/centauro_urdf/meshes/convex_hull/hip-yaw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 scale=0.001 0.001 0.001; visual mesh filename=package://centauro/centauro_urdf/meshes/hip-yaw.stl scale=0.001 0.001 0.001
- link hip1_3: geometry collision mesh filename=package://centauro/centauro_urdf/meshes/convex_hull/hip-yaw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 scale=0.001 0.001 0.001; visual mesh filename=package://centauro/centauro_urdf/meshes/hip-yaw.stl scale=0.001 0.001 0.001
- link hip1_4: geometry collision mesh filename=package://centauro/centauro_urdf/meshes/convex_hull/hip-yaw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 scale=0.001 0.001 0.001; visual mesh filename=package://centauro/centauro_urdf/meshes/hip-yaw.stl scale=0.001 0.001 0.001
- link hip2_1: geometry collision mesh filename=package://centauro/centauro_urdf/meshes/convex_hull/hip-pit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 scale=0.001 0.001 0.001; visual mesh filename=package://centauro/centauro_urdf/meshes/hip-pitch.stl scale=0.001 0.001 0.001
- link hip2_2: geometry collision mesh filename=package://centauro/centauro_urdf/meshes/convex_hull/hip-pit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 scale=0.001 0.001 0.001; visual mesh filename=package://centauro/centauro_urdf/meshes/hip-pitch.stl scale=0.001 0.001 0.001
- link hip2_3: geometry collision cylinder length=0.4 radius=0.05; visual mesh filename=package://centauro/centauro_urdf/meshes/hip-pitch.stl scale=0.001 0.001 0.001
- link hip2_4: geometry collision cylinder length=0.4 radius=0.05; visual mesh filename=package://centauro/centauro_urdf/meshes/hip-pitch.stl scale=0.001 0.001 0.001
- link knee_1: geometry collision mesh filename=package://centauro/centauro_urdf/meshes/convex_hull/knee.stl scale=0.001 0.001 0.001; visual mesh filename=package://centauro/centauro_urdf/meshes/knee.stl scale=0.001 0.001 0.001
- link knee_2: geometry collision mesh filename=package://centauro/centauro_urdf/meshes/convex_hull/knee.stl scale=0.001 0.001 0.001; visual mesh filename=package://centauro/centauro_urdf/meshes/knee.stl scale=0.001 0.001 0.001
- link knee_3: geometry collision cylinder length=0.25 radius=0.05; visual mesh filename=package://centauro/centauro_urdf/meshes/knee.stl scale=0.001 0.001 0.001
- link knee_4: geometry collision cylinder length=0.25 radius=0.05; visual mesh filename=package://centauro/centauro_urdf/meshes/knee.stl scale=0.001 0.001 0.001
- link neck_1: geometry collision mesh filename=package://centauro/centauro_urdf/meshes/convex_hull/neck_ya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 scale=0.001 0.001 0.001; visual mesh filename=package://centauro/centauro_urdf/meshes/neck_yaw.stl scale=0.001 0.001 0.001
- link neck_2: geometry collision mesh filename=package://centauro/centauro_urdf/meshes/convex_hull/neck_pi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 scale=0.001 0.001 0.001; visual mesh filename=package://centauro/centauro_urdf/meshes/neck_pitch.stl scale=0.001 0.001 0.001
- link neck_3: geometry collision mesh filename=package://centauro/centauro_urdf/meshes/convex_hull/velodyn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 scale=0.001 0.001 0.001; visual mesh filename=package://centauro/centauro_urdf/meshes/velodyne.stl scale=0.001 0.001 0.001
- link pelvis: geometry collision mesh filename=package://centauro/centauro_urdf/meshes/convex_hull/pelvis.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 scale=0.001 0.001 0.001; visual mesh filename=package://centauro/centauro_urdf/meshes/pelvis.stl scale=0.001 0.001 0.001
- link torso_2: geometry collision mesh filename=package://centauro/centauro_urdf/meshes/convex_hull/link1.s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 scale=0.001 0.001 0.001; visual mesh filename=package://centauro/centauro_urdf/meshes/link1.stl scale=0.001 0.001 0.001
- link wheel_1: geometry collision mesh filename=package://centauro/centauro_urdf/meshes/convex_hull/wheel.s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 scale=0.001 0.001 0.001; visual mesh filename=package://centauro/centauro_urdf/meshes/wheel.stl scale=0.001 0.001 0.001
- link wheel_2: geometry collision mesh filename=package://centauro/centauro_urdf/meshes/convex_hull/wheel.s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 scale=0.001 0.001 0.001; visual mesh filename=package://centauro/centauro_urdf/meshes/wheel.stl scale=0.001 0.001 0.001
- link wheel_3: geometry collision mesh filename=package://centauro/centauro_urdf/meshes/convex_hull/wheel.s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 scale=0.001 0.001 0.001; visual mesh filename=package://centauro/centauro_urdf/meshes/wheel.stl scale=0.001 0.001 0.001
- link wheel_4: geometry collision mesh filename=package://centauro/centauro_urdf/meshes/convex_hull/wheel.s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 scale=0.001 0.001 0.001; visual mesh filename=package://centauro/centauro_urdf/meshes/wheel.stl scale=0.001 0.001 0.001
Joints:
- removed joint j_camera_central
- removed joint j_camera_left
- removed joint j_camera_right
- removed joint j_kinect
- removed joint j_kinect_optical_frame
- removed joint j_velodyne
- added joint j_foot_fl: type fixed, parent ankle2_1, child foot_fl, origin xyz=0.0 0.0 0.30 rpy=3.1415 0.0 3.1415
- added joint j_foot_fr: type fixed, parent ankle2_2, child foot_fr, origin xyz=0.0 0.0 0.30 rpy=3.1415 0.0 0.0
- added joint j_foot_hl: type fixed, parent ankle2_3, child foot_hl, origin xyz=0.0 0.0 0.30 rpy=3.1415 0.0 3.1415
- added joint j_foot_hr: type fixed, parent ankle2_4, child foot_hr, origin xyz=0.0 0.0 0.30 rpy=3.1415 0.0 0.0
- added joint j_ft_arm1: type fixed, parent arm1_7, child ft_arm1, origin xyz=0.0 0.0 -0.0405 rpy=0.0 3.14159265359 -3.14159265359, axis 1 0 0, limit lower=0.0 upper=0 effort=0 velocity=0
- added joint j_ft_arm2: type fixed, parent arm2_7, child ft_arm2, origin xyz=0.0 0.0 -0.0405 rpy=0.0 3.14159265359 -3.14159265359, axis 1 0 0, limit lower=0.0 upper=0 effort=0 velocity=0
- joint ankle_pitch_1: limit lower=-2.4056 upper=2.3184 effort=147 velocity=8.1 -> lower=-2.61799388 upper=2.61799388 effort=147 velocity=8.1
- joint ankle_pitch_2: limit lower=-2.3266 upper=2.3914 effort=147 velocity=8.1 -> lower=-2.61799388 upper=2.61799388 effort=147 velocity=8.1
- joint ankle_pitch_3: limit lower=-2.4696 upper=2.4464 effort=147 velocity=8.1 -> lower=-2.61799388 upper=2.61799388 effort=147 velocity=8.1
- joint ankle_pitch_4: limit lower=-2.3426 upper=2.3934 effort=147 velocity=8.1 -> lower=-2.61799388 upper=2.61799388 effort=147 velocity=8.1
- joint ankle_yaw_1: limit lower=-2.5626 upper=2.5384 effort=35 velocity=20.0 -> lower=-2.79252680 upper=2.79252680 effort=35 velocity=20.0
- joint ankle_yaw_2: limit lower=-2.5546 upper=2.5484 effort=35 velocity=20.0 -> lower=-2.79252680 upper=2.79252680 effort=35 velocity=20.0
- joint ankle_yaw_3: limit lower=-2.5606 upper=2.5454 effort=35 velocity=20.0 -> lower=-2.79252680 upper=2.79252680 effort=35 velocity=20.0
- joint ankle_yaw_4: limit lower=-2.6046 upper=2.5514 effort=35 velocity=20.0 -> lower=-2.79252680 upper=2.79252680 effort=35 velocity=20.0
- joint hip_pitch_1: limit lower=-2.0226 upper=2.02748 effort=304 velocity=8.8 -> lower=-2.09439510 upper=2.09439510 effort=304 velocity=8.8; origin xyz=0.0 0.0 0.0625 rpy=1.57079632679 0.0 0.46141612323 -> xyz=0.0 0.0 0.059 rpy=1.57079632679 0.0 0.50709869865
- joint hip_pitch_2: limit lower=-2.0156 upper=2.0354 effort=304 velocity=8.8 -> lower=-2.09439510 upper=2.09439510 effort=304 velocity=8.8; origin xyz=0.0 0.0 0.0625 rpy=1.57079632679 0.0 2.68017653036 -> xyz=0.0 0.0 0.059 rpy=1.57079632679 0.0 2.63449395494
- joint hip_pitch_3: limit lower=-2.0126 upper=2.0384 effort=304 velocity=8.8 -> lower=-2.09439510 upper=2.09439510 effort=304 velocity=8.8; origin xyz=0.0 0.0 0.0625 rpy=1.57079632679 0.0 2.68017653036 -> xyz=0.0 0.0 0.059 rpy=1.57079632679 0.0 2.63449395494
- joint hip_pitch_4: limit lower=-2.0326 upper=2.0524 effort=304 velocity=8.8 -> lower=-2.09439510 upper=2.09439510 effort=304 velocity=8.8; origin xyz=0.0 0.0 0.0625 rpy=1.57079632679 0.0 0.46141612323 -> xyz=0.0 0.0 0.059 rpy=1.57079632679 0.0 0.50709869865
- joint hip_yaw_1: limit lower=-0.9432 upper=2.5138 effort=304 velocity=8.8 -> lower=-1.13446401 upper=2.70526034 effort=304 velocity=8.8; origin xyz=0.25 0.125 -0.0566 rpy=3.14159265359 0.0 0.461416123228 -> xyz=0.25 0.125 -0.0566 rpy=3.14159265359 0.0 0.50709869865
- joint hip_yaw_2: limit lower=-2.511 upper=0.943 effort=304 velocity=8.8 -> lower=-2.70526034 upper=1.13446401 effort=304 velocity=8.8; origin xyz=0.25 -0.125 -0.0566 rpy=3.14159265359 0.0 -0.461416123228 -> xyz=0.25 -0.125 -0.0566 rpy=3.14159265359 0.0 -0.50709869865
- joint hip_yaw_3: limit lower=-2.51 upper=0.943 effort=304 velocity=8.8 -> lower=-2.70526034 upper=1.13446401 effort=304 velocity=8.8; origin xyz=-0.25 0.125 -0.0566 rpy=3.14159265359 0.0 2.68017653036 -> xyz=-0.25 0.125 -0.0566 rpy=3.14159265359 0.0 2.63449395494
- joint hip_yaw_4: limit lower=-0.9412 upper=2.5138 effort=304 velocity=8.8 -> lower=-1.13446401 upper=2.70526034 effort=304 velocity=8.8; origin xyz=-0.25 -0.125 -0.0566 rpy=3.14159265359 0.0 3.60300877682 -> xyz=-0.25 -0.125 -0.0566 rpy=3.14159265359 0.0 3.64869135224
- joint j_arm1_1: limit lower=-3.348 upper=1.578 effort=147 velocity=5.7 -> lower=-3.403 upper=1.658 effort=147 velocity=5.7
- joint j_arm1_2: limit lower=-3.42 upper=-0.056 effort=147 velocity=5.7 -> lower=-3.49 upper=-0.25 effort=147 velocity=5.7
- joint j_arm1_3: limit lower=-2.5556 upper=2.5424 effort=147 velocity=8.2 -> lower=-2.618 upper=2.618 effort=147 velocity=8.2
- joint j_arm1_4: limit lower=-2.4636 upper=0.2804 effort=147 velocity=8.2 -> lower=-2.530 upper=0.349 effort=147 velocity=8.2
- joint j_arm1_5: limit lower=-2.5406 upper=2.5534 effort=55 velocity=11.6 -> lower=-2.618 upper=2.618 effort=55 velocity=11.6
- joint j_arm1_6: limit lower=-1.5096 upper=1.5044 effort=55 velocity=11.6 -> lower=-1.570 upper=1.570 effort=55 velocity=11.6
- joint j_arm1_7: limit lower=-2.5376 upper=2.5554 effort=27 velocity=20.3 -> lower=-2.618 upper=2.618 effort=27 velocity=20.3
- joint j_arm1_8: limit (none) -> lower=0.0 upper=0 effort=0 velocity=0; origin xyz=0.0 0.0 -0.0405 rpy=0.0 3.14159265359 3.14159265359 -> xyz=0.0 0.0 -0.0405 rpy=0.0 3.14159265359 -1.5707963268
- joint j_arm2_1: limit lower=-1.6102 upper=3.3138 effort=147 velocity=5.7 -> lower=-1.658 upper=3.403 effort=147 velocity=5.7
- joint j_arm2_2: limit lower=0.0578 upper=3.4288 effort=147 velocity=5.7 -> lower=0.25 upper=3.49 effort=147 velocity=5.7
- joint j_arm2_3: limit lower=-2.5426 upper=2.5524 effort=147 velocity=8.2 -> lower=-2.618 upper=2.618 effort=147 velocity=8.2
- joint j_arm2_4: limit lower=-0.2796 upper=2.4564 effort=147 velocity=8.2 -> lower=-0.349 upper=2.530 effort=147 velocity=8.2
- joint j_arm2_5: limit lower=-2.5626 upper=2.5464 effort=55 velocity=11.6 -> lower=-2.618 upper=2.618 effort=55 velocity=11.6
- joint j_arm2_6: limit lower=-1.4726 upper=1.5364 effort=55 velocity=11.6 -> lower=-1.570 upper=1.570 effort=55 velocity=11.6
- joint j_arm2_7: limit lower=-3.0908 upper=2.0114 effort=27 velocity=20.3 -> lower=-2.618 upper=2.618 effort=27 velocity=20.3
- joint j_arm2_8: limit (none) -> lower=0.0 upper=0 effort=0 velocity=0; origin xyz=0.0 0.0 -0.0405 rpy=0.0 3.14159265359 3.14159265359 -> xyz=0.0 0.0 -0.0405 rpy=0.0 3.14159265359 -1.5707963268
- joint j_wheel_1: axis 0 0 -1 -> 0 0 1; limit effort=35 velocity=20.0 -> lower=-1000000000000000 upper=1000000000000000 effort=35 velocity=20.0; origin xyz=0.0 0.00085 0.23735 rpy=1.57079632679 0.0 3.14159265359 -> xyz=0.0 0.00085 0.235 rpy=1.57079632679 0.0 0.0
- joint j_wheel_2: axis 0 0 -1 -> 0 0 1; limit effort=35 velocity=20.0 -> lower=-1000000000000000 upper=1000000000000000 effort=35 velocity=20.0; origin xyz=0.0 0.00085 0.23735 rpy=1.57079632679 0.0 3.14159265359 -> xyz=0.0 0.00085 0.235 rpy=1.57079632679 0.0 0.0
- joint j_wheel_3: axis 0 0 -1 -> 0 0 1; limit effort=35 velocity=20.0 -> lower=-1000000000000000 upper=1000000000000000 effort=35 velocity=20.0; origin xyz=0.0 0.00085 0.23735 rpy=1.57079632679 0.0 3.14159265359 -> xyz=0.0 0.00085 0.235 rpy=1.57079632679 0.0 0.0
- joint j_wheel_4: axis 0 0 -1 -> 0 0 1; limit effort=35 velocity=20.0 -> lower=-1000000000000000 upper=1000000000000000 effort=35 velocity=20.0; origin xyz=0.0 0.00085 0.23735 rpy=1.57079632679 0.0 3.14159265359 -> xyz=0.0 0.00085 0.235 rpy=1.57079632679 0.0 0.0
- joint knee_pitch_1: limit lower=-2.4056 upper=2.3994 effort=304 velocity=8.8 -> lower=-2.61799388 upper=2.61799388 effort=304 velocity=8.8
- joint knee_pitch_2: limit lower=-2.4006 upper=2.4034 effort=304 velocity=8.8 -> lower=-2.61799388 upper=2.61799388 effort=304 velocity=8.8
- joint knee_pitch_3: limit lower=-2.4056 upper=2.4064 effort=304 velocity=8.8 -> lower=-2.61799388 upper=2.61799388 effort=304 velocity=8.8
- joint knee_pitch_4: limit lower=-2.4176 upper=2.3884 effort=304 velocity=8.8 -> lower=-2.61799388 upper=2.61799388 effort=304 velocity=8.8
- joint neck_velodyne: limit effort=35 velocity=5.7 -> lower=-1000000000000000 upper=1000000000000000 effort=35 velocity=5.7
- joint reference: origin xyz=0.0 0.0 0.93445 -> xyz=0.0 0.0 0.9256; type fixed -> floating
