Commit message: - Updated actuation data for upper-body - Modified ODE solver parameters to stabilize with higher stiffness - Change default end-effector load to 0 - Set default friction coefficients to 0.5

File: centauro/centauro_urdf/urdf/centauro_arm.urdf.xacro (robot description, xacro)
@@ -130,8 +130,8 @@
       <axis xyz="0 ${rot*cos_m10} ${-sin_m10}"/>
       <xacro:unless value="${rot-1}" >
-         <limit lower="-3.403" upper="1.658" effort="1770" velocity="6.5"/>
+         <limit lower="-3.403" upper="1.658" effort="147" velocity="5.7"/>
       </xacro:unless>
       <xacro:unless value="${rot+1}" >
-         <limit lower="-1.658" upper="3.403" effort="1770" velocity="6.5"/>
+         <limit lower="-1.658" upper="3.403" effort="147" velocity="5.7"/>
       </xacro:unless>
    </joint>
@@ -144,8 +144,8 @@
       <axis xyz="-1 0 0"/>
       <xacro:unless value="${rot+1}" >
-         <limit lower="0" upper="3.49" effort="1770" velocity="6.5"/>
+         <limit lower="0" upper="3.49" effort="147" velocity="5.7"/>
       </xacro:unless>
       <xacro:unless value="${rot-1}" >
-         <limit lower="-3.49" upper="0" effort="1770" velocity="6.5"/>
+         <limit lower="-3.49" upper="0" effort="147" velocity="5.7"/>
       </xacro:unless>
    </joint>
@@ -157,5 +157,5 @@
       <origin xyz="${Shoulder_3_Ox} ${Shoulder_3_Oy} ${Shoulder_3_Oz}"/>
       <axis xyz="0 0 -1"/>
-      <limit lower="-2.618" upper="2.618" effort="1770" velocity="6.5"/>
+      <limit lower="-2.618" upper="2.618" effort="147" velocity="8.2"/>
    </joint>
 <!-- /shoulder pitch -->
@@ -167,8 +167,8 @@
       <axis xyz="0 ${rot} 0"/>
       <xacro:unless value="${rot-1}" >
-         <limit lower="-2.530" upper="0.349" effort="1770" velocity="6.5"/>
+         <limit lower="-2.530" upper="0.349" effort="147" velocity="8.2"/>
       </xacro:unless>
       <xacro:unless value="${rot+1}" >
-         <limit lower="-0.349" upper="2.530" effort="1770" velocity="6.5"/>
+         <limit lower="-0.349" upper="2.530" effort="147" velocity="8.2"/>
       </xacro:unless>
    </joint>
@@ -180,5 +180,5 @@
       <origin xyz="${Wrist_1_Ox} ${-rot*Wrist_1_Oy} ${Wrist_1_Oz}"/>
       <axis xyz="0 0 -1"/>
-      <limit lower="-2.618" upper="2.618" effort="950" velocity="6.5"/>
+      <limit lower="-2.618" upper="2.618" effort="55" velocity="11.6"/>
    </joint>
 <!-- /elbow pitch-->
@@ -189,5 +189,5 @@
       <origin xyz="${Wrist_2_Ox} ${rot*Wrist_2_Oy} ${Wrist_2_Oz}"/>
       <axis xyz="0 ${rot} 0"/>
-      <limit lower="-1.570" upper="1.570" effort="950" velocity="6.5"/>
+      <limit lower="-1.570" upper="1.570" effort="55" velocity="11.6"/>
    </joint>
 <!-- /wrist yaw-->
@@ -198,5 +198,5 @@
       <origin xyz="${Wrist_3_Ox} ${-rot*Wrist_3_Oy} ${Wrist_3_Oz}"/>
       <axis xyz="0 0 -1"/>
-      <limit lower="-2.618" upper="2.618" effort="400" velocity="6.5"/>
+      <limit lower="-2.618" upper="2.618" effort="27" velocity="20.3"/>
    </joint>
 <!-- wrist pitch-->

File: centauro/centauro_urdf/urdf/centauro_hand.urdf.xacro (robot description, xacro)
@@ -22,5 +22,5 @@
       <origin xyz="${End_effector_Ox} ${End_effector_Oy} ${End_effector_Oz}" rpy="${End_effector_roll} ${End_effector_pitch} ${End_effector_yaw}"/>
       <axis xyz="1 0 0" />
-      <limit velocity="6.5" effort="400" lower="0.0" upper="1.57075" />
+      <limit velocity="20.3" effort="40" lower="0.0" upper="1.57075" />
    </joint> -->
 <!-- /joints -->

File: centauro/centauro_urdf/urdf/centauro_leg.urdf.xacro (robot description, xacro)
@@ -248,5 +248,5 @@
 	<origin xyz="${origin_x*Leg_1_Ox} ${origin_y*Leg_1_Oy} ${Leg_1_Oz}" rpy="${Leg_1_roll} ${Leg_1_pitch} ${Leg_1_yaw}"/>
 	<axis xyz="0 0 ${-origin_y}"/>
-        <limit lower="-2.09" upper="2.09" effort="1770" velocity="6.5"/> <!-- TODO -->
+        <limit lower="-2.09" upper="2.09" effort="147" velocity="6.5"/> <!-- TODO -->
 </joint>
 <joint name="hip_pitch_${leg_num}" type="revolute">
@@ -255,5 +255,5 @@
 	<origin xyz="${Leg_2_Ox} ${Leg_2_Oy} ${Leg_2_Oz}"/>
 	<axis xyz="0 ${-origin_y} 0"/>
-        <limit lower="-3.14" upper="3.14" effort="3300" velocity="6.5"/> <!-- TODO -->
+        <limit lower="-3.14" upper="3.14" effort="330" velocity="6.5"/> <!-- TODO -->
 </joint>
 <joint name="knee_pitch_${leg_num}" type="revolute">
@@ -262,5 +262,5 @@
 	<origin xyz="${Leg_3_Ox} ${Leg_3_Oy} ${Leg_3_Oz}"/>
 	<axis xyz="0 ${-origin_y} 0"/>
-        <limit  lower="-3.14" upper="3.14" effort="3300" velocity="600.5"/> <!-- TODO -->
+        <limit  lower="-3.14" upper="3.14" effort="330" velocity="6.5"/> <!-- TODO -->
 </joint>
 <!--

File: centauro/centauro_urdf/urdf/centauro_torso.urdf.xacro (robot description, xacro)
@@ -30,5 +30,5 @@
    <child link="torso_2"/>
    <axis xyz="0 0 1"/>
-   <limit lower="-2.618" upper="2.618" effort="1770" velocity="6.5"/> <!-- TODO -->
+   <limit lower="-2.618" upper="2.618" effort="147" velocity="5.7"/> <!-- TODO -->
 </joint>
 <!-- /torso joints -->

Commit message: floating base

File: centauro/centauro_urdf/urdf/centauro_arm.urdf.xacro (robot description, xacro)
@@ -120,8 +120,10 @@
       <axis xyz="0 ${rot*cos_m10} ${-sin_m10}"/>
       <xacro:unless value="${rot-1}" >
-         <limit lower="-3.403" upper="1.658" effort="147" velocity="5.7"/>
+<!--          <limit lower="-3.403" upper="1.658" effort="147" velocity="5.7"/> -->
+         <limit lower="-3.0" upper="3.0" effort="147" velocity="5.7"/>
       </xacro:unless>
       <xacro:unless value="${rot+1}" >
-         <limit lower="-1.658" upper="3.403" effort="147" velocity="5.7"/>
+<!--          <limit lower="-1.658" upper="3.403" effort="147" velocity="5.7"/> -->
+         <limit lower="-3.0" upper="3.0" effort="147" velocity="5.7"/>
       </xacro:unless>
    </joint>
@@ -134,8 +136,10 @@
       <axis xyz="-1 0 0"/>
       <xacro:unless value="${rot+1}" >
-         <limit lower="0" upper="3.49" effort="147" velocity="5.7"/>
+<!--          <limit lower="0" upper="3.49" effort="147" velocity="5.7"/> -->
+         <limit lower="-3.0" upper="3.0" effort="147" velocity="5.7"/>
       </xacro:unless>
       <xacro:unless value="${rot-1}" >
-         <limit lower="-3.49" upper="0" effort="147" velocity="5.7"/>
+<!--          <limit lower="-3.49" upper="0" effort="147" velocity="5.7"/> -->
+         <limit lower="-3.0" upper="3.0" effort="147" velocity="5.7"/>
       </xacro:unless>
    </joint>
@@ -147,5 +151,6 @@
       <origin xyz="${Shoulder_3_Ox} ${Shoulder_3_Oy} ${Shoulder_3_Oz}"/>
       <axis xyz="0 0 -1"/>
-      <limit lower="-2.618" upper="2.618" effort="147" velocity="8.2"/>
+<!--       <limit lower="-2.618" upper="2.618" effort="147" velocity="8.2"/> -->
+         <limit lower="-3.0" upper="3.0" effort="147" velocity="5.7"/>
    </joint>
 <!-- /shoulder pitch -->
@@ -157,8 +162,10 @@
       <axis xyz="0 ${rot} 0"/>
       <xacro:unless value="${rot-1}" >
-         <limit lower="-2.530" upper="0.349" effort="147" velocity="8.2"/>
+<!--          <limit lower="-2.530" upper="0.349" effort="147" velocity="8.2"/> -->
+         <limit lower="-3.0" upper="3.0" effort="147" velocity="5.7"/>
       </xacro:unless>
       <xacro:unless value="${rot+1}" >
-         <limit lower="-0.349" upper="2.530" effort="147" velocity="8.2"/>
+<!--          <limit lower="-0.349" upper="2.530" effort="147" velocity="8.2"/> -->
+         <limit lower="-3.0" upper="3.0" effort="147" velocity="5.7"/>
       </xacro:unless>
    </joint>
@@ -170,5 +177,6 @@
       <origin xyz="${Wrist_1_Ox} ${-rot*Wrist_1_Oy} ${Wrist_1_Oz}"/>
       <axis xyz="0 0 -1"/>
-      <limit lower="-2.618" upper="2.618" effort="55" velocity="11.6"/>
+<!--       <limit lower="-2.618" upper="2.618" effort="55" velocity="11.6"/> -->
+         <limit lower="-3.0" upper="3.0" effort="147" velocity="5.7"/>
    </joint>
 <!-- /elbow pitch-->
@@ -179,5 +187,6 @@
       <origin xyz="${Wrist_2_Ox} ${rot*Wrist_2_Oy} ${Wrist_2_Oz}"/>
       <axis xyz="0 ${rot} 0"/>
-      <limit lower="-1.570" upper="1.570" effort="55" velocity="11.6"/>
+<!--       <limit lower="-1.570" upper="1.570" effort="55" velocity="11.6"/> -->
+         <limit lower="-3.0" upper="3.0" effort="147" velocity="5.7"/>
    </joint>
 <!-- /wrist yaw-->
@@ -188,5 +197,6 @@
       <origin xyz="${Wrist_3_Ox} ${-rot*Wrist_3_Oy} ${Wrist_3_Oz}"/>
       <axis xyz="0 0 -1"/>
-      <limit lower="-2.618" upper="2.618" effort="27" velocity="20.3"/>
+<!--       <limit lower="-2.618" upper="2.618" effort="27" velocity="20.3"/> -->
+         <limit lower="-3.0" upper="3.0" effort="147" velocity="5.7"/>
    </joint>
 <!-- wrist pitch-->
@@ -210,5 +220,11 @@
   <xacro:include filename="$(find centauro)/centauro_urdf/urdf/centauro_stick.urdf.xacro" />
 </xacro:if>
-<xacro:if value="${END_EFFECTOR != 'stick' and END_EFFECTOR != 'soft_hand' }" >
+<xacro:if value="${END_EFFECTOR == 'stick_ball'}">
+   <xacro:include filename="$(find centauro)/centauro_urdf/urdf/centauro_stick_ball.urdf.xacro"/>
+</xacro:if>
+<xacro:if value="${END_EFFECTOR == 'narrow_feet'}">
+  <xacro:include filename="$(find centauro)/centauro_urdf/urdf/centauro_narrow_feet.urdf.xacro"/>
+</xacro:if>
+<xacro:if value="${END_EFFECTOR != 'stick' and END_EFFECTOR != 'soft_hand' and END_EFFECTOR != 'stick_ball' and  END_EFFECTOR != 'narrow_feet'}">
   <xacro:include filename="$(find centauro)/centauro_urdf/urdf/centauro_no_end_effector.urdf.xacro" />
 </xacro:if>

Commit message: change joint angle limits

File: centauro/centauro_urdf/urdf/centauro_arm.urdf.xacro (robot description, xacro)
@@ -120,10 +120,10 @@
       <axis xyz="0 ${rot*cos_m10} ${-sin_m10}"/>
       <xacro:unless value="${rot-1}" >
-<!--          <limit lower="-3.403" upper="1.658" effort="147" velocity="5.7"/> -->
-         <limit lower="-3.0" upper="3.0" effort="147" velocity="5.7"/>
+         <limit lower="-3.403" upper="1.658" effort="147" velocity="5.7"/>
+<!--          <limit lower="-3.0" upper="3.0" effort="147" velocity="5.7"/> -->
       </xacro:unless>
       <xacro:unless value="${rot+1}" >
-<!--          <limit lower="-1.658" upper="3.403" effort="147" velocity="5.7"/> -->
-         <limit lower="-3.0" upper="3.0" effort="147" velocity="5.7"/>
+         <limit lower="-1.658" upper="3.403" effort="147" velocity="5.7"/>
+<!--          <limit lower="-3.0" upper="3.0" effort="147" velocity="5.7"/> -->
       </xacro:unless>
    </joint>
@@ -151,6 +151,6 @@
       <origin xyz="${Shoulder_3_Ox} ${Shoulder_3_Oy} ${Shoulder_3_Oz}"/>
       <axis xyz="0 0 -1"/>
-<!--       <limit lower="-2.618" upper="2.618" effort="147" velocity="8.2"/> -->
-         <limit lower="-3.0" upper="3.0" effort="147" velocity="5.7"/>
+      <limit lower="-2.618" upper="2.618" effort="147" velocity="8.2"/>
+<!--          <limit lower="-3.0" upper="3.0" effort="147" velocity="5.7"/> -->
    </joint>
 <!-- /shoulder pitch -->
@@ -177,6 +177,6 @@
       <origin xyz="${Wrist_1_Ox} ${-rot*Wrist_1_Oy} ${Wrist_1_Oz}"/>
       <axis xyz="0 0 -1"/>
-<!--       <limit lower="-2.618" upper="2.618" effort="55" velocity="11.6"/> -->
-         <limit lower="-3.0" upper="3.0" effort="147" velocity="5.7"/>
+      <limit lower="-2.618" upper="2.618" effort="55" velocity="11.6"/>
+<!--          <limit lower="-3.0" upper="3.0" effort="147" velocity="5.7"/> -->
    </joint>
 <!-- /elbow pitch-->
@@ -187,6 +187,6 @@
       <origin xyz="${Wrist_2_Ox} ${rot*Wrist_2_Oy} ${Wrist_2_Oz}"/>
       <axis xyz="0 ${rot} 0"/>
-<!--       <limit lower="-1.570" upper="1.570" effort="55" velocity="11.6"/> -->
-         <limit lower="-3.0" upper="3.0" effort="147" velocity="5.7"/>
+      <limit lower="-1.570" upper="1.570" effort="55" velocity="11.6"/>
+<!--          <limit lower="-3.0" upper="3.0" effort="147" velocity="5.7"/> -->
    </joint>
 <!-- /wrist yaw-->
@@ -197,6 +197,6 @@
       <origin xyz="${Wrist_3_Ox} ${-rot*Wrist_3_Oy} ${Wrist_3_Oz}"/>
       <axis xyz="0 0 -1"/>
-<!--       <limit lower="-2.618" upper="2.618" effort="27" velocity="20.3"/> -->
-         <limit lower="-3.0" upper="3.0" effort="147" velocity="5.7"/>
+      <limit lower="-2.618" upper="2.618" effort="27" velocity="20.3"/>
+<!--          <limit lower="-3.0" upper="3.0" effort="147" velocity="5.7"/> -->
    </joint>
 <!-- wrist pitch-->

File: centauro/centauro_urdf/urdf/centauro_narrow_feet.urdf.xacro (robot description, xacro)
@@ -5,6 +5,6 @@
         <visual>
             <geometry>
-                <box size="0.4 0.02 0.1"/>
-                <!--box size="0.3 0.1 0.02"/-->
+                <!--box size="0.4 0.02 0.1"/-->
+                <box size="0.3 0.1 0.02"/>
                 <!--cylinder length="0.3" radius="0.02"/-->
             </geometry>
@@ -12,6 +12,6 @@
         <collision>
             <geometry>
-                <box size="0.4 0.02 0.1"/>
-                <!--box size="0.3 0.1 0.02"/-->
+                <!--box size="0.4 0.02 0.1"/-->
+                <box size="0.3 0.1 0.02"/>
                 <!--cylinder length="0.3" radius="0.02"/-->
             </geometry>

Commit message: use the dimension and inertia parameters of real aluminum parts

File: centauro/centauro_urdf/urdf/centauro_arm.urdf.xacro (robot description, xacro)
@@ -136,10 +136,10 @@
       <axis xyz="-1 0 0"/>
       <xacro:unless value="${rot+1}" >
-<!--          <limit lower="0" upper="3.49" effort="147" velocity="5.7"/> -->
-         <limit lower="-3.0" upper="3.0" effort="147" velocity="5.7"/>
+         <limit lower="0" upper="3.49" effort="147" velocity="5.7"/>
+<!--          <limit lower="-3.0" upper="3.0" effort="147" velocity="5.7"/> -->
       </xacro:unless>
       <xacro:unless value="${rot-1}" >
-<!--          <limit lower="-3.49" upper="0" effort="147" velocity="5.7"/> -->
-         <limit lower="-3.0" upper="3.0" effort="147" velocity="5.7"/>
+         <limit lower="-3.49" upper="0" effort="147" velocity="5.7"/>
+<!--          <limit lower="-3.0" upper="3.0" effort="147" velocity="5.7"/> -->
       </xacro:unless>
    </joint>
@@ -162,10 +162,10 @@
       <axis xyz="0 ${rot} 0"/>
       <xacro:unless value="${rot-1}" >
-<!--          <limit lower="-2.530" upper="0.349" effort="147" velocity="8.2"/> -->
-         <limit lower="-3.0" upper="3.0" effort="147" velocity="5.7"/>
+         <limit lower="-2.530" upper="0.349" effort="147" velocity="8.2"/>
+<!--          <limit lower="-3.0" upper="3.0" effort="147" velocity="5.7"/> -->
       </xacro:unless>
       <xacro:unless value="${rot+1}" >
-<!--          <limit lower="-0.349" upper="2.530" effort="147" velocity="8.2"/> -->
-         <limit lower="-3.0" upper="3.0" effort="147" velocity="5.7"/>
+         <limit lower="-0.349" upper="2.530" effort="147" velocity="8.2"/>
+<!--          <limit lower="-3.0" upper="3.0" effort="147" velocity="5.7"/> -->
       </xacro:unless>
    </joint>

File: centauro/centauro_urdf/urdf/centauro_narrow_feet.urdf.xacro (robot description, xacro)
@@ -6,5 +6,5 @@
             <geometry>
                 <!--box size="0.4 0.02 0.1"/-->
-                <box size="0.4 0.06 0.02"/>
+                <box size="0.4 0.03 0.03"/>
                 <!--cylinder length="0.3" radius="0.02"/-->
             </geometry>
@@ -13,19 +13,20 @@
             <geometry>
                 <!--box size="0.4 0.02 0.1"/-->
-                <box size="0.4 0.06 0.02"/>
+                <box size="0.4 0.03 0.03"/>
                 <!--cylinder length="0.3" radius="0.02"/-->
             </geometry>
         </collision>
         <inertial>
-            <mass value="0.01"/>
-            <inertia ixx="0.001" ixy="0.0" ixz="0.0" iyy="0.001" iyz="0.0" izz="0.001"/>
+            <mass value="0.34"/>
+	    <!--origin xyz="0 0 0" rpy="0 0 0"/-->
+            <inertia ixx="5.97e-5" ixy="0.0" ixz="0.0" iyy="4.55e-3" iyz="0.0" izz="4.55e-3"/>
         </inertial>
     </link>
     <!-- /links -->
-    <!--xacro:if value="${arm_num == 1}">
+    <xacro:if value="${arm_num == 1}">
         <joint name="j_arm${arm_num}_8" type="fixed">
             <parent link="arm${arm_num}_7"/>
             <child link="arm${arm_num}_8"/>
-            <origin xyz="0 0 -0.05" rpy="0 0 0.0"/>
+            <origin xyz="0 0 -0.05" rpy="0 0 0.5"/>
         </joint>
     </xacro:if>
@@ -34,14 +35,14 @@
             <parent link="arm${arm_num}_7"/>
             <child link="arm${arm_num}_8"/>
-            <origin xyz="0 0 -0.05" rpy="0 0 -0.0"/>
+            <origin xyz="0 0 -0.05" rpy="0 0 -0.5"/>
         </joint>
-    </xacro:if-->
+    </xacro:if>
     <!--origin xyz="0 0 -0.0605" rpy="0 1.5707 0.5"/-->
     <!--origin xyz="0 0 -0.0605" rpy="0 1.5707 -0.5"/-->
     <!-- /joints -->
-        <joint name="j_arm${arm_num}_8" type="fixed">
+        <!--joint name="j_arm${arm_num}_8" type="fixed">
             <parent link="arm${arm_num}_7"/>
             <child link="arm${arm_num}_8"/>
-            <origin xyz="0 0 -0.08" rpy="0 0 0"/>
-        </joint>
+            <origin xyz="0 0 -0.05" rpy="0 0 0"/>
+        </joint-->
 </robot>
