Commit message: urdf: added joint friction

File: centauro/centauro_urdf/urdf/centauro_arm.urdf.xacro (robot description, xacro)
@@ -125,4 +125,5 @@
          <limit lower="-1.658" upper="3.403" effort="147" velocity="5.7"/>
       </xacro:unless>
+      <dynamics friction="${friction}" />
    </joint>
 <!-- /shoulder yaw -->
@@ -139,4 +140,5 @@
          <limit lower="-3.49" upper="0" effort="147" velocity="5.7"/>
       </xacro:unless>
+      <dynamics friction="${friction}" />
    </joint>
 <!-- /shoulder roll -->
@@ -148,4 +150,5 @@
       <axis xyz="0 0 -1"/>
       <limit lower="-2.618" upper="2.618" effort="147" velocity="8.2"/>
+      <dynamics friction="${friction}" />
    </joint>
 <!-- /shoulder pitch -->
@@ -162,4 +165,5 @@
          <limit lower="-0.349" upper="2.530" effort="147" velocity="8.2"/>
       </xacro:unless>
+      <dynamics friction="${friction}" />
    </joint>
 <!-- /elbow yaw -->
@@ -171,4 +175,5 @@
       <axis xyz="0 0 -1"/>
       <limit lower="-2.618" upper="2.618" effort="55" velocity="11.6"/>
+      <dynamics friction="${friction}" />
    </joint>
 <!-- /elbow pitch-->
@@ -180,4 +185,5 @@
       <axis xyz="0 ${rot} 0"/>
       <limit lower="-1.570" upper="1.570" effort="55" velocity="11.6"/>
+      <dynamics friction="${friction}" />
    </joint>
 <!-- /wrist yaw-->
@@ -189,4 +195,5 @@
       <axis xyz="0 0 -1"/>
       <limit lower="-2.618" upper="2.618" effort="27" velocity="20.3"/>
+      <dynamics friction="${friction}" />
    </joint>
 <!-- wrist pitch-->
@@ -206,9 +213,8 @@
 <xacro:if value="${ft_sensors == 'true'}" >
 <!-- wrist pitch-->
-   <joint name="j_ft_${arm_num}" type="revolute">
+   <joint name="j_ft_${arm_num}" type="fixed">
       <parent link="arm${arm_num}_7"/>
       <child link="ft_arm${arm_num}"/>
       <origin xyz="${Ft_arm_Ox} ${Ft_arm_Oy} ${Ft_arm_Oz}" rpy="${Ft_arm_roll} ${Ft_arm_pitch} ${Ft_arm_yaw}" />
-      <axis xyz="0 0 1"/>
       <limit lower="0.0" upper="0.0" effort="0" velocity="0"/>
    </joint>
@@ -221,7 +227,7 @@
       </inertial>
    </link>
-   <xacro:if value="${arm_actuators}">
+<!--   <xacro:if value="${arm_actuators}">
       <xacro:position_actuator joint="j_ft_${arm_num}" />
-   </xacro:if>
+   </xacro:if>-->
 </xacro:if>
 <xacro:if value="${end_effector == 'soft_hand'}" >

File: centauro/centauro_urdf/urdf/centauro_head.urdf.xacro (robot description, xacro)
@@ -86,4 +86,5 @@
    <axis xyz="0 0 1"/>
    <limit lower="-0.78539816" upper="0.78539816" effort="35" velocity="5.7"/> <!-- TODO -->
+   <dynamics friction="${friction}" />
 </joint>
 <joint name="neck_pitch" type="revolute">
@@ -93,4 +94,5 @@
    <axis xyz="0 1 0"/>
    <limit lower="-0.34906585" upper="0.78539816" effort="35" velocity="5.7"/> <!-- TODO -->
+   <dynamics friction="${friction}" />
 </joint>
 <joint name="neck_velodyne" type="continuous">
@@ -100,4 +102,5 @@
    <axis xyz="0 0 1"/>
    <limit effort="35" velocity="5.7"/> <!-- TODO -->
+   <dynamics friction="${friction}" />
 </joint>
 <!-- /head joints -->

File: centauro/centauro_urdf/urdf/centauro_leg.urdf.xacro (robot description, xacro)
@@ -100,4 +100,5 @@
         <limit lower="-2.70526034" upper="1.13446401" effort="304" velocity="8.8"/>
         </xacro:if>
+	<dynamics friction="${friction}" />
 </joint>
 <joint name="hip_pitch_${leg_num}" type="revolute">
@@ -107,4 +108,5 @@
 	<axis xyz="0 0 1"/>
         <limit lower="-2.09439510" upper="2.09439510" effort="304" velocity="8.8"/>
+	<dynamics friction="${friction}" />
 </joint>
 <joint name="knee_pitch_${leg_num}" type="revolute">
@@ -114,4 +116,5 @@
 	<axis xyz="0 0 1"/>
         <limit  lower="-2.61799388" upper="2.61799388" effort="304" velocity="8.8"/>
+	<dynamics friction="${friction}" />
 </joint>
 <joint name="ankle_pitch_${leg_num}" type="revolute">
@@ -121,4 +124,5 @@
 	<axis xyz="0 0 1"/>
         <limit  lower="-2.61799388" upper="2.61799388" effort="147" velocity="8.1"/>
+	<dynamics friction="${friction}" />
 </joint>
 <joint name="ankle_yaw_${leg_num}" type="revolute">
@@ -128,4 +132,5 @@
 	<axis xyz="0 0 1"/>
         <limit  lower="-2.79252680" upper="2.79252680" effort="35" velocity="20.0"/>
+	<dynamics friction="${friction}" />
 </joint>
 <joint name="j_wheel_${leg_num}" type="continuous">
@@ -135,4 +140,5 @@
 	<axis xyz="0 0 -1"/>
         <limit  effort="35" velocity="20.0"/>
+	<dynamics friction="${friction}" />
 </joint>
 <!--

File: centauro/centauro_urdf/urdf/config.xacro (robot description, xacro)
@@ -59,3 +59,5 @@
 <xacro:property name="kinematic_parameters_file" value="${package + '/centauro_urdf/kinematic_parameters/' + KINEMATIC_PARAM + '.xacro'}"/>
 <xacro:property name="middleware" value="${MIDDLEWARE}"/>
+<xacro:property name="friction" value="10.0" />
+<xacro:property name="friction_schunk" value="3.0" />
 </robot>

File: centauro/centauro_urdf/urdf/models/upper_body/end_effectors/schunk_hand/svh_gazebo.urdf.xacro (robot description, xacro)
@@ -539,7 +539,8 @@
             <parent link="${name}_virtual_a" />
             <child link="${name}_a" />
-            <limit effort="1000.0" lower="0.0" upper="0.9704" velocity="1" />
+            <limit effort="10.0" lower="0.0" upper="0.9704" velocity="1" />
             <origin xyz="0 0 0" rpy="0 0 ${side*(-0.9704)}" />
             <axis xyz="0 0 ${side*(1)}" />
+            <dynamics friction="${friction_schunk}" />
         </joint>
         <xacro:trans_xacro namehand="${name}" jointname="Thumb_Flexion"/>
@@ -564,7 +565,8 @@
             <parent link="${name}_e1" />
             <child link="${name}_z" />
-            <limit effort="1000.0" lower="0.0" upper="0.9879" velocity="1" />
+            <limit effort="10.0" lower="0.0" upper="0.9879" velocity="1" />
             <origin xyz="${side*(-0.01690)} 0.02626 0" rpy="0 0.2618 1.571" />
             <axis xyz="0 0 ${side*(-1)}" />
+            <dynamics friction="${friction_schunk}" />
         </joint>
         <xacro:trans_xacro namehand="${name}" jointname="Thumb_Opposition"/>
@@ -597,8 +599,9 @@
             <parent link="${name}_e1" />
             <child link="${name}_e2" />
-            <limit effort="1000.0" lower="0.0" upper="0.98786" velocity="1" />
+            <limit effort="10.0" lower="0.0" upper="0.98786" velocity="1" />
             <origin xyz="${side*(0.01840)} 0.006 0.0375" rpy="0 0 0" />
             <axis xyz="0 0 ${side*(1)}" />
             <mimic joint="${name}_Thumb_Opposition" multiplier="1" offset="0" />
+            <dynamics friction="${friction_schunk}" />
         </joint>
         <xacro:trans_xacro namehand="${name}" jointname="j5"/>
@@ -631,8 +634,9 @@
             <parent link="${name}_a" />
             <child link="${name}_b" />
-            <limit effort="1000.0" lower="0.0" upper="0.98506" velocity="1" />
+            <limit effort="10.0" lower="0.0" upper="0.98506" velocity="1" />
             <origin xyz="0.0485 0 0" rpy="0 0 0" />
             <axis xyz="0 0 ${side*(1)}" />
             <mimic joint="${name}_Thumb_Flexion" multiplier="1.01511" offset="0" />
+            <dynamics friction="${friction_schunk}" />
         </joint>
         <xacro:trans_xacro namehand="${name}" jointname="j3"/>
@@ -640,8 +644,9 @@
             <parent link="${name}_b" />
             <child link="${name}_c" />
-            <limit effort="1000.0" lower="0.0" upper="1.406" velocity="1" />
+            <limit effort="10.0" lower="0.0" upper="1.406" velocity="1" />
             <origin xyz="0.030 0 0" rpy="0 0 0" />
             <axis xyz="0 0 ${side*(1)}" />
             <mimic joint="${name}_Thumb_Flexion" multiplier="1.44889" offset="0" />
+            <dynamics friction="${friction_schunk}" />
         </joint>
         <xacro:trans_xacro namehand="${name}" jointname="j4"/>
@@ -650,7 +655,8 @@
             <parent link="${name}_l" />
             <child link="${name}_p" />
-            <limit effort="1000.0" lower="0" upper="1.334" velocity="1" />
+            <limit effort="10.0" lower="0" upper="1.334" velocity="1" />
             <origin xyz="0.04804 0 0" rpy="0 0 0" />
             <axis xyz="0 0 1" />
+            <dynamics friction="${friction_schunk}" />
         </joint>
         <xacro:trans_xacro namehand="${name}" jointname="Index_Finger_Distal"/>
@@ -658,7 +664,8 @@
             <parent link="${name}_virtual_l" />
             <child link="${name}_l" />
-            <limit effort="1000.0" lower="0.0" upper="0.79849" velocity="1" />
+            <limit effort="10.0" lower="0.0" upper="0.79849" velocity="1" />
             <origin xyz="0 0 0" rpy="-1.5707 0 0" />
             <axis xyz="0 0 1" />
+            <dynamics friction="${friction_schunk}" />
         </joint>
         <xacro:trans_xacro namehand="${name}" jointname="Index_Finger_Proximal"/>
@@ -667,8 +674,9 @@
             <parent link="${name}_p" />
             <child link="${name}_t" />
-            <limit effort="1000.0" lower="0" upper="1.394" velocity="1" />
+            <limit effort="10.0" lower="0" upper="1.394" velocity="1" />
             <origin xyz="0.026 0 0" rpy="0 0 0" />
             <axis xyz="0 0 1" />
             <mimic joint="${name}_Index_Finger_Distal" multiplier="1.0450" offset="0" />
+            <dynamics friction="${friction_schunk}" />
         </joint>
         <xacro:trans_xacro namehand="${name}" jointname="j14"/>
@@ -677,7 +685,8 @@
             <parent link="${name}_virtual_k" />
             <child link="${name}_k" />
-            <limit effort="1000.0" lower="0.0" upper="0.79849" velocity="1" />
+            <limit effort="10.0" lower="0.0" upper="0.79849" velocity="1" />
             <origin xyz="0 0 0" rpy="-1.5707 0 0" />
             <axis xyz="0 0 1" />
+            <dynamics friction="${friction_schunk}" />
         </joint>
         <xacro:trans_xacro namehand="${name}" jointname="Middle_Finger_Proximal"/>
@@ -685,7 +694,8 @@
             <parent link="${name}_k" />
             <child link="${name}_o" />
-            <limit effort="1000.0" lower="0" upper="1.334" velocity="1" />
+            <limit effort="10.0" lower="0" upper="1.334" velocity="1" />
             <origin xyz="0.05004 0 0" rpy="0 0 0" />
             <axis xyz="0 0 1" />
+            <dynamics friction="${friction_schunk}" />
         </joint>
         <xacro:trans_xacro namehand="${name}" jointname="Middle_Finger_Distal"/>
@@ -693,8 +703,9 @@
             <parent link="${name}_o" />
             <child link="${name}_s" />
-            <limit effort="1000.0" lower="0" upper="1.334" velocity="1" />
+            <limit effort="10.0" lower="0" upper="1.334" velocity="1" />
             <origin xyz="0.032 0 0" rpy="0 0 0" />
             <axis xyz="0 0 1" />
             <mimic joint="${name}_Middle_Finger_Distal" multiplier="1.0454" offset="0" />
+            <dynamics friction="${friction_schunk}" />
         </joint>
         <xacro:trans_xacro namehand="${name}" jointname="j15"/>
@@ -703,7 +714,8 @@
             <parent link="${name}_virtual_j" />
             <child link="${name}_j" />
-            <limit effort="1000.0" lower="0.0" upper="0.98175" velocity="1" />
+            <limit effort="10.0" lower="0.0" upper="0.98175" velocity="1" />
             <origin xyz="0 0 0" rpy="1.5707 0 0" />
             <axis xyz="0 0 1" />
+            <dynamics friction="${friction_schunk}" />
         </joint>
         <xacro:trans_xacro namehand="${name}" jointname="Ring_Finger"/>
@@ -711,8 +723,9 @@
             <parent link="${name}_j" />
             <child link="${name}_n" />
-            <limit effort="1000.0" lower="0" upper="1.334" velocity="1" />
+            <limit effort="10.0" lower="0" upper="1.334" velocity="1" />
             <origin xyz="0.05004 0 0" rpy="0 0 0" />
             <axis xyz="0 0 1" />
             <mimic joint="${name}_Ring_Finger" multiplier="1.3588" offset="0" />
+            <dynamics friction="${friction_schunk}" />
         </joint>
         <xacro:trans_xacro namehand="${name}" jointname="j12"/>
@@ -720,8 +733,9 @@
             <parent link="${name}_n" />
             <child link="${name}_r" />
-            <limit effort="1000.0" lower="0" upper="1.395" velocity="1" />
+            <limit effort="10.0" lower="0" upper="1.395" velocity="1" />
             <origin xyz="0.032 0 0" rpy="0 0 0" />
             <axis xyz="0 0 1" />
             <mimic joint="${name}_Ring_Finger" multiplier="1.42093" offset="0" />
+            <dynamics friction="${friction_schunk}" />
         </joint>
         <xacro:trans_xacro namehand="${name}" jointname="j16"/>
@@ -730,7 +744,8 @@
             <parent link="${name}_virtual_i" />
             <child link="${name}_i" />
-            <limit effort="1000.0" lower="0.0" upper="0.98175" velocity="1" />
+            <limit effort="10.0" lower="0.0" upper="0.98175" velocity="1" />
             <origin xyz="0 0 0" rpy="1.5707 0 0" />
             <axis xyz="0 0 1" />
+            <dynamics friction="${friction_schunk}" />
         </joint>
         <xacro:trans_xacro namehand="${name}" jointname="Pinky"/>
@@ -738,8 +753,9 @@
             <parent link="${name}_i" />
             <child link="${name}_m" />
-            <limit effort="1000.0" lower="0" upper="1.334" velocity="1" />
+            <limit effort="10.0" lower="0" upper="1.334" velocity="1" />
             <origin xyz="0.04454 0 0" rpy="0 0 0" />
             <axis xyz="0 0 1" />
             <mimic joint="${name}_Pinky" multiplier="1.35880" offset="0" />
+            <dynamics friction="${friction_schunk}" />
         </joint>
         <xacro:trans_xacro namehand="${name}" jointname="j13"/>
@@ -747,8 +763,9 @@
             <parent link="${name}_m" />
             <child link="${name}_q" />
-            <limit effort="1000.0" lower="0" upper="1.3971" velocity="1" />
+            <limit effort="10.0" lower="0" upper="1.3971" velocity="1" />
             <origin xyz="0.022 0 0" rpy="0 0 0" />
             <axis xyz="0 0 1" />
             <mimic joint="${name}_Pinky" multiplier="1.42307" offset="0" />
+            <dynamics friction="${friction_schunk}" />
         </joint>
         <xacro:trans_xacro namehand="${name}" jointname="j17"/>
@@ -756,8 +773,9 @@
             <parent link="${name}_d2" />
             <child link="${name}_virtual_l" />
-            <limit effort="1000.0" lower="0.0" upper="0.28833" velocity="1" />
+            <limit effort="10.0" lower="0.0" upper="0.28833" velocity="1" />
             <origin xyz="${side*(-0.025)} 0 0.110" rpy="0 -1.5707 1.5707" />
             <axis xyz="0 0 ${side*(1)}" />
             <mimic joint="${name}_Finger_Spread" multiplier="0.5" offset="0" />
+            <dynamics friction="${friction_schunk}" />
         </joint>
         <xacro:trans_xacro namehand="${name}" jointname="index_spread"/>
@@ -771,8 +789,9 @@
             <parent link="${name}_e5" />
             <child link="${name}_virtual_j" />
-            <limit effort="1000.0" lower="0.0" upper="0.28833" velocity="1" />
+            <limit effort="10.0" lower="0.0" upper="0.28833" velocity="1" />
             <origin xyz="${side*(0.003855)} 0 0.0655" rpy="-1.5707 -1.5707 0" />
             <axis xyz="0 0 ${side*(1)}" />
             <mimic joint="${name}_Finger_Spread" multiplier="0.5" offset="0" />
+            <dynamics friction="${friction_schunk}" />
         </joint>
         <xacro:trans_xacro namehand="${name}" jointname="ring_spread"/>
@@ -780,7 +799,8 @@
             <parent link="${name}_e4" />
             <child link="${name}_virtual_i" />
-            <limit effort="1000.0" lower="0.00" upper="0.5829" velocity="1" />
+            <limit effort="10.0" lower="0.00" upper="0.5829" velocity="1" />
             <origin xyz="${side*(0.025355)} 0 0.056" rpy="-1.5707 -1.5707 0" />
             <axis xyz="0 0 ${side*(1)}" />
+            <dynamics friction="${friction_schunk}" />
         </joint>
         <xacro:trans_xacro namehand="${name}" jointname="Finger_Spread"/>

Commit message: centauro_urdf: ft sensor is a fixed joint

File: centauro/centauro_urdf/urdf/centauro_arm.urdf.xacro (robot description, xacro)
@@ -212,12 +212,9 @@
 <!-- end-effector -->
 <xacro:if value="${ft_sensors == 'true'}" >
-<!-- wrist pitch-->
    <joint name="j_ft_${arm_num}" type="fixed">
       <parent link="arm${arm_num}_7"/>
       <child link="ft_arm${arm_num}"/>
       <origin xyz="${Ft_arm_Ox} ${Ft_arm_Oy} ${Ft_arm_Oz}" rpy="${Ft_arm_roll} ${Ft_arm_pitch} ${Ft_arm_yaw}" />
-      <limit lower="0.0" upper="0.0" effort="0" velocity="0"/>
-   </joint>
-<!-- wrist pitch-->
+   </joint>
    <link name="ft_arm${arm_num}">
       <inertial>
@@ -227,7 +224,4 @@
       </inertial>
    </link>
-<!--   <xacro:if value="${arm_actuators}">
-      <xacro:position_actuator joint="j_ft_${arm_num}" />
-   </xacro:if>-->
 </xacro:if>
 <xacro:if value="${end_effector == 'soft_hand'}" >
