Commit message: centauro_urdf: add friction & damping to joints

File: centauro/centauro_urdf/urdf/centauro_arm.urdf.xacro (robot description, xacro)
@@ -125,5 +125,5 @@
          <limit lower="-1.658" upper="3.403" effort="147" velocity="5.7"/>
       </xacro:unless>
-      <dynamics friction="${friction}" />
+      <dynamics friction="${friction}" damping="${damping_arms}" />
    </joint>
 <!-- /shoulder yaw -->
@@ -140,5 +140,5 @@
          <limit lower="-3.49" upper="0" effort="147" velocity="5.7"/>
       </xacro:unless>
-      <dynamics friction="${friction}" />
+      <dynamics friction="${friction}" damping="${damping_arms}" />
    </joint>
 <!-- /shoulder roll -->
@@ -150,5 +150,5 @@
       <axis xyz="0 0 -1"/>
       <limit lower="-2.618" upper="2.618" effort="147" velocity="8.2"/>
-      <dynamics friction="${friction}" />
+      <dynamics friction="${friction}" damping="${damping_arms}" />
    </joint>
 <!-- /shoulder pitch -->
@@ -165,5 +165,5 @@
          <limit lower="-0.349" upper="2.530" effort="147" velocity="8.2"/>
       </xacro:unless>
-      <dynamics friction="${friction}" />
+      <dynamics friction="${friction}" damping="${damping_arms}" />
    </joint>
 <!-- /elbow yaw -->
@@ -175,5 +175,5 @@
       <axis xyz="0 0 -1"/>
       <limit lower="-2.618" upper="2.618" effort="55" velocity="11.6"/>
-      <dynamics friction="${friction}" />
+      <dynamics friction="${friction}" damping="${damping_arms}" />
    </joint>
 <!-- /elbow pitch-->
@@ -185,5 +185,5 @@
       <axis xyz="0 ${rot} 0"/>
       <limit lower="-1.570" upper="1.570" effort="55" velocity="11.6"/>
-      <dynamics friction="${friction}" />
+      <dynamics friction="${friction}" damping="${damping_arms}" />
    </joint>
 <!-- /wrist yaw-->
@@ -195,5 +195,5 @@
       <axis xyz="0 0 -1"/>
       <limit lower="-2.618" upper="2.618" effort="27" velocity="20.3"/>
-      <dynamics friction="${friction}" />
+      <dynamics friction="${friction}" damping="${0.0*damping_arms}" />
    </joint>
 <!-- wrist pitch-->

File: centauro/centauro_urdf/urdf/centauro_head.urdf.xacro (robot description, xacro)
@@ -102,5 +102,5 @@
    <axis xyz="0 0 1"/>
    <limit effort="35" velocity="5.7"/> <!-- TODO -->
-   <dynamics friction="${friction}" />
+   <dynamics friction="${friction}" damping="${damping_arms}" />
 </joint>
 <!-- /head joints -->

File: centauro/centauro_urdf/urdf/centauro_leg.urdf.xacro (robot description, xacro)
@@ -100,5 +100,5 @@
         <limit lower="-2.70526034" upper="1.13446401" effort="304" velocity="8.8"/>
         </xacro:if>
-	<dynamics friction="${friction}" />
+	<dynamics friction="${friction}" damping="${damping_legs}" />
 </joint>
 <joint name="hip_pitch_${leg_num}" type="revolute">
@@ -108,5 +108,5 @@
 	<axis xyz="0 0 1"/>
         <limit lower="-2.09439510" upper="2.09439510" effort="304" velocity="8.8"/>
-	<dynamics friction="${friction}" />
+	<dynamics friction="${friction}" damping="${damping_legs}" />
 </joint>
 <joint name="knee_pitch_${leg_num}" type="revolute">
@@ -116,5 +116,5 @@
 	<axis xyz="0 0 1"/>
         <limit  lower="-2.61799388" upper="2.61799388" effort="304" velocity="8.8"/>
-	<dynamics friction="${friction}" />
+	<dynamics friction="${friction}" damping="${damping_legs}" />
 </joint>
 <joint name="ankle_pitch_${leg_num}" type="revolute">
@@ -124,5 +124,5 @@
 	<axis xyz="0 0 1"/>
         <limit  lower="-2.61799388" upper="2.61799388" effort="147" velocity="8.1"/>
-	<dynamics friction="${friction}" />
+	<dynamics friction="${friction}" damping="${damping_legs}" />
 </joint>
 <joint name="ankle_yaw_${leg_num}" type="revolute">
@@ -132,5 +132,5 @@
 	<axis xyz="0 0 1"/>
         <limit  lower="-2.79252680" upper="2.79252680" effort="35" velocity="20.0"/>
-	<dynamics friction="${friction}" />
+	<dynamics friction="${friction}" damping="${damping_legs}" />
 </joint>
 <joint name="j_wheel_${leg_num}" type="continuous">
@@ -140,5 +140,5 @@
 	<axis xyz="0 0 -1"/>
         <limit  effort="35" velocity="20.0"/>
-	<dynamics friction="${friction}" />
+	<dynamics friction="${friction}" damping="${damping_legs}" />
 </joint>
 <!--

File: centauro/centauro_urdf/urdf/config.xacro (robot description, xacro)
@@ -60,4 +60,7 @@
 <xacro:property name="middleware" value="${MIDDLEWARE}"/>
 <xacro:property name="friction" value="10.0" />
-<xacro:property name="friction_schunk" value="3.0" />
+<xacro:property name="damping_legs" value="1.0" />
+<xacro:property name="damping_arms" value="0.2" />
+<xacro:property name="friction_schunk" value="1.0" />
+<xacro:property name="damping_schunk" value="0.0" />
 </robot>

File: centauro/centauro_urdf/urdf/models/upper_body/end_effectors/schunk_hand/svh_gazebo.urdf.xacro (robot description, xacro)
@@ -12,11 +12,29 @@
         </inertial>
     </xacro:macro>
+	<xacro:macro name="cylinder_inertial_y" params="radius length mass *origin">
+        <inertial>
+            <mass value="${mass}" />
+            <xacro:insert_block name="origin" />
+            <inertia ixx="${0.0833333 * mass * (3 * radius * radius + length * length)}" ixy="0.0" ixz="0.0"
+                iyy="${0.5 * mass * radius * radius}" iyz="0.0"
+                izz="${0.0833333 * mass * (3 * radius * radius + length * length)}" />
+        </inertial>
+    </xacro:macro>
+	<xacro:macro name="cylinder_inertial_x" params="radius length mass *origin">
+        <inertial>
+            <mass value="${mass}" />
+            <xacro:insert_block name="origin" />
+            <inertia ixx="${0.5 * mass * radius * radius}" ixy="0.0" ixz="0.0"
+                iyy="${0.0833333 * mass * (3 * radius * radius + length * length)}" iyz="0.0"
+                izz="${0.0833333 * mass * (3 * radius * radius + length * length)}" />
+        </inertial>
+    </xacro:macro>
     <xacro:macro name="dummy_inertial">
-        <inertial>
-            <mass value="0.03" />
-            <inertia ixx="0.00001" ixy="0.0" ixz="0.0"
-                iyy="0.00001" iyz="0.0"
-                izz="0.00001" />
-        </inertial>
+		<inertial>
+			<mass value="0.01" />
+			<inertia ixx="1e-6" ixy="0" ixz="0"
+				iyy="1e-6" iyz="0"
+				izz="1e-6" />
+		</inertial>
     </xacro:macro>
     <xacro:macro name="trans_xacro" params="namehand jointname">
@@ -86,5 +104,5 @@
                <origin rpy="0 0 0" xyz="0 0 0" />
                 <geometry>
-                    <mesh filename="package://centauro/centauro_urdf/meshes/schunk_hand/camera_link.STL" />
+					<mesh filename="package://centauro/centauro_urdf/meshes/schunk_hand/camera_link.STL" /> <!-- FIXME: convex hull? -->
                 </geometry>
             </collision>
@@ -127,5 +145,7 @@
         <!-- LENGTH NOT FOUND IN DATASHEET! GUESSED!!! -->
         <link name="${name}_e1">
-            <xacro:dummy_inertial />
+			<xacro:cylinder_inertial radius="0.025" length="0.12" mass="0.03">
+				<origin rpy="0 0 0" xyz="-0.00368 0.0 0.06" />
+			</xacro:cylinder_inertial>
             <visual>
                 <origin rpy="0 0 0" xyz="0 0.01313 0" />
@@ -199,5 +219,7 @@
         <!-- THUMB LINKS -->
         <link name="${name}_z">
-            <xacro:dummy_inertial />
+            <xacro:cylinder_inertial radius="0.018796440353616439" length="0.01042481810366226" mass="0.03">
+				<origin rpy="2.9985 8.56161e-08 1.19461e-06" xyz="4.8053e-09 0.000609069 0.0461834" />
+			</xacro:cylinder_inertial>
             <visual>
                 <origin xyz="0 0 0.02442" />
@@ -218,5 +240,7 @@
         </link>
         <link name="${name}_a">
-            <xacro:dummy_inertial />
+			<xacro:cylinder_inertial radius="0.016759180858870293" length="0.047241541605838461" mass="0.03">
+				<origin rpy="-1.57079 1.53946 -1.53946" xyz="0.0234125 -0.000744623 -1.94586e-05" />
+			</xacro:cylinder_inertial>
             <visual>
                 <geometry>
@@ -232,5 +256,7 @@
         </link>
         <link name="${name}_b">
-            <xacro:dummy_inertial />
+            <xacro:cylinder_inertial radius="0.015792729610253044" length="0.023014525532768428" mass="0.03">
+				<origin rpy="1.56836 1.57067 1.56823" xyz="0.0115211 -7.34551e-06 2.67722e-06" />
+			</xacro:cylinder_inertial>
             <visual>
                 <geometry>
@@ -246,5 +272,7 @@
         </link>
         <link name="${name}_c">
-            <xacro:dummy_inertial />
+             <xacro:cylinder_inertial radius="0.010704766923000805" length="0.015173140958556149" mass="0.03">
+				<origin rpy="1.5708 1.55113 1.55114" xyz="0.0096433 -0.000617283 1.28171e-10" />
+			</xacro:cylinder_inertial>
             <visual>
                 <geometry>
@@ -542,5 +570,5 @@
             <origin xyz="0 0 0" rpy="0 0 ${side*(-0.9704)}" />
             <axis xyz="0 0 ${side*(1)}" />
-            <dynamics friction="${friction_schunk}" />
+            <dynamics friction="${friction_schunk}" damping="${damping_schunk}" />
         </joint>
         <xacro:trans_xacro namehand="${name}" jointname="Thumb_Flexion"/>
@@ -568,5 +596,5 @@
             <origin xyz="${side*(-0.01690)} 0.02626 0" rpy="0 0.2618 1.571" />
             <axis xyz="0 0 ${side*(-1)}" />
-            <dynamics friction="${friction_schunk}" />
+            <dynamics friction="${friction_schunk}" damping="${damping_schunk}" />
         </joint>
         <xacro:trans_xacro namehand="${name}" jointname="Thumb_Opposition"/>
@@ -603,5 +631,5 @@
             <axis xyz="0 0 ${side*(1)}" />
             <mimic joint="${name}_Thumb_Opposition" multiplier="1" offset="0" />
-            <dynamics friction="${friction_schunk}" />
+            <dynamics friction="${friction_schunk}" damping="${damping_schunk}" />
         </joint>
         <xacro:trans_xacro namehand="${name}" jointname="j5"/>
@@ -638,5 +666,5 @@
             <axis xyz="0 0 ${side*(1)}" />
             <mimic joint="${name}_Thumb_Flexion" multiplier="1.01511" offset="0" />
-            <dynamics friction="${friction_schunk}" />
+            <dynamics friction="${friction_schunk}" damping="${damping_schunk}" />
         </joint>
         <xacro:trans_xacro namehand="${name}" jointname="j3"/>
@@ -648,5 +676,5 @@
             <axis xyz="0 0 ${side*(1)}" />
             <mimic joint="${name}_Thumb_Flexion" multiplier="1.44889" offset="0" />
-            <dynamics friction="${friction_schunk}" />
+            <dynamics friction="${friction_schunk}" damping="${damping_schunk}" />
         </joint>
         <xacro:trans_xacro namehand="${name}" jointname="j4"/>
@@ -658,5 +686,5 @@
             <origin xyz="0.04804 0 0" rpy="0 0 0" />
             <axis xyz="0 0 1" />
-            <dynamics friction="${friction_schunk}" />
+            <dynamics friction="${friction_schunk}" damping="${damping_schunk}" />
         </joint>
         <xacro:trans_xacro namehand="${name}" jointname="Index_Finger_Distal"/>
@@ -667,5 +695,5 @@
             <origin xyz="0 0 0" rpy="-1.5707 0 0" />
             <axis xyz="0 0 1" />
-            <dynamics friction="${friction_schunk}" />
+            <dynamics friction="${friction_schunk}" damping="${damping_schunk}" />
         </joint>
         <xacro:trans_xacro namehand="${name}" jointname="Index_Finger_Proximal"/>
@@ -678,5 +706,5 @@
             <axis xyz="0 0 1" />
             <mimic joint="${name}_Index_Finger_Distal" multiplier="1.0450" offset="0" />
-            <dynamics friction="${friction_schunk}" />
+            <dynamics friction="${friction_schunk}" damping="${damping_schunk}" />
         </joint>
         <xacro:trans_xacro namehand="${name}" jointname="j14"/>
@@ -688,5 +716,5 @@
             <origin xyz="0 0 0" rpy="-1.5707 0 0" />
             <axis xyz="0 0 1" />
-            <dynamics friction="${friction_schunk}" />
+            <dynamics friction="${friction_schunk}" damping="${damping_schunk}" />
         </joint>
         <xacro:trans_xacro namehand="${name}" jointname="Middle_Finger_Proximal"/>
@@ -697,5 +725,5 @@
             <origin xyz="0.05004 0 0" rpy="0 0 0" />
             <axis xyz="0 0 1" />
-            <dynamics friction="${friction_schunk}" />
+            <dynamics friction="${friction_schunk}" damping="${damping_schunk}" />
         </joint>
         <xacro:trans_xacro namehand="${name}" jointname="Middle_Finger_Distal"/>
@@ -707,5 +735,5 @@
             <axis xyz="0 0 1" />
             <mimic joint="${name}_Middle_Finger_Distal" multiplier="1.0454" offset="0" />
-            <dynamics friction="${friction_schunk}" />
+            <dynamics friction="${friction_schunk}" damping="${damping_schunk}" />
         </joint>
         <xacro:trans_xacro namehand="${name}" jointname="j15"/>
@@ -717,5 +745,5 @@
             <origin xyz="0 0 0" rpy="1.5707 0 0" />
             <axis xyz="0 0 1" />
-            <dynamics friction="${friction_schunk}" />
+            <dynamics friction="${friction_schunk}" damping="${damping_schunk}" />
         </joint>
         <xacro:trans_xacro namehand="${name}" jointname="Ring_Finger"/>
@@ -727,5 +755,5 @@
             <axis xyz="0 0 1" />
             <mimic joint="${name}_Ring_Finger" multiplier="1.3588" offset="0" />
-            <dynamics friction="${friction_schunk}" />
+            <dynamics friction="${friction_schunk}" damping="${damping_schunk}" />
         </joint>
         <xacro:trans_xacro namehand="${name}" jointname="j12"/>
@@ -737,5 +765,5 @@
             <axis xyz="0 0 1" />
             <mimic joint="${name}_Ring_Finger" multiplier="1.42093" offset="0" />
-            <dynamics friction="${friction_schunk}" />
+            <dynamics friction="${friction_schunk}" damping="${damping_schunk}" />
         </joint>
         <xacro:trans_xacro namehand="${name}" jointname="j16"/>
@@ -747,5 +775,5 @@
             <origin xyz="0 0 0" rpy="1.5707 0 0" />
             <axis xyz="0 0 1" />
-            <dynamics friction="${friction_schunk}" />
+            <dynamics friction="${friction_schunk}" damping="${damping_schunk}" />
         </joint>
         <xacro:trans_xacro namehand="${name}" jointname="Pinky"/>
@@ -757,5 +785,5 @@
             <axis xyz="0 0 1" />
             <mimic joint="${name}_Pinky" multiplier="1.35880" offset="0" />
-            <dynamics friction="${friction_schunk}" />
+            <dynamics friction="${friction_schunk}" damping="${damping_schunk}" />
         </joint>
         <xacro:trans_xacro namehand="${name}" jointname="j13"/>
@@ -767,5 +795,5 @@
             <axis xyz="0 0 1" />
             <mimic joint="${name}_Pinky" multiplier="1.42307" offset="0" />
-            <dynamics friction="${friction_schunk}" />
+            <dynamics friction="${friction_schunk}" damping="${damping_schunk}" />
         </joint>
         <xacro:trans_xacro namehand="${name}" jointname="j17"/>
@@ -777,5 +805,5 @@
             <axis xyz="0 0 ${side*(1)}" />
             <mimic joint="${name}_Finger_Spread" multiplier="0.5" offset="0" />
-            <dynamics friction="${friction_schunk}" />
+            <dynamics friction="${friction_schunk}" damping="${damping_schunk}" />
         </joint>
         <xacro:trans_xacro namehand="${name}" jointname="index_spread"/>
@@ -793,5 +821,5 @@
             <axis xyz="0 0 ${side*(1)}" />
             <mimic joint="${name}_Finger_Spread" multiplier="0.5" offset="0" />
-            <dynamics friction="${friction_schunk}" />
+            <dynamics friction="${friction_schunk}" damping="${damping_schunk}" />
         </joint>
         <xacro:trans_xacro namehand="${name}" jointname="ring_spread"/>
@@ -802,5 +830,5 @@
             <origin xyz="${side*(0.025355)} 0 0.056" rpy="-1.5707 -1.5707 0" />
             <axis xyz="0 0 ${side*(1)}" />
-            <dynamics friction="${friction_schunk}" />
+            <dynamics friction="${friction_schunk}" damping="${damping_schunk}" />
         </joint>
         <xacro:trans_xacro namehand="${name}" jointname="Finger_Spread"/>

Commit message: urdf: correct model of centauro with only right arm

File: centauro/centauro_urdf/urdf/centauro_arm.urdf.xacro (robot description, xacro)
@@ -237,5 +237,5 @@
     </xacro:svh>
 </xacro:if>
-<xacro:if value="${end_effector != 'stick' and end_effector != 'soft_hand' and end_effector != 'schunk_hand'}" >
+<xacro:if value="${end_effector != 'stick' and end_effector != 'soft_hand' and end_effector != 'schunk_hand' and end_effector != 'no_end_effector_joint'}" >
   <xacro:include filename="$(find centauro)/centauro_urdf/urdf/centauro_no_end_effector.urdf.xacro" />
 </xacro:if>

File: centauro/centauro_urdf/urdf/centauro_right_arm.urdf.xacro (robot description, xacro)
@@ -21,7 +21,7 @@
   <xacro:include filename="$(find centauro)/centauro_urdf/urdf/centauro_arm.urdf.xacro"/>
 </xacro:if>
+<xacro:include filename="$(find centauro)/centauro_urdf/urdf/models/upper_body/end_effectors/schunk_hand/svh_gazebo.urdf.xacro" />
+<xacro:include filename="$(find centauro)/centauro_urdf/urdf/centauro_eef.urdf.xacro"/>
 <!-- /other files -->
-<!-- reference -->
-<link name="world"/>
 <xacro:if value="${pelvis}">
    <link name="pelvis">
@@ -53,41 +53,27 @@
    <link name="pelvis"/>
 </xacro:unless>
-<joint name="reference" type="${reference}">
-   <origin xyz="${Pelvis_Ox} ${Pelvis_Oy} ${Pelvis_Oz}"/>
-   <parent link="world"/>
-   <child link="pelvis"/>
+<link name="base_link" />
+<joint name="base_pelvis" type="fixed">
+   <parent link="base_link" />
+   <child link="pelvis" />
+   <origin xyz="0 0 0" rpy="0 0 0" />
 </joint>
+<xacro:if value="${include_world}">
+   <!-- reference -->
+   <link name="world"/>
+   <joint name="reference" type="${reference}">
+      <origin xyz="${Pelvis_Ox} ${Pelvis_Oy} ${Pelvis_Oz}"/>
+      <parent link="world"/>
+      <child link="base_link"/>
+   </joint>
+</xacro:if>
 <!-- /reference  -->
 <!-- torso -->
-<xacro:if value="${torso == 'true'}">
    <xacro:include filename="$(find centauro)/centauro_urdf/urdf/centauro_torso_fixed.urdf.xacro"/>
-</xacro:if>
-<xacro:if value="${head == 'true'}">
-   <xacro:include filename="$(find centauro)/centauro_urdf/urdf/centauro_head.urdf.xacro"/>
-</xacro:if>
 <!-- /torso -->
-<!-- arms -->
-<xacro:if value="${arms == 'true'}">
+<!-- arm -->
    <xacro:centauro_arm arm_num="2" rot="-1"  parent="torso_2" end_effector="${RIGHT_END_EFFECTOR}">
       <origin xyz="${Shoulder_1_Ox} ${-Shoulder_1_Oy} ${Shoulder_1_Oz}" rpy="${Shoulder_1_roll} ${Shoulder_1_pitch} ${-Shoulder_1_yaw}" />
    </xacro:centauro_arm>
-</xacro:if>
-<xacro:if value="${arm == 'true' and arms == 'false'}">
-        <xacro:centauro_arm arm_num="1"  rot="1" parent="world">
-           <origin xyz="${Shoulder_1_Ox + Pelvis_Ox + Torso_2_Ox} ${Shoulder_1_Oy + Pelvis_Oy + Torso_2_Oy} ${Shoulder_1_Oz + Pelvis_Oz + Torso_2_Oz}" rpy="${Shoulder_1_roll} ${Shoulder_1_pitch} ${Shoulder_1_yaw}"/>
-        </xacro:centauro_arm>
-</xacro:if>
-<!-- /arms -->
-<!-- legs -->
-<xacro:if value="${legs}">
-<xacro:centauro_leg leg_num="1" origin_x="1" origin_y="-1">
-</xacro:centauro_leg>
-<xacro:centauro_leg leg_num="2" origin_x="1" origin_y="1">
-</xacro:centauro_leg>
-<xacro:centauro_leg leg_num="3" origin_x="-1" origin_y="-1">
-</xacro:centauro_leg>
-<xacro:centauro_leg leg_num="4" origin_x="-1" origin_y="1">
-</xacro:centauro_leg>
-</xacro:if>
-<!-- /legs -->
+<!-- /arm -->
 </robot>

Commit message: Added damping to all the joints

File: centauro/centauro_urdf/urdf/centauro_arm.urdf.xacro (robot description, xacro)
@@ -125,4 +125,5 @@
          <limit lower="-1.658" upper="3.403" effort="147" velocity="5.7"/>
       </xacro:unless>
+      <dynamics friction="0" damping="0.5"/>
    </joint>
 <!-- /shoulder yaw -->
@@ -139,4 +140,5 @@
          <limit lower="-3.49" upper="0" effort="147" velocity="5.7"/>
       </xacro:unless>
+      <dynamics friction="0" damping="0.5"/>
    </joint>
 <!-- /shoulder roll -->
@@ -148,4 +150,5 @@
       <axis xyz="0 0 -1"/>
       <limit lower="-2.618" upper="2.618" effort="147" velocity="8.2"/>
+      <dynamics friction="0" damping="0.5"/>
    </joint>
 <!-- /shoulder pitch -->
@@ -162,4 +165,5 @@
          <limit lower="-0.349" upper="2.530" effort="147" velocity="8.2"/>
       </xacro:unless>
+      <dynamics friction="0" damping="0.5"/>
    </joint>
 <!-- /elbow yaw -->
@@ -171,4 +175,5 @@
       <axis xyz="0 0 -1"/>
       <limit lower="-2.618" upper="2.618" effort="55" velocity="11.6"/>
+      <dynamics friction="0" damping="0.5"/>
    </joint>
 <!-- /elbow pitch-->
@@ -180,4 +185,5 @@
       <axis xyz="0 ${rot} 0"/>
       <limit lower="-1.570" upper="1.570" effort="55" velocity="11.6"/>
+      <dynamics friction="0" damping="0.5"/>
    </joint>
 <!-- /wrist yaw-->
@@ -189,4 +195,5 @@
       <axis xyz="0 0 -1"/>
       <limit lower="-2.618" upper="2.618" effort="27" velocity="20.3"/>
+      <dynamics friction="0" damping="0.5"/>
    </joint>
 <!-- wrist pitch-->

File: centauro/centauro_urdf/urdf/centauro_head.urdf.xacro (robot description, xacro)
@@ -87,4 +87,5 @@
    <axis xyz="0 0 1"/>
    <limit lower="-0.78539816" upper="0.78539816" effort="35" velocity="5.7"/> <!-- TODO -->
+   <dynamics friction="0" damping="0.3"/>
 </joint>
 <joint name="neck_pitch" type="revolute">
@@ -94,4 +95,5 @@
    <axis xyz="0 1 0"/>
    <limit lower="-0.34906585" upper="0.78539816" effort="35" velocity="5.7"/> <!-- TODO -->
+   <dynamics friction="0" damping="0.5"/>
 </joint>
 <joint name="neck_velodyne" type="continuous">
@@ -101,4 +103,5 @@
    <axis xyz="0 0 1"/>
    <limit effort="35" velocity="5.7"/> <!-- TODO -->
+   <dynamics friction="0" damping="0.3"/>
 </joint>
 <!-- /head joints -->

File: centauro/centauro_urdf/urdf/centauro_leg.urdf.xacro (robot description, xacro)
@@ -100,4 +100,5 @@
         <limit lower="-2.70526034" upper="1.13446401" effort="304" velocity="8.8"/>
         </xacro:if>
+        <dynamics friction="0" damping="0.3"/>
 </joint>
 <joint name="hip_pitch_${leg_num}" type="revolute">
@@ -107,4 +108,5 @@
 	<axis xyz="0 0 1"/>
         <limit lower="-2.09439510" upper="2.09439510" effort="304" velocity="8.8"/>
+        <dynamics friction="0" damping="0.3"/>
 </joint>
 <joint name="knee_pitch_${leg_num}" type="revolute">
@@ -114,4 +116,5 @@
 	<axis xyz="0 0 1"/>
         <limit  lower="-2.61799388" upper="2.61799388" effort="304" velocity="8.8"/>
+        <dynamics friction="0" damping="0.3"/>
 </joint>
 <joint name="ankle_pitch_${leg_num}" type="revolute">
@@ -121,4 +124,5 @@
 	<axis xyz="0 0 1"/>
         <limit  lower="-2.61799388" upper="2.61799388" effort="147" velocity="8.1"/>
+        <dynamics friction="0" damping="0.3"/>
 </joint>
 <joint name="ankle_yaw_${leg_num}" type="revolute">
@@ -128,4 +132,5 @@
 	<axis xyz="0 0 1"/>
         <limit  lower="-2.79252680" upper="2.79252680" effort="35" velocity="20.0"/>
+        <dynamics friction="0" damping="0.3"/>
 </joint>
 <joint name="j_wheel_${leg_num}" type="continuous">
@@ -135,4 +140,5 @@
 	<axis xyz="0 0 1"/>
         <limit  effort="35" velocity="20.0"/>
+        <dynamics friction="0" damping="0.3"/>
 </joint>
 <!--

File: centauro/centauro_urdf/urdf/centauro_torso.urdf.xacro (robot description, xacro)
@@ -29,4 +29,5 @@
    <axis xyz="0 0 1"/>
    <limit lower="-2.618" upper="2.618" effort="147" velocity="5.7"/> <!-- TODO -->
+   <dynamics friction="0" damping="0.3"/>
 </joint>
 <!-- /torso joints -->
