Commit message: Add modified version for generation of centauro urdf used in robolearn: https://github.com/ADVRHumanoids/robolearn

File: centauro/centauro_urdf/urdf/centauro_arm.urdf.xacro (robot description, xacro)
@@ -29,4 +29,5 @@
       <visual>
          <xacro:visual_model.arm2 />
+         <material name="dark_grey"/>
       </visual>
       <collision>
@@ -60,4 +61,5 @@
       <visual>
          <xacro:visual_model.arm4 />
+         <material name="dark_grey"/>
       </visual>
       <collision>
@@ -91,4 +93,5 @@
       <visual>
          <xacro:visual_model.arm6 />
+         <material name="dark_grey"/>
       </visual>
       <collision>
@@ -118,6 +121,12 @@
       <child link="arm${arm_num}_1"/>
       <xacro:insert_block name="origin"/>
-      <axis xyz="0 ${rot*cos_m10} ${-sin_m10}"/>
+      <axis xyz="0. ${rot*cos_m10} ${-sin_m10}"/>
       <limit lower="${j_arm_1_lower[arm_num-1]}" upper="${j_arm_1_upper[arm_num-1]}" effort="147" velocity="5.7"/>
+      <!--<xacro:unless value="${rot-1}" >-->
+         <!--<limit lower="-3.403" upper="1.658" effort="147" velocity="5.7"/>-->
+      <!--</xacro:unless>-->
+      <!--<xacro:unless value="${rot+1}" >-->
+         <!--<limit lower="-1.658" upper="3.403" effort="147" velocity="5.7"/>-->
+      <!--</xacro:unless>-->
    </joint>
 <!-- /shoulder yaw -->
@@ -129,4 +138,11 @@
       <axis xyz="-1 0 0"/>
       <limit lower="${j_arm_2_lower[arm_num-1]}" upper="${j_arm_2_upper[arm_num-1]}" effort="147" velocity="5.7"/>
+      <!--<xacro:unless value="${rot+1}" >-->
+      <!--<limit lower="0" upper="3.49" effort="147" velocity="5.7"/>-->
+      <xacro:unless value="${rot+1}" > <limit lower="0" upper="3.49" effort="147" velocity="5.7"/>
+      </xacro:unless>
+      <xacro:unless value="${rot-1}" >
+         <limit lower="-3.49" upper="0" effort="147" velocity="5.7"/>
+      </xacro:unless>
    </joint>
 <!-- /shoulder roll -->
@@ -137,4 +153,5 @@
       <origin xyz="${Shoulder_3_Ox} ${Shoulder_3_Oy} ${Shoulder_3_Oz}"/>
       <axis xyz="0 0 -1"/>
+      <!--<limit lower="-2.618" upper="2.618" effort="147" velocity="8.2"/>-->
       <limit lower="${j_arm_3_lower[arm_num-1]}" upper="${j_arm_3_upper[arm_num-1]}" effort="147" velocity="8.2"/>
    </joint>
@@ -147,4 +164,12 @@
       <axis xyz="0 ${rot} 0"/>
       <limit lower="${j_arm_4_lower[arm_num-1]}" upper="${j_arm_4_upper[arm_num-1]}" effort="147" velocity="8.2"/>
+      <!--<xacro:unless value="${rot-1}" >-->
+         <!--<limit lower="-2.530" upper="0.349" effort="147" velocity="8.2"/>-->
+      <!--</xacro:unless>-->
+      <xacro:unless value="${rot-1}" > <limit lower="-2.530" upper="0.349" effort="147" velocity="8.2"/>
+      </xacro:unless>
+      <xacro:unless value="${rot+1}" >
+         <limit lower="-0.349" upper="2.530" effort="147" velocity="8.2"/>
+      </xacro:unless>
    </joint>
 <!-- /elbow yaw -->
@@ -155,4 +180,5 @@
       <origin xyz="${Wrist_1_Ox} ${-rot*Wrist_1_Oy} ${Wrist_1_Oz}"/>
       <axis xyz="0 0 -1"/>
+      <!--<limit lower="-2.618" upper="2.618" effort="55" velocity="11.6"/>-->
       <limit lower="${j_arm_5_lower[arm_num-1]}" upper="${j_arm_5_upper[arm_num-1]}" effort="55" velocity="11.6"/>
    </joint>
@@ -164,4 +190,5 @@
       <origin xyz="${Wrist_2_Ox} ${rot*Wrist_2_Oy} ${Wrist_2_Oz}"/>
       <axis xyz="0 ${rot} 0"/>
+      <!--<limit lower="-1.570" upper="1.570" effort="55" velocity="11.6"/>-->
       <limit lower="${j_arm_6_lower[arm_num-1]}" upper="${j_arm_6_upper[arm_num-1]}" effort="55" velocity="11.6"/>
    </joint>
@@ -173,4 +200,5 @@
       <origin xyz="${Wrist_3_Ox} ${-rot*Wrist_3_Oy} ${Wrist_3_Oz}"/>
       <axis xyz="0 0 -1"/>
+      <!--<limit lower="-2.618" upper="2.618" effort="27" velocity="20.3"/>-->
       <limit lower="${j_arm_7_lower[arm_num-1]}" upper="${j_arm_7_upper[arm_num-1]}" effort="27" velocity="20.3"/>
    </joint>

File: centauro/centauro_urdf/urdf/centauro_hand_fakelink.urdf.xacro (robot description, xacro)
@@ -6,19 +6,22 @@
 <!-- /constants -->
 <!-- other files -->
-<xacro:include filename="$(find centauro)/centauro_urdf/urdf/config.xacro"/>
+<xacro:include filename="config.xacro"/>
 <xacro:if value="${GAZEBO}">
-  <xacro:include filename="$(find centauro_gazebo)/urdf/centauro.gazebo"/>
+  <xacro:include filename="centauro.gazebo"/>
 </xacro:if>
 <xacro:include filename="${inertia_parameters_file}"/>
 <xacro:include filename="${kinematic_parameters_file}"/>
-<xacro:include filename="$(find centauro)/centauro_urdf/limits/default.xacro"/>
-<xacro:include filename="$(find centauro)/centauro_urdf/materials.xacro"/>
-<xacro:include filename="$(find centauro)/centauro_urdf/urdf/models/model.xacro"/>
-<xacro:include filename="$(find centauro)/centauro_urdf/urdf/centauro_actuators.urdf.xacro" />
+<xacro:include filename="../materials.xacro"/>
+<xacro:include filename="models/model.xacro"/>
+<xacro:include filename="centauro_actuators.urdf.xacro" />
 <xacro:if value="${LEGS}">
-  <xacro:include filename="$(find centauro)/centauro_urdf/urdf/centauro_leg.urdf.xacro"/>
+  <xacro:include filename="centauro_leg.urdf.xacro"/>
 </xacro:if>
 <xacro:if value="${arms}">
-  <xacro:include filename="$(find centauro)/centauro_urdf/urdf/centauro_arm.urdf.xacro"/>
+  <xacro:include filename="centauro_arm.urdf.xacro"/>
+</xacro:if>
+<xacro:property name="HAND_FAKELINK" value="$(arg HAND_FAKELINK)"/>
+<xacro:if value="${HAND_FAKELINK}">
+    <xacro:include filename="hand_fakelink.urdf.xacro"/>
 </xacro:if>
 <!-- /other files -->
@@ -67,5 +70,4 @@
    <!--<child link="pelvis"/>-->
 <!--</joint>-->
-<!-- /reference  -->
 <link name="base_link">
     <inertial>
@@ -81,8 +83,8 @@
 <!-- torso -->
 <xacro:if value="${torso == 'true'}">
-   <xacro:include filename="$(find centauro)/centauro_urdf/urdf/centauro_torso.urdf.xacro"/>
+   <xacro:include filename="centauro_torso.urdf.xacro"/>
 </xacro:if>
 <xacro:if value="${head == 'true'}">
-   <xacro:include filename="$(find centauro)/centauro_urdf/urdf/centauro_head.urdf.xacro"/>
+   <xacro:include filename="centauro_head.urdf.xacro"/>
 </xacro:if>
 <!-- /torso -->

File: centauro/centauro_urdf/urdf/centauro_head.urdf.xacro (robot description, xacro)
@@ -9,8 +9,9 @@
         </inertial>
 	<visual>
-                <xacro:visual_model.neck_yaw />
+        <xacro:visual_model.neck_yaw />
+        <material name="dark_grey"/>
 	</visual>
 	<collision>
-                <xacro:collision_model.neck_yaw />
+        <xacro:collision_model.neck_yaw />
 	</collision>
 </link>
@@ -22,8 +23,9 @@
         </inertial>
 	<visual>
-                <xacro:visual_model.neck_pitch />
+        <xacro:visual_model.neck_pitch />
+        <material name="dark_grey"/>
 	</visual>
 	<collision>
-                <xacro:collision_model.neck_pitch />
+        <xacro:collision_model.neck_pitch />
 	</collision>
 </link>
@@ -35,5 +37,6 @@
         </inertial>
 	<visual>
-                <xacro:visual_model.velodyne />
+        <xacro:visual_model.velodyne />
+        <material name="dark_grey"/>
 	</visual>
 	<collision>
@@ -71,5 +74,11 @@
         </inertial>
 </link>
-<link name="kinect2_rgb_optical_frame" />
+<link name="kinect2_rgb_optical_frame">
+    <inertial>
+        <origin xyz="0.0 0.0 0.0"/>
+        <mass value="1e-6"/>
+        <inertia ixx="1e-06" ixy="0.0" ixz="0.0" iyy="1e-06" iyz="0.0" izz="1e-06"/>
+    </inertial>
+</link>
 <link name="velodyne_mount">
 	<inertial>

File: centauro/centauro_urdf/urdf/centauro_leg.urdf.xacro (robot description, xacro)
@@ -27,4 +27,5 @@
       <visual>
          <xacro:visual_model.leg2 />
+		  <material name="dark_grey"/>
       </visual>
       <collision>
@@ -56,4 +57,5 @@
       <visual>
          <xacro:visual_model.ankle1 />
+		  <material name="dark_grey"/>
       </visual>
       <collision>
@@ -95,4 +97,10 @@
 	<axis xyz="0 0 1"/>
         <limit lower="${hip_yaw_lower[leg_num-1]}" upper="${hip_yaw_upper[leg_num-1]}" effort="304" velocity="8.8"/>
+	<!--<xacro:if value="${origin_y*origin_x == -1}">-->
+		<!--<limit lower="-1.13446401" upper="2.70526034" effort="304" velocity="8.8"/>-->
+	<!--</xacro:if>-->
+	<!--<xacro:if value="${origin_y*origin_x == 1}">-->
+		<!--<limit lower="-2.70526034" upper="1.13446401" effort="304" velocity="8.8"/>-->
+	<!--</xacro:if>-->
 </joint>
 <joint name="hip_pitch_${leg_num}" type="revolute">
@@ -101,4 +109,5 @@
 	<origin xyz="${Leg_2_Ox} ${Leg_2_Oy} ${Leg_2_Oz}" rpy="${Leg_2_roll} ${Leg_2_pitch} ${origin_x*origin_y*Leg_2_yaw-origin_x*origin_y*PI/2 + PI/2}"/>
 	<axis xyz="0 0 1"/>
+        <!--<limit lower="-2.09439510" upper="2.09439510" effort="304" velocity="8.8"/> -->
         <limit lower="${hip_pitch_lower[leg_num-1]}" upper="${hip_pitch_upper[leg_num-1]}" effort="304" velocity="8.8"/>
 </joint>
@@ -108,4 +117,5 @@
 	<origin xyz="${Leg_3_Ox} ${Leg_3_Oy} ${Leg_3_Oz}" rpy="${Leg_3_roll} ${Leg_3_pitch} ${Leg_3_yaw}"/>
 	<axis xyz="0 0 1"/>
+        <!--<limit  lower="-2.61799388" upper="2.61799388" effort="304" velocity="8.8"/>-->
         <limit lower="${knee_pitch_lower[leg_num-1]}" upper="${knee_pitch_upper[leg_num-1]}" effort="304" velocity="8.8"/>
 </joint>
@@ -115,4 +125,5 @@
 	<origin xyz="${Ankle_1_Ox} ${Ankle_1_Oy} ${Ankle_1_Oz}" rpy="${Ankle_1_roll} ${Ankle_1_pitch} ${Ankle_1_yaw}"/>
 	<axis xyz="0 0 1"/>
+        <!--<limit  lower="-2.61799388" upper="2.61799388" effort="147" velocity="8.1"/> -->
         <limit lower="${ankle_pitch_lower[leg_num-1]}" upper="${ankle_pitch_upper[leg_num-1]}" effort="147" velocity="8.1"/>
 </joint>
@@ -122,4 +133,5 @@
 	<origin xyz="${Ankle_2_Ox} ${Ankle_2_Oy} ${Ankle_2_Oz}" rpy="${Ankle_2_roll} ${Ankle_2_pitch} ${Ankle_2_yaw}"/>
 	<axis xyz="0 0 1"/>
+        <!--<limit  lower="-2.58308729" upper="2.58308729" effort="35" velocity="20.0"/> -->
         <limit lower="${ankle_yaw_lower[leg_num-1]}" upper="${ankle_yaw_upper[leg_num-1]}" effort="35" velocity="20.0"/>
 </joint>
@@ -128,4 +140,5 @@
 	<child link="wheel_${leg_num}"/>
 	<origin xyz="${Wheel_Ox} ${Wheel_Oy} ${Wheel_Oz}" rpy="${Wheel_roll} ${Wheel_pitch} ${Wheel_yaw}"/>
+	<!--<axis xyz="0 0 1"/>-->
 	<axis xyz="0 0 -1"/>
         <limit  effort="35" velocity="20.0"/>

File: centauro/centauro_urdf/urdf/centauro_right_arm.urdf.xacro (robot description, xacro)
@@ -32,5 +32,6 @@
       </inertial>
       <visual>
-         <xacro:visual_model.pelvis />
+          <xacro:visual_model.pelvis />
+          <material name="dark_grey"/>
       </visual>
       <collision>

File: centauro/centauro_urdf/urdf/centauro_torso.urdf.xacro (robot description, xacro)
@@ -9,5 +9,6 @@
         </inertial>
 	<visual>
-                <xacro:visual_model.torso />
+        <xacro:visual_model.torso />
+        <material name="dark_grey"/>
 	</visual>
 	<collision>
@@ -28,5 +29,6 @@
    <child link="torso_2"/>
    <axis xyz="0 0 1"/>
-   <limit lower="${torso_yaw_lower}" upper="${torso_yaw_upper}" effort="147" velocity="5.7"/> <!-- TODO -->
+    <!--<limit lower="-2.618" upper="2.618" effort="147" velocity="5.7"/> &lt;!&ndash; TODO &ndash;&gt;-->
+    <limit lower="${torso_yaw_lower}" upper="${torso_yaw_upper}" effort="147" velocity="5.7"/> <!-- TODO -->
 </joint>
 <!-- /torso joints -->

File: centauro/centauro_urdf/urdf/centauro_tray.urdf.xacro (robot description, xacro)
@@ -6,19 +6,22 @@
 <!-- /constants -->
 <!-- other files -->
-<xacro:include filename="$(find centauro)/centauro_urdf/urdf/config.xacro"/>
+<xacro:include filename="config.xacro"/>
 <xacro:if value="${GAZEBO}">
-  <xacro:include filename="$(find centauro_gazebo)/urdf/centauro.gazebo"/>
+  <xacro:include filename="centauro.gazebo"/>
 </xacro:if>
 <xacro:include filename="${inertia_parameters_file}"/>
 <xacro:include filename="${kinematic_parameters_file}"/>
-<xacro:include filename="$(find centauro)/centauro_urdf/limits/default.xacro"/>
-<xacro:include filename="$(find centauro)/centauro_urdf/materials.xacro"/>
-<xacro:include filename="$(find centauro)/centauro_urdf/urdf/models/model.xacro"/>
-<xacro:include filename="$(find centauro)/centauro_urdf/urdf/centauro_actuators.urdf.xacro" />
+<xacro:include filename="../materials.xacro"/>
+<xacro:include filename="models/model.xacro"/>
+<xacro:include filename="centauro_actuators.urdf.xacro" />
 <xacro:if value="${LEGS}">
-  <xacro:include filename="$(find centauro)/centauro_urdf/urdf/centauro_leg.urdf.xacro"/>
+  <xacro:include filename="centauro_leg.urdf.xacro"/>
 </xacro:if>
 <xacro:if value="${arms}">
-  <xacro:include filename="$(find centauro)/centauro_urdf/urdf/centauro_arm.urdf.xacro"/>
+  <xacro:include filename="centauro_arm.urdf.xacro"/>
+</xacro:if>
+<xacro:property name="TRAY" value="$(arg TRAY)"/>
+<xacro:if value="${TRAY}">
+    <xacro:include filename="hand_tray.urdf.xacro"/>
 </xacro:if>
 <!-- /other files -->
@@ -67,5 +70,4 @@
    <!--<child link="pelvis"/>-->
 <!--</joint>-->
-<!-- /reference  -->
 <link name="base_link">
     <inertial>
@@ -81,8 +83,8 @@
 <!-- torso -->
 <xacro:if value="${torso == 'true'}">
-   <xacro:include filename="$(find centauro)/centauro_urdf/urdf/centauro_torso.urdf.xacro"/>
+   <xacro:include filename="centauro_torso.urdf.xacro"/>
 </xacro:if>
 <xacro:if value="${head == 'true'}">
-   <xacro:include filename="$(find centauro)/centauro_urdf/urdf/centauro_head.urdf.xacro"/>
+   <xacro:include filename="centauro_head.urdf.xacro"/>
 </xacro:if>
 <!-- /torso -->

File: centauro/centauro_urdf/urdf/models/upper_body/end_effectors/schunk_hand/svh_gazebo.urdf.xacro (robot description, xacro)
@@ -82,4 +82,5 @@
                     <mesh filename="package://centauro/centauro_urdf/meshes/schunk_hand/camera_link.STL" />
                 </geometry>
+                <material name="dark_grey"/>
             </visual>
             <collision>
@@ -108,4 +109,5 @@
                     <mesh filename="package://centauro/centauro_urdf/meshes/schunk_hand/base10.dae" />
                 </geometry>
+                <material name="dark_grey"/>
             </visual>
             <collision>
@@ -133,4 +135,5 @@
                     <mesh scale="${side*(1)} 1 1" filename="package://centauro/centauro_urdf/meshes/schunk_hand/h10.dae" />
                 </geometry>
+                <material name="dark_grey"/>
             </visual>
             <collision>
@@ -152,4 +155,5 @@
                     <mesh scale="${side*(1)} 1 1" filename="package://centauro/centauro_urdf/meshes/schunk_hand/h11.dae" />
                 </geometry>
+                <material name="dark_grey"/>
             </visual>
             <collision>
@@ -205,4 +209,5 @@
                     <mesh scale="1 ${side*(1)} 1" filename="package://centauro/centauro_urdf/meshes/schunk_hand/d10.dae" />
                 </geometry>
+                <material name="dark_grey"/>
             </visual>
             <!--collision>
@@ -223,4 +228,5 @@
                     <mesh scale="1 ${side*(1)} ${side*(1)}" filename="package://centauro/centauro_urdf/meshes/schunk_hand/d11.dae" />
                 </geometry>
+                <material name="dark_grey"/>
             </visual>
             <!--collision>
@@ -237,4 +243,5 @@
                     <mesh scale="1 ${side*(1)} ${side*(1)}" filename="package://centauro/centauro_urdf/meshes/schunk_hand/d12.dae" />
                 </geometry>
+                <material name="dark_grey"/>
             </visual>
             <!--collision>
@@ -251,4 +258,5 @@
                     <mesh scale="1 ${side*(1)} ${side*(1)}" filename="package://centauro/centauro_urdf/meshes/schunk_hand/d13.dae" />
                 </geometry>
+                <material name="dark_grey"/>
             </visual>
             <!--collision>
@@ -269,4 +277,5 @@
                     <mesh filename="package://centauro/centauro_urdf/meshes/schunk_hand/f10.dae" />
                 </geometry>
+                <material name="dark_grey"/>
             </visual>
             <!--collision>
@@ -284,4 +293,5 @@
                     <mesh filename="package://centauro/centauro_urdf/meshes/schunk_hand/f11.dae" />
                 </geometry>
+                <material name="dark_grey"/>
             </visual>
             <!--collision>
@@ -300,4 +310,5 @@
                     <mesh filename="package://centauro/centauro_urdf/meshes/schunk_hand/f12.dae" />
                 </geometry>
+                <material name="dark_grey"/>
             </visual>
             <!--collision>
@@ -318,4 +329,5 @@
                     <mesh filename="package://centauro/centauro_urdf/meshes/schunk_hand/f13.dae" />
                 </geometry>
+                <material name="dark_grey"/>
             </visual>
             <!--collision>
@@ -337,4 +349,5 @@
                     <mesh filename="package://centauro/centauro_urdf/meshes/schunk_hand/f20.dae" />
                 </geometry>
+                <material name="dark_grey"/>
             </visual>
             <!--collision>
@@ -352,4 +365,5 @@
                     <mesh filename="package://centauro/centauro_urdf/meshes/schunk_hand/f21.dae" />
                 </geometry>
+                <material name="dark_grey"/>
             </visual>
             <!--collision>
@@ -369,4 +383,5 @@
                     <mesh filename="package://centauro/centauro_urdf/meshes/schunk_hand/f22.dae" />
                 </geometry>
+                <material name="dark_grey"/>
             </visual>
             <!--collision>
@@ -387,4 +402,5 @@
                     <mesh filename="package://centauro/centauro_urdf/meshes/schunk_hand/f23.dae" />
                 </geometry>
+                <material name="dark_grey"/>
             </visual>
             <!--collision>

File: centauro/centauro_urdf/urdf/models/upper_body/end_effectors/soft_hand/convex_hull.xacro (robot description, xacro)
@@ -1,3 +1,9 @@
 <?xml version="1.0" ?>
 <robot name="centauro" xmlns:xacro="http://www.ros.org/wiki/xacro">
+<xacro:macro name="soft_hand">
+    <origin xyz="0.0 0.0 -0.038"  rpy="0.0 0.0  ${PI/2+rot*PI/2}"/>
+    <geometry>
+        <mesh filename="package://centauro/centauro_urdf/meshes/convex_hull/soft_hand_open.stl" scale="${-rot*0.001} 0.001 0.001" />
+    </geometry>
+</xacro:macro>
 </robot>
