Commit message: Updated joint limits for hip yaw joints
Modify primitive position for a soft_hand

Update contact assumptions

File: centauro/centauro_urdf/urdf/centauro_leg.urdf.xacro (robot description, xacro)
@@ -94,9 +94,9 @@
 	<origin xyz="${origin_x*Leg_1_Ox} ${origin_y*Leg_1_Oy} ${Leg_1_Oz}" rpy="${Leg_1_roll} ${Leg_1_pitch} ${PI/2-origin_x*PI/2+origin_x*origin_y*Leg_1_yaw}"/>
 	<axis xyz="0 0 1"/>
+        <xacro:if value="${origin_y*origin_x == -1}">
+        <limit lower="-1.13446401" upper="2.70526034" effort="304" velocity="8.8"/>
+        </xacro:if>
         <xacro:if value="${origin_y*origin_x == 1}">
-        <limit lower="-2.35619449" upper="0.78539816" effort="304" velocity="8.8"/>
-        </xacro:if>
-        <xacro:if value="${origin_y*origin_x == -1}">
-        <limit lower="-0.78539816" upper="2.35619449" effort="304" velocity="8.8"/>
+        <limit lower="-2.70526034" upper="1.13446401" effort="304" velocity="8.8"/>
         </xacro:if>
 </joint>

File: centauro/centauro_urdf/urdf/models/upper_body/end_effectors/soft_hand/primitives.xacro (robot description, xacro)
@@ -2,5 +2,5 @@
 <robot name="centauro" xmlns:xacro="http://www.ros.org/wiki/xacro">
 <xacro:macro name="soft_hand" >
-   <origin xyz="0 0 0.10" rpy="0 0 0" />
+   <origin xyz="0 0 0.0" rpy="0 0 0" />
    <geometry>
       <box size="0.07 0.07 0.07" />

Commit message: centauro_urdf: fix wheel joint direction

File: centauro/centauro_urdf/urdf/centauro_leg.urdf.xacro (robot description, xacro)
@@ -133,5 +133,5 @@
 	<child link="wheel_${leg_num}"/>
 	<origin xyz="${Wheel_Ox} ${Wheel_Oy} ${Wheel_Oz}" rpy="${Wheel_roll} ${Wheel_pitch} ${Wheel_yaw}"/>
-	<axis xyz="0 0 1"/>
+	<axis xyz="0 0 -1"/>
         <limit  effort="35" velocity="20.0"/>
 </joint>

Commit message: centauro_urdf: centauro_leg: invert wheel joint again

File: centauro/centauro_urdf/urdf/centauro_leg.urdf.xacro (robot description, xacro)
@@ -138,5 +138,5 @@
 	<child link="wheel_${leg_num}"/>
 	<origin xyz="${Wheel_Ox} ${Wheel_Oy} ${Wheel_Oz}" rpy="${Wheel_roll} ${Wheel_pitch} ${Wheel_yaw}"/>
-	<axis xyz="0 0 -1"/>
+	<axis xyz="0 0 1"/>
         <limit  effort="35" velocity="20.0"/>
 	<dynamics friction="${friction}" damping="${damping_legs}" />

Commit message: centauro_gazebo/urdf: import of momaro wheel actuator settings
Seems to work much better.

File: centauro/centauro_urdf/urdf/centauro_leg.urdf.xacro (robot description, xacro)
@@ -139,6 +139,6 @@
 	<origin xyz="${Wheel_Ox} ${Wheel_Oy} ${Wheel_Oz}" rpy="${Wheel_roll} ${Wheel_pitch} ${Wheel_yaw}"/>
 	<axis xyz="0 0 1"/>
-        <limit  effort="35" velocity="20.0"/>
-	<dynamics friction="${friction}" damping="${damping_legs}" />
+        <limit  effort="180" velocity="2.0"/>
+<!-- 	<dynamics friction="${friction}" damping="${damping_legs}" /> -->
 </joint>
 <!--

Commit message: Added option to have fixed wheels

File: centauro/centauro_urdf/urdf/centauro_leg.urdf.xacro (robot description, xacro)
@@ -129,5 +129,5 @@
         <limit  lower="-2.79252680" upper="2.79252680" effort="35" velocity="20.0"/>
 </joint>
-<joint name="j_wheel_${leg_num}" type="continuous">
+<joint name="j_wheel_${leg_num}" type="${wheel_joint}">
 	<parent link="ankle2_${leg_num}"/>
 	<child link="wheel_${leg_num}"/>

File: centauro/centauro_urdf/urdf/config.xacro (robot description, xacro)
@@ -42,4 +42,5 @@
 <xacro:property name="reference" value="${'fixed' if (static == 'true') else 'floating'}" />
 <xacro:property name="torso_joint" value="${'fixed' if ('fixed' in [TORSO]) else 'revolute'}"/>
+<xacro:property name="wheel_joint" value="${'fixed' if ('fixed' in [WHEELS]) else 'continuous'}"/>
 <!-- ACTUATION -->
 <xacro:property name="torso_actuators" value="${'true' if ('false' not in [TORSO_ACTUATORS, TORSO]) else 'false'}"/>

Commit message: Introduced fixed link corresponding to feet FT sensors

File: centauro/centauro_urdf/urdf/centauro_leg.urdf.xacro (robot description, xacro)
@@ -136,11 +136,16 @@
         <limit  effort="35" velocity="20.0"/>
 </joint>
-<!--
-<joint name="ft_foot_${leg_num}_joint" type="fixed">
-  <parent link="knee_${leg_num}"/>
+<joint name="j_ft_foot_${leg_num}" type="fixed">
+  <parent link="ankle2_${leg_num}"/>
   <child link="ft_foot_${leg_num}"/>
-  <origin xyz="0 0 -0.3" rpy="0 0 0"/>
+  <origin xyz="${Wheel_Ox} ${Wheel_Oy} ${Wheel_Oz}" rpy="0 0 0"/>
 </joint>
--->
+<link name="ft_foot_${leg_num}">
+    <inertial>
+        <origin xyz="0 0 0"/>
+        <mass value="0"/>  <!-- org: 3.5, foot un modeled-->
+        <inertia ixx="0" ixy="0" ixz="0" iyy="0" iyz="0" izz="0"/>
+    </inertial>
+</link>
 <!-- actuators -->
 <xacro:if	value="${leg_actuators}">

Commit message: add i2r demo scene and remove joint limits temporarily

File: centauro/centauro_urdf/urdf/centauro_leg.urdf.xacro (robot description, xacro)
@@ -94,10 +94,11 @@
 	<origin xyz="${origin_x*Leg_1_Ox} ${origin_y*Leg_1_Oy} ${Leg_1_Oz}" rpy="${Leg_1_roll} ${Leg_1_pitch} ${PI/2-origin_x*PI/2+origin_x*origin_y*Leg_1_yaw}"/>
 	<axis xyz="0 0 1"/>
-        <xacro:if value="${origin_y*origin_x == -1}">
+        <!--xacro:if value="${origin_y*origin_x == -1}">
         <limit lower="-1.13446401" upper="2.70526034" effort="304" velocity="8.8"/>
         </xacro:if>
         <xacro:if value="${origin_y*origin_x == 1}">
         <limit lower="-2.70526034" upper="1.13446401" effort="304" velocity="8.8"/>
-        </xacro:if>
+        </xacro:if-->
+        <limit lower="-3" upper="3" effort="304" velocity="8.8"/>
 </joint>
 <joint name="hip_pitch_${leg_num}" type="revolute">
@@ -106,5 +107,6 @@
 	<origin xyz="${Leg_2_Ox} ${Leg_2_Oy} ${Leg_2_Oz}" rpy="${Leg_2_roll} ${Leg_2_pitch} ${origin_x*origin_y*Leg_2_yaw-origin_x*origin_y*PI/2 + PI/2}"/>
 	<axis xyz="0 0 1"/>
-        <limit lower="-2.09439510" upper="2.09439510" effort="304" velocity="8.8"/>
+        <!--limit lower="-2.09439510" upper="2.09439510" effort="304" velocity="8.8"/-->
+        <limit lower="-3" upper="3" effort="304" velocity="8.8"/>
 </joint>
 <joint name="knee_pitch_${leg_num}" type="revolute">
@@ -113,5 +115,6 @@
 	<origin xyz="${Leg_3_Ox} ${Leg_3_Oy} ${Leg_3_Oz}" rpy="${Leg_3_roll} ${Leg_3_pitch} ${Leg_3_yaw}"/>
 	<axis xyz="0 0 1"/>
-        <limit  lower="-2.61799388" upper="2.61799388" effort="304" velocity="8.8"/>
+        <!--limit  lower="-2.61799388" upper="2.61799388" effort="304" velocity="8.8"/-->
+        <limit lower="-3" upper="3" effort="304" velocity="8.8"/>
 </joint>
 <joint name="ankle_pitch_${leg_num}" type="revolute">
@@ -120,5 +123,6 @@
 	<origin xyz="${Ankle_1_Ox} ${Ankle_1_Oy} ${Ankle_1_Oz}" rpy="${Ankle_1_roll} ${Ankle_1_pitch} ${Ankle_1_yaw}"/>
 	<axis xyz="0 0 1"/>
-        <limit  lower="-2.61799388" upper="2.61799388" effort="147" velocity="8.1"/>
+        <!--limit  lower="-2.61799388" upper="2.61799388" effort="147" velocity="8.1"/-->
+        <limit lower="-3" upper="3" effort="304" velocity="8.8"/>
 </joint>
 <joint name="ankle_yaw_${leg_num}" type="revolute">
@@ -127,5 +131,6 @@
 	<origin xyz="${Ankle_2_Ox} ${Ankle_2_Oy} ${Ankle_2_Oz}" rpy="${Ankle_2_roll} ${Ankle_2_pitch} ${Ankle_2_yaw}"/>
 	<axis xyz="0 0 1"/>
-        <limit  lower="-2.79252680" upper="2.79252680" effort="35" velocity="20.0"/>
+        <!--limit  lower="-2.79252680" upper="2.79252680" effort="35" velocity="20.0"/-->
+        <limit lower="-3" upper="3" effort="304" velocity="8.8"/>
 </joint>
 <joint name="j_wheel_${leg_num}" type="continuous">
@@ -135,4 +140,5 @@
 	<axis xyz="0 0 1"/>
         <limit  effort="35" velocity="20.0"/>
+        <dynamics friction="5" damping="2.0"/>
 </joint>
 <!--

Commit message: add dustbin and box

File: centauro/centauro_urdf/urdf/centauro_leg.urdf.xacro (robot description, xacro)
@@ -107,6 +107,6 @@
 	<origin xyz="${Leg_2_Ox} ${Leg_2_Oy} ${Leg_2_Oz}" rpy="${Leg_2_roll} ${Leg_2_pitch} ${origin_x*origin_y*Leg_2_yaw-origin_x*origin_y*PI/2 + PI/2}"/>
 	<axis xyz="0 0 1"/>
-        <!--limit lower="-2.09439510" upper="2.09439510" effort="304" velocity="8.8"/-->
-        <limit lower="-3" upper="3" effort="304" velocity="8.8"/>
+        <limit lower="-2.09439510" upper="2.09439510" effort="304" velocity="8.8"/>
+        <!--limit lower="-3" upper="3" effort="304" velocity="8.8"/-->
 </joint>
 <joint name="knee_pitch_${leg_num}" type="revolute">
@@ -115,6 +115,6 @@
 	<origin xyz="${Leg_3_Ox} ${Leg_3_Oy} ${Leg_3_Oz}" rpy="${Leg_3_roll} ${Leg_3_pitch} ${Leg_3_yaw}"/>
 	<axis xyz="0 0 1"/>
-        <!--limit  lower="-2.61799388" upper="2.61799388" effort="304" velocity="8.8"/-->
-        <limit lower="-3" upper="3" effort="304" velocity="8.8"/>
+        <limit  lower="-2.61799388" upper="2.61799388" effort="304" velocity="8.8"/>
+        <!--limit lower="-3" upper="3" effort="304" velocity="8.8"/-->
 </joint>
 <joint name="ankle_pitch_${leg_num}" type="revolute">
@@ -123,6 +123,6 @@
 	<origin xyz="${Ankle_1_Ox} ${Ankle_1_Oy} ${Ankle_1_Oz}" rpy="${Ankle_1_roll} ${Ankle_1_pitch} ${Ankle_1_yaw}"/>
 	<axis xyz="0 0 1"/>
-        <!--limit  lower="-2.61799388" upper="2.61799388" effort="147" velocity="8.1"/-->
-        <limit lower="-3" upper="3" effort="304" velocity="8.8"/>
+        <limit  lower="-2.61799388" upper="2.61799388" effort="147" velocity="8.1"/>
+        <!--limit lower="-3" upper="3" effort="304" velocity="8.8"/-->
 </joint>
 <joint name="ankle_yaw_${leg_num}" type="revolute">
@@ -131,6 +131,6 @@
 	<origin xyz="${Ankle_2_Ox} ${Ankle_2_Oy} ${Ankle_2_Oz}" rpy="${Ankle_2_roll} ${Ankle_2_pitch} ${Ankle_2_yaw}"/>
 	<axis xyz="0 0 1"/>
-        <!--limit  lower="-2.79252680" upper="2.79252680" effort="35" velocity="20.0"/-->
-        <limit lower="-3" upper="3" effort="304" velocity="8.8"/>
+        <limit  lower="-2.79252680" upper="2.79252680" effort="35" velocity="20.0"/>
+        <!--limit lower="-3" upper="3" effort="304" velocity="8.8"/-->
 </joint>
 <joint name="j_wheel_${leg_num}" type="continuous">
@@ -140,5 +140,5 @@
 	<axis xyz="0 0 1"/>
         <limit  effort="35" velocity="20.0"/>
-        <dynamics friction="5" damping="2.0"/>
+        <!--dynamics friction="10" damping="1.0"/-->
 </joint>
 <!--

Commit message: demo1

File: centauro/centauro_urdf/urdf/centauro_leg.urdf.xacro (robot description, xacro)
@@ -140,5 +140,5 @@
 	<axis xyz="0 0 1"/>
         <limit  effort="35" velocity="20.0"/>
-        <!--dynamics friction="10" damping="1.0"/-->
+        <dynamics friction="10" damping="1.0"/>
 </joint>
 <!--

Commit message: add grasp world file

File: centauro/centauro_urdf/urdf/centauro_leg.urdf.xacro (robot description, xacro)
@@ -107,6 +107,6 @@
 	<origin xyz="${Leg_2_Ox} ${Leg_2_Oy} ${Leg_2_Oz}" rpy="${Leg_2_roll} ${Leg_2_pitch} ${origin_x*origin_y*Leg_2_yaw-origin_x*origin_y*PI/2 + PI/2}"/>
 	<axis xyz="0 0 1"/>
-        <limit lower="-2.09439510" upper="2.09439510" effort="304" velocity="8.8"/>
-        <!--limit lower="-3" upper="3" effort="304" velocity="8.8"/-->
+        <!--limit lower="-2.09439510" upper="2.09439510" effort="304" velocity="8.8"/-->
+        <limit lower="-3" upper="3" effort="304" velocity="8.8"/>
 </joint>
 <joint name="knee_pitch_${leg_num}" type="revolute">
@@ -115,6 +115,6 @@
 	<origin xyz="${Leg_3_Ox} ${Leg_3_Oy} ${Leg_3_Oz}" rpy="${Leg_3_roll} ${Leg_3_pitch} ${Leg_3_yaw}"/>
 	<axis xyz="0 0 1"/>
-        <limit  lower="-2.61799388" upper="2.61799388" effort="304" velocity="8.8"/>
-        <!--limit lower="-3" upper="3" effort="304" velocity="8.8"/-->
+        <!--limit  lower="-2.61799388" upper="2.61799388" effort="304" velocity="8.8"/-->
+        <limit lower="-3" upper="3" effort="304" velocity="8.8"/>
 </joint>
 <joint name="ankle_pitch_${leg_num}" type="revolute">
@@ -123,6 +123,6 @@
 	<origin xyz="${Ankle_1_Ox} ${Ankle_1_Oy} ${Ankle_1_Oz}" rpy="${Ankle_1_roll} ${Ankle_1_pitch} ${Ankle_1_yaw}"/>
 	<axis xyz="0 0 1"/>
-        <limit  lower="-2.61799388" upper="2.61799388" effort="147" velocity="8.1"/>
-        <!--limit lower="-3" upper="3" effort="304" velocity="8.8"/-->
+        <!--limit  lower="-2.61799388" upper="2.61799388" effort="147" velocity="8.1"/-->
+        <limit lower="-3" upper="3" effort="304" velocity="8.8"/>
 </joint>
 <joint name="ankle_yaw_${leg_num}" type="revolute">

Commit message: add grasp world file

File: centauro/centauro_urdf/urdf/centauro_leg.urdf.xacro (robot description, xacro)
@@ -140,5 +140,5 @@
 	<axis xyz="0 0 1"/>
         <limit  effort="35" velocity="20.0"/>
-        <dynamics friction="10" damping="1.0"/>
+        <dynamics friction="1" damping="1.0"/>
 </joint>
 <!--

Commit message: use a bigger pallet

File: centauro/centauro_urdf/urdf/centauro_leg.urdf.xacro (robot description, xacro)
@@ -100,5 +100,5 @@
         <limit lower="-2.70526034" upper="1.13446401" effort="304" velocity="8.8"/>
         </xacro:if-->
-        <limit lower="-3" upper="3" effort="304" velocity="8.8"/>
+        <limit lower="-2.7" upper="2.7" effort="304" velocity="8.8"/>
 </joint>
 <joint name="hip_pitch_${leg_num}" type="revolute">
@@ -107,6 +107,6 @@
 	<origin xyz="${Leg_2_Ox} ${Leg_2_Oy} ${Leg_2_Oz}" rpy="${Leg_2_roll} ${Leg_2_pitch} ${origin_x*origin_y*Leg_2_yaw-origin_x*origin_y*PI/2 + PI/2}"/>
 	<axis xyz="0 0 1"/>
-        <!--limit lower="-2.09439510" upper="2.09439510" effort="304" velocity="8.8"/-->
-        <limit lower="-3" upper="3" effort="304" velocity="8.8"/>
+        <limit lower="-2.09439510" upper="2.09439510" effort="304" velocity="8.8"/>
+        <!--limit lower="-3" upper="3" effort="304" velocity="8.8"/-->
 </joint>
 <joint name="knee_pitch_${leg_num}" type="revolute">
@@ -115,6 +115,6 @@
 	<origin xyz="${Leg_3_Ox} ${Leg_3_Oy} ${Leg_3_Oz}" rpy="${Leg_3_roll} ${Leg_3_pitch} ${Leg_3_yaw}"/>
 	<axis xyz="0 0 1"/>
-        <!--limit  lower="-2.61799388" upper="2.61799388" effort="304" velocity="8.8"/-->
-        <limit lower="-3" upper="3" effort="304" velocity="8.8"/>
+        <limit  lower="-2.61799388" upper="2.61799388" effort="304" velocity="8.8"/>
+        <!--limit lower="-3" upper="3" effort="304" velocity="8.8"/-->
 </joint>
 <joint name="ankle_pitch_${leg_num}" type="revolute">
@@ -123,6 +123,6 @@
 	<origin xyz="${Ankle_1_Ox} ${Ankle_1_Oy} ${Ankle_1_Oz}" rpy="${Ankle_1_roll} ${Ankle_1_pitch} ${Ankle_1_yaw}"/>
 	<axis xyz="0 0 1"/>
-        <!--limit  lower="-2.61799388" upper="2.61799388" effort="147" velocity="8.1"/-->
-        <limit lower="-3" upper="3" effort="304" velocity="8.8"/>
+        <limit  lower="-2.61799388" upper="2.61799388" effort="147" velocity="8.1"/>
+        <!--limit lower="-3" upper="3" effort="304" velocity="8.8"/-->
 </joint>
 <joint name="ankle_yaw_${leg_num}" type="revolute">
@@ -140,5 +140,5 @@
 	<axis xyz="0 0 1"/>
         <limit  effort="35" velocity="20.0"/>
-        <dynamics friction="1" damping="1.0"/>
+        <dynamics friction="5" damping="1.0"/>
 </joint>
 <!--

Commit message: fixing wheel joints z axis sign.

File: centauro/centauro_urdf/urdf/centauro_leg.urdf.xacro (robot description, xacro)
@@ -128,5 +128,5 @@
 	<child link="wheel_${leg_num}"/>
 	<origin xyz="${Wheel_Ox} ${Wheel_Oy} ${Wheel_Oz}" rpy="${Wheel_roll} ${Wheel_pitch} ${Wheel_yaw}"/>
-	<axis xyz="0 0 1"/>
+	<axis xyz="0 0 -1"/>
         <limit  effort="35" velocity="20.0"/>
 </joint>

Commit message: try box collision shapes

File: centauro/centauro_urdf/urdf/centauro_leg.urdf.xacro (robot description, xacro)
@@ -45,4 +45,8 @@
       <collision>
          <xacro:collision_model.leg3 />
+        <origin xyz="0.1 0.0 0.0" rpy="0 0 0"/>
+        <!--geometry>
+          <box size="0.3 0.06 0.06"/>
+        </geometry-->
       </collision>
 </link>
@@ -94,11 +98,11 @@
 	<origin xyz="${origin_x*Leg_1_Ox} ${origin_y*Leg_1_Oy} ${Leg_1_Oz}" rpy="${Leg_1_roll} ${Leg_1_pitch} ${PI/2-origin_x*PI/2+origin_x*origin_y*Leg_1_yaw}"/>
 	<axis xyz="0 0 1"/>
-        <!--xacro:if value="${origin_y*origin_x == -1}">
+        <xacro:if value="${origin_y*origin_x == -1}">
         <limit lower="-1.13446401" upper="2.70526034" effort="304" velocity="8.8"/>
         </xacro:if>
         <xacro:if value="${origin_y*origin_x == 1}">
         <limit lower="-2.70526034" upper="1.13446401" effort="304" velocity="8.8"/>
-        </xacro:if-->
-        <limit lower="-2.7" upper="2.7" effort="304" velocity="8.8"/>
+        </xacro:if>
+        <!--limit lower="-2.7" upper="2.7" effort="304" velocity="8.8"/-->
 </joint>
 <joint name="hip_pitch_${leg_num}" type="revolute">

Commit message: Restore correct wheel orientation

File: centauro/centauro_urdf/urdf/centauro_leg.urdf.xacro (robot description, xacro)
@@ -128,5 +128,5 @@
 	<child link="wheel_${leg_num}"/>
 	<origin xyz="${Wheel_Ox} ${Wheel_Oy} ${Wheel_Oz}" rpy="${Wheel_roll} ${Wheel_pitch} ${Wheel_yaw}"/>
-	<axis xyz="0 0 -1"/>
+	<axis xyz="0 0 1"/>
         <limit  effort="35" velocity="20.0"/>
 </joint>
