Commit message: strange local changes (imu pos)

File: centauro/centauro_urdf/urdf/centauro_temp1.urdf (robot description, URDF)
Before this commit: robot centauro, 93 links, 92 joints
Links:
- removed link kinect2_rgb_frame
- removed link velodyne_calib
Joints:
- removed joint j_kinect2_rgb_frame
- removed joint velodyne_calib
- joint imu_joint: origin xyz=0.248316 0.0 0.015 rpy=0.0 0.0 0.0 -> xyz=0.0 0.0 0.0 rpy=0.0 0.0 0.0
- joint j_kinect_optical_frame: origin rpy= -1.5707963268 0 -1.5707963268 -> xyz=0.050 -0.110 -0.035 rpy= -1.5707963268 0 -1.5707963268; parent kinect2_rgb_frame -> kinect
