Commit message: Hand/stick must be a fixed joint

File: centauro/centauro_urdf/urdf/centauro_hand.urdf.xacro (robot description, xacro)
@@ -17,5 +17,5 @@
    </link>
 <!-- /links -->
-   <joint name="j_arm${arm_num}_8" type="revolute">
+   <joint name="j_arm${arm_num}_8" type="fixed">
       <parent link="arm${arm_num}_7"/>
       <child link="arm${arm_num}_8"/>

File: centauro/centauro_urdf/urdf/centauro_stick.urdf.xacro (robot description, xacro)
@@ -19,5 +19,5 @@
 <!-- /links -->
 <!-- joints -->
-   <joint name="j_arm${arm_num}_8" type="revolute">
+   <joint name="j_arm${arm_num}_8" type="fixed">
       <parent link="arm${arm_num}_7"/>
       <child link="arm${arm_num}_8"/>

Commit message: some little changes to the simulation again

File: centauro/centauro_urdf/urdf/centauro_hand.urdf.xacro (robot description, xacro)
@@ -17,4 +17,5 @@
    </link>
 <!-- /links -->
+<!-- joints -->
    <joint name="j_arm${arm_num}_8" type="revolute">
       <parent link="arm${arm_num}_7"/>
@@ -22,9 +23,6 @@
       <origin xyz="${End_effector_Ox} ${End_effector_Oy} ${End_effector_Oz}" rpy="${End_effector_roll} ${End_effector_pitch} ${End_effector_yaw}"/>
       <axis xyz="1 0 0" />
-      <limit velocity="20.3" effort="40" lower="0.0" upper="1.57075" />
+      <limit velocity="0" effort="0" lower="0.0" upper="0" />
    </joint> -->
 <!-- /joints -->
-<!-- actuators -->
-   <xacro:position_actuator joint="j_arm${arm_num}_8" />
-<!-- /actuators -->
 </robot>

Commit message: Modified limits on soft_hand. Added debris removal task launch and world

File: centauro/centauro_urdf/urdf/centauro_hand.urdf.xacro (robot description, xacro)
@@ -30,5 +30,5 @@
       <xacro:if value="${joint not in ['fixed']}" >
          <axis xyz="0 1 0" />
-         <limit velocity="20.3" effort="40" lower="0.0" upper="1.57075" />
+         <limit velocity="20.3" effort="40" lower="0.0" upper="0.0" />
       </xacro:if>
    </joint> -->

Commit message: back

File: centauro/centauro_urdf/urdf/centauro_hand.urdf.xacro (robot description, xacro)
@@ -30,5 +30,5 @@
       <xacro:if value="${joint not in ['fixed']}" >
          <axis xyz="0 1 0" />
-         <limit velocity="20.3" effort="40" lower="0.0" upper="0.0" />
+         <limit velocity="20.3" effort="40" lower="0.0" upper="1.57075" />
       </xacro:if>
    </joint> -->

Commit message: If false for ft_sensors produce the fixed joint else revolute

File: centauro/centauro_urdf/urdf/centauro_hand.urdf.xacro (robot description, xacro)
@@ -19,12 +19,12 @@
 <!-- /links -->
    <joint name="j_arm${arm_num}_8" type="${joint}">
-      <xacro:if value="${ft_sensors == 'true'}" >
+<!--      <xacro:if value="${ft_sensors == 'true'}" > -->
          <parent link="ft_arm${arm_num}"/>
          <origin xyz="${Hand_ft_Ox} ${Hand_ft_Oy} ${Hand_ft_Oz}" rpy="${Hand_ft_roll} ${Hand_ft_pitch} ${Hand_ft_yaw}"/>
-      </xacro:if>
-      <xacro:unless value="${ft_sensors == 'true'}" >
+<!--      </xacro:if> -->
+<!--      <xacro:unless value="${ft_sensors == 'true'}" >
          <parent link="arm${arm_num}_7"/>
          <origin xyz="${Hand_Ox} ${Hand_Oy} ${Hand_Oz}" rpy="${Hand_roll} ${Hand_pitch} ${Hand_yaw}"/>
-      </xacro:unless>
+      </xacro:unless> -->
       <child link="arm${arm_num}_8"/>
       <xacro:if value="${joint not in ['fixed']}" >

File: centauro/centauro_urdf/urdf/centauro_heri.urdf.xacro (robot description, xacro)
@@ -20,12 +20,12 @@
 <!-- joints -->
    <joint name="j_arm${arm_num}_8" type="fixed">
-      <xacro:if value="${ft_sensors == 'true'}" >
+<!--      <xacro:if value="${ft_sensors == 'true'}" > -->
          <parent link="ft_arm${arm_num}"/>
          <origin xyz="${Heri_ft_Ox} ${Heri_ft_Oy} ${Heri_ft_Oz}" rpy="${Heri_ft_roll} ${Heri_ft_pitch} ${Heri_ft_yaw}"/>
-      </xacro:if>
+<!--      </xacro:if>
       <xacro:unless value="${ft_sensors == 'true'}" >
          <parent link="arm${arm_num}_7"/>
          <origin xyz="${Heri_Ox} ${Heri_Oy} ${Heri_Oz}" rpy="${Heri_roll} ${Heri_pitch} ${Heri_yaw}"/>
-      </xacro:unless>
+      </xacro:unless> -->
       <child link="arm${arm_num}_8"/>
       <axis xyz="1 0 0" />

File: centauro/centauro_urdf/urdf/centauro_no_end_effector.urdf.xacro (robot description, xacro)
@@ -5,12 +5,12 @@
 <!-- /links -->
    <joint name="j_arm${arm_num}_8" type="revolute">
-      <xacro:if value="${ft_sensors == 'true'}" >
+<!--      <xacro:if value="${ft_sensors == 'true'}" > -->
          <parent link="ft_arm${arm_num}"/>
          <origin xyz="${No_end_ft_Ox} ${No_end_ft_Oy} ${No_end_ft_Oz}" rpy="${No_end_ft_roll} ${No_end_ft_pitch} ${No_end_ft_yaw}"/>
-      </xacro:if>
-      <xacro:unless value="${ft_sensors == 'true'}" >
+<!--      </xacro:if> -->
+<!--      <xacro:unless value="${ft_sensors == 'true'}" >
          <parent link="arm${arm_num}_7"/>
          <origin xyz="${No_end_Ox} ${No_end_Oy} ${No_end_Oz}" rpy="${No_end_roll} ${No_end_pitch} ${No_end_yaw}"/>
-      </xacro:unless>
+      </xacro:unless> -->
       <child link="arm${arm_num}_8"/>
       <axis xyz="1 0 0" />

File: centauro/centauro_urdf/urdf/centauro_stick.urdf.xacro (robot description, xacro)
@@ -20,12 +20,12 @@
 <!-- joints -->
    <joint name="j_arm${arm_num}_8" type="fixed">
-      <xacro:if value="${ft_sensors == 'true'}" >
+<!--      <xacro:if value="${ft_sensors == 'true'}" > -->
          <parent link="ft_arm${arm_num}"/>
          <origin xyz="${Stick_ft_Ox} ${Stick_ft_Oy} ${Stick_ft_Oz}" rpy="${Stick_ft_roll} ${Stick_ft_pitch} ${Stick_ft_yaw}"/>
-      </xacro:if>
+<!--      </xacro:if>
       <xacro:unless value="${ft_sensors == 'true'}" >
          <parent link="arm${arm_num}_7"/>
          <origin xyz="${Stick_Ox} ${Stick_Oy} ${Stick_Oz}" rpy="${Stick_roll} ${Stick_pitch} ${Stick_yaw}"/>
-      </xacro:unless>
+      </xacro:unless> -->
       <child link="arm${arm_num}_8"/>
       <axis xyz="1 0 0" />

File: centauro/centauro_urdf/urdf/config.xacro (robot description, xacro)
@@ -57,5 +57,5 @@
 <xacro:property name="arm_sensors" value="${'true' if ('false' not in [ARM_SENSORS, arms]) else 'false'}"/>
 <xacro:property name="leg_sensors" value="${'true' if ('false' not in [LEG_SENSORS, legs]) else 'false'}"/>
-<xacro:property name="ft_sensors" value="${'true' if ('false' not in [FT_SENSORS]) else 'false'}"/>
+<xacro:property name="ft_sensors" value="${'revolute' if ('false' not in [FT_SENSORS]) else 'fixed'}"/>
 <xacro:property name="bumbers" value="${'true' if ('false' not in [BUMBERS]) else 'false'}"/>
 <xacro:property name="imu" value="${'true' if ('false' not in [IMU, pelvis]) else 'false'}"/>

File: centauro_gazebo/sensors/config.xacro (robot description, xacro)
@@ -15,5 +15,5 @@
    </xacro:macro>
 <!-- Load all controllers macros -->
-<xacro:if value="${ft_sensors}">
+<xacro:if value="${ft_sensors == 'revolute'}">
         <xacro:load_model middleware="${middleware}" sensor="ft_sensor" arm_sensors="${arm_sensors}" leg_sensors="${leg_sensors}" head_sensors="false"/>
 </xacro:if>

File: centauro_gazebo/sensors/ros_control/ft_sensor/load/legs.xacro (robot description, xacro)
@@ -1,3 +1,7 @@
 <!--<?xml version="1.0"?>-->
 <robot  xmlns:xacro="http://www.ros.org/wiki/xacro">
+  <xacro:force-torque_sensor joint="ankle_yaw_1" robot="centauro"/>
+  <xacro:force-torque_sensor joint="ankle_yaw_2" robot="centauro"/>
+  <xacro:force-torque_sensor joint="ankle_yaw_3" robot="centauro"/>
+  <xacro:force-torque_sensor joint="ankle_yaw_4" robot="centauro"/>
 </robot>
