Commit message: Adding IMU to pelvis link

File: centauro/centauro_urdf/urdf/centauro.urdf.xacro (robot description, xacro)
@@ -12,4 +12,5 @@
 <xacro:include filename="${inertia_parameters_file}"/>
 <xacro:include filename="${kinematic_parameters_file}"/>
+<xacro:include filename="${sensor_parameters_file}"/>
 <xacro:include filename="$(find centauro)/centauro_urdf/materials.xacro"/>
 <xacro:include filename="$(find centauro)/centauro_urdf/urdf/models/model.xacro"/>

File: centauro/centauro_urdf/urdf/centauro_torso.urdf.xacro (robot description, xacro)
@@ -17,4 +17,10 @@
 	</collision>
 </link>
+<link name="imu_link">
+    <inertial>
+        <mass value="0.0"/> <!-- mass  7: torso_1 (2) + torso_2 (5), head un_modelled -->
+        <inertia ixx="0.0" ixy="0.0" ixz="0.0" iyy="0.0" iyz="0.0" izz="0.0"/>
+    </inertial>
+</link>
 <!-- /torso links -->
 <!-- torso joints -->
@@ -32,4 +38,15 @@
    <limit lower="-2.618" upper="2.618" effort="147" velocity="5.7"/> <!-- TODO -->
 </joint>
+<joint name="imu_joint" type="fixed">
+   <xacro:if value="${pelvis}">
+      <parent link="pelvis"/>
+      <origin xyz="${Imu_x} ${Imu_y} ${Imu_z}"/>
+   </xacro:if>
+   <xacro:unless value="${pelvis}">
+      <parent link="world"/>
+      <origin xyz="${Imu_x + Pelvis_Ox} ${Imu_y + Pelvis_Oy} ${Imu_z + Pelvis_Oz}"/>
+   </xacro:unless>
+   <child link="imu_link"/>
+</joint>
 <!-- /torso joints -->
 <xacro:if	value="${torso_actuators}">

File: centauro/centauro_urdf/urdf/config.xacro (robot description, xacro)
@@ -40,3 +40,4 @@
 <xacro:property name="inertia_parameters_file" value="${package + '/centauro_urdf/inertia_parameters/' + INERTIA_PARAM + '.xacro'}"/>
 <xacro:property name="kinematic_parameters_file" value="${package + '/centauro_urdf/kinematic_parameters/' + KINEMATIC_PARAM + '.xacro'}"/>
+<xacro:property name="sensor_parameters_file" value="${package + '/centauro_urdf/sensor_parameters/' + 'original.xacro'}"/>
 </robot>

Commit message: Imu is now attached to pelvis

File: centauro/centauro_urdf/urdf/centauro.urdf.xacro (robot description, xacro)
@@ -39,8 +39,25 @@
       </collision>
    </link>
+   <link name="imu_link">
+     <inertial>
+        <mass value="0.0"/> <!-- mass  7: torso_1 (2) + torso_2 (5), head un_modelled -->
+        <inertia ixx="0.0" ixy="0.0" ixz="0.0" iyy="0.0" iyz="0.0" izz="0.0"/>
+     </inertial>
+   </link>
 </xacro:if>
 <xacro:unless value="${pelvis}">
    <link name="pelvis"/>
 </xacro:unless>
+<joint name="imu_joint" type="fixed">
+   <xacro:if value="${pelvis}">
+      <parent link="pelvis"/>
+      <origin xyz="${Imu_x} ${Imu_y} ${Imu_z}"/>
+   </xacro:if>
+   <xacro:unless value="${pelvis}">
+      <parent link="world"/>
+      <origin xyz="${Imu_x + Pelvis_Ox} ${Imu_y + Pelvis_Oy} ${Imu_z + Pelvis_Oz}"/>
+   </xacro:unless>
+   <child link="imu_link"/>
+</joint>
 <joint name="reference" type="${reference}">
    <origin xyz="${Pelvis_Ox} ${Pelvis_Oy} ${Pelvis_Oz}"/>

File: centauro/centauro_urdf/urdf/centauro_torso.urdf.xacro (robot description, xacro)
@@ -15,10 +15,4 @@
 	</collision>
 </link>
-<link name="imu_link">
-    <inertial>
-        <mass value="0.0"/> <!-- mass  7: torso_1 (2) + torso_2 (5), head un_modelled -->
-        <inertia ixx="0.0" ixy="0.0" ixz="0.0" iyy="0.0" iyz="0.0" izz="0.0"/>
-    </inertial>
-</link>
 <!-- /torso links -->
 <!-- torso joints -->
@@ -36,15 +30,4 @@
    <limit lower="-2.618" upper="2.618" effort="147" velocity="5.7"/> <!-- TODO -->
 </joint>
-<joint name="imu_joint" type="fixed">
-   <xacro:if value="${pelvis}">
-      <parent link="pelvis"/>
-      <origin xyz="${Imu_x} ${Imu_y} ${Imu_z}"/>
-   </xacro:if>
-   <xacro:unless value="${pelvis}">
-      <parent link="world"/>
-      <origin xyz="${Imu_x + Pelvis_Ox} ${Imu_y + Pelvis_Oy} ${Imu_z + Pelvis_Oz}"/>
-   </xacro:unless>
-   <child link="imu_link"/>
-</joint>
 <!-- /torso joints -->
 <xacro:if	value="${torso_actuators}">

Commit message: Revert "Imu is now attached to pelvis"
This reverts commit 51695f9f89b7bc254a93e32ab88b08c9a2354bbc.

File: centauro/centauro_urdf/urdf/centauro.urdf.xacro (robot description, xacro)
@@ -39,25 +39,8 @@
       </collision>
    </link>
-   <link name="imu_link">
-     <inertial>
-        <mass value="0.0"/> <!-- mass  7: torso_1 (2) + torso_2 (5), head un_modelled -->
-        <inertia ixx="0.0" ixy="0.0" ixz="0.0" iyy="0.0" iyz="0.0" izz="0.0"/>
-     </inertial>
-   </link>
 </xacro:if>
 <xacro:unless value="${pelvis}">
    <link name="pelvis"/>
 </xacro:unless>
-<joint name="imu_joint" type="fixed">
-   <xacro:if value="${pelvis}">
-      <parent link="pelvis"/>
-      <origin xyz="${Imu_x} ${Imu_y} ${Imu_z}"/>
-   </xacro:if>
-   <xacro:unless value="${pelvis}">
-      <parent link="world"/>
-      <origin xyz="${Imu_x + Pelvis_Ox} ${Imu_y + Pelvis_Oy} ${Imu_z + Pelvis_Oz}"/>
-   </xacro:unless>
-   <child link="imu_link"/>
-</joint>
 <joint name="reference" type="${reference}">
    <origin xyz="${Pelvis_Ox} ${Pelvis_Oy} ${Pelvis_Oz}"/>

File: centauro/centauro_urdf/urdf/centauro_torso.urdf.xacro (robot description, xacro)
@@ -15,4 +15,10 @@
 	</collision>
 </link>
+<link name="imu_link">
+    <inertial>
+        <mass value="0.0"/> <!-- mass  7: torso_1 (2) + torso_2 (5), head un_modelled -->
+        <inertia ixx="0.0" ixy="0.0" ixz="0.0" iyy="0.0" iyz="0.0" izz="0.0"/>
+    </inertial>
+</link>
 <!-- /torso links -->
 <!-- torso joints -->
@@ -30,4 +36,15 @@
    <limit lower="-2.618" upper="2.618" effort="147" velocity="5.7"/> <!-- TODO -->
 </joint>
+<joint name="imu_joint" type="fixed">
+   <xacro:if value="${pelvis}">
+      <parent link="pelvis"/>
+      <origin xyz="${Imu_x} ${Imu_y} ${Imu_z}"/>
+   </xacro:if>
+   <xacro:unless value="${pelvis}">
+      <parent link="world"/>
+      <origin xyz="${Imu_x + Pelvis_Ox} ${Imu_y + Pelvis_Oy} ${Imu_z + Pelvis_Oz}"/>
+   </xacro:unless>
+   <child link="imu_link"/>
+</joint>
 <!-- /torso joints -->
 <xacro:if	value="${torso_actuators}">

Commit message: Fix issue with imu & legs:=false

File: centauro/centauro_urdf/urdf/centauro.urdf.xacro (robot description, xacro)
@@ -45,9 +45,5 @@
      </inertial>
    </link>
-</xacro:if>
-<xacro:unless value="${pelvis}">
-   <link name="pelvis"/>
-</xacro:unless>
-<joint name="imu_joint" type="fixed">
+   <joint name="imu_joint" type="fixed">
    <xacro:if value="${pelvis}">
       <parent link="pelvis"/>
@@ -60,4 +56,8 @@
    <child link="imu_link"/>
 </joint>
+</xacro:if>
+<xacro:unless value="${pelvis}">
+   <link name="pelvis"/>
+</xacro:unless>
 <joint name="reference" type="${reference}">
    <origin xyz="${Pelvis_Ox} ${Pelvis_Oy} ${Pelvis_Oz}"/>

Commit message: Integration with XBot

File: centauro/centauro_urdf/urdf/centauro.urdf.xacro (robot description, xacro)
@@ -38,4 +38,15 @@
       </collision>
    </link>
+    <link name="imu_link">
+        <inertial>
+            <mass value="0.0"/>
+            <inertia ixx="0.0" ixy="0.0" ixz="0.0" iyy="0.0" iyz="0.0" izz="0.0"/>
+        </inertial>
+    </link>
+    <joint name="imu_joint" type="fixed">
+        <parent link="pelvis"/>
+        <origin xyz="${Imu_Ox} ${Imu_Oy} ${Imu_Oz}" rpy="${Imu_raw} ${Imu_pitch} ${Imu_yaw}"/>
+        <child link="imu_link"/>
+    </joint>
 </xacro:if>
 <xacro:unless value="${pelvis}">

File: centauro/centauro_urdf/urdf/config.xacro (robot description, xacro)
@@ -14,5 +14,5 @@
 <xacro:property name="ONE_ARM" value="$(arg ONE_ARM)"/>
 <xacro:property name="GAZEBO" value="$(arg GAZEBO)"/>
-<xacro:property name="CONTROLLER" value="$(arg CONTROLLER)"/>
+<xacro:property name="MIDDLEWARE" value="$(arg MIDDLEWARE)"/>
 <xacro:property name="INERTIA_PARAM" value="$(arg INERTIA_PARAM)"/>
 <xacro:property name="KINEMATIC_PARAM" value="$(arg KINEMATIC_PARAM)"/>
@@ -22,4 +22,8 @@
 <xacro:property name="WHEELS_ACTUATORS" value="$(arg WHEELS_ACTUATORS)"/>
 <xacro:property name="ARM_SENSORS" value="$(arg ARM_SENSORS)"/>
+<xacro:property name="LEG_SENSORS" value="$(arg LEG_SENSORS)"/>
+<xacro:property name="FT_SENSORS" value="$(arg FT_SENSORS)"/>
+<xacro:property name="BUMBERS" value="$(arg BUMBERS)"/>
+<xacro:property name="IMU" value="$(arg IMU)"/>
 <xacro:property name="MASS" value="$(arg MASS)"/>
 <!-- dependend arguments -->
@@ -32,12 +36,19 @@
 <xacro:property name="static" value="${'true' if ('true' in [STATIC, ONE_ARM] or 'false' in [legs, LEG_ACTUATORS]) else 'false'}"/>
 <xacro:property name="reference" value="${'fixed' if (static == 'true') else 'floating'}" />
+<!-- ACTUATION -->
 <xacro:property name="torso_actuators" value="${'true' if ('false' not in [TORSO_ACTUATORS, TORSO]) else 'false'}"/>
 <xacro:property name="arm_actuators" value="${'true' if ('false' not in [ARM_ACTUATORS, TORSO_ACTUATORS, arm]) else 'false'}"/>
 <xacro:property name="leg_actuators" value="${'true' if ('false' not in [LEG_ACTUATORS, legs]) else 'false'}"/>
 <xacro:property name="wheels_actuators" value="${'true' if ('false' not in [WHEELS_ACTUATORS, LEG_ACTUATORS, wheels]) else 'false'}"/>
+<!-- SENSORS -->
 <xacro:property name="arm_sensors" value="${'true' if ('false' not in [ARM_SENSORS, arm]) else 'false'}"/>
-<xacro:property name="leg_sensors" value="${'true' if ('false' not in [legs]) else 'false'}"/>
+<xacro:property name="leg_sensors" value="${'true' if ('false' not in [LEG_SENSORS, legs]) else 'false'}"/>
+<xacro:property name="ft_sensors" value="${'true' if ('false' not in [FT_SENSORS]) else 'false'}"/>
+<xacro:property name="bumbers" value="${'true' if ('false' not in [BUMBERS]) else 'false'}"/>
+<xacro:property name="imu" value="${'true' if ('false' not in [IMU, pelvis]) else 'false'}"/>
+<!-- LOAD PARAMETERS -->
 <xacro:property name="package" value="$(find centauro)"/>
 <xacro:property name="inertia_parameters_file" value="${package + '/centauro_urdf/inertia_parameters/' + INERTIA_PARAM + '.xacro'}"/>
 <xacro:property name="kinematic_parameters_file" value="${package + '/centauro_urdf/kinematic_parameters/' + KINEMATIC_PARAM + '.xacro'}"/>
+<xacro:property name="middleware" value="${MIDDLEWARE}"/>
 </robot>

File: centauro/centauro_urdf/urdf/models/model_config.xacro (robot description, xacro)
@@ -5,22 +5,13 @@
    <xacro:macro name="load_model" params="path model">
    <!-- load proper collision model -->
-      <xacro:include filename="$(find centauro)/centauro_urdf/urdf/models/${path}/primitives.xacro"/>
-      <xacro:if value="${model == 'mesh'}">
-         <xacro:include filename="$(find centauro)/centauro_urdf/urdf/models/${path}/meshes.xacro"/>
-      </xacro:if>
-      <xacro:if value="${model == 'capsule'}">
-         <xacro:include filename="$(find centauro)/centauro_urdf/urdf/models/${path}/capsules.xacro"/>
-      </xacro:if>
-      <xacro:if value="${model == 'convex_hull'}">
-         <xacro:include filename="$(find centauro)/centauro_urdf/urdf/models/${path}/convex_hull.xacro"/>
+      <xacro:include filename="$(find centauro)/centauro_urdf/urdf/models/${path}/primitive.xacro"/>
+      <xacro:if value="${model in ['mesh', 'capsule', 'convex_hull']}">
+         <xacro:include filename="$(find centauro)/centauro_urdf/urdf/models/${path}/${model}.xacro"/>
       </xacro:if>
    </xacro:macro>
    <xacro:load_model path="upper_body" model="${model}"/>
    <xacro:load_model path="lower_body" model="${model}"/>
-   <xacro:if value="${END_EFFECTOR == 'soft_hand'}" >
-      <xacro:load_model path="upper_body/end_effectors/soft_hand"  model="${model}"/>
-   </xacro:if>
-   <xacro:if value="${END_EFFECTOR == 'stick'}">
-     <xacro:load_model path="upper_body/end_effectors/stick"  model="${model}"/>
+   <xacro:if value="${END_EFFECTOR in ['soft_hand', 'stick']}" >
+      <xacro:load_model path="upper_body/end_effectors/${END_EFFECTOR}"  model="${model}"/>
    </xacro:if>
 </xacro:macro>

Commit message: Revised changes for xbot integration
Major modifications:
* Add sensors configuration for each middleware
* Add automatic choice of control plugin depending on middleware

Minor modification:
* Clear out files loading model

File: centauro/centauro_urdf/urdf/centauro.urdf.xacro (robot description, xacro)
@@ -46,5 +46,5 @@
     <joint name="imu_joint" type="fixed">
         <parent link="pelvis"/>
-        <origin xyz="${Imu_x} ${Imu_y} ${Imu_z}" rpy="${Imu_r} ${Imu_p} ${Imu_yaw}"/>
+        <origin xyz="${Imu_Ox} ${Imu_Oy} ${Imu_Oz}" rpy="${Imu_raw} ${Imu_pitch} ${Imu_yaw}"/>
         <child link="imu_link"/>
     </joint>

File: centauro/centauro_urdf/urdf/config.xacro (robot description, xacro)
@@ -14,5 +14,5 @@
 <xacro:property name="ONE_ARM" value="$(arg ONE_ARM)"/>
 <xacro:property name="GAZEBO" value="$(arg GAZEBO)"/>
-<xacro:property name="CONTROLLER" value="$(arg CONTROLLER)"/>
+<xacro:property name="MIDDLEWARE" value="$(arg MIDDLEWARE)"/>
 <xacro:property name="INERTIA_PARAM" value="$(arg INERTIA_PARAM)"/>
 <xacro:property name="KINEMATIC_PARAM" value="$(arg KINEMATIC_PARAM)"/>
@@ -22,4 +22,8 @@
 <xacro:property name="WHEELS_ACTUATORS" value="$(arg WHEELS_ACTUATORS)"/>
 <xacro:property name="ARM_SENSORS" value="$(arg ARM_SENSORS)"/>
+<xacro:property name="LEG_SENSORS" value="$(arg LEG_SENSORS)"/>
+<xacro:property name="FT_SENSORS" value="$(arg FT_SENSORS)"/>
+<xacro:property name="BUMBERS" value="$(arg BUMBERS)"/>
+<xacro:property name="IMU" value="$(arg IMU)"/>
 <xacro:property name="MASS" value="$(arg MASS)"/>
 <!-- dependend arguments -->
@@ -32,14 +36,19 @@
 <xacro:property name="static" value="${'true' if ('true' in [STATIC, ONE_ARM] or 'false' in [legs, LEG_ACTUATORS]) else 'false'}"/>
 <xacro:property name="reference" value="${'fixed' if (static == 'true') else 'floating'}" />
+<!-- ACTUATION -->
 <xacro:property name="torso_actuators" value="${'true' if ('false' not in [TORSO_ACTUATORS, TORSO]) else 'false'}"/>
 <xacro:property name="arm_actuators" value="${'true' if ('false' not in [ARM_ACTUATORS, TORSO_ACTUATORS, arm]) else 'false'}"/>
 <xacro:property name="leg_actuators" value="${'true' if ('false' not in [LEG_ACTUATORS, legs]) else 'false'}"/>
 <xacro:property name="wheels_actuators" value="${'true' if ('false' not in [WHEELS_ACTUATORS, LEG_ACTUATORS, wheels]) else 'false'}"/>
+<!-- SENSORS -->
 <xacro:property name="arm_sensors" value="${'true' if ('false' not in [ARM_SENSORS, arm]) else 'false'}"/>
-<xacro:property name="leg_sensors" value="${'true' if ('false' not in [legs]) else 'false'}"/>
+<xacro:property name="leg_sensors" value="${'true' if ('false' not in [LEG_SENSORS, legs]) else 'false'}"/>
+<xacro:property name="ft_sensors" value="${'true' if ('false' not in [FT_SENSORS]) else 'false'}"/>
+<xacro:property name="bumbers" value="${'true' if ('false' not in [BUMBERS]) else 'false'}"/>
+<xacro:property name="imu" value="${'true' if ('false' not in [IMU, pelvis]) else 'false'}"/>
+<!-- LOAD PARAMETERS -->
 <xacro:property name="package" value="$(find centauro)"/>
 <xacro:property name="inertia_parameters_file" value="${package + '/centauro_urdf/inertia_parameters/' + INERTIA_PARAM + '.xacro'}"/>
 <xacro:property name="kinematic_parameters_file" value="${package + '/centauro_urdf/kinematic_parameters/' + KINEMATIC_PARAM + '.xacro'}"/>
-<xacro:property name="xbotcore" value="${'true' if ('xbotcore' == CONTROLLER) else 'false'}"/>
-<xacro:property name="ros_control" value="${'true' if ('ros_control' == CONTROLLER) else 'false'}"/>
+<xacro:property name="middleware" value="${MIDDLEWARE}"/>
 </robot>
