Commit message: Simplified sensor integration for ros and xbot to minimize code repetitions and provide common parameters

File: centauro/centauro_urdf/urdf/centauro.urdf.xacro (robot description, xacro)
@@ -38,15 +38,4 @@
       </collision>
    </link>
-    <link name="imu_link">
-        <inertial>
-            <mass value="0.0"/>
-            <inertia ixx="0.0" ixy="0.0" ixz="0.0" iyy="0.0" iyz="0.0" izz="0.0"/>
-        </inertial>
-    </link>
-    <joint name="imu_joint" type="fixed">
-        <parent link="pelvis"/>
-        <origin xyz="${Imu_Ox} ${Imu_Oy} ${Imu_Oz}" rpy="${Imu_raw} ${Imu_pitch} ${Imu_yaw}"/>
-        <child link="imu_link"/>
-    </joint>
 </xacro:if>
 <xacro:unless value="${pelvis}">

File: centauro/centauro_urdf/urdf/config.xacro (robot description, xacro)
@@ -25,7 +25,10 @@
 <xacro:property name="ARM_SENSORS" value="$(arg ARM_SENSORS)"/>
 <xacro:property name="LEG_SENSORS" value="$(arg LEG_SENSORS)"/>
+<xacro:property name="HEAD_SENSORS" value="$(arg HEAD_SENSORS)"/>
 <xacro:property name="FT_SENSORS" value="$(arg FT_SENSORS)"/>
-<xacro:property name="BUMBERS" value="$(arg BUMBERS)"/>
+<xacro:property name="BUMPERS" value="$(arg BUMPERS)"/>
 <xacro:property name="IMU" value="$(arg IMU)"/>
+<xacro:property name="KINECT" value="$(arg KINECT)"/>
+<xacro:property name="VELODYNE" value="$(arg VELODYNE)"/>
 <xacro:property name="MASS" value="$(arg MASS)"/>
 <!-- dependend arguments -->
@@ -44,11 +47,13 @@
 <xacro:property name="leg_actuators" value="${'true' if ('false' not in [LEG_ACTUATORS, legs]) else 'false'}"/>
 <xacro:property name="head_actuators" value="${'true' if ('false' not in [HEAD_ACTUATORS, head]) else 'false'}"/>
-<xacro:property name="torso_actuators" value="${'true' if ('false' not in [TORSO_ACTUATORS, TORSO]) else 'false'}"/>
 <!-- SENSORS -->
 <xacro:property name="arm_sensors" value="${'true' if ('false' not in [ARM_SENSORS, arm]) else 'false'}"/>
 <xacro:property name="leg_sensors" value="${'true' if ('false' not in [LEG_SENSORS, legs]) else 'false'}"/>
+<xacro:property name="head_sensors" value="${'true' if ('false' not in [HEAD_SENSORS, head]) else 'false'}"/>
 <xacro:property name="ft_sensors" value="${'true' if ('false' not in [FT_SENSORS]) else 'false'}"/>
-<xacro:property name="bumbers" value="${'true' if ('false' not in [BUMBERS]) else 'false'}"/>
+<xacro:property name="bumpers" value="${'true' if ('false' not in [BUMPERS]) else 'false'}"/>
 <xacro:property name="imu" value="${'true' if ('false' not in [IMU, pelvis]) else 'false'}"/>
+<xacro:property name="kinect" value="${'true' if ('false' not in [KINECT]) else 'false'}"/>
+<xacro:property name="velodyne" value="${'true' if ('false' not in [VELODYNE]) else 'false'}"/>
 <!-- LOAD PARAMETERS -->
 <xacro:property name="package" value="$(find centauro)"/>

File: centauro_gazebo/sensors/config.xacro (robot description, xacro)
@@ -2,22 +2,32 @@
 <robot  xmlns:xacro="http://www.ros.org/wiki/xacro">
 <xacro:include filename="$(find centauro)/centauro_urdf/urdf/config.xacro"/>
-   <xacro:macro name="load_model" params="middleware sensor arm_sensors leg_sensors">
-      <xacro:include filename="$(find centauro_gazebo)/sensors/${middleware}/${sensor}/plugin.xacro"/>
+   <xacro:macro name="load_model" params="middleware sensor arm_sensors leg_sensors head_sensors">
+      <xacro:include filename="$(find centauro_gazebo)/sensors/gazebo/${sensor}/sensor.xacro"/>
+      <xacro:include filename="$(find centauro_gazebo)/sensors/${middleware}/plugin.xacro"/>
       <xacro:if value="${arm_sensors}">
-         <xacro:include filename="$(find centauro_gazebo)/sensors/${middleware}/${sensor}/load/arms.xacro"/>
+         <xacro:include filename="$(find centauro_gazebo)/sensors/gazebo/${sensor}/load/arms.xacro"/>
       </xacro:if>
       <xacro:if value="${leg_sensors}">
-         <xacro:include filename="$(find centauro_gazebo)/sensors/${middleware}/${sensor}/load/legs.xacro"/>
+         <xacro:include filename="$(find centauro_gazebo)/sensors/gazebo/${sensor}/load/legs.xacro"/>
+      </xacro:if>
+      <xacro:if value="${head_sensors}">
+         <xacro:include filename="$(find centauro_gazebo)/sensors/gazebo/${sensor}/load/head.xacro"/>
       </xacro:if>
    </xacro:macro>
 <!-- Load all controllers macros -->
 <xacro:if value="${ft_sensors}">
-        <xacro:load_model middleware="${middleware}" sensor="ft_sensor" arm_sensors="${arm_sensors}" leg_sensors="${leg_sensors}"/>
+        <xacro:load_model middleware="${middleware}" sensor="ft_sensor" arm_sensors="${arm_sensors}" leg_sensors="${leg_sensors}" head_sensors="${head_sensors}"/>
 </xacro:if>
-<xacro:if value="${bumbers}">
-        <xacro:load_model middleware="${middleware}" sensor="bumber" arm_sensors="${arm_sensors}" leg_sensors="${leg_sensors}"/>
+<xacro:if value="${bumpers}">
+        <xacro:load_model middleware="${middleware}" sensor="bumper" arm_sensors="${arm_sensors}" leg_sensors="${leg_sensors}" head_sensors="${head_sensors}"/>
 </xacro:if>
 <xacro:if value="${imu}">
-        <xacro:load_model middleware="${middleware}" sensor="imu" arm_sensors="${arm_sensors}" leg_sensors="${leg_sensors}"/>
+        <xacro:load_model middleware="${middleware}" sensor="imu" arm_sensors="${arm_sensors}" leg_sensors="${leg_sensors}" head_sensors="${head_sensors}"/>
+</xacro:if>
+<xacro:if value="${kinect}">
+        <xacro:load_model middleware="${middleware}" sensor="kinect" arm_sensors="${arm_sensors}" leg_sensors="${leg_sensors}" head_sensors="${head_sensors}"/>
+</xacro:if>
+<xacro:if value="${velodyne}">
+        <xacro:load_model middleware="${middleware}" sensor="velodyne" arm_sensors="${arm_sensors}" leg_sensors="${leg_sensors}" head_sensors="${head_sensors}"/>
 </xacro:if>
 </robot>

File: centauro_gazebo/sensors/gazebo/ft_sensor/load/arms.xacro (robot description, xacro)
@@ -2,7 +2,7 @@
 <robot  xmlns:xacro="http://www.ros.org/wiki/xacro">
 <xacro:include filename="$(find centauro)/centauro_urdf/urdf/config.xacro"/>
-  <xacro:force-torque_sensor joint="j_arm1_8" robot="centauro"/>
+  <xacro:middleware joint="j_arm1_8"  robot="centauro"  ft_name="left_arm_ft"/>
   <xacro:if value="${arms}">
-    <xacro:force-torque_sensor joint="j_arm2_8" robot="centauro"/>
+    <xacro:middleware joint="j_arm2_8" robot="centauro" ft_name="right_arm_ft" />
   </xacro:if>
 </robot>

File: centauro_gazebo/sensors/gazebo/ft_sensor/sensor.xacro (robot description, xacro)
@@ -1,5 +1,5 @@
 <!--<?xml version="1.0"?>-->
 <robot xmlns:xacro="http://www.ros.org/wiki/xacro">
-<xacro:macro name="imu_sensor" params="link robot">
+<xacro:macro name="force-torque_sensor" params="joint robot">
 </xacro:macro>
 </robot>

File: centauro_gazebo/sensors/gazebo/imu/load/legs.xacro (robot description, xacro)
@@ -2,6 +2,7 @@
 <robot  xmlns:xacro="http://www.ros.org/wiki/xacro">
 <xacro:include filename="$(find centauro)/centauro_urdf/urdf/config.xacro"/>
+<xacro:include filename="${kinematic_parameters_file}"/>
 <xacro:if value="${pelvis}">
-    <xacro:imu_sensor link="imu_link" robot="centauro"/>
+    <xacro:imu_sensor link="pelvis" robot="centauro" xyz="${Imu_Ox} ${Imu_Oy} ${Imu_Oz}" rpy="${Imu_raw} ${Imu_pitch} ${Imu_yaw}"/>
 </xacro:if>
 </robot>

File: centauro_gazebo/sensors/gazebo/imu/sensor.xacro (robot description, xacro)
@@ -1,7 +1,18 @@
 <!--<?xml version="1.0"?>-->
 <robot xmlns:xacro="http://www.ros.org/wiki/xacro">
-<xacro:macro name="imu_sensor" params="link robot">
+<xacro:macro name="imu_sensor" params="link robot xyz rpy">
+    <link name="${link}_imu_link">
+        <inertial>
+            <mass value="0.0"/>
+            <inertia ixx="1e-6" ixy="0.0" ixz="0.0" iyy="1e-6" iyz="0.0" izz="1e-6"/>
+        </inertial>
+    </link>
+    <joint name="${link}_imu_joint" type="fixed">
+        <parent link="${link}"/>
+        <origin xyz="${xyz}" rpy="${rpy}"/>
+        <child link="${link}_imu_link"/>
+    </joint>
     <gazebo reference="${link}">
-        <sensor name="${link}" type="imu">
+        <sensor name="${link}_imu" type="imu">
             <always_on>1</always_on>
             <update_rate>500</update_rate>
@@ -9,5 +20,4 @@
             <topic>__default_topic__</topic>
             <imu>
-                <!--
                 <noise>
                 <type>gaussian</type>
@@ -25,6 +35,6 @@
                 </accel>
                 </noise>
-                -->
             </imu>
+            <xacro:middleware link="${link}" robot="${robot}" />
         </sensor>
     </gazebo>

File: centauro_gazebo/sensors/gazebo/kinect/load/legs.xacro (robot description, xacro)
@@ -1,3 +1,4 @@
 <!--<?xml version="1.0"?>-->
 <robot  xmlns:xacro="http://www.ros.org/wiki/xacro">
+<xacro:include filename="$(find centauro)/centauro_urdf/urdf/config.xacro"/>
 </robot>

File: centauro_gazebo/sensors/gazebo/velodyne/load/legs.xacro (robot description, xacro)
@@ -2,6 +2,3 @@
 <robot  xmlns:xacro="http://www.ros.org/wiki/xacro">
 <xacro:include filename="$(find centauro)/centauro_urdf/urdf/config.xacro"/>
-<xacro:if value="${pelvis}">
-    <xacro:imu_sensor link="imu_link" robot="centauro"/>
-</xacro:if>
 </robot>

File: centauro_gazebo/sensors/ros_control/ft_sensor.xacro (robot description, xacro)
@@ -1,13 +1,14 @@
 <!--<?xml version="1.0"?>-->
 <robot xmlns:xacro="http://www.ros.org/wiki/xacro">
-<xacro:macro name="force-torque_sensor" params="joint robot">
+<xacro:macro name="middleware" params="joint robot ft_name">
         <gazebo reference="${joint}">
             <provideFeedback>true</provideFeedback>
         </gazebo>
         <gazebo>
-            <plugin name="${joint}_ft_sensor" filename="libgazebo_ros_ft_sensor.so">
+            <plugin name="${ft_name}" filename="libgazebo_ros_ft_sensor.so">
                 <updateRate>100.0</updateRate>
-                <topicName>${robot}/${joint}_ft_sensor</topicName>
+                <topicName>${robot}/${ft_name}</topicName>
                 <jointName>${joint}</jointName>
+                <gaussianNoise>0.0</gaussianNoise>
             </plugin>
         </gazebo>

File: centauro_gazebo/sensors/xbotcore/ft_sensor.xacro (robot description, xacro)
@@ -1,5 +1,5 @@
 <!--<?xml version="1.0"?>-->
 <robot xmlns:xacro="http://www.ros.org/wiki/xacro">
-<xacro:macro name="force-torque_sensor" params="joint robot ft_name pose">
+<xacro:macro name="middleware" params="joint robot ft_name">
         <gazebo reference="${joint}">
             <sensor type="force_torque" name="${ft_name}">
@@ -11,5 +11,5 @@
                 <visualize>true</visualize>
                 <update_rate>1000</update_rate>
-                <pose>${pose}</pose>
+                <pose>0 0 0 0 0 0</pose>
             </sensor>
         </gazebo>

Commit message: Decouple hand end-effectors

File: centauro/centauro_urdf/urdf/centauro.urdf.xacro (robot description, xacro)
@@ -69,8 +69,8 @@
 <!-- arms -->
 <xacro:if value="${arms == 'true'}">
-   <xacro:centauro_arm arm_num="1"  rot="1"  parent="torso_2">
+   <xacro:centauro_arm arm_num="1"  rot="1"  parent="torso_2" end_effector="${LEFT_END_EFFECTOR}">
       <origin xyz="${Shoulder_1_Ox} ${Shoulder_1_Oy} ${Shoulder_1_Oz}" rpy="${Shoulder_1_roll} ${Shoulder_1_pitch} ${Shoulder_1_yaw}"/>
    </xacro:centauro_arm>
-   <xacro:centauro_arm arm_num="2" rot="-1"  parent="torso_2">
+   <xacro:centauro_arm arm_num="2" rot="-1"  parent="torso_2" end_effector="${RIGHT_END_EFFECTOR}">
       <origin xyz="${Shoulder_1_Ox} ${-Shoulder_1_Oy} ${Shoulder_1_Oz}" rpy="${Shoulder_1_roll} ${Shoulder_1_pitch} ${-Shoulder_1_yaw}" />
    </xacro:centauro_arm>

File: centauro/centauro_urdf/urdf/centauro_arm.urdf.xacro (robot description, xacro)
@@ -2,5 +2,5 @@
 <robot xmlns:xacro="http://www.ros.org/wiki/xacro">
 <!-- macro arms -->
-<xacro:macro name="centauro_arm" params="arm_num rot parent *origin">
+<xacro:macro name="centauro_arm" params="arm_num rot parent end_effector *origin">
 <!-- LINKS -->
 <!-- shoulder yaw-roll-->
@@ -225,11 +225,11 @@
    </xacro:if>
 </xacro:if>
-<xacro:if value="${END_EFFECTOR == 'soft_hand'}" >
+<xacro:if value="${end_effector == 'soft_hand'}" >
   <xacro:include filename="$(find centauro)/centauro_urdf/urdf/centauro_hand.urdf.xacro" />
 </xacro:if>
-<xacro:if value="${END_EFFECTOR == 'stick'}" >
+<xacro:if value="${end_effector == 'stick'}" >
   <xacro:include filename="$(find centauro)/centauro_urdf/urdf/centauro_stick.urdf.xacro" />
 </xacro:if>
-<xacro:if value="${END_EFFECTOR != 'stick' and END_EFFECTOR != 'soft_hand' }" >
+<xacro:if value="${end_effector != 'stick' and end_effector != 'soft_hand' }" >
   <xacro:include filename="$(find centauro)/centauro_urdf/urdf/centauro_no_end_effector.urdf.xacro" />
 </xacro:if>

File: centauro/centauro_urdf/urdf/config.xacro (robot description, xacro)
@@ -4,5 +4,6 @@
      Also all the parameter dependencies are resolved-->
 <!-- basic arguments -->
-<xacro:property name="END_EFFECTOR" value="$(arg END_EFFECTOR)"/>
+<xacro:property name="LEFT_END_EFFECTOR" value="$(arg LEFT_END_EFFECTOR)"/>
+<xacro:property name="RIGHT_END_EFFECTOR" value="$(arg RIGHT_END_EFFECTOR)"/>
 <xacro:property name="COLLISION_MODEL" value="$(arg COLLISION_MODEL)"/>
 <xacro:property name="VISUAL_MODEL" value="$(arg VISUAL_MODEL)"/>

File: centauro/centauro_urdf/urdf/models/model_config.xacro (robot description, xacro)
@@ -12,6 +12,9 @@
    <xacro:load_model path="upper_body" model="${model}"/>
    <xacro:load_model path="lower_body" model="${model}"/>
-   <xacro:if value="${END_EFFECTOR in ['soft_hand', 'stick']}" >
-      <xacro:load_model path="upper_body/end_effectors/${END_EFFECTOR}"  model="${model}"/>
+   <xacro:if value="${LEFT_END_EFFECTOR in ['soft_hand', 'stick']}" >
+      <xacro:load_model path="upper_body/end_effectors/${LEFT_END_EFFECTOR}"  model="${model}"/>
+   </xacro:if>
+   <xacro:if value="${RIGHT_END_EFFECTOR in ['soft_hand', 'stick']}" >
+      <xacro:load_model path="upper_body/end_effectors/${RIGHT_END_EFFECTOR}"  model="${model}"/>
    </xacro:if>
    <xacro:if value="${head == 'true'}" >

Commit message: centauro_urdf: added eef_links and schunk hand

File: centauro/centauro_urdf/urdf/centauro.urdf.xacro (robot description, xacro)
@@ -21,4 +21,6 @@
   <xacro:include filename="$(find centauro)/centauro_urdf/urdf/centauro_arm.urdf.xacro"/>
 </xacro:if>
+<xacro:include filename="$(find centauro)/centauro_urdf/urdf/models/upper_body/end_effectors/schunk_hand/svh_gazebo.urdf.xacro" />
+<xacro:include filename="$(find centauro)/centauro_urdf/urdf/centauro_eef.urdf.xacro"/>
 <!-- /other files -->
 <!-- reference -->
@@ -75,4 +77,16 @@
       <origin xyz="${Shoulder_1_Ox} ${-Shoulder_1_Oy} ${Shoulder_1_Oz}" rpy="${Shoulder_1_roll} ${Shoulder_1_pitch} ${-Shoulder_1_yaw}" />
    </xacro:centauro_arm>
+   <!-- hand eef -->
+   <xacro:hand_eef prefix="left_hand" parent="arm1_7">
+	   <origin xyz="0 0 -0.1" rpy="0 0 0" />
+   </xacro:hand_eef>
+   <!-- schunk hand -->
+   <xacro:svh parent="arm2_7" name="right_hand" side="1">
+        <origin xyz="0 0 -0.04"  rpy= "${PI} 0 ${PI}" />
+    </xacro:svh>
+	<xacro:hand_eef prefix="right_hand" parent="right_hand_base_link">
+	   <origin xyz="0.0 0.02 0.08" rpy="0 0 0" />
+   </xacro:hand_eef>
+	<!-- schunk hand eef -->
 </xacro:if>
 <xacro:if value="${arm == 'true' and arms == 'false'}">
@@ -92,4 +106,9 @@
 <xacro:centauro_leg leg_num="4" origin_x="-1" origin_y="1">
 </xacro:centauro_leg>
+<!-- leg eef -->
+<xacro:leg_eef prefix="front_left" parent="ankle2_1"/>
+<xacro:leg_eef prefix="front_right" parent="ankle2_2"/>
+<xacro:leg_eef prefix="back_left" parent="ankle2_3"/>
+<xacro:leg_eef prefix="back_right" parent="ankle2_4"/>
 </xacro:if>
 <!-- /legs -->

Commit message: centauro_urdf: moved schunk hand to correct position & added hand_camera link

File: centauro/centauro_urdf/urdf/centauro.urdf.xacro (robot description, xacro)
@@ -81,11 +81,4 @@
 	   <origin xyz="0 0 -0.1" rpy="0 0 0" />
    </xacro:hand_eef>
-   <!-- schunk hand -->
-   <xacro:svh parent="arm2_7" name="right_hand" side="1">
-        <origin xyz="0 0 -0.04"  rpy= "${PI} 0 ${PI}" />
-    </xacro:svh>
-	<xacro:hand_eef prefix="right_hand" parent="right_hand_base_link">
-	   <origin xyz="0.0 0.02 0.08" rpy="0 0 0" />
-   </xacro:hand_eef>
 	<!-- schunk hand eef -->
 </xacro:if>

File: centauro/centauro_urdf/urdf/centauro_arm.urdf.xacro (robot description, xacro)
@@ -231,5 +231,14 @@
   <xacro:include filename="$(find centauro)/centauro_urdf/urdf/centauro_stick.urdf.xacro" />
 </xacro:if>
-<xacro:if value="${end_effector != 'stick' and end_effector != 'soft_hand' }" >
+<xacro:if value="${end_effector == 'schunk_hand'}" >
+	 <!-- schunk hand -->
+   <xacro:svh parent="arm2_7" name="right_hand" side="1">
+        <origin xyz="0 0 -0.04"  rpy= "${PI} 0 ${PI/2}" />
+    </xacro:svh>
+   	<xacro:hand_eef prefix="right_hand" parent="right_hand_base_link">
+	   <origin xyz="0.0 0.02 0.08" rpy="0 0 0" />
+   </xacro:hand_eef>
+</xacro:if>
+<xacro:if value="${end_effector != 'stick' and end_effector != 'soft_hand' and end_effector != 'schunk_hand'}" >
   <xacro:include filename="$(find centauro)/centauro_urdf/urdf/centauro_no_end_effector.urdf.xacro" />
 </xacro:if>

File: centauro/centauro_urdf/urdf/models/upper_body/end_effectors/schunk_hand/svh_gazebo.urdf.xacro (robot description, xacro)
@@ -75,7 +75,27 @@
         <!-- RIGHT HAND = 1, LEFT HAND = -1 -->
         <!-- BASE_LINE LINKS -->
+		<link name="${name}_camera_link">
+			<xacro:dummy_inertial />
+            <visual>
+                <origin rpy="0 0 0" xyz="0 0 0" />
+                <geometry>
+                    <mesh filename="package://schunk_svh_driver/description/meshes/camera_link.STL" />
+                </geometry>
+            </visual>
+            <collision>
+               <origin rpy="0 0 0" xyz="0 0 0" />
+                <geometry>
+                    <mesh filename="package://schunk_svh_driver/description/meshes/camera_link.STL" />
+                </geometry>
+            </collision>
+		</link>
+		<joint name="${name}_camera_joint" type="fixed" >
+			<xacro:insert_block name="origin" />
+            <parent link="${parent}" />
+			<child link="${name}_camera_link"/>
+		</joint>
         <joint name="${name}_base_joint" type="fixed" >
-            <xacro:insert_block name="origin" />
-            <parent link="${parent}" />
+			<origin xyz="0 0 ${0.011 + 0.0065 + 0.032}" rpy="0 0 -${PI/2}" />
+            <parent link="${name}_camera_link" />
             <child link="${name}_base_link" />
         </joint>

Commit message: get gazebo running

File: centauro/centauro_urdf/urdf/centauro.urdf.xacro (robot description, xacro)
@@ -106,3 +106,30 @@
 </xacro:if>
 <!-- /legs -->
+<gazebo>
+	<plugin name="gazebo_ros_control" filename="libgazebo_ros_control.so">
+	<robotNamespace>centauro</robotNamespace>
+	</plugin>
+</gazebo>
+<xacro:macro name="gz_wheel" params="wheel_link_name" >
+<gazebo reference="${wheel_link_name}">
+			<!--<material>Gazebo/FlatBlack</material>
+			<kp>10.0</kp>
+			<kd>10.0</kd>
+			<mu1>1.0</mu1>
+			<mu2>1.0</mu2>
+			<fdir1>1 0 0</fdir1>
+			<maxVel>1.0</maxVel>
+			<minDepth>0.00</minDepth>-->
+			<mu1>10000.0</mu1>
+			<mu2>10000.0</mu2>
+			<fdir1>1 0 0</fdir1>
+			<maxVel>0.0</maxVel>
+			<minDepth>0.001</minDepth>
+			<material>Gazebo/Black</material>
+</gazebo>
+</xacro:macro>
+<xacro:gz_wheel wheel_link_name="wheel_1" />
+<xacro:gz_wheel wheel_link_name="wheel_2" />
+<xacro:gz_wheel wheel_link_name="wheel_3" />
+<xacro:gz_wheel wheel_link_name="wheel_4" />
 </robot>

File: centauro/centauro_urdf/urdf/centauro_actuators.urdf.xacro (robot description, xacro)
@@ -5,8 +5,8 @@
 	<type> transmission_interface/SimpleTransmission</type>
 	<joint name="${joint}">
-		<hardwareInterface>hardware_interface/EffortJointInterface</hardwareInterface>
+		<hardwareInterface>EffortJointInterface</hardwareInterface>
 	</joint>
 	<actuator name="motor_${joint}">
-		<hardwareInterface>hardware_interface/EffortJointInterface</hardwareInterface>
+		<hardwareInterface>EffortJointInterface</hardwareInterface>
 		<machanicalReduction>1</machanicalReduction>
 	</actuator>

File: centauro/centauro_urdf/urdf/models/upper_body/end_effectors/schunk_hand/svh_gazebo.urdf.xacro (robot description, xacro)
@@ -24,9 +24,9 @@
             <type>transmission_interface/SimpleTransmission</type>
             <joint name="${namehand}_${jointname}">
-                <hardwareInterface>hardware_interface/EffortJointInterface</hardwareInterface>
+                <hardwareInterface>EffortJointInterface</hardwareInterface>
             </joint>
             <actuator name="motor_${namehand}_${jointname}">
                 <mechanicalReduction>1</mechanicalReduction>
-                <hardwareInterface>hardware_interface/EffortJointInterface</hardwareInterface>
+                <hardwareInterface>EffortJointInterface</hardwareInterface>
             </actuator>
         </transmission>
@@ -547,9 +547,9 @@
             <type>transmission_interface/SimpleTransmission</type>
             <joint name="${name}_Thumb_Flexion">
-                <hardwareInterface>hardware_interface/EffortJointInterface</hardwareInterface>
+                <hardwareInterface>EffortJointInterface</hardwareInterface>
             </joint>
             <actuator name="motor_${name}_Thumb_Flexion">
                 <mechanicalReduction>1</mechanicalReduction>
-                <hardwareInterface>hardware_interface/EffortJointInterface</hardwareInterface>
+                <hardwareInterface>EffortJointInterface</hardwareInterface>
             </actuator>
         </transmission-->

Commit message: added ankle chains

File: centauro/centauro_urdf/urdf/centauro.urdf.xacro (robot description, xacro)
@@ -100,8 +100,8 @@
 </xacro:centauro_leg>
 <!-- leg eef -->
-<xacro:leg_eef prefix="front_left" parent="ankle2_1"/>
-<xacro:leg_eef prefix="front_right" parent="ankle2_2"/>
-<xacro:leg_eef prefix="back_left" parent="ankle2_3"/>
-<xacro:leg_eef prefix="back_right" parent="ankle2_4"/>
+<xacro:leg_eef prefix="front_left" parent="ankle1_1"/>
+<xacro:leg_eef prefix="front_right" parent="ankle1_2"/>
+<xacro:leg_eef prefix="back_right" parent="ankle1_3"/>
+<xacro:leg_eef prefix="back_left" parent="ankle1_4"/>
 </xacro:if>
 <!-- /legs -->

File: centauro/centauro_urdf/urdf/centauro_eef.urdf.xacro (robot description, xacro)
@@ -16,5 +16,5 @@
 			<parent link="${parent}"/>
 			<child link="${prefix}_eef_link"/>
-			<origin rpy="1.57079632679 0.0 0.0" xyz="0.0 0.00085 0.235"/>
+			<origin rpy="0 0.0 0.0" xyz="0.0 0.0 0.0"/>
 		</joint>
 		<link name="${prefix}_dummy_link"/>
