Commit message: centauro_urdf: define end effector link for all hands consistently

File: centauro/centauro_urdf/urdf/centauro.urdf.xacro (robot description, xacro)
@@ -79,7 +79,9 @@
    <!-- hand eef -->
    <xacro:hand_eef prefix="left_hand" parent="arm1_7">
-	   <origin xyz="0 0 -0.1" rpy="0 0 0" />
+      <origin xyz="0 0.020 -0.169" rpy="${pi} 0 ${-pi}" />
    </xacro:hand_eef>
-	<!-- schunk hand eef -->
+   <xacro:hand_eef prefix="right_hand" parent="arm2_7">
+      <origin xyz="0 0.020 -0.169" rpy="${pi} 0 ${-pi}" />
+   </xacro:hand_eef>
 </xacro:if>
 <xacro:if value="${arm == 'true' and arms == 'false'}">

File: centauro/centauro_urdf/urdf/centauro_arm.urdf.xacro (robot description, xacro)
@@ -236,7 +236,4 @@
         <origin xyz="0 0 -0.04"  rpy= "${PI} 0 ${PI/2}" />
     </xacro:svh>
-   	<xacro:hand_eef prefix="right_hand" parent="right_hand_base_link">
-	   <origin xyz="0.0 0.02 0.08" rpy="0 0 0" />
-   </xacro:hand_eef>
 </xacro:if>
 <xacro:if value="${end_effector != 'stick' and end_effector != 'soft_hand' and end_effector != 'schunk_hand'}" >

Commit message: centauro_urdf: move leg endeffectors into wheel centers

File: centauro/centauro_urdf/urdf/centauro.urdf.xacro (robot description, xacro)
@@ -102,8 +102,16 @@
 </xacro:centauro_leg>
 <!-- leg eef -->
-<xacro:leg_eef prefix="front_left" parent="ankle1_1"/>
-<xacro:leg_eef prefix="front_right" parent="ankle1_2"/>
-<xacro:leg_eef prefix="back_left" parent="ankle1_3"/>
-<xacro:leg_eef prefix="back_right" parent="ankle1_4"/>
+<xacro:leg_eef prefix="front_left" parent="ankle1_1">
+	<origin xyz="0.237 -0.001 0.000" />
+</xacro:leg_eef>
+<xacro:leg_eef prefix="front_right" parent="ankle1_2">
+	<origin xyz="0.237 0.001 0.000" />
+</xacro:leg_eef>
+<xacro:leg_eef prefix="back_left" parent="ankle1_3">
+	<origin xyz="0.237 0.001 0.000" />
+</xacro:leg_eef>
+<xacro:leg_eef prefix="back_right" parent="ankle1_4">
+	<origin xyz="0.237 -0.001 0.000" />
+</xacro:leg_eef>
 </xacro:if>
 <!-- /legs -->

File: centauro/centauro_urdf/urdf/centauro_eef.urdf.xacro (robot description, xacro)
@@ -16,5 +16,5 @@
 			<parent link="${parent}"/>
 			<child link="${prefix}_eef_link"/>
-			<origin rpy="0 0.0 0.0" xyz="0.0 0.0 0.0"/>
+			<xacro:insert_block name="origin" />
 		</joint>
 		<link name="${prefix}_dummy_link"/>

Commit message: centauro_urdf: introduce "base_link" and make world link optional

File: centauro/centauro_urdf/urdf/centauro.urdf.xacro (robot description, xacro)
@@ -24,6 +24,4 @@
 <xacro:include filename="$(find centauro)/centauro_urdf/urdf/centauro_eef.urdf.xacro"/>
 <!-- /other files -->
-<!-- reference -->
-<link name="world"/>
 <xacro:if value="${pelvis}">
    <link name="pelvis">
@@ -55,9 +53,19 @@
    <link name="pelvis"/>
 </xacro:unless>
-<joint name="reference" type="${reference}">
-   <origin xyz="${Pelvis_Ox} ${Pelvis_Oy} ${Pelvis_Oz}"/>
-   <parent link="world"/>
-   <child link="pelvis"/>
+<link name="base_link" />
+<joint name="base_pelvis" type="fixed">
+   <parent link="base_link" />
+   <child link="pelvis" />
+   <origin xyz="0 0 0" rpy="0 0 0" />
 </joint>
+<xacro:if value="${include_world}">
+   <!-- reference -->
+   <link name="world"/>
+   <joint name="reference" type="${reference}">
+      <origin xyz="${Pelvis_Ox} ${Pelvis_Oy} ${Pelvis_Oz}"/>
+      <parent link="world"/>
+      <child link="base_link"/>
+   </joint>
+</xacro:if>
 <!-- /reference  -->
 <!-- torso -->

File: centauro/centauro_urdf/urdf/config.xacro (robot description, xacro)
@@ -31,4 +31,6 @@
 <xacro:property name="IMU" value="$(arg IMU)"/>
 <xacro:property name="MASS" value="$(arg MASS)"/>
+<xacro:arg name="INCLUDE_WORLD" default="true" />
+<xacro:property name="INCLUDE_WORLD" value="$(arg INCLUDE_WORLD)"/>
 <!-- dependend arguments -->
 <xacro:property name="arms" value="${'true' if ('false' not in [TORSO, ARMS] and 'false' in [ONE_ARM]) else 'false'}"/>
@@ -41,4 +43,5 @@
 <xacro:property name="static" value="${'true' if ('true' in [STATIC, ONE_ARM] or 'false' in [legs, LEG_ACTUATORS]) else 'false'}"/>
 <xacro:property name="reference" value="${'fixed' if (static == 'true') else 'floating'}" />
+<xacro:property name="include_world" value="${INCLUDE_WORLD}" />
 <!-- ACTUATION -->
 <xacro:property name="torso_actuators" value="${'true' if ('false' not in [TORSO_ACTUATORS, TORSO]) else 'false'}"/>

Commit message: introduce individual wheel frictions to avoid unstable behavior of wheel-to-ground contact

File: centauro/centauro_urdf/urdf/centauro.urdf.xacro (robot description, xacro)
@@ -129,16 +129,16 @@
 	</plugin>
 </gazebo>
-<xacro:macro name="gz_wheel" params="wheel_link_name" >
+<xacro:macro name="gz_wheel" params="wheel_link_name wheel_friction" >
 <gazebo reference="${wheel_link_name}">
 			<!--<material>Gazebo/FlatBlack</material>
 			<kp>10.0</kp>
 			<kd>10.0</kd>
-			<mu1>1.0</mu1>
-			<mu2>1.0</mu2>
+			<mu1>${wheel_friction}</mu1>
+			<mu2>${wheel_friction}</mu2>
 			<fdir1>1 0 0</fdir1>
 			<maxVel>1.0</maxVel>
 			<minDepth>0.00</minDepth>-->
-			<mu1>10000.0</mu1>
-			<mu2>10000.0</mu2>
+			<mu1>${wheel_friction}</mu1>
+			<mu2>${wheel_friction}</mu2>
 			<fdir1>1 0 0</fdir1>
 			<maxVel>0.0</maxVel>
@@ -147,7 +147,7 @@
 </gazebo>
 </xacro:macro>
-<xacro:gz_wheel wheel_link_name="wheel_1" />
-<xacro:gz_wheel wheel_link_name="wheel_2" />
-<xacro:gz_wheel wheel_link_name="wheel_3" />
-<xacro:gz_wheel wheel_link_name="wheel_4" />
+<xacro:gz_wheel wheel_link_name="wheel_1" wheel_friction="1000.0" />
+<xacro:gz_wheel wheel_link_name="wheel_2" wheel_friction="0.1"/>
+<xacro:gz_wheel wheel_link_name="wheel_3" wheel_friction="0.1"/>
+<xacro:gz_wheel wheel_link_name="wheel_4" wheel_friction="0.1"/>
 </robot>

Commit message: Add mesh file for soft hand and add 'fixed_soft_hand' to simulate soft hand without additional DoFs

File: centauro/centauro_urdf/urdf/centauro.urdf.xacro (robot description, xacro)
@@ -23,4 +23,11 @@
 <!-- /other files -->
 <!-- reference -->
+<!-- <link name="base_link"/>
+<joint name="base_joint" type="fixed">
+   <origin xyz="0 0 0"/>
+   <parent link="base_link"/>
+   <child link="world"/>
+</joint>
+-->
 <link name="world"/>
 <xacro:if value="${pelvis}">
@@ -69,10 +76,10 @@
 <!-- arms -->
 <xacro:if value="${left_arm == 'true'}">
-   <xacro:centauro_arm arm_num="1"  rot="1"  parent="torso_2" end_effector="${LEFT_END_EFFECTOR}">
+   <xacro:centauro_arm arm_num="1"  rot="1"  parent="torso_2" end_effector="${left_end_effector}" mount="${left_arm_mount}">
       <origin xyz="${Shoulder_1_Ox} ${Shoulder_1_Oy} ${Shoulder_1_Oz}" rpy="${Shoulder_1_roll} ${Shoulder_1_pitch} ${Shoulder_1_yaw}"/>
    </xacro:centauro_arm>
 </xacro:if>
 <xacro:if value="${right_arm == 'true'}">
-   <xacro:centauro_arm arm_num="2" rot="-1"  parent="torso_2" end_effector="${RIGHT_END_EFFECTOR}">
+   <xacro:centauro_arm arm_num="2" rot="-1"  parent="torso_2" end_effector="${right_end_effector}" mount="${right_arm_mount}">
       <origin xyz="${Shoulder_1_Ox} ${-Shoulder_1_Oy} ${Shoulder_1_Oz}" rpy="${Shoulder_1_roll} ${Shoulder_1_pitch} ${-Shoulder_1_yaw}" />
    </xacro:centauro_arm>

File: centauro/centauro_urdf/urdf/centauro_arm.urdf.xacro (robot description, xacro)
@@ -2,5 +2,5 @@
 <robot xmlns:xacro="http://www.ros.org/wiki/xacro">
 <!-- macro arms -->
-<xacro:macro name="centauro_arm" params="arm_num rot parent end_effector *origin">
+<xacro:macro name="centauro_arm" params="arm_num rot parent end_effector mount *origin">
 <!-- LINKS -->
 <!-- shoulder yaw-roll-->
@@ -227,4 +227,5 @@
 <xacro:if value="${end_effector == 'soft_hand'}" >
   <xacro:include filename="$(find centauro)/centauro_urdf/urdf/centauro_hand.urdf.xacro" />
+  <xacro:soft_hand arm_num="${arm_num}"  rot="${rot}"  joint="${mount}"/>
 </xacro:if>
 <xacro:if value="${end_effector == 'stick'}" >

File: centauro/centauro_urdf/urdf/centauro_hand.urdf.xacro (robot description, xacro)
@@ -2,4 +2,5 @@
 <robot xmlns:xacro="http://www.ros.org/wiki/xacro">
 <!-- links -->
+<xacro:macro name="soft_hand" params="arm_num rot joint">
    <link name="arm${arm_num}_8">
       <inertial>
@@ -17,5 +18,5 @@
    </link>
 <!-- /links -->
-   <joint name="j_arm${arm_num}_8" type="revolute">
+   <joint name="j_arm${arm_num}_8" type="${joint}">
       <xacro:if value="${ft_sensors == 'true'}" >
          <parent link="ft_arm${arm_num}"/>
@@ -27,10 +28,15 @@
       </xacro:unless>
       <child link="arm${arm_num}_8"/>
-      <axis xyz="0 1 0" />
-      <limit velocity="20.3" effort="40" lower="0.0" upper="1.57075" />
+      <xacro:if value="${joint not in ['fixed']}" >
+         <axis xyz="0 1 0" />
+         <limit velocity="20.3" effort="40" lower="0.0" upper="1.57075" />
+      </xacro:if>
    </joint> -->
 <!-- /joints -->
 <!-- actuators -->
-   <xacro:position_actuator joint="j_arm${arm_num}_8" />
+   <xacro:if value="${joint not in ['fixed']}" >
+     <xacro:position_actuator joint="j_arm${arm_num}_8" />
+   </xacro:if>
 <!-- /actuators -->
+</xacro:macro>
 </robot>

File: centauro/centauro_urdf/urdf/config.xacro (robot description, xacro)
@@ -42,4 +42,8 @@
 <xacro:property name="reference" value="${'fixed' if (static == 'true') else 'floating'}" />
 <xacro:property name="torso_joint" value="${'fixed' if ('fixed' in [TORSO]) else 'revolute'}"/>
+<xacro:property name="left_arm_mount" value= "${'revolute' if LEFT_END_EFFECTOR in ['soft_hand'] else 'fixed'}" />
+<xacro:property name="right_arm_mount" value= "${'revolute' if RIGHT_END_EFFECTOR in ['soft_hand'] else 'fixed'}" />
+<xacro:property name="left_end_effector" value= "${LEFT_END_EFFECTOR.split('fixed_', 2).pop()}" />
+<xacro:property name="right_end_effector" value= "${RIGHT_END_EFFECTOR.split('fixed_', 2).pop()}" />
 <!-- ACTUATION -->
 <xacro:property name="torso_actuators" value="${'true' if ('false' not in [TORSO_ACTUATORS, TORSO]) else 'false'}"/>

File: centauro/centauro_urdf/urdf/models/model_config.xacro (robot description, xacro)
@@ -12,9 +12,9 @@
    <xacro:load_model path="upper_body" model="${model}"/>
    <xacro:load_model path="lower_body" model="${model}"/>
-   <xacro:if value="${LEFT_END_EFFECTOR in ['soft_hand', 'stick']}" >
-      <xacro:load_model path="upper_body/end_effectors/${LEFT_END_EFFECTOR}"  model="${model}"/>
+   <xacro:if value="${left_end_effector in ['soft_hand', 'stick']}" >
+      <xacro:load_model path="upper_body/end_effectors/${left_end_effector}"  model="${model}"/>
    </xacro:if>
-   <xacro:if value="${RIGHT_END_EFFECTOR in ['soft_hand', 'stick']}" >
-      <xacro:load_model path="upper_body/end_effectors/${RIGHT_END_EFFECTOR}"  model="${model}"/>
+   <xacro:if value="${right_end_effector in ['soft_hand', 'stick']}" >
+      <xacro:load_model path="upper_body/end_effectors/${right_end_effector}"  model="${model}"/>
    </xacro:if>
    <xacro:if value="${head == 'true'}" >

File: centauro/centauro_urdf/urdf/models/upper_body/end_effectors/soft_hand/mesh.xacro (robot description, xacro)
@@ -1,3 +1,9 @@
 <?xml version="1.0" ?>
 <robot name="centauro" xmlns:xacro="http://www.ros.org/wiki/xacro">
+<xacro:macro name="soft_hand">
+   <origin xyz="0.0 0.0 -0.038"  rpy="0.0 0.0  ${PI/2+rot*PI/2}"/>
+   <geometry>
+      <mesh filename="package://centauro/centauro_urdf/meshes/soft_hand_open.stl" scale="0.001 0.001 0.001" />
+   </geometry>
+</xacro:macro>
 </robot>

Commit message: updated joint limits

File: centauro/centauro_urdf/urdf/centauro.urdf.xacro (robot description, xacro)
@@ -12,4 +12,5 @@
 <xacro:include filename="${inertia_parameters_file}"/>
 <xacro:include filename="${kinematic_parameters_file}"/>
+<xacro:include filename="$(find centauro)/centauro_urdf/limits/default.xacro"/>
 <xacro:include filename="$(find centauro)/centauro_urdf/materials.xacro"/>
 <xacro:include filename="$(find centauro)/centauro_urdf/urdf/models/model.xacro"/>

File: centauro/centauro_urdf/urdf/centauro_arm.urdf.xacro (robot description, xacro)
@@ -119,10 +119,5 @@
       <xacro:insert_block name="origin"/>
       <axis xyz="0 ${rot*cos_m10} ${-sin_m10}"/>
-      <xacro:unless value="${rot-1}" >
-         <limit lower="-3.403" upper="1.658" effort="147" velocity="5.7"/>
-      </xacro:unless>
-      <xacro:unless value="${rot+1}" >
-         <limit lower="-1.658" upper="3.403" effort="147" velocity="5.7"/>
-      </xacro:unless>
+      <limit lower="${j_arm_1_lower[arm_num-1]}" upper="${j_arm_1_upper[arm_num-1]}" effort="147" velocity="5.7"/>
    </joint>
 <!-- /shoulder yaw -->
@@ -133,10 +128,5 @@
       <origin xyz="${Shoulder_2_Ox} ${rot*Shoulder_2_Oy} ${Shoulder_2_Oz}"/>
       <axis xyz="-1 0 0"/>
-      <xacro:unless value="${rot+1}" >
-         <limit lower="0" upper="3.49" effort="147" velocity="5.7"/>
-      </xacro:unless>
-      <xacro:unless value="${rot-1}" >
-         <limit lower="-3.49" upper="0" effort="147" velocity="5.7"/>
-      </xacro:unless>
+      <limit lower="${j_arm_2_lower[arm_num-1]}" upper="${j_arm_2_upper[arm_num-1]}" effort="147" velocity="5.7"/>
    </joint>
 <!-- /shoulder roll -->
@@ -147,5 +137,5 @@
       <origin xyz="${Shoulder_3_Ox} ${Shoulder_3_Oy} ${Shoulder_3_Oz}"/>
       <axis xyz="0 0 -1"/>
-      <limit lower="-2.618" upper="2.618" effort="147" velocity="8.2"/>
+      <limit lower="${j_arm_3_lower[arm_num-1]}" upper="${j_arm_3_upper[arm_num-1]}" effort="147" velocity="8.2"/>
    </joint>
 <!-- /shoulder pitch -->
@@ -156,10 +146,5 @@
       <origin xyz="${Elbow_1_Ox} ${rot*Elbow_1_Oy} ${Elbow_1_Oz}"/>
       <axis xyz="0 ${rot} 0"/>
-      <xacro:unless value="${rot-1}" >
-         <limit lower="-2.530" upper="0.349" effort="147" velocity="8.2"/>
-      </xacro:unless>
-      <xacro:unless value="${rot+1}" >
-         <limit lower="-0.349" upper="2.530" effort="147" velocity="8.2"/>
-      </xacro:unless>
+      <limit lower="${j_arm_4_lower[arm_num-1]}" upper="${j_arm_4_upper[arm_num-1]}" effort="147" velocity="8.2"/>
    </joint>
 <!-- /elbow yaw -->
@@ -170,5 +155,5 @@
       <origin xyz="${Wrist_1_Ox} ${-rot*Wrist_1_Oy} ${Wrist_1_Oz}"/>
       <axis xyz="0 0 -1"/>
-      <limit lower="-2.618" upper="2.618" effort="55" velocity="11.6"/>
+      <limit lower="${j_arm_5_lower[arm_num-1]}" upper="${j_arm_5_upper[arm_num-1]}" effort="55" velocity="11.6"/>
    </joint>
 <!-- /elbow pitch-->
@@ -179,5 +164,5 @@
       <origin xyz="${Wrist_2_Ox} ${rot*Wrist_2_Oy} ${Wrist_2_Oz}"/>
       <axis xyz="0 ${rot} 0"/>
-      <limit lower="-1.570" upper="1.570" effort="55" velocity="11.6"/>
+      <limit lower="${j_arm_6_lower[arm_num-1]}" upper="${j_arm_6_upper[arm_num-1]}" effort="55" velocity="11.6"/>
    </joint>
 <!-- /wrist yaw-->
@@ -188,5 +173,5 @@
       <origin xyz="${Wrist_3_Ox} ${-rot*Wrist_3_Oy} ${Wrist_3_Oz}"/>
       <axis xyz="0 0 -1"/>
-      <limit lower="-2.618" upper="2.618" effort="27" velocity="20.3"/>
+      <limit lower="${j_arm_7_lower[arm_num-1]}" upper="${j_arm_7_upper[arm_num-1]}" effort="27" velocity="20.3"/>
    </joint>
 <!-- wrist pitch-->

File: centauro/centauro_urdf/urdf/centauro_leg.urdf.xacro (robot description, xacro)
@@ -94,10 +94,5 @@
 	<origin xyz="${origin_x*Leg_1_Ox} ${origin_y*Leg_1_Oy} ${Leg_1_Oz}" rpy="${Leg_1_roll} ${Leg_1_pitch} ${PI/2-origin_x*PI/2+origin_x*origin_y*Leg_1_yaw}"/>
 	<axis xyz="0 0 1"/>
-        <xacro:if value="${origin_y*origin_x == -1}">
-        <limit lower="-1.13446401" upper="2.70526034" effort="304" velocity="8.8"/>
-        </xacro:if>
-        <xacro:if value="${origin_y*origin_x == 1}">
-        <limit lower="-2.70526034" upper="1.13446401" effort="304" velocity="8.8"/>
-        </xacro:if>
+        <limit lower="${hip_yaw_lower[leg_num-1]}" upper="${hip_yaw_upper[leg_num-1]}" effort="304" velocity="8.8"/>
 </joint>
 <joint name="hip_pitch_${leg_num}" type="revolute">
@@ -106,5 +101,5 @@
 	<origin xyz="${Leg_2_Ox} ${Leg_2_Oy} ${Leg_2_Oz}" rpy="${Leg_2_roll} ${Leg_2_pitch} ${origin_x*origin_y*Leg_2_yaw-origin_x*origin_y*PI/2 + PI/2}"/>
 	<axis xyz="0 0 1"/>
-        <limit lower="-2.09439510" upper="2.09439510" effort="304" velocity="8.8"/>
+        <limit lower="${hip_pitch_lower[leg_num-1]}" upper="${hip_pitch_upper[leg_num-1]}" effort="304" velocity="8.8"/>
 </joint>
 <joint name="knee_pitch_${leg_num}" type="revolute">
@@ -113,5 +108,5 @@
 	<origin xyz="${Leg_3_Ox} ${Leg_3_Oy} ${Leg_3_Oz}" rpy="${Leg_3_roll} ${Leg_3_pitch} ${Leg_3_yaw}"/>
 	<axis xyz="0 0 1"/>
-        <limit  lower="-2.61799388" upper="2.61799388" effort="304" velocity="8.8"/>
+        <limit lower="${knee_pitch_lower[leg_num-1]}" upper="${knee_pitch_upper[leg_num-1]}" effort="304" velocity="8.8"/>
 </joint>
 <joint name="ankle_pitch_${leg_num}" type="revolute">
@@ -120,5 +115,5 @@
 	<origin xyz="${Ankle_1_Ox} ${Ankle_1_Oy} ${Ankle_1_Oz}" rpy="${Ankle_1_roll} ${Ankle_1_pitch} ${Ankle_1_yaw}"/>
 	<axis xyz="0 0 1"/>
-        <limit  lower="-2.61799388" upper="2.61799388" effort="147" velocity="8.1"/>
+        <limit lower="${ankle_pitch_lower[leg_num-1]}" upper="${ankle_pitch_upper[leg_num-1]}" effort="147" velocity="8.1"/>
 </joint>
 <joint name="ankle_yaw_${leg_num}" type="revolute">
@@ -127,5 +122,5 @@
 	<origin xyz="${Ankle_2_Ox} ${Ankle_2_Oy} ${Ankle_2_Oz}" rpy="${Ankle_2_roll} ${Ankle_2_pitch} ${Ankle_2_yaw}"/>
 	<axis xyz="0 0 1"/>
-        <limit  lower="-2.58308729" upper="2.58308729" effort="35" velocity="20.0"/>
+        <limit lower="${ankle_yaw_lower[leg_num-1]}" upper="${ankle_yaw_upper[leg_num-1]}" effort="35" velocity="20.0"/>
 </joint>
 <joint name="j_wheel_${leg_num}" type="continuous">

File: centauro/centauro_urdf/urdf/centauro_torso.urdf.xacro (robot description, xacro)
@@ -28,5 +28,5 @@
    <child link="torso_2"/>
    <axis xyz="0 0 1"/>
-   <limit lower="-2.618" upper="2.618" effort="147" velocity="5.7"/> <!-- TODO -->
+   <limit lower="${torso_yaw_lower}" upper="${torso_yaw_upper}" effort="147" velocity="5.7"/> <!-- TODO -->
 </joint>
 <!-- /torso joints -->

Commit message: read the velocity and torque limits from the external file

File: centauro/centauro_urdf/urdf/centauro.urdf.xacro (robot description, xacro)
@@ -12,5 +12,5 @@
 <xacro:include filename="${inertia_parameters_file}"/>
 <xacro:include filename="${kinematic_parameters_file}"/>
-<xacro:include filename="$(find centauro)/centauro_urdf/limits/default.xacro"/>
+<xacro:include filename="$(find centauro)/centauro_urdf/limits/${limits}.xacro"/>
 <xacro:include filename="$(find centauro)/centauro_urdf/materials.xacro"/>
 <xacro:include filename="$(find centauro)/centauro_urdf/urdf/models/model.xacro"/>
@@ -83,5 +83,5 @@
 <xacro:if value="${right_arm == 'true'}">
    <xacro:centauro_arm arm_num="2" rot="-1"  parent="torso_2" end_effector="${right_end_effector}" mount="${right_arm_mount}">
-      <origin xyz="${Shoulder_1_Ox} ${-Shoulder_1_Oy} ${Shoulder_1_Oz}" rpy="${Shoulder_1_roll} ${Shoulder_1_pitch} ${-Shoulder_1_yaw}" />
+      <origin xyz="${Shoulder_1_Ox} ${-Shoulder_1_Oy} ${Shoulder_1_Oz}" rpy="${-Shoulder_1_roll} ${Shoulder_1_pitch} ${-Shoulder_1_yaw}" />
    </xacro:centauro_arm>
 </xacro:if>
