Commit message: provide support for gazebo9

File: centauro/centauro_urdf/urdf/centauro.urdf.xacro (robot description, xacro)
@@ -16,5 +16,5 @@
 <xacro:include filename="$(find centauro)/centauro_urdf/urdf/models/model.xacro"/>
 <xacro:include filename="$(find centauro)/centauro_urdf/urdf/centauro_actuators.urdf.xacro" />
-<xacro:if value="${LEGS}">
+<xacro:if value="${legs}">
   <xacro:include filename="$(find centauro)/centauro_urdf/urdf/centauro_leg.urdf.xacro"/>
 </xacro:if>
@@ -68,18 +68,18 @@
 <!-- /reference  -->
 <!-- torso -->
-<xacro:if value="${torso == 'true'}">
+<xacro:if value="${torso in [True, 'true']}">
    <xacro:include filename="$(find centauro)/centauro_urdf/urdf/centauro_torso.urdf.xacro"/>
 </xacro:if>
-<xacro:if value="${head == 'true'}">
+<xacro:if value="${head in [True, 'true']}">
    <xacro:include filename="$(find centauro)/centauro_urdf/urdf/centauro_head.urdf.xacro"/>
 </xacro:if>
 <!-- /torso -->
 <!-- arms -->
-<xacro:if value="${left_arm == 'true'}">
+<xacro:if value="${left_arm in [True, 'true']}">
    <xacro:centauro_arm arm_num="1"  rot="1"  parent="torso_2" end_effector="${left_end_effector}" mount="${left_arm_mount}">
       <origin xyz="${Shoulder_1_Ox} ${Shoulder_1_Oy} ${Shoulder_1_Oz}" rpy="${Shoulder_1_roll} ${Shoulder_1_pitch} ${Shoulder_1_yaw}"/>
    </xacro:centauro_arm>
 </xacro:if>
-<xacro:if value="${right_arm == 'true'}">
+<xacro:if value="${right_arm in [True, 'true']}">
    <xacro:centauro_arm arm_num="2" rot="-1"  parent="torso_2" end_effector="${right_end_effector}" mount="${right_arm_mount}">
       <origin xyz="${Shoulder_1_Ox} ${-Shoulder_1_Oy} ${Shoulder_1_Oz}" rpy="${Shoulder_1_roll} ${Shoulder_1_pitch} ${-Shoulder_1_yaw}" />

File: centauro/centauro_urdf/urdf/centauro_right_arm.urdf.xacro (robot description, xacro)
@@ -60,18 +60,18 @@
 <!-- /reference  -->
 <!-- torso -->
-<xacro:if value="${torso == 'true'}">
+<xacro:if value="${torso in [True, 'true']}">
    <xacro:include filename="$(find centauro)/centauro_urdf/urdf/centauro_torso_fixed.urdf.xacro"/>
 </xacro:if>
-<xacro:if value="${head == 'true'}">
+<xacro:if value="${head in [True, 'true']}">
    <xacro:include filename="$(find centauro)/centauro_urdf/urdf/centauro_head.urdf.xacro"/>
 </xacro:if>
 <!-- /torso -->
 <!-- arms -->
-<xacro:if value="${arms == 'true'}">
+<xacro:if value="${arms in [True, 'true']}">
    <xacro:centauro_arm arm_num="2" rot="-1"  parent="torso_2" end_effector="${RIGHT_END_EFFECTOR}">
       <origin xyz="${Shoulder_1_Ox} ${-Shoulder_1_Oy} ${Shoulder_1_Oz}" rpy="${Shoulder_1_roll} ${Shoulder_1_pitch} ${-Shoulder_1_yaw}" />
    </xacro:centauro_arm>
 </xacro:if>
-<xacro:if value="${arm == 'true' and arms == 'false'}">
+<xacro:if value="${arm in [True, 'true'] and arms in [False, 'false']}">
         <xacro:centauro_arm arm_num="1"  rot="1" parent="world">
            <origin xyz="${Shoulder_1_Ox + Pelvis_Ox + Torso_2_Ox} ${Shoulder_1_Oy + Pelvis_Oy + Torso_2_Oy} ${Shoulder_1_Oz + Pelvis_Oz + Torso_2_Oz}" rpy="${Shoulder_1_roll} ${Shoulder_1_pitch} ${Shoulder_1_yaw}"/>

File: centauro/centauro_urdf/urdf/config.xacro (robot description, xacro)
@@ -34,14 +34,14 @@
 <xacro:property name="MASS" value="$(arg MASS)"/>
 <!-- dependend arguments -->
-<xacro:property name="torso" value="${'true' if ('true' in [TORSO] or 'fixed' in [TORSO]) else 'false'}"/>
-<xacro:property name="head" value="${'true' if ('false' not in [torso, HEAD]) else 'false'}"/>
-<xacro:property name="arms" value="${'true' if ('false' not in [TORSO, ARMS]) else 'false'}"/>
-<xacro:property name="left_arm" value= "${'true' if ('true' in [arms] and ('true' in [ARMS] or 'left' in [ARMS])) else 'false'}" />
-<xacro:property name="right_arm" value= "${'true' if ('true' in [arms] and ('true' in [ARMS] or 'right' in [ARMS])) else 'false'}" />
-<xacro:property name="legs" value="${'true' if ('false' not in [LEGS]) else 'false'}"/>
-<xacro:property name="pelvis" value= "${'true' if ('true' in [legs]) else 'false'}" />
-<xacro:property name="wheels" value="${'true' if ('false' not in [WHEELS, legs]) else 'false'}"/>
-<xacro:property name="static" value="${'true' if ('true' in [STATIC] or 'false' in [legs, LEG_ACTUATORS]) else 'false'}"/>
-<xacro:property name="reference" value="${'fixed' if (static == 'true') else 'floating'}" />
+<xacro:property name="torso" value="${'true' if (TORSO in [True, 'true', 'fixed'] ) else 'false'}"/>
+<xacro:property name="head" value="${'true' if (False not in [torso, HEAD] and 'false' not in [torso, HEAD]) else 'false'}"/>
+<xacro:property name="arms" value="${'true' if (False not in [TORSO, ARMS] and 'false' not in [TORSO, ARMS]) else 'false'}"/>
+<xacro:property name="left_arm" value= "${'true' if (arms in [True, 'true'] and (ARMS in [True, 'true', 'left'] )) else 'false'}" />
+<xacro:property name="right_arm" value= "${'true' if (arms in [True, 'true'] and (ARMS in [True, 'true', 'right'] )) else 'false'}" />
+<xacro:property name="legs" value="${'true' if (LEGS not in [False, 'false']) else 'false'}"/>
+<xacro:property name="pelvis" value= "${'true' if (legs in [True, 'true']) else 'false'}" />
+<xacro:property name="wheels" value="${'true' if (False not in [WHEELS, legs] and 'false' not in [WHEELS, legs]) else 'false'}"/>
+<xacro:property name="static" value="${'true' if (STATIC in [True, 'true'] or False in [legs, LEG_ACTUATORS]) else 'false'}"/>
+<xacro:property name="reference" value="${'fixed' if (static in [True, 'true']) else 'floating'}" />
 <xacro:property name="torso_joint" value="${'fixed' if ('fixed' in [TORSO]) else 'revolute'}"/>
 <xacro:property name="left_arm_mount" value= "${'revolute' if LEFT_END_EFFECTOR in ['soft_hand'] else 'fixed'}" />
@@ -50,17 +50,18 @@
 <xacro:property name="right_end_effector" value= "${RIGHT_END_EFFECTOR.split('fixed_', 2).pop()}" />
 <!-- ACTUATION -->
-<xacro:property name="torso_actuators" value="${'true' if ('false' not in [TORSO_ACTUATORS, TORSO]) else 'false'}"/>
-<xacro:property name="arm_actuators" value="${'true' if ('false' not in [ARM_ACTUATORS, TORSO_ACTUATORS, arms]) else 'false'}"/>
-<xacro:property name="leg_actuators" value="${'true' if ('false' not in [LEG_ACTUATORS, legs]) else 'false'}"/>
-<xacro:property name="head_actuators" value="${'true' if ('false' not in [HEAD_ACTUATORS, head]) else 'false'}"/>
-<xacro:property name="torso_actuators" value="${'true' if ('false' not in [TORSO_ACTUATORS, TORSO]) else 'false'}"/>
+<xacro:property name="torso_actuators" value="${'true' if (False not in [TORSO_ACTUATORS, TORSO] and 'false' not in [TORSO_ACTUATORS, TORSO]) else 'false'}"/>
+<xacro:property name="arm_actuators" value="${'true' if (False not in [ARM_ACTUATORS, TORSO_ACTUATORS, arms] and 'false' not in [ARM_ACTUATORS, TORSO_ACTUATORS, arms]) else 'false'}"/>
+<xacro:property name="leg_actuators" value="${'true' if (False not in [LEG_ACTUATORS, legs] and 'false' not in [LEG_ACTUATORS, legs]) else 'false'}"/>
+<xacro:property name="head_actuators" value="${'true' if (False not in [HEAD_ACTUATORS, head] and 'false' not in [HEAD_ACTUATORS, head]) else 'false'}"/>
+<xacro:property name="torso_actuators" value="${'true' if (False not in [TORSO_ACTUATORS, TORSO] and 'false' not in [TORSO_ACTUATORS, TORSO]) else 'false'}"/>
 <!-- SENSORS -->
-<xacro:property name="arm_sensors" value="${'true' if ('false' not in [ARM_SENSORS, arms]) else 'false'}"/>
-<xacro:property name="leg_sensors" value="${'true' if ('false' not in [LEG_SENSORS, legs]) else 'false'}"/>
-<xacro:property name="ft_sensors" value="${'revolute' if ('false' not in [FT_SENSORS]) else 'fixed'}"/>
-<xacro:property name="bumbers" value="${'true' if ('false' not in [BUMBERS]) else 'false'}"/>
-<xacro:property name="imu" value="${'true' if ('false' not in [IMU, pelvis]) else 'false'}"/>
-<xacro:property name="kinect" value="${'true' if ('false' not in [KINECT, head]) else 'false'}"/>
-<xacro:property name="velodyne" value="${'true' if ('false' not in [VELODYNE, head]) else 'false'}"/>
+<xacro:property name="arm_sensors" value="${'true' if (False not in [ARM_SENSORS, arms] and 'false' not in [ARM_SENSORS, arms]) else 'false'}"/>
+<xacro:property name="leg_sensors" value="${'true' if (False not in [LEG_SENSORS, legs] and 'false' not in [LEG_SENSORS, legs]) else 'false'}"/>
+<xacro:property name="ft_sensors" value="${'revolute' if (False not in [FT_SENSORS]) else 'fixed'}"/>
+<xacro:property name="bumbers" value="${'true' if (BUMBERS not in [False, 'false']) else 'false'}"/>
+<xacro:property name="imu" value="${'true' if (False not in [IMU, pelvis] and 'false' not in [IMU, pelvis]) else 'false'}"/>
+<xacro:property name="kinect" value="${'true' if (False not in [KINECT, head] and 'false' not in [KINECT, head]) else 'false'}"/>
+<xacro:property name="velodyne" value="${'true' if (False not in [VELODYNE, head] and 'false' not in [VELODYNE, head]) else 'false'}"/>
+<!--xacro:property name="velodyne" value="false"/-->
 <!-- LOAD PARAMETERS -->
 <xacro:property name="package" value="$(find centauro)"/>

File: centauro/centauro_urdf/urdf/models/model_config.xacro (robot description, xacro)
@@ -18,5 +18,5 @@
       <xacro:load_model path="upper_body/end_effectors/${right_end_effector}"  model="${model}"/>
    </xacro:if>
-   <xacro:if value="${head == 'true'}" >
+   <xacro:if value="${head in [True, 'true']}" >
       <xacro:load_model path="upper_body/head"  model="${model}"/>
    </xacro:if>

File: centauro_gazebo/sensors/config.xacro (robot description, xacro)
@@ -1,32 +1,3 @@
 <!--<?xml version="1.0"?>-->
 <robot  xmlns:xacro="http://www.ros.org/wiki/xacro">
-<xacro:include filename="$(find centauro)/centauro_urdf/urdf/config.xacro"/>
-   <xacro:macro name="load_model" params="middleware sensor arm_sensors leg_sensors head_sensors">
-      <xacro:include filename="$(find centauro_gazebo)/sensors/${middleware}/${sensor}/plugin.xacro"/>
-      <xacro:if value="${arm_sensors}">
-         <xacro:include filename="$(find centauro_gazebo)/sensors/${middleware}/${sensor}/load/arms.xacro"/>
-      </xacro:if>
-      <xacro:if value="${leg_sensors}">
-         <xacro:include filename="$(find centauro_gazebo)/sensors/${middleware}/${sensor}/load/legs.xacro"/>
-      </xacro:if>
-      <xacro:if value="${head_sensors}" >
-         <xacro:include filename="$(find centauro_gazebo)/sensors/${middleware}/${sensor}/load/head.xacro"/>
-      </xacro:if>
-   </xacro:macro>
-<!-- Load all controllers macros -->
-<xacro:if value="${ft_sensors == 'revolute'}">
-        <xacro:load_model middleware="${middleware}" sensor="ft_sensor" arm_sensors="${arm_sensors}" leg_sensors="${leg_sensors}" head_sensors="false"/>
-</xacro:if>
-<xacro:if value="${bumbers}">
-        <xacro:load_model middleware="${middleware}" sensor="bumber" arm_sensors="${arm_sensors}" leg_sensors="${leg_sensors}" head_sensors="false"/>
-</xacro:if>
-<xacro:if value="${imu}">
-        <xacro:load_model middleware="${middleware}" sensor="imu" arm_sensors="${arm_sensors}" leg_sensors="${leg_sensors}" head_sensors="false"/>
-</xacro:if>
-<xacro:if value="${kinect}">
-        <xacro:load_model middleware="${middleware}" sensor="kinect" arm_sensors="false" leg_sensors="false" head_sensors="${head}"/>
-</xacro:if>
-<xacro:if value="${velodyne}">
-        <xacro:load_model middleware="${middleware}" sensor="velodyne" arm_sensors="false" leg_sensors="false" head_sensors="${head}"/>
-</xacro:if>
 </robot>

Commit message: Restore sensors update

File: centauro/centauro_urdf/urdf/centauro.urdf.xacro (robot description, xacro)
@@ -32,5 +32,5 @@
 -->
 <link name="world"/>
-<xacro:if value="${pelvis}">
+<xacro:if value="${pelvis in [True, 'true']}">
    <link name="pelvis">
       <inertial>
@@ -58,7 +58,7 @@
     </joint>
 </xacro:if>
-<xacro:unless value="${pelvis}">
+<xacro:if value="${pelvis not in [True, 'true']}">
    <link name="pelvis"/>
-</xacro:unless>
+</xacro:if>
 <joint name="reference" type="${reference}">
    <origin xyz="${Pelvis_Ox} ${Pelvis_Oy} ${Pelvis_Oz}"/>

File: centauro/centauro_urdf/urdf/centauro_torso.urdf.xacro (robot description, xacro)
@@ -18,12 +18,12 @@
 <!-- torso joints -->
 <joint name="torso_yaw" type="${torso_joint}">
-   <xacro:if value="${pelvis}">
+   <xacro:if value="${pelvis in [True, 'true']}">
       <parent link="pelvis"/>
       <origin xyz="${Torso_2_Ox} ${Torso_2_Oy} ${Torso_2_Oz}"/>
    </xacro:if>
-   <xacro:unless value="${pelvis}">
+   <xacro:if value="${pelvis not  in [True, 'true']}">
       <parent link="world"/>
       <origin xyz="${Torso_2_Ox + Pelvis_Ox} ${Torso_2_Oy + Pelvis_Oy} ${Torso_2_Oz + Pelvis_Oz}"/>
-   </xacro:unless>
+   </xacro:if>
    <child link="torso_2"/>
    <axis xyz="0 0 1"/>

File: centauro_gazebo/sensors/config.xacro (robot description, xacro)
@@ -1,3 +1,32 @@
 <!--<?xml version="1.0"?>-->
 <robot  xmlns:xacro="http://www.ros.org/wiki/xacro">
+<xacro:include filename="$(find centauro)/centauro_urdf/urdf/config.xacro"/>
+   <xacro:macro name="load_model" params="middleware sensor arm_sensors leg_sensors head_sensors">
+      <xacro:include filename="$(find centauro_gazebo)/sensors/${middleware}/${sensor}/plugin.xacro"/>
+      <xacro:if value="${arm_sensors}">
+         <xacro:include filename="$(find centauro_gazebo)/sensors/${middleware}/${sensor}/load/arms.xacro"/>
+      </xacro:if>
+      <xacro:if value="${leg_sensors}">
+         <xacro:include filename="$(find centauro_gazebo)/sensors/${middleware}/${sensor}/load/legs.xacro"/>
+      </xacro:if>
+      <xacro:if value="${head_sensors}" >
+         <xacro:include filename="$(find centauro_gazebo)/sensors/${middleware}/${sensor}/load/head.xacro"/>
+      </xacro:if>
+   </xacro:macro>
+<!-- Load all controllers macros -->
+<xacro:if value="${ft_sensors == 'revolute'}">
+        <xacro:load_model middleware="${middleware}" sensor="ft_sensor" arm_sensors="${arm_sensors}" leg_sensors="${leg_sensors}" head_sensors="false"/>
+</xacro:if>
+<xacro:if value="${bumbers}">
+        <xacro:load_model middleware="${middleware}" sensor="bumber" arm_sensors="${arm_sensors}" leg_sensors="${leg_sensors}" head_sensors="false"/>
+</xacro:if>
+<xacro:if value="${imu}">
+        <xacro:load_model middleware="${middleware}" sensor="imu" arm_sensors="${arm_sensors}" leg_sensors="${leg_sensors}" head_sensors="false"/>
+</xacro:if>
+<xacro:if value="${kinect}">
+        <xacro:load_model middleware="${middleware}" sensor="kinect" arm_sensors="false" leg_sensors="false" head_sensors="${head}"/>
+</xacro:if>
+<xacro:if value="${velodyne}">
+        <xacro:load_model middleware="${middleware}" sensor="velodyne" arm_sensors="false" leg_sensors="false" head_sensors="${head}"/>
+</xacro:if>
 </robot>
