Commit message: Introduced flag for selecting gazebo control plugin (xbotcore or ros_control)

File: centauro/centauro_urdf/urdf/config.xacro (robot description, xacro)
@@ -14,4 +14,5 @@
 <xacro:property name="ONE_ARM" value="$(arg ONE_ARM)"/>
 <xacro:property name="GAZEBO" value="$(arg GAZEBO)"/>
+<xacro:property name="CONTROLLER" value="$(arg CONTROLLER)"/>
 <xacro:property name="INERTIA_PARAM" value="$(arg INERTIA_PARAM)"/>
 <xacro:property name="KINEMATIC_PARAM" value="$(arg KINEMATIC_PARAM)"/>
@@ -40,3 +41,5 @@
 <xacro:property name="inertia_parameters_file" value="${package + '/centauro_urdf/inertia_parameters/' + INERTIA_PARAM + '.xacro'}"/>
 <xacro:property name="kinematic_parameters_file" value="${package + '/centauro_urdf/kinematic_parameters/' + KINEMATIC_PARAM + '.xacro'}"/>
+<xacro:property name="xbotcore" value="${'true' if ('xbotcore' == CONTROLLER) else 'false'}"/>
+<xacro:property name="ros_control" value="${'true' if ('ros_control' == CONTROLLER) else 'false'}"/>
 </robot>

Commit message: add xbot_config_file parameter with default to advr_shared

File: centauro/centauro_urdf/urdf/config.xacro (robot description, xacro)
@@ -17,4 +17,5 @@
 <xacro:property name="GAZEBO" value="$(arg GAZEBO)"/>
 <xacro:property name="MIDDLEWARE" value="$(arg MIDDLEWARE)"/>
+<xacro:property name="XBOT_CONFIG_FILE" value="$(arg XBOT_CONFIG_FILE)"/>
 <xacro:property name="INERTIA_PARAM" value="$(arg INERTIA_PARAM)"/>
 <xacro:property name="KINEMATIC_PARAM" value="$(arg KINEMATIC_PARAM)"/>
@@ -54,4 +55,5 @@
 <!-- LOAD PARAMETERS -->
 <xacro:property name="package" value="$(find centauro)"/>
+<xacro:property name="xbot_config_file" value="${XBOT_CONFIG_FILE}"/>
 <xacro:property name="inertia_parameters_file" value="${package + '/centauro_urdf/inertia_parameters/' + INERTIA_PARAM + '.xacro'}"/>
 <xacro:property name="kinematic_parameters_file" value="${package + '/centauro_urdf/kinematic_parameters/' + KINEMATIC_PARAM + '.xacro'}"/>

Commit message: centauro/centauro_gazebo: tuning for schunk simulation

File: centauro/centauro_urdf/urdf/config.xacro (robot description, xacro)
@@ -62,5 +62,5 @@
 <xacro:property name="damping_legs" value="1.0" />
 <xacro:property name="damping_arms" value="0.2" />
-<xacro:property name="friction_schunk" value="1.0" />
+<xacro:property name="friction_schunk" value="2.0" />
 <xacro:property name="damping_schunk" value="0.0" />
 </robot>

File: centauro/centauro_urdf/urdf/models/upper_body/end_effectors/schunk_hand/svh_gazebo.urdf.xacro (robot description, xacro)
@@ -32,8 +32,9 @@
     <xacro:macro name="dummy_inertial">
 		<inertial>
-			<mass value="0.01" />
-			<inertia ixx="1e-6" ixy="0" ixz="0"
-				iyy="1e-6" iyz="0"
-				izz="1e-6" />
+			<mass value="0.05" />
+			<!-- solid sphere -->
+			<inertia ixx="${2.0 / 5.0 * 0.05 * (0.01*0.01)}" ixy="0" ixz="0"
+				iyy="${2.0 / 5.0 * 0.05 * (0.01*0.01)}" iyz="0"
+				izz="${2.0 / 5.0 * 0.05 * (0.01*0.01)}" />
 		</inertial>
     </xacro:macro>
@@ -104,5 +105,5 @@
                <origin rpy="0 0 0" xyz="0 0 0" />
                 <geometry>
-					<mesh filename="package://centauro/centauro_urdf/meshes/schunk_hand/camera_link.STL" /> <!-- FIXME: convex hull? -->
+					<mesh filename="package://centauro/centauro_urdf/meshes/schunk_hand/camera_link_convex.stl" /> <!-- FIXME: convex hull? -->
                 </geometry>
             </collision>

Commit message: correct evaluation of the static model with the gazbo9 support

File: centauro/centauro_urdf/urdf/config.xacro (robot description, xacro)
@@ -42,5 +42,5 @@
 <xacro:property name="pelvis" value= "${'true' if (legs in [True, 'true']) else 'false'}" />
 <xacro:property name="wheels" value="${'true' if (False not in [WHEELS, legs] and 'false' not in [WHEELS, legs]) else 'false'}"/>
-<xacro:property name="static" value="${'true' if (STATIC in [True, 'true'] or False in [legs, LEG_ACTUATORS]) else 'false'}"/>
+<xacro:property name="static" value="${'true' if (STATIC in [True, 'true'] or False in [legs, LEG_ACTUATORS] or 'false' in [legs, LEG_ACTUATORS]) else 'false'}"/>
 <xacro:property name="reference" value="${'fixed' if (static in [True, 'true']) else 'floating'}" />
 <xacro:property name="torso_joint" value="${'fixed' if ('fixed' in [TORSO]) else 'revolute'}"/>
