Commit message: neck joints limits

File: centauro/centauro_urdf/urdf/centauro_head.urdf.xacro (robot description, xacro)
@@ -48,5 +48,5 @@
    <child link="neck_1"/>
    <axis xyz="0 0 1"/>
-   <limit lower="-2.618" upper="2.618" effort="147" velocity="5.7"/> <!-- TODO -->
+   <limit lower="-0.78539816" upper="0.78539816" effort="35" velocity="5.7"/> <!-- TODO -->
 </joint>
 <joint name="neck_pitch" type="revolute">
@@ -55,5 +55,5 @@
    <child link="neck_2"/>
    <axis xyz="0 1 0"/>
-   <limit lower="-2.618" upper="2.618" effort="147" velocity="5.7"/> <!-- TODO -->
+   <limit lower="-0.34906585" upper="0.78539816" effort="35" velocity="5.7"/> <!-- TODO -->
 </joint>
 <joint name="neck_velodyne" type="revolute">
@@ -62,5 +62,5 @@
    <child link="neck_3"/>
    <axis xyz="0 0 1"/>
-   <limit lower="-2.618" upper="2.618" effort="147" velocity="5.7"/> <!-- TODO -->
+   <limit lower="-2.618" upper="2.618" effort="35" velocity="5.7"/> <!-- TODO -->
 </joint>
 <!-- /head joints -->

Commit message: Change velodyne joint to continuous

File: centauro/centauro_urdf/urdf/centauro_head.urdf.xacro (robot description, xacro)
@@ -57,10 +57,10 @@
    <limit lower="-0.34906585" upper="0.78539816" effort="35" velocity="5.7"/> <!-- TODO -->
 </joint>
-<joint name="neck_velodyne" type="revolute">
+<joint name="neck_velodyne" type="continuous">
    <parent link="torso_2"/>
    <origin xyz="${Neck_3_Ox} ${Neck_3_Oy} ${Neck_3_Oz}"/>
    <child link="neck_3"/>
    <axis xyz="0 0 1"/>
-   <limit lower="-2.618" upper="2.618" effort="35" velocity="5.7"/> <!-- TODO -->
+   <limit effort="35" velocity="5.7"/> <!-- TODO -->
 </joint>
 <!-- /head joints -->

Commit message: added kinect optical_frame link for calibration

File: centauro/centauro_urdf/urdf/centauro_head.urdf.xacro (robot description, xacro)
@@ -123,4 +123,11 @@
    <child link="kinect"/>
 </joint>
+<link name="kinect2_rgb_optical_frame" />
+<link name="cali_dummy" />
+<joint name="j_kinect_optical_frame" type="fixed">
+	<parent link="kinect"/>
+	<child link="cali_dummy" />
+	<origin xyz="0 0 0" rpy=" -${PI/2} 0 -${PI/2}"/>
+</joint>
 <joint name="j_velodyne" type="fixed">
    <parent link="neck_3"/>

Commit message: add Velodyne and laser rotator

File: centauro/centauro_urdf/urdf/centauro_head.urdf.xacro (robot description, xacro)
@@ -71,5 +71,5 @@
         </inertial>
 </link>
-<link name="velodyne">
+<link name="velodyne_mount">
 	<inertial>
 		<origin xyz="${Dummy_x} ${Dummy_y} ${Dummy_z}"/>
@@ -132,7 +132,11 @@
    <parent link="neck_3"/>
    <origin xyz="${Velodyne_Ox} ${Velodyne_Oy} ${Velodyne_Oz}" rpy="${Velodyne_roll} ${Velodyne_pitch} ${Velodyne_yaw}"/>
-   <child link="velodyne"/>
+   <child link="velodyne_mount"/>
 </joint>
 <!-- /sensors transformations -->
+<xacro:include filename="$(find velodyne_description)/urdf/VLP-16.urdf.xacro"/>
+<VLP-16 parent="velodyne_mount" name="velodyne" topic="/velodyne_points" hz="10" samples="440">
+	<origin xyz="0 0 0" rpy="-1.57079 0 -1.57079" />
+</VLP-16>
 <xacro:if value="${head_actuators}">
 <!-- torso actuators -->

Commit message: centauro: kinect2 extrinsic calibration

File: centauro/centauro_urdf/urdf/centauro_head.urdf.xacro (robot description, xacro)
@@ -124,9 +124,8 @@
 </joint>
 <link name="kinect2_rgb_optical_frame" />
-<link name="cali_dummy" />
 <joint name="j_kinect_optical_frame" type="fixed">
 	<parent link="kinect"/>
-	<child link="cali_dummy" />
-	<origin xyz="0 0 0" rpy=" -${PI/2} 0 -${PI/2}"/>
+	<child link="kinect2_rgb_optical_frame" />
+	<origin xyz="0.040 -0.040 -0.045" rpy=" -${PI/2} 0 -${PI/2}"/>
 </joint>
 <joint name="j_velodyne" type="fixed">

Commit message: centauro_urdf: kinect2 extrinsics update
to match iai_kinect2 driver

File: centauro/centauro_urdf/urdf/centauro_head.urdf.xacro (robot description, xacro)
@@ -127,5 +127,5 @@
 	<parent link="kinect"/>
 	<child link="kinect2_rgb_optical_frame" />
-	<origin xyz="0.040 -0.040 -0.045" rpy=" -${PI/2} 0 -${PI/2}"/>
+	<origin xyz="0.050 -0.110 -0.035" rpy=" -${PI/2} 0 -${PI/2}"/>
 </joint>
 <joint name="j_velodyne" type="fixed">

Commit message: velodyne orientation

File: centauro/centauro_urdf/urdf/centauro_head.urdf.xacro (robot description, xacro)
@@ -98,5 +98,5 @@
 <joint name="neck_velodyne" type="continuous">
    <parent link="torso_2"/>
-   <origin xyz="${Neck_3_Ox} ${Neck_3_Oy} ${Neck_3_Oz}"/>
+   <origin xyz="${Neck_3_Ox} ${Neck_3_Oy} ${Neck_3_Oz}" rpy="0.0 0.0 ${pi}"/>
    <child link="neck_3"/>
    <axis xyz="0 0 1"/>

Commit message: Revert "velodyne orientation"
This reverts commit bcc3bec248d4336dddac279fa7ccdf2dca0988f9.

File: centauro/centauro_urdf/urdf/centauro_head.urdf.xacro (robot description, xacro)
@@ -98,5 +98,5 @@
 <joint name="neck_velodyne" type="continuous">
    <parent link="torso_2"/>
-   <origin xyz="${Neck_3_Ox} ${Neck_3_Oy} ${Neck_3_Oz}" rpy="0.0 0.0 ${pi}"/>
+   <origin xyz="${Neck_3_Ox} ${Neck_3_Oy} ${Neck_3_Oz}"/>
    <child link="neck_3"/>
    <axis xyz="0 0 1"/>

Commit message: velodyne calib

File: centauro/centauro_urdf/urdf/centauro_head.urdf.xacro (robot description, xacro)
@@ -142,4 +142,10 @@
 	<origin xyz="0 0 0" rpy="-1.57079 0 -1.57079" />
 </VLP-16>
+<link name="velodyne_calib" />
+<joint name="velodyne_calib" type="fixed">
+   <parent link="velodyne"/>
+   <origin xyz="0 0 0" rpy="0 0 0.015"/>
+   <child link="velodyne_calib"/>
+</joint>
 <xacro:if value="${head_actuators}">
 <!-- torso actuators -->

Commit message: Update ankle yaw joint limits

File: centauro/centauro_urdf/urdf/centauro_head.urdf.xacro (robot description, xacro)
@@ -42,5 +42,5 @@
 </link>
 <!-- /head links -->
-<!-- sensors links -->
+<!-- sensors links
 <link name="camera_central">
 	<inertial>
@@ -79,4 +79,5 @@
         </inertial>
 </link>
+-->
 <!-- /sensors links -->
 <!-- head joints -->
@@ -103,5 +104,5 @@
 </joint>
 <!-- /head joints -->
-<!-- sensors transformations -->
+<!-- sensors transformations
 <joint name="j_camera_central" type="fixed">
    <parent link="torso_2"/>
@@ -134,4 +135,5 @@
    <child link="velodyne_mount"/>
 </joint>
+-->
 <!-- /sensors transformations -->
 <xacro:if value="${head_actuators}">

File: centauro/centauro_urdf/urdf/centauro_leg.urdf.xacro (robot description, xacro)
@@ -127,5 +127,5 @@
 	<origin xyz="${Ankle_2_Ox} ${Ankle_2_Oy} ${Ankle_2_Oz}" rpy="${Ankle_2_roll} ${Ankle_2_pitch} ${Ankle_2_yaw}"/>
 	<axis xyz="0 0 1"/>
-        <limit  lower="-2.79252680" upper="2.79252680" effort="35" velocity="20.0"/>
+        <limit  lower="-2.58308729" upper="2.58308729" effort="35" velocity="20.0"/>
 </joint>
 <joint name="j_wheel_${leg_num}" type="continuous">

Commit message: Update ankle yaw joint limits

File: centauro/centauro_urdf/urdf/centauro_head.urdf.xacro (robot description, xacro)
@@ -42,5 +42,5 @@
 </link>
 <!-- /head links -->
-<!-- sensors links
+<!-- sensors links -->
 <link name="camera_central">
 	<inertial>
@@ -79,5 +79,4 @@
         </inertial>
 </link>
--->
 <!-- /sensors links -->
 <!-- head joints -->
@@ -104,5 +103,5 @@
 </joint>
 <!-- /head joints -->
-<!-- sensors transformations
+<!-- sensors transformations  -->
 <joint name="j_camera_central" type="fixed">
    <parent link="torso_2"/>
@@ -135,5 +134,4 @@
    <child link="velodyne_mount"/>
 </joint>
--->
 <!-- /sensors transformations -->
 <xacro:if value="${head_actuators}">

File: centauro/centauro_urdf/urdf/centauro_mass.urdf.xacro (robot description, xacro)
@@ -13,5 +13,5 @@
         <origin xyz="0.0 0.0 0"  rpy="0.0 0.0 0.0"/>
         <geometry>
-          <box size="0.05 0.05 0.05"/>
+          <box size="0.1 0.1 0.1"/>
          </geometry>
          <material name="blue"/>
@@ -23,5 +23,5 @@
       <parent link="arm${arm_num}_8"/>
       <child link="arm${arm_num}_9"/>
-      <origin xyz="${rot*0.1} 0 0.1" rpy="0 0 0"/>
+      <origin xyz="${rot*0.065} 0 0.1" rpy="0 0 0"/>
    </joint> -->
 <!-- /joints -->

Commit message: initial commit to correct for velodyne frames so that pointcloud frames match that of the real robot

File: centauro/centauro_urdf/urdf/centauro_head.urdf.xacro (robot description, xacro)
@@ -153,9 +153,3 @@
 <!-- Kinect simulation -->
 <!-- /sensors transformations -->
-<link name="velodyne_calib" />
-<joint name="velodyne_calib" type="fixed">
-   <parent link="neck_3"/>
-  <origin xyz="-0.175768 0 -0.034219" rpy="-1.57772 0.0128311 1.57073"/>
-   <child link="velodyne_calib"/>
-</joint>
 </robot>

File: centauro_gazebo/sensors/ros_control/velodyne/load/head.xacro (robot description, xacro)
@@ -1,6 +1,6 @@
 <!--<?xml version="1.0"?>-->
 <robot  xmlns:xacro="http://www.ros.org/wiki/xacro">
-        <VLP-16 parent="velodyne_mount" name="velodyne" topic="/velodyne_points" hz="10" samples="440">
-        	<origin xyz="0 0 0" rpy="-1.57079 0 -1.57079" />
-        </VLP-16>
+      <VLP-16 parent="neck_3" name="velodyne_calib" topic="/velodyne_points" hz="10" samples="440">
+        <origin xyz="0.032768 -0.01 0.048219" rpy="0 1.5709 -0.316519  " />
+      </VLP-16>
 </robot>

File: centauro_gazebo/sensors/xbotcore/velodyne/load/head.xacro (robot description, xacro)
@@ -1,6 +1,6 @@
 <!--<?xml version="1.0"?>-->
 <robot  xmlns:xacro="http://www.ros.org/wiki/xacro">
-        <VLP-16 parent="velodyne_mount" name="velodyne" topic="/velodyne_points" hz="10" samples="440">
-        	<origin xyz="0 0 0" rpy="-1.57079 0 -1.57079" />
+        <VLP-16 parent="neck_3" name="velodyne_calib" topic="/velodyne_points" hz="10" samples="440">
+        	<origin xyz="0.032768 -0.01 0.048219" rpy="0 1.5709 -0.316519  " />
         </VLP-16>
 </robot>
