Commit message: Updated generated urdf

File: centauro/centauro_urdf/urdf/centauro.urdf (robot description, URDF)
Before this commit: robot centauro, 43 links, 42 joints
Links:
- added link imu_link, mass 0.0
Joints:
- added joint imu_joint: type fixed, parent pelvis, child imu_link, origin xyz=0.0 0.0 0.0 rpy=0.0 0.0 0.0
- joint hip_yaw_1: limit lower=-0.78539816 upper=2.35619449 effort=304 velocity=8.8 -> lower=-1.13446401 upper=2.70526034 effort=304 velocity=8.8
- joint hip_yaw_2: limit lower=-2.35619449 upper=0.78539816 effort=304 velocity=8.8 -> lower=-2.70526034 upper=1.13446401 effort=304 velocity=8.8
- joint hip_yaw_3: limit lower=-2.35619449 upper=0.78539816 effort=304 velocity=8.8 -> lower=-2.70526034 upper=1.13446401 effort=304 velocity=8.8
- joint hip_yaw_4: limit lower=-0.78539816 upper=2.35619449 effort=304 velocity=8.8 -> lower=-1.13446401 upper=2.70526034 effort=304 velocity=8.8

Commit message: Monday Final

File: centauro/centauro_urdf/urdf/centauro.urdf (robot description, URDF)
Before this commit: robot centauro, 53 links, 52 joints
Links:
- link arm1_8: mass 1.8366865 -> 0.15; geometry collision cylinder length=0.13 radius=0.013; visual mesh filename=package://centauro/centauro_urdf/meshes/simplified/link9.stl scale=0.001 -0.001 -0.001
- link arm2_8: mass 1.8366865 -> 0.15; geometry collision cylinder length=0.13 radius=0.013; visual mesh filename=package://centauro/centauro_urdf/meshes/simplified/link9.stl scale=0.001 0.001 -0.001
Joints:
- joint j_arm1_8: origin xyz=0.0 0.0 -0.0405 rpy=0.0 3.14159265359 3.14159265359 -> xyz=0.0 0.0 -0.0405 rpy=0.0 3.14159265359 -1.5707963268
- joint j_arm2_8: origin xyz=0.0 0.0 -0.0405 rpy=0.0 3.14159265359 3.14159265359 -> xyz=0.0 0.0 -0.0405 rpy=0.0 3.14159265359 -1.5707963268

Commit message: Added new arms

File: centauro/centauro_urdf/urdf/centauro.urdf (robot description, URDF)
Before this commit: robot centauro, 91 links, 90 joints
Links:
- removed link ft_arm1
- removed link ft_arm2
- removed link right_hand_a
- removed link right_hand_b
- removed link right_hand_base_link
- removed link right_hand_c
- removed link right_hand_camera_link
- removed link right_hand_d
- removed link right_hand_d2
- removed link right_hand_e
- removed link right_hand_e1
- removed link right_hand_e2
- removed link right_hand_e3
- removed link right_hand_e4
- removed link right_hand_e5
- removed link right_hand_h
- removed link right_hand_i
- removed link right_hand_index_tip_ee
- removed link right_hand_j
- removed link right_hand_k
- removed link right_hand_l
- removed link right_hand_m
- removed link right_hand_middle_tip_ee
- removed link right_hand_n
- removed link right_hand_o
- removed link right_hand_p
- removed link right_hand_pinky_tip_ee
- removed link right_hand_q
- removed link right_hand_r
- removed link right_hand_ring_tip_ee
- removed link right_hand_s
- removed link right_hand_t
- removed link right_hand_thumb_tip_ee
- removed link right_hand_virtual_a
- removed link right_hand_virtual_i
- removed link right_hand_virtual_j
- removed link right_hand_virtual_k
- removed link right_hand_virtual_l
- removed link right_hand_z
- added link DWYTorso
- added link LElb, mass 1.3157289; collision mesh filename=package://cogimon_urdf/meshes/simple/Elbow.STL scale=0.001 -0.001 0.001; visual mesh filename=package://cogimon_urdf/meshes/Elbow.STL scale=0.001 -0.001 0.001
- added link LForearm, mass 1.4908547; collision mesh filename=package://cogimon_urdf/meshes/simple/Forearm.STL scale=0.001 -0.001 0.001; visual mesh filename=package://cogimon_urdf/meshes/Forearm.STL scale=0.001 -0.001 0.001
- added link LShp, mass 1.9628675; collision mesh filename=package://cogimon_urdf/meshes/simple/ShoulderPitch.STL scale=0.001 -0.001 0.001; visual mesh filename=package://cogimon_urdf/meshes/ShoulderPitch.STL scale=0.001 -0.001 0.001
- added link LShr, mass 1.8595811; collision mesh filename=package://cogimon_urdf/meshes/simple/ShoulderRoll.STL scale=0.001 -0.001 0.001; visual mesh filename=package://cogimon_urdf/meshes/ShoulderRoll.STL scale=0.001 -0.001 0.001
- added link LShy, mass 1.6678109; collision mesh filename=package://cogimon_urdf/meshes/simple/ShoulderYaw.STL scale=0.001 -0.001 0.001; visual mesh filename=package://cogimon_urdf/meshes/ShoulderYaw.STL scale=0.001 -0.001 0.001
- added link LWrMot2, mass 1.1263612; collision mesh filename=package://cogimon_urdf/meshes/simple/ForearmPitch.STL scale=0.001 -0.001 0.001; visual mesh filename=package://cogimon_urdf/meshes/ForearmPitch.STL scale=0.001 -0.001 0.001
- added link LWrMot3, mass 2.7966428e-01; collision mesh filename=package://cogimon_urdf/meshes/simple/ForearmYaw.STL scale=0.001 -0.001 0.001; visual mesh filename=package://cogimon_urdf/meshes/ForearmYaw.STL scale=0.001 -0.001 0.001
- added link RElb, mass 1.3157289; collision mesh filename=package://cogimon_urdf/meshes/simple/Elbow.STL scale=0.001 0.001 0.001; visual mesh filename=package://cogimon_urdf/meshes/Elbow.STL scale=0.001 0.001 0.001
- added link RForearm, mass 1.4908547; collision mesh filename=package://cogimon_urdf/meshes/simple/Forearm.STL scale=0.001 0.001 0.001; visual mesh filename=package://cogimon_urdf/meshes/Forearm.STL scale=0.001 0.001 0.001
- added link RShp, mass 1.9628675; collision mesh filename=package://cogimon_urdf/meshes/simple/ShoulderPitch.STL scale=0.001 0.001 0.001; visual mesh filename=package://cogimon_urdf/meshes/ShoulderPitch.STL scale=0.001 0.001 0.001
- added link RShr, mass 1.8595811; collision mesh filename=package://cogimon_urdf/meshes/simple/ShoulderRoll.STL scale=0.001 0.001 0.001; visual mesh filename=package://cogimon_urdf/meshes/ShoulderRoll.STL scale=0.001 0.001 0.001
- added link RShy, mass 1.6678109; collision mesh filename=package://cogimon_urdf/meshes/simple/ShoulderYaw.STL scale=0.001 0.001 0.001; visual mesh filename=package://cogimon_urdf/meshes/ShoulderYaw.STL scale=0.001 0.001 0.001
- added link RWrMot2, mass 1.1263612; collision mesh filename=package://cogimon_urdf/meshes/simple/ForearmPitch.STL scale=0.001 0.001 0.001; visual mesh filename=package://cogimon_urdf/meshes/ForearmPitch.STL scale=0.001 0.001 0.001
- added link RWrMot3, mass 2.7966428e-01; collision mesh filename=package://cogimon_urdf/meshes/simple/ForearmYaw.STL scale=0.001 0.001 0.001; visual mesh filename=package://cogimon_urdf/meshes/ForearmYaw.STL scale=0.001 0.001 0.001
- added link arm2_8
- added link kinect2_rgb_frame
- added link l_wrist, mass 3.7827821e-01; collision mesh filename=package://cogimon_urdf/meshes/simple/Wrist.STL scale=0.001 -0.001 0.001; visual mesh filename=package://cogimon_urdf/meshes/Wrist.STL scale=0.001 -0.001 0.001
- added link r_wrist, mass 3.7827821e-01; collision mesh filename=package://cogimon_urdf/meshes/simple/Wrist.STL scale=0.001 0.001 0.001; visual mesh filename=package://cogimon_urdf/meshes/Wrist.STL scale=0.001 0.001 0.001
- added link velodyne_calib
- link arm1_1: mass 1.5583338 -> None; geometry 
- link arm1_2: mass 1.515061 -> None; geometry 
- link arm1_3: mass 1.5088101 -> None; geometry 
- link arm1_4: mass 0.96297329 -> None; geometry 
- link arm1_5: mass 1.4703698 -> None; geometry 
- link arm1_6: mass 0.94693868 -> None; geometry 
- link arm1_7: mass 0.55981036 -> None; geometry 
- link arm1_8: mass 1.8366865 -> None; geometry 
- link arm2_1: mass 1.5583338 -> None; geometry 
- link arm2_2: mass 1.515061 -> None; geometry 
- link arm2_3: mass 1.5088101 -> None; geometry 
- link arm2_4: mass 0.96297329 -> None; geometry 
- link arm2_5: mass 1.4703698 -> None; geometry 
- link arm2_6: mass 0.94693868 -> None; geometry 
- link arm2_7: mass 0.55981036 -> None; geometry 
Joints:
- removed joint j_arm1_1
- removed joint j_arm1_2
- removed joint j_arm1_3
- removed joint j_arm1_4
- removed joint j_arm1_5
- removed joint j_arm1_6
- removed joint j_arm1_7
- removed joint j_arm1_8
- removed joint j_arm2_1
- removed joint j_arm2_2
- removed joint j_arm2_3
- removed joint j_arm2_4
- removed joint j_arm2_5
- removed joint j_arm2_6
- removed joint j_arm2_7
- removed joint j_ft_1
- removed joint j_ft_2
- removed joint right_hand_Finger_Spread
- removed joint right_hand_Index_Finger_Distal
- removed joint right_hand_Index_Finger_Proximal
- removed joint right_hand_Middle_Finger_Distal
- removed joint right_hand_Middle_Finger_Proximal
- removed joint right_hand_Pinky
- removed joint right_hand_Ring_Finger
- removed joint right_hand_Thumb_Flexion
- removed joint right_hand_Thumb_Helper
- removed joint right_hand_Thumb_Opposition
- removed joint right_hand_base_joint
- removed joint right_hand_camera_joint
- removed joint right_hand_f1
- removed joint right_hand_f2
- removed joint right_hand_f3
- removed joint right_hand_f4
- removed joint right_hand_f5
- removed joint right_hand_f6
- removed joint right_hand_f7
- removed joint right_hand_f8
- removed joint right_hand_index_spread
- removed joint right_hand_index_tip_joint
- removed joint right_hand_j12
- removed joint right_hand_j13
- removed joint right_hand_j14
- removed joint right_hand_j15
- removed joint right_hand_j16
- removed joint right_hand_j17
- removed joint right_hand_j3
- removed joint right_hand_j4
- removed joint right_hand_j5
- removed joint right_hand_middle_spread_dummy
- removed joint right_hand_middle_tip_joint
- removed joint right_hand_pinky_tip_joint
- removed joint right_hand_ring_spread
- removed joint right_hand_ring_tip_joint
- removed joint right_hand_thumb_tip_joint
- added joint LElbj: type revolute, parent LShy, child LElb, origin xyz=0.045 0.05515 -0.074 rpy=0 0 0, axis 0 1 0, limit lower=-2.492 upper=0.298 effort=120 velocity=6.283
- added joint LForearmPlate: type revolute, parent LElb, child LForearm, origin xyz=-0.015 -0.05515 -0.095 rpy=0 0 0, axis 0 0 1, limit lower=-2.55 upper=2.55 effort=35 velocity=6.283
- added joint LShLat: type revolute, parent LShp, child LShr, origin xyz=-0.09015 0.062 0 rpy=-0.1745327 0 0, axis 1 0 0, limit lower=0.0 upper=3.517 effort=140 velocity=6.283
- added joint LShSag: type revolute, parent DWYTorso, child LShp, origin xyz=0.0457475 0.169137 0.155126 rpy=0.174533 0 -0.5235988, axis 0 1 0, limit lower=-3.352 upper=1.603 effort=140 velocity=6.283
- added joint LShYaw: type revolute, parent LShr, child LShy, origin xyz=0.09015 0 -0.21815 rpy=0 0 0, axis 0 0 1, limit lower=-2.55 upper=2.55 effort=120 velocity=6.283
- added joint LWrj1: type revolute, parent LForearm, child LWrMot2, origin xyz=0 0.049 -0.156 rpy=0 0 0, axis 0 1 0, limit lower=-1.562 upper=1.478 effort=35 velocity=6.283
- added joint LWrj2: type revolute, parent LWrMot2, child LWrMot3, origin xyz=0 -0.049 -0.174 rpy=0 0 0, axis 0 0 1, limit lower=-2.55 upper=2.55 effort=20 velocity=6.283
- added joint RElbj: type revolute, parent RShy, child RElb, origin xyz=0.045 -0.05515 -0.074 rpy=0 0 0, axis 0 1 0, limit lower=-2.488 upper=0.292 effort=120 velocity=6.283
- added joint RForearmPlate: type revolute, parent RElb, child RForearm, origin xyz=-0.015 0.05515 -0.095 rpy=0 0 0, axis 0 0 1, limit lower=-2.55 upper=2.55 effort=35 velocity=6.283
- added joint RShLat: type revolute, parent RShp, child RShr, origin xyz=-0.09015 -0.062 0 rpy=0.1745327 0 0, axis 1 0 0, limit lower=-3.43 upper=0.0 effort=140 velocity=6.283
- added joint RShSag: type revolute, parent DWYTorso, child RShp, origin xyz=0.0457475 -0.169137 0.155126 rpy=-0.174533 0 0.5235988, axis 0 1 0, limit lower=-3.359 upper=1.606 effort=140 velocity=6.283
- added joint RShYaw: type revolute, parent RShr, child RShy, origin xyz=0.09015 0 -0.21815 rpy=0 0 0, axis 0 0 1, limit lower=-2.55 upper=2.55 effort=120 velocity=6.283
- added joint RWrj1: type revolute, parent RForearm, child RWrMot2, origin xyz=0 -0.049 -0.156 rpy=0 0 0, axis 0 1 0, limit lower=-1.542 upper=1.508 effort=35 velocity=6.283
- added joint RWrj2: type revolute, parent RWrMot2, child RWrMot3, origin xyz=0 0.049 -0.174 rpy=0 0 0, axis 0 0 1, limit lower=-2.55 upper=2.55 effort=20 velocity=6.283
- added joint j_kinect2_rgb_frame: type fixed, parent kinect, child kinect2_rgb_frame, origin xyz=0.050 -0.110 -0.035
- added joint jf1: type fixed, parent LShp, child arm1_1, origin xyz=0 0 0 rpy=0 0 0
- added joint jf10: type fixed, parent RShr, child arm2_2, origin xyz=0 0 0 rpy=0 0 0
- added joint jf11: type fixed, parent RShy, child arm2_3, origin xyz=0 0 0 rpy=0 0 0
- added joint jf12: type fixed, parent RElb, child arm2_4, origin xyz=0 0 0 rpy=0 0 0
- added joint jf13: type fixed, parent RForearm, child arm2_5, origin xyz=0 0 0 rpy=0 0 0
- added joint jf14: type fixed, parent RWrMot2, child arm2_6, origin xyz=0 0 0 rpy=0 0 0
- added joint jf15: type fixed, parent RWrMot3, child arm2_7, origin xyz=0 0 0 rpy=0 0 0
- added joint jf16: type fixed, parent arm2_7, child arm2_8, origin xyz=0 0 0 rpy=0 0 0
- added joint jf2: type fixed, parent LShr, child arm1_2, origin xyz=0 0 0 rpy=0 0 0
- added joint jf3: type fixed, parent LShy, child arm1_3, origin xyz=0 0 0 rpy=0 0 0
- added joint jf4: type fixed, parent LElb, child arm1_4, origin xyz=0 0 0 rpy=0 0 0
- added joint jf5: type fixed, parent LForearm, child arm1_5, origin xyz=0 0 0 rpy=0 0 0
- added joint jf6: type fixed, parent LWrMot2, child arm1_6, origin xyz=0 0 0 rpy=0 0 0
- added joint jf7: type fixed, parent LWrMot3, child arm1_7, origin xyz=0 0 0 rpy=0 0 0
- added joint jf8: type fixed, parent arm1_7, child arm1_8, origin xyz=0 0 0 rpy=0 0 0
- added joint jf9: type fixed, parent RShp, child arm2_1, origin xyz=0 0 0 rpy=0 0 0
- added joint l_wrist_joint: type fixed, parent LWrMot3, child l_wrist, origin xyz=0 0 0 rpy=0 0 0
- added joint r_wrist_joint: type fixed, parent RWrMot3, child r_wrist, origin xyz=0 0 0 rpy=0 0 0
- added joint torso_renaming: type fixed, parent torso_2, child DWYTorso, origin xyz=0 0 -0.0385 rpy=0 0 0
- added joint velodyne_calib: type fixed, parent neck_3, child velodyne_calib, origin xyz=-0.175768 0 -0.034219 rpy=-1.57772 0.0128311 1.57073
- joint imu_joint: origin xyz=0.0 0.0 0.0 rpy=0.0 0.0 0.0 -> xyz=0.248316 0.0 0.015 rpy=0.0 0.0 0.0
- joint j_kinect_optical_frame: origin xyz=0.050 -0.110 -0.035 rpy= -1.5707963268 0 -1.5707963268 -> rpy= -1.5707963268 0 -1.5707963268; parent kinect -> kinect2_rgb_frame

File: centauro/centauro_urdf/urdf/centauro.urdf.xacro (robot description, xacro)
@@ -19,7 +19,7 @@
   <xacro:include filename="$(find centauro)/centauro_urdf/urdf/centauro_leg.urdf.xacro"/>
 </xacro:if>
-<xacro:if value="${arms}">
+<!--xacro:if value="${arms}">
   <xacro:include filename="$(find centauro)/centauro_urdf/urdf/centauro_arm.urdf.xacro"/>
-</xacro:if>
+</xacro:if-->
 <!-- /other files -->
 <!-- reference -->
@@ -76,4 +76,5 @@
 <!-- /torso -->
 <!-- arms -->
+<!--
 <xacro:if value="${left_arm == 'true'}">
    <xacro:centauro_arm arm_num="1"  rot="1"  parent="torso_2" end_effector="${left_end_effector}" mount="${left_arm_mount}">
@@ -86,4 +87,16 @@
    </xacro:centauro_arm>
 </xacro:if>
+-->
+<xacro:property name="COGIMON_LEFT_ARM" value="true" />
+<xacro:property name="COGIMON_RIGHT_ARM" value="true" />
+<link name="DWYTorso"/>
+<joint name="torso_renaming" type="fixed">
+       <parent link="torso_2"/>
+       <child link="DWYTorso"/>
+       <origin xyz="0 0 -0.0385" rpy="0 0 0" />
+</joint>
+<xacro:include filename="$(find cogimon_urdf)/urdf/conversions.urdf.xacro" />
+<xacro:include filename="$(find cogimon_urdf)/urdf/parts/arms.urdf.xacro" />
+<xacro:include filename="$(find centauro)/centauro_urdf/urdf/centauro_arm_frames.urdf.xacro" />
 <!-- /arms -->
 <!-- legs -->
