Commit message: Added new arms

File: centauro/centauro_urdf/urdf/centauro_capsules.urdf (robot description, URDF)
Before this commit: robot centauro, 17 links, 16 joints
Links:
- added link DWYTorso
- added link LElb, mass 1.3157289; collision cylinder length=0.0871341857294 radius=0.0600429; visual mesh filename=package://cogimon_urdf/meshes/Elbow.STL scale=0.001 -0.001 0.001
- added link LForearm, mass 1.4908547; collision cylinder length=0.0843473974771 radius=0.0804108; visual mesh filename=package://cogimon_urdf/meshes/Forearm.STL scale=0.001 -0.001 0.001
- added link LShp, mass 1.9628675; collision cylinder length=0.0373976849456 radius=0.0698859; visual mesh filename=package://cogimon_urdf/meshes/ShoulderPitch.STL scale=0.001 -0.001 0.001
- added link LShr, mass 1.8595811; collision cylinder length=0.127992690725 radius=0.0700645; visual mesh filename=package://cogimon_urdf/meshes/ShoulderRoll.STL scale=0.001 -0.001 0.001
- added link LShy, mass 1.6678109; collision cylinder length=0.060822526466 radius=0.0896121; visual mesh filename=package://cogimon_urdf/meshes/ShoulderYaw.STL scale=0.001 -0.001 0.001
- added link LWrMot2, mass 1.1263612; collision cylinder length=0.114251418714 radius=0.0583263; visual mesh filename=package://cogimon_urdf/meshes/ForearmPitch.STL scale=0.001 -0.001 0.001
- added link LWrMot3, mass 0.27966428; collision cylinder length=0.00916730749359 radius=0.0207073; visual mesh filename=package://cogimon_urdf/meshes/ForearmYaw.STL scale=0.001 -0.001 0.001
- added link RElb, mass 1.3157289; collision cylinder length=0.0871341857294 radius=0.0600429; visual mesh filename=package://cogimon_urdf/meshes/Elbow.STL scale=0.001 0.001 0.001
- added link RForearm, mass 1.4908547; collision cylinder length=0.0843473974771 radius=0.0804108; visual mesh filename=package://cogimon_urdf/meshes/Forearm.STL scale=0.001 0.001 0.001
- added link RShp, mass 1.9628675; collision cylinder length=0.0373976849456 radius=0.0698859; visual mesh filename=package://cogimon_urdf/meshes/ShoulderPitch.STL scale=0.001 0.001 0.001
- added link RShr, mass 1.8595811; collision cylinder length=0.127992690725 radius=0.0700645; visual mesh filename=package://cogimon_urdf/meshes/ShoulderRoll.STL scale=0.001 0.001 0.001
- added link RShy, mass 1.6678109; collision cylinder length=0.060822526466 radius=0.0896121; visual mesh filename=package://cogimon_urdf/meshes/ShoulderYaw.STL scale=0.001 0.001 0.001
- added link RWrMot2, mass 1.1263612; collision cylinder length=0.114251418714 radius=0.0583263; visual mesh filename=package://cogimon_urdf/meshes/ForearmPitch.STL scale=0.001 0.001 0.001
- added link RWrMot3, mass 0.27966428; collision cylinder length=0.00916730749359 radius=0.0207073; visual mesh filename=package://cogimon_urdf/meshes/ForearmYaw.STL scale=0.001 0.001 0.001
- added link ankle1_1, mass 1.2380744; collision cylinder length=0.0427933218169 radius=0.0763963; visual mesh filename=package://centauro/centauro_urdf/meshes/simplified/ankle-pi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 scale=0.001 0.001 0.001
- added link ankle1_2, mass 1.2380744; collision cylinder length=0.0427933218169 radius=0.0763963; visual mesh filename=package://centauro/centauro_urdf/meshes/simplified/ankle-pi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 scale=0.001 0.001 0.001
- added link ankle1_3, mass 1.2380744; collision cylinder length=0.0427933218169 radius=0.0763963; visual mesh filename=package://centauro/centauro_urdf/meshes/simplified/ankle-pi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 scale=0.001 0.001 0.001
- added link ankle1_4, mass 1.2380744; collision cylinder length=0.0427933218169 radius=0.0763963; visual mesh filename=package://centauro/centauro_urdf/meshes/simplified/ankle-pi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 scale=0.001 0.001 0.001
- added link ankle2_1, mass 1.1565926; collision cylinder length=0.014473082934 radius=0.101494; visual mesh filename=package://centauro/centauro_urdf/meshes/simplified/ankle-ya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 scale=0.001 0.001 0.001
- added link ankle2_2, mass 1.1565926; collision cylinder length=0.014473082934 radius=0.101494; visual mesh filename=package://centauro/centauro_urdf/meshes/simplified/ankle-ya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 scale=0.001 0.001 0.001
- added link ankle2_3, mass 1.1565926; collision cylinder length=0.014473082934 radius=0.101494; visual mesh filename=package://centauro/centauro_urdf/meshes/simplified/ankle-ya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 scale=0.001 0.001 0.001
- added link ankle2_4, mass 1.1565926; collision cylinder length=0.014473082934 radius=0.101494; visual mesh filename=package://centauro/centauro_urdf/meshes/simplified/ankle-ya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 scale=0.001 0.001 0.001
- added link arm1_8
- added link arm2_8
- added link camera_central, mass 0.1
- added link camera_left, mass 0.1
- added link camera_right, mass 0.1
- added link hip1_1, mass 1.9194403; collision cylinder length=0.0345165338408 radius=0.0653044; visual mesh filename=package://centauro/centauro_urdf/meshes/simplified/hip-yaw.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 scale=0.001 0.001 0.001
- added link hip1_2, mass 1.9194403; collision cylinder length=0.0345165338408 radius=0.0653044; visual mesh filename=package://centauro/centauro_urdf/meshes/simplified/hip-yaw.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 scale=0.001 0.001 0.001
- added link hip1_3, mass 1.9194403; collision cylinder length=0.0345165338408 radius=0.0653044; visual mesh filename=package://centauro/centauro_urdf/meshes/simplified/hip-yaw.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 scale=0.001 0.001 0.001
- added link hip1_4, mass 1.9194403; collision cylinder length=0.0345165338408 radius=0.0653044; visual mesh filename=package://centauro/centauro_urdf/meshes/simplified/hip-yaw.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 scale=0.001 0.001 0.001
- added link hip2_1, mass 2.7264471; collision cylinder length=0.292249159884 radius=0.0847444; visual mesh filename=package://centauro/centauro_urdf/meshes/simplified/hip-pitc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 scale=0.001 0.001 0.001
- added link hip2_2, mass 2.7264471; collision cylinder length=0.292249159884 radius=0.0847444; visual mesh filename=package://centauro/centauro_urdf/meshes/simplified/hip-pitc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 scale=0.001 0.001 0.001
- added link hip2_3, mass 2.7264471; collision cylinder length=0.292249159884 radius=0.0847444; visual mesh filename=package://centauro/centauro_urdf/meshes/simplified/hip-pitc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 scale=0.001 0.001 0.001
- added link hip2_4, mass 2.7264471; collision cylinder length=0.292249159884 radius=0.0847444; visual mesh filename=package://centauro/centauro_urdf/meshes/simplified/hip-pitc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 scale=0.001 0.001 0.001
- added link imu_link, mass 0.0
- added link kinect, mass 0.1
- added link kinect2_rgb_frame
- added link kinect2_rgb_optical_frame
- added link knee_1, mass 1.9356754; collision cylinder length=0.192525790304 radius=0.066434; visual mesh filename=package://centauro/centauro_urdf/meshes/simplified/knee.stl scale=0.001 0.001 0.001
- added link knee_2, mass 1.9356754; collision cylinder length=0.192525790304 radius=0.066434; visual mesh filename=package://centauro/centauro_urdf/meshes/simplified/knee.stl scale=0.001 0.001 0.001
- added link knee_3, mass 1.9356754; collision cylinder length=0.192525790304 radius=0.066434; visual mesh filename=package://centauro/centauro_urdf/meshes/simplified/knee.stl scale=0.001 0.001 0.001
- added link knee_4, mass 1.9356754; collision cylinder length=0.192525790304 radius=0.066434; visual mesh filename=package://centauro/centauro_urdf/meshes/simplified/knee.stl scale=0.001 0.001 0.001
- added link l_wrist, mass 0.37827821; collision cylinder length=0.0628232385677 radius=0.0468649; visual mesh filename=package://cogimon_urdf/meshes/Wrist.STL scale=0.001 -0.001 0.001
- added link neck_1, mass 0.33878686; collision cylinder length=0.10965536987 radius=0.0257769; visual mesh filename=package://centauro/centauro_urdf/meshes/simplified/neck_yaw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 scale=0.001 0.001 0.001
- added link neck_2, mass 0.78526942; collision cylinder length=0.111328782421 radius=0.0423975; visual mesh filename=package://centauro/centauro_urdf/meshes/simplified/neck_pit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 scale=0.001 0.001 0.001
- added link neck_3, mass 0.78526942; collision cylinder length=0.114524744064 radius=0.0519914; visual mesh filename=package://centauro/centauro_urdf/meshes/simplified/velodyne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 scale=0.001 0.001 0.001
- added link r_wrist, mass 0.37827821; collision cylinder length=0.0628232385677 radius=0.0468649; visual mesh filename=package://cogimon_urdf/meshes/Wrist.STL scale=0.001 0.001 0.001
- added link velodyne_calib
- added link velodyne_mount, mass 0.1
- added link wheel_1, mass 1.7289003; collision cylinder length=0.00108743512283 radius=0.08665; visual mesh filename=package://centauro/centauro_urdf/meshes/simplified/wheel.stl scale=0.001 0.001 0.001
- added link wheel_2, mass 1.7289003; collision cylinder length=0.00108743512283 radius=0.08665; visual mesh filename=package://centauro/centauro_urdf/meshes/simplified/wheel.stl scale=0.001 0.001 0.001
- added link wheel_3, mass 1.7289003; collision cylinder length=0.00108743512283 radius=0.08665; visual mesh filename=package://centauro/centauro_urdf/meshes/simplified/wheel.stl scale=0.001 0.001 0.001
- added link wheel_4, mass 1.7289003; collision cylinder length=0.00108743512283 radius=0.08665; visual mesh filename=package://centauro/centauro_urdf/meshes/simplified/wheel.stl scale=0.001 0.001 0.001
- link arm1_1: mass 1.7 -> None; geometry 
- link arm1_2: mass 2.0 -> None; geometry 
- link arm1_3: mass 2.0 -> None; geometry 
- link arm1_4: mass 1.3 -> None; geometry 
- link arm1_5: mass 1.4 -> None; geometry 
- link arm1_6: mass 1.1 -> None; geometry 
- link arm1_7: mass 1.7 -> None; geometry 
- link arm2_1: mass 1.7 -> None; geometry 
- link arm2_2: mass 2.0 -> None; geometry 
- link arm2_3: mass 2.0 -> None; geometry 
- link arm2_4: mass 1.3 -> None; geometry 
- link arm2_5: mass 1.4 -> None; geometry 
- link arm2_6: mass 1.1 -> None; geometry 
- link arm2_7: mass 1.7 -> None; geometry 
- link pelvis: mass 25.0 -> 16.097574; geometry collision cylinder length=0.385941397914 radius=0.213204; visual mesh filename=package://centauro/centauro_urdf/meshes/simplified/pelvis.s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 scale=0.001 0.001 0.001
- link torso_2: mass 3.0 -> 11.492689; geometry collision cylinder length=0.128018449088 radius=0.200841; visual mesh filename=package://centauro/centauro_urdf/meshes/simplified/link1.stl scale=0.001 0.001 0.001
Joints:
- removed joint j_arm1_1
- removed joint j_arm1_2
- removed joint j_arm1_3
- removed joint j_arm1_4
- removed joint j_arm1_5
- removed joint j_arm1_6
- removed joint j_arm1_7
- removed joint j_arm2_1
- removed joint j_arm2_2
- removed joint j_arm2_3
- removed joint j_arm2_4
- removed joint j_arm2_5
- removed joint j_arm2_6
- removed joint j_arm2_7
- added joint LElbj: type revolute, parent LShy, child LElb, origin xyz=0.045 0.05515 -0.074 rpy=0.0 0.0 0.0, axis 0.0 1.0 0.0, limit lower=-2.492 upper=0.298 effort=120.0 velocity=6.283
- added joint LForearmPlate: type revolute, parent LElb, child LForearm, origin xyz=-0.015 -0.05515 -0.095 rpy=0.0 0.0 0.0, axis 0.0 0.0 1.0, limit lower=-2.55 upper=2.55 effort=35.0 velocity=6.283
- added joint LShLat: type revolute, parent LShp, child LShr, origin xyz=-0.09015 0.062 0.0 rpy=-0.1745327 0.0 0.0, axis 1.0 0.0 0.0, limit lower=0.0 upper=3.517 effort=140.0 velocity=6.283
- added joint LShSag: type revolute, parent DWYTorso, child LShp, origin xyz=0.0457475 0.169137 0.155126 rpy=0.174533 0.0 -0.5235988, axis 0.0 1.0 0.0, limit lower=-3.352 upper=1.603 effort=140.0 velocity=6.283
- added joint LShYaw: type revolute, parent LShr, child LShy, origin xyz=0.09015 0.0 -0.21815 rpy=0.0 0.0 0.0, axis 0.0 0.0 1.0, limit lower=-2.55 upper=2.55 effort=120.0 velocity=6.283
- added joint LWrj1: type revolute, parent LForearm, child LWrMot2, origin xyz=0.0 0.049 -0.156 rpy=0.0 0.0 0.0, axis 0.0 1.0 0.0, limit lower=-1.562 upper=1.478 effort=35.0 velocity=6.283
- added joint LWrj2: type revolute, parent LWrMot2, child LWrMot3, origin xyz=0.0 -0.049 -0.174 rpy=0.0 0.0 0.0, axis 0.0 0.0 1.0, limit lower=-2.55 upper=2.55 effort=20.0 velocity=6.283
- added joint RElbj: type revolute, parent RShy, child RElb, origin xyz=0.045 -0.05515 -0.074 rpy=0.0 0.0 0.0, axis 0.0 1.0 0.0, limit lower=-2.488 upper=0.292 effort=120.0 velocity=6.283
- added joint RForearmPlate: type revolute, parent RElb, child RForearm, origin xyz=-0.015 0.05515 -0.095 rpy=0.0 0.0 0.0, axis 0.0 0.0 1.0, limit lower=-2.55 upper=2.55 effort=35.0 velocity=6.283
- added joint RShLat: type revolute, parent RShp, child RShr, origin xyz=-0.09015 -0.062 0.0 rpy=0.1745327 0.0 0.0, axis 1.0 0.0 0.0, limit lower=-3.43 upper=0.0 effort=140.0 velocity=6.283
- added joint RShSag: type revolute, parent DWYTorso, child RShp, origin xyz=0.0457475 -0.169137 0.155126 rpy=-0.174533 0.0 0.5235988, axis 0.0 1.0 0.0, limit lower=-3.359 upper=1.606 effort=140.0 velocity=6.283
- added joint RShYaw: type revolute, parent RShr, child RShy, origin xyz=0.09015 0.0 -0.21815 rpy=0.0 0.0 0.0, axis 0.0 0.0 1.0, limit lower=-2.55 upper=2.55 effort=120.0 velocity=6.283
- added joint RWrj1: type revolute, parent RForearm, child RWrMot2, origin xyz=0.0 -0.049 -0.156 rpy=0.0 0.0 0.0, axis 0.0 1.0 0.0, limit lower=-1.542 upper=1.508 effort=35.0 velocity=6.283
- added joint RWrj2: type revolute, parent RWrMot2, child RWrMot3, origin xyz=0.0 0.049 -0.174 rpy=0.0 0.0 0.0, axis 0.0 0.0 1.0, limit lower=-2.55 upper=2.55 effort=20.0 velocity=6.283
- added joint ankle_pitch_1: type revolute, parent knee_1, child ankle1_1, origin xyz=0.2 0.0 -0.10015 rpy=3.14159265359 0.0 0.0, axis 0.0 0.0 1.0, limit lower=-2.4056 upper=2.3184 effort=147.0 velocity=8.1
- added joint ankle_pitch_2: type revolute, parent knee_2, child ankle1_2, origin xyz=0.2 0.0 -0.10015 rpy=3.14159265359 0.0 0.0, axis 0.0 0.0 1.0, limit lower=-2.3266 upper=2.3914 effort=147.0 velocity=8.1
- added joint ankle_pitch_3: type revolute, parent knee_3, child ankle1_3, origin xyz=0.2 0.0 -0.10015 rpy=3.14159265359 0.0 0.0, axis 0.0 0.0 1.0, limit lower=-2.4696 upper=2.4464 effort=147.0 velocity=8.1
- added joint ankle_pitch_4: type revolute, parent knee_4, child ankle1_4, origin xyz=0.2 0.0 -0.10015 rpy=3.14159265359 0.0 0.0, axis 0.0 0.0 1.0, limit lower=-2.3426 upper=2.3934 effort=147.0 velocity=8.1
- added joint ankle_yaw_1: type revolute, parent ankle1_1, child ankle2_1, origin xyz=0.0 0.0 0.0 rpy=1.57079632679 0.0 1.57079632679, axis 0.0 0.0 1.0, limit lower=-2.5626 upper=2.5384 effort=35.0 velocity=20.0
- added joint ankle_yaw_2: type revolute, parent ankle1_2, child ankle2_2, origin xyz=0.0 0.0 0.0 rpy=1.57079632679 0.0 1.57079632679, axis 0.0 0.0 1.0, limit lower=-2.5546 upper=2.5484 effort=35.0 velocity=20.0
- added joint ankle_yaw_3: type revolute, parent ankle1_3, child ankle2_3, origin xyz=0.0 0.0 0.0 rpy=1.57079632679 0.0 1.57079632679, axis 0.0 0.0 1.0, limit lower=-2.5606 upper=2.5454 effort=35.0 velocity=20.0
- added joint ankle_yaw_4: type revolute, parent ankle1_4, child ankle2_4, origin xyz=0.0 0.0 0.0 rpy=1.57079632679 0.0 1.57079632679, axis 0.0 0.0 1.0, limit lower=-2.6046 upper=2.5514 effort=35.0 velocity=20.0
- added joint hip_pitch_1: type revolute, parent hip1_1, child hip2_1, origin xyz=0.0 0.0 0.0625 rpy=1.57079632679 0.0 0.46141612323, axis 0.0 0.0 1.0, limit lower=-2.0226 upper=2.02748 effort=304.0 velocity=8.8
- added joint hip_pitch_2: type revolute, parent hip1_2, child hip2_2, origin xyz=0.0 0.0 0.0625 rpy=1.57079632679 0.0 2.68017653036, axis 0.0 0.0 1.0, limit lower=-2.0156 upper=2.0354 effort=304.0 velocity=8.8
- added joint hip_pitch_3: type revolute, parent hip1_3, child hip2_3, origin xyz=0.0 0.0 0.0625 rpy=1.57079632679 0.0 2.68017653036, axis 0.0 0.0 1.0, limit lower=-2.0126 upper=2.0384 effort=304.0 velocity=8.8
- added joint hip_pitch_4: type revolute, parent hip1_4, child hip2_4, origin xyz=0.0 0.0 0.0625 rpy=1.57079632679 0.0 0.46141612323, axis 0.0 0.0 1.0, limit lower=-2.0326 upper=2.0524 effort=304.0 velocity=8.8
- added joint hip_yaw_1: type revolute, parent pelvis, child hip1_1, origin xyz=0.25 0.125 -0.0566 rpy=3.14159265359 0.0 0.461416123228, axis 0.0 0.0 1.0, limit lower=-0.9432 upper=2.5138 effort=304.0 velocity=8.8
- added joint hip_yaw_2: type revolute, parent pelvis, child hip1_2, origin xyz=0.25 -0.125 -0.0566 rpy=3.14159265359 0.0 -0.461416123228, axis 0.0 0.0 1.0, limit lower=-2.511 upper=0.943 effort=304.0 velocity=8.8
- added joint hip_yaw_3: type revolute, parent pelvis, child hip1_3, origin xyz=-0.25 0.125 -0.0566 rpy=3.14159265359 0.0 2.68017653036, axis 0.0 0.0 1.0, limit lower=-2.51 upper=0.943 effort=304.0 velocity=8.8
- added joint hip_yaw_4: type revolute, parent pelvis, child hip1_4, origin xyz=-0.25 -0.125 -0.0566 rpy=3.14159265359 0.0 3.60300877682, axis 0.0 0.0 1.0, limit lower=-0.9412 upper=2.5138 effort=304.0 velocity=8.8
- added joint imu_joint: type fixed, parent pelvis, child imu_link, origin xyz=0.248316 0.0 0.015 rpy=0.0 0.0 0.0
- added joint j_camera_central: type fixed, parent torso_2, child camera_central, origin xyz=0.0559593 5e-12 0.390626 rpy=0.0 0.349065586018 0.0
- added joint j_camera_left: type fixed, parent torso_2, child camera_left, origin xyz=0.0191392 0.0525845 0.390626 rpy=0.0 0.349065586018 1.2217302006
- added joint j_camera_right: type fixed, parent torso_2, child camera_right, origin xyz=0.0191392 -0.0525845 0.390626 rpy=0.0 0.349065586018 -1.2217302006
- added joint j_kinect: type fixed, parent neck_2, child kinect, origin xyz=0.03 -0.0596 0.045855 rpy=0.0 0.0 0.0
- added joint j_kinect2_rgb_frame: type fixed, parent kinect, child kinect2_rgb_frame, origin xyz=0.05 -0.11 -0.035
- added joint j_kinect_optical_frame: type fixed, parent kinect2_rgb_frame, child kinect2_rgb_optical_frame, origin rpy=-1.5707963268 0.0 -1.5707963268
- added joint j_velodyne: type fixed, parent neck_3, child velodyne_mount, origin xyz=-0.138 0.0 -0.033 rpy=0.0 0.0 -3.14159265359
- added joint j_wheel_1: type continuous, parent ankle2_1, child wheel_1, origin xyz=0.0 0.00085 0.23735 rpy=1.57079632679 0.0 3.14159265359, axis 0.0 0.0 1.0, limit effort=35.0 velocity=20.0
- added joint j_wheel_2: type continuous, parent ankle2_2, child wheel_2, origin xyz=0.0 0.00085 0.23735 rpy=1.57079632679 0.0 3.14159265359, axis 0.0 0.0 1.0, limit effort=35.0 velocity=20.0
- added joint j_wheel_3: type continuous, parent ankle2_3, child wheel_3, origin xyz=0.0 0.00085 0.23735 rpy=1.57079632679 0.0 3.14159265359, axis 0.0 0.0 1.0, limit effort=35.0 velocity=20.0
- added joint j_wheel_4: type continuous, parent ankle2_4, child wheel_4, origin xyz=0.0 0.00085 0.23735 rpy=1.57079632679 0.0 3.14159265359, axis 0.0 0.0 1.0, limit effort=35.0 velocity=20.0
- added joint jf1: type fixed, parent LShp, child arm1_1, origin xyz=0.0 0.0 0.0 rpy=0.0 0.0 0.0
- added joint jf10: type fixed, parent RShr, child arm2_2, origin xyz=0.0 0.0 0.0 rpy=0.0 0.0 0.0
- added joint jf11: type fixed, parent RShy, child arm2_3, origin xyz=0.0 0.0 0.0 rpy=0.0 0.0 0.0
- added joint jf12: type fixed, parent RElb, child arm2_4, origin xyz=0.0 0.0 0.0 rpy=0.0 0.0 0.0
- added joint jf13: type fixed, parent RForearm, child arm2_5, origin xyz=0.0 0.0 0.0 rpy=0.0 0.0 0.0
- added joint jf14: type fixed, parent RWrMot2, child arm2_6, origin xyz=0.0 0.0 0.0 rpy=0.0 0.0 0.0
- added joint jf15: type fixed, parent RWrMot3, child arm2_7, origin xyz=0.0 0.0 0.0 rpy=0.0 0.0 0.0
- added joint jf16: type fixed, parent arm2_7, child arm2_8, origin xyz=0.0 0.0 0.0 rpy=0.0 0.0 0.0
- added joint jf2: type fixed, parent LShr, child arm1_2, origin xyz=0.0 0.0 0.0 rpy=0.0 0.0 0.0
- added joint jf3: type fixed, parent LShy, child arm1_3, origin xyz=0.0 0.0 0.0 rpy=0.0 0.0 0.0
- added joint jf4: type fixed, parent LElb, child arm1_4, origin xyz=0.0 0.0 0.0 rpy=0.0 0.0 0.0
- added joint jf5: type fixed, parent LForearm, child arm1_5, origin xyz=0.0 0.0 0.0 rpy=0.0 0.0 0.0
- added joint jf6: type fixed, parent LWrMot2, child arm1_6, origin xyz=0.0 0.0 0.0 rpy=0.0 0.0 0.0
- added joint jf7: type fixed, parent LWrMot3, child arm1_7, origin xyz=0.0 0.0 0.0 rpy=0.0 0.0 0.0
- added joint jf8: type fixed, parent arm1_7, child arm1_8, origin xyz=0.0 0.0 0.0 rpy=0.0 0.0 0.0
- added joint jf9: type fixed, parent RShp, child arm2_1, origin xyz=0.0 0.0 0.0 rpy=0.0 0.0 0.0
- added joint knee_pitch_1: type revolute, parent hip2_1, child knee_1, origin xyz=0.0 0.3 -0.0036 rpy=3.14159265359 0.0 1.57079632679, axis 0.0 0.0 1.0, limit lower=-2.4056 upper=2.3994 effort=304.0 velocity=8.8
- added joint knee_pitch_2: type revolute, parent hip2_2, child knee_2, origin xyz=0.0 0.3 -0.0036 rpy=3.14159265359 0.0 1.57079632679, axis 0.0 0.0 1.0, limit lower=-2.4006 upper=2.4034 effort=304.0 velocity=8.8
- added joint knee_pitch_3: type revolute, parent hip2_3, child knee_3, origin xyz=0.0 0.3 -0.0036 rpy=3.14159265359 0.0 1.57079632679, axis 0.0 0.0 1.0, limit lower=-2.4056 upper=2.4064 effort=304.0 velocity=8.8
- added joint knee_pitch_4: type revolute, parent hip2_4, child knee_4, origin xyz=0.0 0.3 -0.0036 rpy=3.14159265359 0.0 1.57079632679, axis 0.0 0.0 1.0, limit lower=-2.4176 upper=2.3884 effort=304.0 velocity=8.8
- added joint l_wrist_joint: type fixed, parent LWrMot3, child l_wrist, origin xyz=0.0 0.0 0.0 rpy=0.0 0.0 0.0
- added joint neck_pitch: type revolute, parent neck_1, child neck_2, origin xyz=0.054 0.0596 -0.0124975, axis 0.0 1.0 0.0, limit lower=-0.34906585 upper=0.78539816 effort=35.0 velocity=5.7
- added joint neck_velodyne: type continuous, parent torso_2, child neck_3, origin xyz=0.055 0.0 0.473262, axis 0.0 0.0 1.0, limit effort=35.0 velocity=5.7
- added joint neck_yaw: type revolute, parent torso_2, child neck_1, origin xyz=0.0 0.0 0.2795, axis 0.0 0.0 1.0, limit lower=-0.78539816 upper=0.78539816 effort=35.0 velocity=5.7
- added joint r_wrist_joint: type fixed, parent RWrMot3, child r_wrist, origin xyz=0.0 0.0 0.0 rpy=0.0 0.0 0.0
- added joint torso_renaming: type fixed, parent torso_2, child DWYTorso, origin xyz=0.0 0.0 -0.0385 rpy=0.0 0.0 0.0
- added joint velodyne_calib: type fixed, parent neck_3, child velodyne_calib, origin xyz=-0.175768 0.0 -0.034219 rpy=-1.57772 0.0128311 1.57073
- joint reference: origin xyz=0.0 0.0 0.85 -> xyz=0.0 0.0 0.93445; type fixed -> floating
- joint torso_yaw: limit lower=-2.618 upper=2.618 effort=350.0 velocity=6.5 -> lower=-2.618 upper=2.618 effort=147.0 velocity=5.7; origin xyz=0.3 0.0 0.0 -> xyz=0.2 0.0 0.256
