Commit message: changed names in arms according to old convension

File: centauro/centauro_urdf/urdf/centauro.urdf (robot description, URDF)
Before this commit: robot centauro, 72 links, 71 joints
Joints:
- removed joint LElbj
- removed joint LForearmPlate
- removed joint LShLat
- removed joint LShSag
- removed joint LShYaw
- removed joint LWrj1
- removed joint LWrj2
- removed joint RElbj
- removed joint RForearmPlate
- removed joint RShLat
- removed joint RShSag
- removed joint RShYaw
- removed joint RWrj1
- removed joint RWrj2
- added joint j_arm1_1: type revolute, parent DWYTorso, child LShp, origin xyz=0.0457475 0.169137 0.155126 rpy=0.174533 0 -0.5235988, axis 0 1 0, limit lower=-3.352 upper=1.603 effort=140 velocity=6.283
- added joint j_arm1_2: type revolute, parent LShp, child LShr, origin xyz=-0.09015 0.062 0 rpy=-0.1745327 0 0, axis 1 0 0, limit lower=0.0 upper=3.517 effort=140 velocity=6.283
- added joint j_arm1_3: type revolute, parent LShr, child LShy, origin xyz=0.09015 0 -0.21815 rpy=0 0 0, axis 0 0 1, limit lower=-2.55 upper=2.55 effort=120 velocity=6.283
- added joint j_arm1_4: type revolute, parent LShy, child LElb, origin xyz=0.045 0.05515 -0.074 rpy=0 0 0, axis 0 1 0, limit lower=-2.492 upper=0.298 effort=120 velocity=6.283
- added joint j_arm1_5: type revolute, parent LElb, child LForearm, origin xyz=-0.015 -0.05515 -0.095 rpy=0 0 0, axis 0 0 1, limit lower=-2.55 upper=2.55 effort=35 velocity=6.283
- added joint j_arm1_6: type revolute, parent LForearm, child LWrMot2, origin xyz=0 0.049 -0.156 rpy=0 0 0, axis 0 1 0, limit lower=-1.562 upper=1.478 effort=35 velocity=6.283
- added joint j_arm1_7: type revolute, parent LWrMot2, child LWrMot3, origin xyz=0 -0.049 -0.174 rpy=0 0 0, axis 0 0 1, limit lower=-2.55 upper=2.55 effort=20 velocity=6.283
- added joint j_arm2_1: type revolute, parent DWYTorso, child RShp, origin xyz=0.0457475 -0.169137 0.155126 rpy=-0.174533 0 0.5235988, axis 0 1 0, limit lower=-3.359 upper=1.606 effort=140 velocity=6.283
- added joint j_arm2_2: type revolute, parent RShp, child RShr, origin xyz=-0.09015 -0.062 0 rpy=0.1745327 0 0, axis 1 0 0, limit lower=-3.43 upper=0.0 effort=140 velocity=6.283
- added joint j_arm2_3: type revolute, parent RShr, child RShy, origin xyz=0.09015 0 -0.21815 rpy=0 0 0, axis 0 0 1, limit lower=-2.55 upper=2.55 effort=120 velocity=6.283
- added joint j_arm2_4: type revolute, parent RShy, child RElb, origin xyz=0.045 -0.05515 -0.074 rpy=0 0 0, axis 0 1 0, limit lower=-2.488 upper=0.292 effort=120 velocity=6.283
- added joint j_arm2_5: type revolute, parent RElb, child RForearm, origin xyz=-0.015 0.05515 -0.095 rpy=0 0 0, axis 0 0 1, limit lower=-2.55 upper=2.55 effort=35 velocity=6.283
- added joint j_arm2_6: type revolute, parent RForearm, child RWrMot2, origin xyz=0 -0.049 -0.156 rpy=0 0 0, axis 0 1 0, limit lower=-1.542 upper=1.508 effort=35 velocity=6.283
- added joint j_arm2_7: type revolute, parent RWrMot2, child RWrMot3, origin xyz=0 0.049 -0.174 rpy=0 0 0, axis 0 0 1, limit lower=-2.55 upper=2.55 effort=20 velocity=6.283

File: centauro/centauro_urdf/urdf/centauro.urdf.xacro (robot description, xacro)
@@ -88,6 +88,8 @@
 </xacro:if>
 -->
-<xacro:property name="COGIMON_LEFT_ARM" value="true" />
-<xacro:property name="COGIMON_RIGHT_ARM" value="true" />
+<xacro:include filename="$(find cogimon_urdf)/urdf/conversions.urdf.xacro" />
+<xacro:include filename="$(find cogimon_urdf)/urdf/parts/arms_macro.urdf.xacro" />
+<xacro:right_arm joint1_name="j_arm2_1" joint2_name="j_arm2_2" joint3_name="j_arm2_3" joint4_name="j_arm2_4" joint5_name="j_arm2_5" joint6_name="j_arm2_6" joint7_name="j_arm2_7" />
+<xacro:left_arm joint1_name="j_arm1_1" joint2_name="j_arm1_2" joint3_name="j_arm1_3" joint4_name="j_arm1_4" joint5_name="j_arm1_5" joint6_name="j_arm1_6" joint7_name="j_arm1_7" />
 <link name="DWYTorso"/>
 <joint name="torso_renaming" type="fixed">
@@ -96,6 +98,4 @@
        <origin xyz="0 0 -0.0385" rpy="0 0 0" />
 </joint>
-<xacro:include filename="$(find cogimon_urdf)/urdf/conversions.urdf.xacro" />
-<xacro:include filename="$(find cogimon_urdf)/urdf/parts/arms.urdf.xacro" />
 <xacro:include filename="$(find centauro)/centauro_urdf/urdf/centauro_arm_frames.urdf.xacro" />
 <!-- /arms -->

File: centauro/centauro_urdf/urdf/centauro_capsules.urdf (robot description, URDF)
Before this commit: robot centauro, 72 links, 71 joints
Joints:
- removed joint LElbj
- removed joint LForearmPlate
- removed joint LShLat
- removed joint LShSag
- removed joint LShYaw
- removed joint LWrj1
- removed joint LWrj2
- removed joint RElbj
- removed joint RForearmPlate
- removed joint RShLat
- removed joint RShSag
- removed joint RShYaw
- removed joint RWrj1
- removed joint RWrj2
- added joint j_arm1_1: type revolute, parent DWYTorso, child LShp, origin xyz=0.0457475 0.169137 0.155126 rpy=0.174533 0.0 -0.5235988, axis 0.0 1.0 0.0, limit lower=-3.352 upper=1.603 effort=140.0 velocity=6.283
- added joint j_arm1_2: type revolute, parent LShp, child LShr, origin xyz=-0.09015 0.062 0.0 rpy=-0.1745327 0.0 0.0, axis 1.0 0.0 0.0, limit lower=0.0 upper=3.517 effort=140.0 velocity=6.283
- added joint j_arm1_3: type revolute, parent LShr, child LShy, origin xyz=0.09015 0.0 -0.21815 rpy=0.0 0.0 0.0, axis 0.0 0.0 1.0, limit lower=-2.55 upper=2.55 effort=120.0 velocity=6.283
- added joint j_arm1_4: type revolute, parent LShy, child LElb, origin xyz=0.045 0.05515 -0.074 rpy=0.0 0.0 0.0, axis 0.0 1.0 0.0, limit lower=-2.492 upper=0.298 effort=120.0 velocity=6.283
- added joint j_arm1_5: type revolute, parent LElb, child LForearm, origin xyz=-0.015 -0.05515 -0.095 rpy=0.0 0.0 0.0, axis 0.0 0.0 1.0, limit lower=-2.55 upper=2.55 effort=35.0 velocity=6.283
- added joint j_arm1_6: type revolute, parent LForearm, child LWrMot2, origin xyz=0.0 0.049 -0.156 rpy=0.0 0.0 0.0, axis 0.0 1.0 0.0, limit lower=-1.562 upper=1.478 effort=35.0 velocity=6.283
- added joint j_arm1_7: type revolute, parent LWrMot2, child LWrMot3, origin xyz=0.0 -0.049 -0.174 rpy=0.0 0.0 0.0, axis 0.0 0.0 1.0, limit lower=-2.55 upper=2.55 effort=20.0 velocity=6.283
- added joint j_arm2_1: type revolute, parent DWYTorso, child RShp, origin xyz=0.0457475 -0.169137 0.155126 rpy=-0.174533 0.0 0.5235988, axis 0.0 1.0 0.0, limit lower=-3.359 upper=1.606 effort=140.0 velocity=6.283
- added joint j_arm2_2: type revolute, parent RShp, child RShr, origin xyz=-0.09015 -0.062 0.0 rpy=0.1745327 0.0 0.0, axis 1.0 0.0 0.0, limit lower=-3.43 upper=0.0 effort=140.0 velocity=6.283
- added joint j_arm2_3: type revolute, parent RShr, child RShy, origin xyz=0.09015 0.0 -0.21815 rpy=0.0 0.0 0.0, axis 0.0 0.0 1.0, limit lower=-2.55 upper=2.55 effort=120.0 velocity=6.283
- added joint j_arm2_4: type revolute, parent RShy, child RElb, origin xyz=0.045 -0.05515 -0.074 rpy=0.0 0.0 0.0, axis 0.0 1.0 0.0, limit lower=-2.488 upper=0.292 effort=120.0 velocity=6.283
- added joint j_arm2_5: type revolute, parent RElb, child RForearm, origin xyz=-0.015 0.05515 -0.095 rpy=0.0 0.0 0.0, axis 0.0 0.0 1.0, limit lower=-2.55 upper=2.55 effort=35.0 velocity=6.283
- added joint j_arm2_6: type revolute, parent RForearm, child RWrMot2, origin xyz=0.0 -0.049 -0.156 rpy=0.0 0.0 0.0, axis 0.0 1.0 0.0, limit lower=-1.542 upper=1.508 effort=35.0 velocity=6.283
- added joint j_arm2_7: type revolute, parent RWrMot2, child RWrMot3, origin xyz=0.0 0.049 -0.174 rpy=0.0 0.0 0.0, axis 0.0 0.0 1.0, limit lower=-2.55 upper=2.55 effort=20.0 velocity=6.283

Commit message: Updated armx_8 links according to old ones

File: centauro/centauro_urdf/urdf/centauro.urdf (robot description, URDF)
Before this commit: robot centauro, 72 links, 71 joints
Joints:
- joint jf16: origin xyz=0 0 0 rpy=0 0 0 -> xyz=0 0 0 rpy=0 3.14159265359 -1.57079632679
- joint jf8: origin xyz=0 0 0 rpy=0 0 0 -> xyz=0 0 0 rpy=0 3.14159265359 -1.57079632679

File: centauro/centauro_urdf/urdf/centauro_arm_frames.urdf.xacro (robot description, xacro)
@@ -55,5 +55,5 @@
        <parent link="arm1_7"/>
        <child link="arm1_8"/>
-       <origin xyz="0 0 0" rpy="0 0 0" />
+       <origin xyz="0 0 0" rpy="0 ${PI} ${-PI_2}" />
 </joint>
 <joint name="jf9" type="fixed">
@@ -95,5 +95,5 @@
        <parent link="arm2_7"/>
        <child link="arm2_8"/>
-       <origin xyz="0 0 0" rpy="0 0 0" />
+       <origin xyz="0 0 0" rpy="0 ${PI} ${-PI_2}" />
 </joint>
 </robot>

File: centauro/centauro_urdf/urdf/centauro_capsules.urdf (robot description, URDF)
Before this commit: robot centauro, 72 links, 71 joints
Joints:
- joint jf16: origin xyz=0.0 0.0 0.0 rpy=0.0 0.0 0.0 -> xyz=0.0 0.0 0.0 rpy=0.0 3.14159265359 -1.57079632679
- joint jf8: origin xyz=0.0 0.0 0.0 rpy=0.0 0.0 0.0 -> xyz=0.0 0.0 0.0 rpy=0.0 3.14159265359 -1.57079632679

Commit message: updated linear part

File: centauro/centauro_urdf/urdf/centauro.urdf (robot description, URDF)
Before this commit: robot centauro, 72 links, 71 joints
Joints:
- joint jf16: origin xyz=0 0 0 rpy=0 3.14159265359 -1.57079632679 -> xyz=0 0 -0.0405 rpy=0 3.14159265359 -1.57079632679
- joint jf8: origin xyz=0 0 0 rpy=0 3.14159265359 -1.57079632679 -> xyz=0 0 -0.0405 rpy=0 3.14159265359 -1.57079632679

File: centauro/centauro_urdf/urdf/centauro_arm_frames.urdf.xacro (robot description, xacro)
@@ -55,5 +55,5 @@
        <parent link="arm1_7"/>
        <child link="arm1_8"/>
-       <origin xyz="0 0 0" rpy="0 ${PI} ${-PI_2}" />
+       <origin xyz="0 0 -0.0405" rpy="0 ${PI} ${-PI_2}" />
 </joint>
 <joint name="jf9" type="fixed">
@@ -95,5 +95,5 @@
        <parent link="arm2_7"/>
        <child link="arm2_8"/>
-       <origin xyz="0 0 0" rpy="0 ${PI} ${-PI_2}" />
+       <origin xyz="0 0 -0.0405" rpy="0 ${PI} ${-PI_2}" />
 </joint>
 </robot>

File: centauro/centauro_urdf/urdf/centauro_capsules.urdf (robot description, URDF)
Before this commit: robot centauro, 72 links, 71 joints
Joints:
- joint jf16: origin xyz=0.0 0.0 0.0 rpy=0.0 3.14159265359 -1.57079632679 -> xyz=0.0 0.0 -0.0405 rpy=0.0 3.14159265359 -1.57079632679
- joint jf8: origin xyz=0.0 0.0 0.0 rpy=0.0 3.14159265359 -1.57079632679 -> xyz=0.0 0.0 -0.0405 rpy=0.0 3.14159265359 -1.57079632679

Commit message: faster verion of simulation with simpler wheels and control from Enrico plus realsense sensors

File: centauro/centauro_urdf/urdf/centauro.urdf (robot description, URDF)
Before this commit: robot centauro, 91 links, 90 joints
Joints:
- removed joint j_ft_1
- removed joint j_ft_2
- added joint j_ft_arm1: type revolute, parent arm1_7, child ft_arm1, origin xyz=0.0 0.0 -0.0405 rpy=0.0 3.14159265359 -3.14159265359, axis 0 0 1, limit lower=0.0 upper=0.0 effort=0 velocity=0
- added joint j_ft_arm2: type revolute, parent arm2_7, child ft_arm2, origin xyz=0.0 0.0 -0.0405 rpy=0.0 3.14159265359 -3.14159265359, axis 0 0 1, limit lower=0.0 upper=0.0 effort=0 velocity=0

File: centauro/centauro_urdf/urdf/centauro.urdf.xacro (robot description, xacro)
@@ -21,4 +21,7 @@
 <xacro:if value="${arms}">
   <xacro:include filename="$(find centauro)/centauro_urdf/urdf/centauro_arm.urdf.xacro"/>
+</xacro:if>
+<xacro:if value="${realsense}">
+  <xacro:include filename="$(find realsense_gazebo_plugin)/urdf/d435.urdf.xacro"/>
 </xacro:if>
 <!-- /other files -->

File: centauro/centauro_urdf/urdf/centauro_arm.urdf.xacro (robot description, xacro)
@@ -190,10 +190,10 @@
 <!-- end-effector -->
 <!-- wrist pitch-->
-   <joint name="j_ft_${arm_num}" type="${ft_sensors}">
+   <joint name="j_ft_arm${arm_num}" type="${ft_sensors}">
       <parent link="arm${arm_num}_7"/>
       <child link="ft_arm${arm_num}"/>
       <origin xyz="${Ft_arm_Ox} ${Ft_arm_Oy} ${Ft_arm_Oz}" rpy="${Ft_arm_roll} ${Ft_arm_pitch} ${Ft_arm_yaw}" />
       <axis xyz="0 0 1"/>
-      <limit lower="0.0" upper="0.0" effort="0" velocity="0"/>
+      <limit lower="0.0" upper="5.0" effort="5" velocity="5"/>
    </joint>
 <!-- wrist pitch-->
@@ -213,5 +213,5 @@
 <xacro:if value="${ft_sensors == 'revolute'}" >
    <xacro:if value="${arm_actuators}">
-      <xacro:position_actuator joint="j_ft_${arm_num}" />
+      <xacro:position_actuator joint="j_ft_arm${arm_num}" />
    </xacro:if>
 </xacro:if>

File: centauro/centauro_urdf/urdf/config.xacro (robot description, xacro)
@@ -32,4 +32,5 @@
 <xacro:property name="KINECT" value="$(arg KINECT)"/>
 <xacro:property name="VELODYNE" value="$(arg VELODYNE)"/>
+<xacro:property name="REALSENSE" value="$(arg REALSENSE)"/>
 <xacro:property name="MASS" value="$(arg MASS)"/>
 <!-- dependend arguments -->
@@ -64,4 +65,5 @@
 <xacro:property name="velodyne" value="${'true' if (False not in [VELODYNE, head] and 'false' not in [VELODYNE, head]) else 'false'}"/>
 <!--xacro:property name="velodyne" value="false"/-->
+<xacro:property name="realsense" value="${'true' if (False not in [REALSENSE, head] and 'false' not in [REALSENSE, head]) else 'false'}"/>
 <!-- LOAD PARAMETERS -->
 <xacro:property name="package" value="$(find centauro)"/>

File: centauro/centauro_urdf/urdf/models/lower_body/convex_hull.xacro (robot description, xacro)
@@ -40,5 +40,6 @@
    <origin xyz="0.0 0.0 0.0"  rpy="0.0 0.0 0.0"/>
    <geometry>
-      <mesh filename="package://centauro/centauro_urdf/meshes/convex_hull/wheel.stl" scale="0.001 ${0.001} 0.001" />
+      <!--<mesh filename="package://centauro/centauro_urdf/meshes/convex_hull/wheel.stl" scale="0.001 ${0.001} 0.001" />-->
+      <cylinder length="0.06" radius="${0.14/2.}"/>
    </geometry>
 </xacro:macro>

File: centauro/centauro_urdf/urdf/models/lower_body/mesh.xacro (robot description, xacro)
@@ -40,5 +40,6 @@
    <origin xyz="0.0 0.0 0.0"  rpy="0.0 0.0 0.0"/>
    <geometry>
-      <mesh filename="package://centauro/centauro_urdf/meshes/wheel.stl" scale="0.001 ${0.001} 0.001" />
+      <!--<mesh filename="package://centauro/centauro_urdf/meshes/wheel.stl" scale="0.001 ${0.001} 0.001" />-->
+      <cylinder length="0.06" radius="${0.14/2.}"/>
    </geometry>
 </xacro:macro>

File: centauro/centauro_urdf/urdf/models/lower_body/primitive.xacro (robot description, xacro)
@@ -40,5 +40,5 @@
 		<origin xyz="0 0 0" />
 		<geometry>
-			<sphere radius="0.078"/>
+      <cylinder length="0.06" radius="${0.14/2.0}"/>
 		</geometry>
 </xacro:macro>

File: centauro/centauro_urdf/urdf/models/lower_body/simplified.xacro (robot description, xacro)
@@ -40,5 +40,6 @@
    <origin xyz="0.0 0.0 0.0"  rpy="0.0 0.0 0.0"/>
    <geometry>
-      <mesh filename="package://centauro/centauro_urdf/meshes/simplified/wheel.stl" scale="0.001 ${0.001} 0.001" />
+      <!--<mesh filename="package://centauro/centauro_urdf/meshes/simplified/wheel.stl" scale="0.001 ${0.001} 0.001" />-->
+      <cylinder length="0.06" radius="${0.14/2.0}"/>
    </geometry>
 </xacro:macro>

File: centauro_gazebo/sensors/config.xacro (robot description, xacro)
@@ -30,3 +30,6 @@
         <xacro:load_model middleware="${middleware}" sensor="velodyne" arm_sensors="false" leg_sensors="false" head_sensors="${head}"/>
 </xacro:if>
+<xacro:if value="${realsense}">
+        <xacro:load_model middleware="${middleware}" sensor="realsense" arm_sensors="false" leg_sensors="false" head_sensors="${head}"/>
+</xacro:if>
 </robot>

File: centauro_gazebo/sensors/ros_control/ft_sensor/load/arms.xacro (robot description, xacro)
@@ -2,7 +2,7 @@
 <robot  xmlns:xacro="http://www.ros.org/wiki/xacro">
 <xacro:include filename="$(find centauro)/centauro_urdf/urdf/config.xacro"/>
-  <xacro:force-torque_sensor joint="j_ft_1" robot="centauro"/>
+  <xacro:force-torque_sensor joint="j_ft_arm1" robot="centauro"/>
   <xacro:if value="${arms}">
-    <xacro:force-torque_sensor joint="j_ft_2" robot="centauro"/>
+    <xacro:force-torque_sensor joint="j_ft_arm2" robot="centauro"/>
   </xacro:if>
 </robot>

File: centauro_gazebo/sensors/xbotcore/ft_sensor/load/arms.xacro (robot description, xacro)
@@ -2,7 +2,7 @@
 <robot  xmlns:xacro="http://www.ros.org/wiki/xacro">
 <xacro:include filename="$(find centauro)/centauro_urdf/urdf/config.xacro"/>
-  <xacro:force-torque_sensor joint="j_ft_1" robot="centauro" ft_name="left_arm_ft" pose="0 0 0 0 0 0"/>
+  <xacro:force-torque_sensor joint="j_ft_arm1" robot="centauro" ft_name="left_arm_ft" pose="0 0 0 0 0 0"/>
   <xacro:if value="${arms}">
-    <xacro:force-torque_sensor joint="j_ft_2" robot="centauro" ft_name="right_arm_ft" pose="0 0 0 0 0 0"/>
+    <xacro:force-torque_sensor joint="j_ft_arm2" robot="centauro" ft_name="right_arm_ft" pose="0 0 0 0 0 0"/>
   </xacro:if>
 </robot>
