Commit message: continuous joints changed in fixed

File: centauro/centauro_urdf/urdf/centauro_control.urdf (robot description, URDF)
Before this commit: robot centauro, 59 links, 58 joints
Joints:
- joint j_wheel_1: type continuous -> fixed
- joint j_wheel_2: type continuous -> fixed
- joint j_wheel_3: type continuous -> fixed
- joint j_wheel_4: type continuous -> fixed
- joint neck_velodyne: type continuous -> fixed
