Commit message: Update contact sensors and lower body primitives model

File: centauro/centauro_urdf/urdf/models/lower_body/primitives.xacro (robot description, xacro)
@@ -2,25 +2,43 @@
 <robot name="centauro" xmlns:xacro="http://www.ros.org/wiki/xacro">
 <xacro:macro name="pelvis" >
-   <origin xyz="0 0 0"  rpy="0.0 0.0 0.0"/>
+   <origin xyz="0 0.02 0.18"  rpy="0.0 0.0 0.0"/>
    <geometry>
-      <box size="0.70 0.40 0.20"/>
+      <box size="0.52 0.38 0.30"/>
    </geometry>
 </xacro:macro>
 <xacro:macro name="leg1">
-		<origin xyz="0 0 -0.1"/>
+		<origin xyz="0 0 0.05" />
 		<geometry>
-			<box size="${link_visual} ${link_visual} 0.2"/> <!-- OK: from hip-yaw to pelvis (0.1) + from plevis to hip-pitch (0.1)-->
+			<box size="0.1 0.1 0.1"/>
 		</geometry>
 </xacro:macro>
 <xacro:macro name="leg2">
-		<origin xyz="0 0 -${0.35/2}"/>
+		<origin xyz="0.0 0.15 0.1" />
 		<geometry>
-			<box size="${link_visual} ${link_visual} 0.35"/> <!-- OK -->
+			<box size="0.1 0.40 0.1"/>
 		</geometry>
 </xacro:macro>
 <xacro:macro name="leg3">
-		<origin xyz="0 0 -${0.3-link_width/2}" />
+		<origin xyz="0.10 0 0.0" />
 		<geometry>
-			<sphere radius="${link_width/2}"/>
+			<box size="0.30 0.1 0.1"/>
+		</geometry>
+</xacro:macro>
+<xacro:macro name="ankle1">
+		<origin xyz="0.05 0 0" />
+		<geometry>
+			<box size="0.1 0.1 0.1"/>
+		</geometry>
+</xacro:macro>
+<xacro:macro name="ankle2">
+		<origin xyz="0.0 0.0 0.2" />
+		<geometry>
+			<box size="0.1 0.1 0.1"/>
+		</geometry>
+</xacro:macro>
+<xacro:macro name="wheel">
+		<origin xyz="0 0 0" />
+		<geometry>
+			<cylinder radius="0.075" length="0.1"/>
 		</geometry>
 </xacro:macro>
