Commit message: change the default setting for the collision model to primitives

File: centauro/centauro_urdf/urdf/models/lower_body/primitive.xacro (robot description, xacro)
@@ -2,7 +2,7 @@
 <robot name="centauro" xmlns:xacro="http://www.ros.org/wiki/xacro">
 <xacro:macro name="pelvis" >
-   <origin xyz="0 0.02 0.18"  rpy="0.0 0.0 0.0"/>
+   <origin xyz="0 0.02 0.07"  rpy="0.0 0.0 0.0"/>
    <geometry>
-      <box size="0.52 0.38 0.30"/>
+      <box size="0.52 0.38 0.25"/>
    </geometry>
 </xacro:macro>
@@ -10,5 +10,5 @@
 		<origin xyz="0 0 0.05" />
 		<geometry>
-			<box size="0.1 0.1 0.1"/>
+			<box size="0.05 0.05 0.05"/>
 		</geometry>
 </xacro:macro>
@@ -26,13 +26,13 @@
 </xacro:macro>
 <xacro:macro name="ankle1">
-		<origin xyz="0.05 0 0" />
+		<origin xyz="0.0 0 0.0" />
 		<geometry>
-			<box size="0.1 0.1 0.1"/>
+			<box size="0.09 0.09 0.09"/>
 		</geometry>
 </xacro:macro>
 <xacro:macro name="ankle2">
-		<origin xyz="0.0 0.0 0.2" />
+		<origin xyz="0.0 0.0 0.1" />
 		<geometry>
-			<box size="0.1 0.1 0.1"/>
+			<box size="0.09 0.09 0.09"/>
 		</geometry>
 </xacro:macro>
@@ -40,5 +40,6 @@
 		<origin xyz="0 0 0" />
 		<geometry>
-			<cylinder radius="0.075" length="0.1"/>
+<!--			<cylinder radius="0.075" length="0.1"/> -->
+			<sphere radius="0.078"/>
 		</geometry>
 </xacro:macro>

File: centauro/centauro_urdf/urdf/models/upper_body/head/primitive.xacro (robot description, xacro)
@@ -3,19 +3,19 @@
 <xacro:macro name="neck_yaw">
    <origin xyz="0.0 0 0.0"  rpy="0.0 0.0 0.0"/>
-   <geometry>
+<!--   <geometry>
       <box size="0.05 0.05 0.05"/>
-   </geometry>
+   </geometry> -->
 </xacro:macro>
 <xacro:macro name="neck_pitch">
    <origin xyz="0.0 0 0.0"  rpy="0.0 0.0 0.0"/>
-   <geometry>
-       <box size="0.05 0.05 0.05"/>
-   </geometry>
+<!--   <geometry>
+      <box size="0.05 0.05 0.05"/>
+   </geometry> -->
 </xacro:macro>
 <xacro:macro name="velodyne">
    <origin xyz="0.0 0 0.0"  rpy="0.0 0.0 0.0"/>
-   <geometry>
-        <box size="0.05 0.05 0.05"/>
-   </geometry>
+<!--   <geometry>
+      <box size="0.05 0.05 0.05"/>
+   </geometry> -->
 </xacro:macro>
 </robot>

File: centauro/centauro_urdf/urdf/models/upper_body/primitive.xacro (robot description, xacro)
@@ -8,5 +8,5 @@
 </xacro:macro>
 <xacro:macro name="arm1">
-   <origin xyz="0.0 0.05 0.0"  rpy="0.0 0.0 0.0"/>
+   <origin xyz="0.0 ${rot*0.05} 0.0"  rpy="0.0 0.0 0.0"/>
    <geometry>
       <box size="${link_visual} 0.1 ${link_visual}"/>
@@ -22,5 +22,5 @@
    <origin xyz="0.0 0.0 -0.075"  rpy="0.0 0.0 0.0"/>
    <geometry>
-      <box size="${link_visual} ${link_visual} 0.15"/>
+      <box size="${link_visual} ${link_visual} 0.10"/>
    </geometry>
 </xacro:macro>
@@ -28,5 +28,5 @@
    <origin xyz="0 0.0 -0.065"  rpy="0.0 0.0 0.0"/>
    <geometry>
-      <box size="${link_visual} ${link_visual} 0.13"/>
+      <box size="${link_visual} ${link_visual} 0.10"/>
    </geometry>
 </xacro:macro>
@@ -44,5 +44,5 @@
 </xacro:macro>
 <xacro:macro name="arm7">
-   <origin xyz="0.0 0.0 -0.020"  rpy="0.0 0.0 0.0"/>
+   <origin xyz="0.0 0.0 0.0"  rpy="0.0 0.0 0.0"/>
    <geometry>
       <box size="${link_visual} ${link_visual} ${link_visual}"/>

Commit message: set-up previous wheel radius

File: centauro/centauro_urdf/urdf/models/lower_body/primitive.xacro (robot description, xacro)
@@ -41,5 +41,5 @@
 		<geometry>
 <!--			<cylinder radius="0.075" length="0.1"/> -->
-			<sphere radius="0.078"/>
+			<sphere radius="0.075"/>
 		</geometry>
 </xacro:macro>

Commit message: lower body merge conflict

File: centauro/centauro_urdf/urdf/models/lower_body/primitive.xacro (robot description, xacro)
@@ -2,7 +2,7 @@
 <robot name="centauro" xmlns:xacro="http://www.ros.org/wiki/xacro">
 <xacro:macro name="pelvis" >
-   <origin xyz="0 0.02 0.18"  rpy="0.0 0.0 0.0"/>
+   <origin xyz="0 0.02 0.07"  rpy="0.0 0.0 0.0"/>
    <geometry>
-      <box size="0.52 0.38 0.30"/>
+      <box size="0.52 0.38 0.25"/>
    </geometry>
 </xacro:macro>
@@ -10,5 +10,5 @@
 		<origin xyz="0 0 0.05" />
 		<geometry>
-			<box size="0.1 0.1 0.1"/>
+			<box size="0.05 0.05 0.05"/>
 		</geometry>
 </xacro:macro>
@@ -26,13 +26,13 @@
 </xacro:macro>
 <xacro:macro name="ankle1">
-		<origin xyz="0.05 0 0" />
+		<origin xyz="0.0 0 0.0" />
 		<geometry>
-			<box size="0.1 0.1 0.1"/>
+			<box size="0.09 0.09 0.09"/>
 		</geometry>
 </xacro:macro>
 <xacro:macro name="ankle2">
-		<origin xyz="0.0 0.0 0.2" />
+		<origin xyz="0.0 0.0 0.1" />
 		<geometry>
-			<box size="0.1 0.1 0.1"/>
+			<box size="0.09 0.09 0.09"/>
 		</geometry>
 </xacro:macro>
@@ -40,6 +40,6 @@
 		<origin xyz="0 0 0" />
 		<geometry>
-<!--			<cylinder radius="0.078" length="0.1"/> -->
-                        <sphere radius="0.078"/>
+<!--			<cylinder radius="0.075" length="0.1"/> -->
+			<sphere radius="0.075"/>
 		</geometry>
 </xacro:macro>
