Commit message: Updated lower-body inertia parameters

File: centauro/centauro_urdf/inertia_parameters/primitives.xacro (robot description, xacro)
@@ -11,94 +11,94 @@
 <xacro:property name="wheel_weight" value=" 2.000000 "/>
 <!-- Center of Mass -->
-<xacro:property name="Pelvis_x" value=" -0.0135413420 "/>
-<xacro:property name="Pelvis_y" value=" -0.0029098264 "/>
-<xacro:property name="Pelvis_z" value=" 0.1806072100 "/>
-<!-- Inertia -->
-<xacro:property name="Pelvis_xx" value=" 0.2002111900 "/>
-<xacro:property name="Pelvis_yy" value=" 0.5113621400 "/>
-<xacro:property name="Pelvis_zz" value=" 0.5440141100 "/>
-<xacro:property name="Pelvis_xy" value=" -0.0038421093 "/>
-<xacro:property name="Pelvis_xz" value=" -0.0332988490 "/>
-<xacro:property name="Pelvis_yz" value=" 0.0044698470 "/>
-<!-- Mass -->
-<xacro:property name="Pelvis_mass" value=" 24.1909450000 "/>
-<!-- Center of Mass -->
-<xacro:property name="Leg_1_x" value=" 0.0102141990 "/>
-<xacro:property name="Leg_1_y" value=" 0.0183483590 "/>
-<xacro:property name="Leg_1_z" value=" 0.0380909870 "/>
-<!-- Inertia -->
-<xacro:property name="Leg_1_xx" value=" 0.0047439572 "/>
-<xacro:property name="Leg_1_yy" value=" 0.0040551878 "/>
-<xacro:property name="Leg_1_zz" value=" 0.0034146219 "/>
-<xacro:property name="Leg_1_xy" value=" -0.0005747047 "/>
-<xacro:property name="Leg_1_xz" value=" -0.0003784138 "/>
-<xacro:property name="Leg_1_yz" value=" -0.0007407508 "/>
-<!-- Mass -->
-<xacro:property name="Leg_1_mass" value=" 1.9194403000 "/>
-<!-- Center of Mass -->
-<xacro:property name="Leg_2_x" value=" 0.0000257966 "/>
-<xacro:property name="Leg_2_y" value=" 0.1810266000 "/>
-<xacro:property name="Leg_2_z" value=" 0.0856697560 "/>
-<!-- Inertia -->
-<xacro:property name="Leg_2_xx" value=" 0.0485186900 "/>
-<xacro:property name="Leg_2_yy" value=" 0.0042420550 "/>
-<xacro:property name="Leg_2_zz" value=" 0.0482558300 "/>
-<xacro:property name="Leg_2_xy" value=" -0.0000411894 "/>
-<xacro:property name="Leg_2_xz" value=" -0.0000168778 "/>
-<xacro:property name="Leg_2_yz" value=" 0.0032243188 "/>
-<!-- Mass -->
-<xacro:property name="Leg_2_mass" value=" 2.7264471000 "/>
-<!-- Center of Mass -->
-<xacro:property name="Leg_3_x" value="0.1088166700 "/>
-<xacro:property name="Leg_3_y" value="0.0001089081 "/>
-<xacro:property name="Leg_3_z" value="-0.0226389960 "/>
-<!-- Inertia -->
-<xacro:property name="Leg_3_xx" value=" 0.0030534242 "/>
-<xacro:property name="Leg_3_yy" value=" 0.0196033210 "/>
-<xacro:property name="Leg_3_zz" value=" 0.0198498170 "/>
-<xacro:property name="Leg_3_xy" value=" -0.0000422079 "/>
-<xacro:property name="Leg_3_xz" value=" 0.0013679297 "/>
-<xacro:property name="Leg_3_yz" value=" 0.0000069941 "/>
-<!-- Mass -->
-<xacro:property name="Leg_3_mass" value="1.9356754000 "/>
-<!-- Center of Mass -->
-<xacro:property name="Ankle_1_x" value=" 0.0321373180 "/>
-<xacro:property name="Ankle_1_y" value=" 0.0000973572 "/>
-<xacro:property name="Ankle_1_z" value=" -0.0044222206 "/>
-<!-- Inertia -->
-<xacro:property name="Ankle_1_xx" value=" 0.0015610452 "/>
-<xacro:property name="Ankle_1_yy" value=" 0.0037423211 "/>
-<xacro:property name="Ankle_1_zz" value=" 0.0038312442 "/>
-<xacro:property name="Ankle_1_xy" value=" 0.0000330597 "/>
-<xacro:property name="Ankle_1_xz" value=" -0.0001314174 "/>
-<xacro:property name="Ankle_1_yz" value=" -0.0000212589 "/>
-<!-- Mass -->
-<xacro:property name="Ankle_1_mass" value="1.2380744000 "/>
-<!-- Center of Mass -->
-<xacro:property name="Ankle_2_x" value=" 0.0004435803 "/>
-<xacro:property name="Ankle_2_y" value=" 0.0004389911 "/>
-<xacro:property name="Ankle_2_z" value=" 0.1939209200 "/>
-<!-- Inertia -->
-<xacro:property name="Ankle_2_xx" value=" 0.0049019475 "/>
-<xacro:property name="Ankle_2_yy" value=" 0.0038724162 "/>
-<xacro:property name="Ankle_2_zz" value=" 0.0021783198 "/>
-<xacro:property name="Ankle_2_xy" value=" 0.0000043032 "/>
-<xacro:property name="Ankle_2_xz" value=" 0.0000346491 "/>
-<xacro:property name="Ankle_2_yz" value=" 0.0000170990 "/>
-<!-- Mass -->
-<xacro:property name="Ankle_2_mass" value=" 1.1565926000 "/>
-<!-- Center of Mass -->
-<xacro:property name="Wheel_x" value=" 0.0000000000 "/>
+<xacro:property name="Pelvis_x" value=" 0.0 "/>
+<xacro:property name="Pelvis_y" value=" 0.02 "/>
+<xacro:property name="Pelvis_z" value=" 0.18 "/>
+<!-- Inertia -->
+<xacro:property name="Pelvis_xx" value=" 0.488 "/>
+<xacro:property name="Pelvis_yy" value=" 0.751 "/>
+<xacro:property name="Pelvis_zz" value=" 0.864 "/>
+<xacro:property name="Pelvis_xy" value=" 0.000000 "/>
+<xacro:property name="Pelvis_xz" value=" 0.000000 "/>
+<xacro:property name="Pelvis_yz" value=" 0.000000 "/>
+<!-- Mass -->
+<xacro:property name="Pelvis_mass" value=" 25.000000 "/>
+<!-- Center of Mass -->
+<xacro:property name="Leg_1_x" value=" 0.000000 "/>
+<xacro:property name="Leg_1_y" value=" 0.000000 "/>
+<xacro:property name="Leg_1_z" value=" 0.05 "/>
+<!-- Inertia -->
+<xacro:property name="Leg_1_xx" value=" 0.0033 "/>
+<xacro:property name="Leg_1_yy" value=" 0.0033 "/>
+<xacro:property name="Leg_1_zz" value=" 0.0033 "/>
+<xacro:property name="Leg_1_xy" value=" 0.000000 "/>
+<xacro:property name="Leg_1_xz" value=" 0.000000 "/>
+<xacro:property name="Leg_1_yz" value=" -0.000000 "/>
+<!-- Mass -->
+<xacro:property name="Leg_1_mass" value=" 2.000000 "/>
+<!-- Center of Mass -->
+<xacro:property name="Leg_2_x" value=" 0.000000 "/>
+<xacro:property name="Leg_2_y" value=" 0.15 "/>
+<xacro:property name="Leg_2_z" value=" 0.1 "/>
+<!-- Inertia -->
+<xacro:property name="Leg_2_xx" value=" 0.064 "/>
+<xacro:property name="Leg_2_yy" value=" 0.0075 "/>
+<xacro:property name="Leg_2_zz" value=" 0.064 "/>
+<xacro:property name="Leg_2_xy" value=" 0.000000 "/>
+<xacro:property name="Leg_2_xz" value=" 0.000000 "/>
+<xacro:property name="Leg_2_yz" value=" -0.000000 "/>
+<!-- Mass -->
+<xacro:property name="Leg_2_mass" value=" 4.500000 "/>
+<!-- Center of Mass -->
+<xacro:property name="Leg_3_x" value=" 0.1 "/>
+<xacro:property name="Leg_3_y" value=" 0.000000 "/>
+<xacro:property name="Leg_3_z" value=" 0.0000 "/>
+<!-- Inertia -->
+<xacro:property name="Leg_3_xx" value=" 0.0058 "/>
+<xacro:property name="Leg_3_yy" value=" 0.0292 "/>
+<xacro:property name="Leg_3_zz" value=" 0.0292 "/>
+<xacro:property name="Leg_3_xy" value=" 0.000000 "/>
+<xacro:property name="Leg_3_xz" value=" 0.000000 "/>
+<xacro:property name="Leg_3_yz" value=" 0.000000 "/>
+<!-- Mass -->
+<xacro:property name="Leg_3_mass" value=" 3.500000 "/>
+<!-- Center of Mass -->
+<xacro:property name="Ankle_1_x" value=" 0.05 "/>
+<xacro:property name="Ankle_1_y" value=" 0.000000 "/>
+<xacro:property name="Ankle_1_z" value=" 0.0000 "/>
+<!-- Inertia -->
+<xacro:property name="Ankle_1_xx" value=" 0.0033 "/>
+<xacro:property name="Ankle_1_yy" value=" 0.0033 "/>
+<xacro:property name="Ankle_1_zz" value=" 0.0033 "/>
+<xacro:property name="Ankle_1_xy" value=" 0.000000 "/>
+<xacro:property name="Ankle_1_xz" value=" 0.000000 "/>
+<xacro:property name="Ankle_1_yz" value=" 0.000000 "/>
+<!-- Mass -->
+<xacro:property name="Ankle_1_mass" value=" 2.00000 "/>
+<!-- Center of Mass -->
+<xacro:property name="Ankle_2_x" value=" 0.0 "/>
+<xacro:property name="Ankle_2_y" value=" 0.000000 "/>
+<xacro:property name="Ankle_2_z" value=" 0.150 "/>
+<!-- Inertia -->
+<xacro:property name="Ankle_2_xx" value=" 0.0033 "/>
+<xacro:property name="Ankle_2_yy" value=" 0.0033 "/>
+<xacro:property name="Ankle_2_zz" value=" 0.0033 "/>
+<xacro:property name="Ankle_2_xy" value=" 0.000000 "/>
+<xacro:property name="Ankle_2_xz" value=" 0.000000 "/>
+<xacro:property name="Ankle_2_yz" value=" 0.000000 "/>
+<!-- Mass -->
+<xacro:property name="Ankle_2_mass" value=" 2.00000 "/>
+<!-- Center of Mass -->
+<xacro:property name="Wheel_x" value=" 0.00 "/>
 <xacro:property name="Wheel_y" value=" 0.000000 "/>
-<xacro:property name="Wheel_z" value=" 0.0024271906 "/>
-<!-- Inertia -->
-<xacro:property name="Wheel_xx" value=" 0.0046864297 "/>
-<xacro:property name="Wheel_yy" value=" 0.0046713489 "/>
-<xacro:property name="Wheel_zz" value=" 0.0053126029 "/>
+<xacro:property name="Wheel_z" value=" 0.0000 "/>
+<!-- Inertia -->
+<xacro:property name="Wheel_xx" value=" 0.00365 "/>
+<xacro:property name="Wheel_yy" value=" 0.00365 "/>
+<xacro:property name="Wheel_zz" value=" 0.0048 "/>
 <xacro:property name="Wheel_xy" value=" 0.000000 "/>
 <xacro:property name="Wheel_xz" value=" 0.000000 "/>
 <xacro:property name="Wheel_yz" value=" 0.000000 "/>
 <!-- Mass -->
-<xacro:property name="Wheel_mass" value=" 1.7289003000 "/>
+<xacro:property name="Wheel_mass" value=" 1.500000 "/>
 <!-- Center of Mass -->
 <xacro:property name="Torso_2_x" value=" 0.0047281261 "/>

File: centauro/centauro_urdf/urdf/centauro_leg.urdf.xacro (robot description, xacro)
@@ -5,7 +5,7 @@
 <link name="hip1_${leg_num}">
 	<inertial>
-		<origin xyz="${Leg_1_x} ${Leg_1_y} ${Leg_1_z}"/>
+		<origin xyz="${Leg_1_x} ${origin_x*origin_y*Leg_1_y} ${Leg_1_z}" />
 		<mass value="${Leg_1_mass}"/> <!-- org: 2 -->
-		<inertia ixx="${Leg_1_xx}" ixy="${Leg_1_xy}" ixz="${Leg_1_xz}" iyy="${Leg_1_yy}" iyz="${Leg_1_yz}" izz="${Leg_1_zz}"/>
+		<inertia ixx="${Leg_1_xx}" ixy="${origin_x*origin_y*Leg_1_xy}" ixz="${Leg_1_xz}" iyy="${Leg_1_yy}" iyz="${origin_x*origin_y*Leg_1_yz}" izz="${Leg_1_zz}"/>
 		<!-- <inertia ixx="0.01" ixy="0.01" ixz="0.01" iyy="0.01" iyz="0.01" izz="0.01"/> -->
 	</inertial>
@@ -49,7 +49,7 @@
 <link name="ankle1_${leg_num}">
 	<inertial>
-		<origin xyz="${Wrist_3_x} ${Wrist_3_y} ${Wrist_3_z}"/>
-		<mass value="${Wrist_3_mass}"/>  <!-- org: 3.5, foot un modeled-->
-		<inertia ixx="${Wrist_3_xx}" ixy="${Wrist_3_xy}" ixz="${Wrist_3_xz}" iyy="${Wrist_3_yy}" iyz="${Wrist_3_yz}" izz="${Wrist_3_zz}"/>
+		<origin xyz="${Ankle_1_x} ${Ankle_1_y} ${Ankle_1_z}"/>
+		<mass value="${Ankle_1_mass}"/>  <!-- org: 3.5, foot un modeled-->
+		<inertia ixx="${Ankle_1_xx}" ixy="${Ankle_1_xy}" ixz="${Ankle_1_xz}" iyy="${Ankle_1_yy}" iyz="${Ankle_1_yz}" izz="${Ankle_1_zz}"/>
 	<!--	<inertia ixx="0.01" ixy="0.01" ixz="0.01" iyy="0.01" iyz="0.01" izz="0.01"/>  -->
 	</inertial>
@@ -63,7 +63,7 @@
 <link name="ankle2_${leg_num}">
 	<inertial>
-		<origin xyz="${Wrist_3_x} ${Wrist_3_y} ${Wrist_3_z}"/>
-		<mass value="${Wrist_3_mass}"/>  <!-- org: 3.5, foot un modeled-->
-		<inertia ixx="${Wrist_3_xx}" ixy="${Wrist_3_xy}" ixz="${Wrist_3_xz}" iyy="${Wrist_3_yy}" iyz="${Wrist_3_yz}" izz="${Wrist_3_zz}"/>
+		<origin xyz="${Ankle_2_x} ${Ankle_2_y} ${Ankle_2_z}"/>
+		<mass value="${Ankle_2_mass}"/>  <!-- org: 3.5, foot un modeled-->
+		<inertia ixx="${Ankle_2_xx}" ixy="${Ankle_2_xy}" ixz="${Ankle_2_xz}" iyy="${Ankle_2_yy}" iyz="${Ankle_2_yz}" izz="${Ankle_2_zz}"/>
 	</inertial>
       <visual>
@@ -77,7 +77,7 @@
 <link name="wheel_${leg_num}">
 	<inertial>
-		<origin xyz="${Wrist_3_x} ${Wrist_3_y} ${Wrist_3_z}"/>
-		<mass value="${Wrist_3_mass}"/>  <!-- org: 3.5, foot un modeled-->
-		<inertia ixx="${Wrist_3_xx}" ixy="${Wrist_3_xy}" ixz="${Wrist_3_xz}" iyy="${Wrist_3_yy}" iyz="${Wrist_3_yz}" izz="${Wrist_3_zz}"/>
+		<origin xyz="${Wheel_x} ${Wheel_y} ${Wheel_z}"/>
+		<mass value="${Wheel_mass}"/>  <!-- org: 3.5, foot un modeled-->
+		<inertia ixx="${Wheel_xx}" ixy="${Wheel_xy}" ixz="${Wheel_xz}" iyy="${Wheel_yy}" iyz="${Wheel_yz}" izz="${Wheel_zz}"/>
 	</inertial>
       <visual>
@@ -89,104 +89,4 @@
       </collision>
 </link>
-<!-- wheels -->
-<xacro:if	value="${wheels}">
-	<!-- links -->
-	<link name="wheel_hip_${leg_num}">
-		<inertial>
-			<origin xyz="${Wheel_x} ${Wheel_y} ${Wheel_z}"/>	<!-- TODO -->
-			<mass value="${Wheel_mass}"/>  <!-- org: 3.5, foot un modeled-->
-			<inertia ixx="${Wheel_xx}" ixy="${Wheel_xy}" ixz="${Wheel_xz}" iyy="${Wheel_yy}" iyz="${Wheel_yz}" izz="${Wheel_zz}"/>
-		</inertial>
-		<visual>
-			<origin xyz="0 0 0" rpy="${PI/2} 0 0" />
-			<geometry>
-				<cylinder length="${wheel_length}" radius="${wheel_radius}"/>
-			</geometry>
-		</visual>
-		<collision>
-			<origin xyz="0 0 0" rpy="${PI/2} 0 0" />
-			<geometry>
-				<cylinder length="${wheel_length}" radius="${wheel_radius}"/>
-			</geometry>
-		</collision>
-	</link>
-	<link name="wheel_hip_reference_${leg_num}">
-		<inertial>
-			<origin xyz="0 0 0"/>	<!-- TODO -->
-			<mass value="${0.01}"/>  <!-- org: 3.5, foot un modeled-->
-			<inertia ixx="${0.01/12*(0.01*0.01+0.01*0.01)}" ixy="0" ixz="0" iyy="${0.01/12*(wheel_radius*wheel_radius+0.01*0.01)}" iyz="0" izz="${0.01/12*(wheel_radius*wheel_radius+0.01*0.01)}"/>
-		</inertial>
-		<visual>
-			<origin xyz="0 0 0" rpy="0 0 0" />
-			<geometry>
-				<box size="${wheel_radius} 0.01 0.01"/>
-			</geometry>
-		</visual>
-	</link>
-	<link name="wheel_knee_${leg_num}">
-		<inertial>
-			<origin xyz="${Wheel_x} ${Wheel_y} ${Wheel_z}"/>	<!-- TODO -->
-			<mass value="${Wheel_mass}"/>  <!-- org: 3.5, foot un modeled-->
-			<inertia ixx="${Wheel_xx}" ixy="${Wheel_xy}" ixz="${Wheel_xz}" iyy="${Wheel_yy}" iyz="${Wheel_yz}" izz="${Wheel_zz}"/>
-		</inertial>
-		<visual>
-			<origin xyz="0 0 0" rpy="${PI/2} 0 0" />
-			<geometry>
-				<cylinder length="${wheel_length}" radius="${wheel_radius}"/>
-			</geometry>
-		</visual>
-		<collision>
-			<origin xyz="0 0 0" rpy="${PI/2} 0 0" />
-			<geometry>
-				<cylinder length="${wheel_length}" radius="${wheel_radius}"/>
-			</geometry>
-		</collision>
-	</link>
-	<link name="wheel_knee_reference_${leg_num}">
-		<inertial>
-			<origin xyz="0 0 0"/>	<!-- TODO -->
-			<mass value="${0.01}"/>  <!-- org: 3.5, foot un modeled-->
-			<inertia ixx="${0.01/12*(0.01*0.01+0.01*0.01)}" ixy="0" ixz="0" iyy="${0.01/12*(wheel_radius*wheel_radius+0.01*0.01)}" iyz="0" izz="${0.01/12*(wheel_radius*wheel_radius+0.01*0.01)}"/>
-		</inertial>
-		<visual>
-			<origin xyz="0 0 0" rpy="0 0 0" />
-			<geometry>
-				<box size="${wheel_radius} 0.01 0.01"/>
-			</geometry>
-		</visual>
-	</link>
-	<!-- /links -->
-	<!-- joints -->
-	<joint name="j_wheel_hip_${leg_num}" type="continuous">
-		<parent link="hip2_${leg_num}"/>
-		<child link="wheel_hip_${leg_num}"/>
-		<origin xyz = "0 ${origin_x*(motors_length+wheel_length)/2} 0"/>
-		<axis xyz="0 ${origin_x*origin_y} 0"/>
-	</joint>
-	<joint name="j_wheel_hip_reeferece_${leg_num}" type="fixed">
-		<origin xyz="0 ${origin_y*(wheel_length+0.005)} 0"/>
-		<parent link="wheel_hip_${leg_num}"/>
-		<child link="wheel_hip_reference_${leg_num}"/>
-	</joint>
-	<joint name="j_wheel_knee_${leg_num}" type="continuous">
-		<parent link="knee_${leg_num}"/>
-		<child link="wheel_knee_${leg_num}"/>
-		<origin xyz = "0 ${origin_x*(motors_length+wheel_length)/2} 0"/>
-		<axis xyz="0 ${origin_x*origin_y} 0"/>
-	</joint>
-	<joint name="j_wheel_knee_reeferece_${leg_num}" type="fixed">
-		<origin xyz="0 ${origin_y*(wheel_length+0.005)} 0"/>
-		<parent link="wheel_knee_${leg_num}"/>
-		<child link="wheel_knee_reference_${leg_num}"/>
-	</joint>
-	<!-- /joints -->
-	<!-- actuators -->
-<xacro:if	value="${wheels_actuators}">
-	<xacro:position_actuator joint="j_wheel_hip_${leg_num}" />
-	<xacro:position_actuator joint="j_wheel_knee_${leg_num}" />
-	<!-- /actuators -->
-</xacro:if>
-</xacro:if>
-<!-- /wheels -->
 <joint name="hip_yaw_${leg_num}" type="revolute">
 	<parent link="pelvis"/>
