Commit message: Major changes: - adjust physics engine parameters to stabilize the simulation with updated inertia parameters - add mass at the arm end that facilitate stabilization of a simulation (see wiki for details) - add script publishing transform for a floating base used by rviz - add script publishing static transform for a false fixed joints (with 0 limits) for rviz visualization
Minor changes:
- change friction parameters for world and knee joints
- add convex_hull and STP-BV models for an additional link
- update Allowed Collision Matrix to consider additional link
- change xacro call to use an --inorder model used in scripts
- move kinematic_parameters to external file
- provide a script to read/modify inertia/kinematic parameters
- provide option of simulating perturbed inertia/kinematic parameters

File: centauro/centauro_urdf/inertia_parameters/original.xacro (robot description, xacro)
@@ -179,3 +179,32 @@
 <!-- Mass -->
 <xacro:property name="Wheel_mass" value=" 2.000000 "/>
+<!-- END-EFFECTORS-->
+<!-- SOFT HAND-->
+<!-- Center of Mass -->
+<xacro:property name="Hand_x" value=" 0 "/>
+<xacro:property name="Hand_y" value=" 0 "/>
+<xacro:property name="Hand_z" value=" 0.10 "/>
+<!-- Inertia -->
+<xacro:property name="Hand_xx" value=" 0.00024500 "/>
+<xacro:property name="Hand_yy" value=" 0.00024500 "/>
+<xacro:property name="Hand_zz" value=" 0.00024500 "/>
+<xacro:property name="Hand_xy" value=" 0 "/>
+<xacro:property name="Hand_xz" value=" 0 "/>
+<xacro:property name="Hand_yz" value=" 0 "/>
+<!-- Mass -->
+<xacro:property name="Hand_mass" value=" 0.3 "/>
+<!-- STICK-->
+<!-- Center of Mass -->
+<xacro:property name="Stick_x" value=" 0.001 "/>
+<xacro:property name="Stick_y" value=" 0.0 "/>
+<xacro:property name="Stick_z" value=" 0.006 "/>
+<!-- Inertia -->
+<xacro:property name="Stick_xx" value=" 0.0002 "/>
+<xacro:property name="Stick_yy" value=" 0.0002 "/>
+<xacro:property name="Stick_zz" value=" 0.00001 "/>
+<xacro:property name="Stick_xy" value=" 0.0 "/>
+<xacro:property name="Stick_xz" value=" 0.0 "/>
+<xacro:property name="Stick_yz" value=" 0.0 "/>
+<!-- Mass -->
+<xacro:property name="Stick_mass" value=" 0.150 "/>
 </robot>

File: centauro/centauro_urdf/urdf/centauro.urdf.xacro (robot description, xacro)
@@ -10,5 +10,6 @@
   <xacro:include filename="$(find centauro_gazebo)/urdf/centauro.gazebo"/>
 </xacro:if>
-<xacro:include filename="$(find centauro)/centauro_urdf/parameters.xacro"/>
+<xacro:include filename="${inertia_parameters_file}"/>
+<xacro:include filename="${kinematic_parameters_file}"/>
 <xacro:include filename="$(find centauro)/centauro_urdf/materials.xacro"/>
 <xacro:include filename="$(find centauro)/centauro_urdf/urdf/models/model.xacro"/>
@@ -39,10 +40,13 @@
       </collision>
    </link>
-   <joint name="reference" type="${reference}">
-      <origin xyz="0 0 0.85"/>
-      <parent link="world"/>
-      <child link="pelvis"/>
-   </joint>
 </xacro:if>
+<xacro:unless value="${pelvis}">
+   <link name="pelvis"/>
+</xacro:unless>
+<joint name="reference" type="${reference}">
+   <origin xyz="${Pelvis_Ox} ${Pelvis_Oy} ${Pelvis_Oz}"/>
+   <parent link="world"/>
+   <child link="pelvis"/>
+</joint>
 <!-- /reference  -->
 <!-- torso -->
@@ -54,13 +58,13 @@
 <xacro:if value="${arms == 'true'}">
    <xacro:centauro_arm arm_num="1"  rot="1"  parent="torso_2">
-      <origin xyz="0.04576 0.169137 0.190626" rpy="0.0 0 -0.5236026689864071"/>
+      <origin xyz="${Shoulder_1_Ox} ${Shoulder_1_Oy} ${Shoulder_1_Oz}" rpy="${Shoulder_1_roll} ${Shoulder_1_pitch} ${Shoulder_1_yaw}"/>
    </xacro:centauro_arm>
    <xacro:centauro_arm arm_num="2" rot="-1"  parent="torso_2">
-      <origin xyz="0.0457475 -0.169137 0.190626" rpy="0.0 0 0.5236026689864071" />
+      <origin xyz="${Shoulder_1_Ox} ${-Shoulder_1_Oy} ${Shoulder_1_Oz}" rpy="${Shoulder_1_roll} ${Shoulder_1_pitch} ${-Shoulder_1_yaw}" />
    </xacro:centauro_arm>
 </xacro:if>
 <xacro:if value="${arm == 'true' and arms == 'false'}">
         <xacro:centauro_arm arm_num="1"  rot="1" parent="world">
-           <origin xyz="${0.04576 + 0.3} ${0.169137} ${1.1+0.190626}" rpy="0.0 0 -0.5236026689864071"/>
+           <origin xyz="${Shoulder_1_Ox + Pelvis_Ox + Torso_2_Ox} ${Shoulder_1_Oy + Pelvis_Oy + Torso_2_Oy} ${Shoulder_1_Oz + Pelvis_Oz + Torso_2_Oz}" rpy="${Shoulder_1_roll} ${Shoulder_1_pitch} ${Shoulder_1_yaw}"/>
         </xacro:centauro_arm>
 </xacro:if>

File: centauro/centauro_urdf/urdf/centauro_arm.urdf.xacro (robot description, xacro)
@@ -1,5 +1,4 @@
+<?xml version="1.0"?>
 <robot xmlns:xacro="http://www.ros.org/wiki/xacro">
-<xacro:property name="cos_m10" value="0.984807753012208"/>
-<xacro:property name="sin_m10" value="-0.17364817766693033"/>
 <!-- macro arms -->
 <xacro:macro name="centauro_arm" params="arm_num rot parent *origin">
@@ -62,5 +61,5 @@
          <mass value="${Elbow_1_mass}"/>
          <inertia ixx="${Elbow_1_xx}" ixy="${-rot*Elbow_1_xy}" ixz="${Elbow_1_xz}" iyy="${Elbow_1_yy}" iyz="${-rot*Elbow_1_yz}" izz="${Elbow_1_zz}"/>
-</inertial>
+      </inertial>
       <visual>
          <xacro:visual_model.arm4 />
@@ -122,20 +121,4 @@
       </collision>
    </link>
-<!-- mass -->
-<!--   <link name="mass${arm_num}_body">
-      <inertial>
-         <origin xyz="0 0 0"/> -->
-<!--         <mass value="10"/> -->
-<!--         <inertia ixx="0.001" ixy="0.00" ixz="0.00" iyy="0.001" iyz="0.00" izz="0.001"/>
-      </inertial>
-      <visual>
-         <origin xyz="0.0 0.0 0"/>
-         <geometry>
-            <box size="0.10 0.10 0.10"/>--> <!-- OK -->
-<!--         </geometry>
-         <material name="red"/>
-      </visual>
-   </link> -->
-<!-- /mass -->
 <!-- /LINKS -->
 <!-- JOINTS -->
@@ -158,5 +141,5 @@
       <parent link="arm${arm_num}_1"/>
       <child link="arm${arm_num}_2"/>
-      <origin xyz="-0.09115 ${rot*0.06106} 0.010766"/>
+      <origin xyz="${Shoulder_2_Ox} ${rot*Shoulder_2_Oy} ${Shoulder_2_Oz}"/>
       <axis xyz="-1 0 0"/>
       <xacro:unless value="${rot+1}" >
@@ -172,5 +155,5 @@
       <parent link="arm${arm_num}_2"/>
       <child link="arm${arm_num}_3"/>
-      <origin xyz="0.09115 0 -0.21915"/>
+      <origin xyz="${Shoulder_3_Ox} ${Shoulder_3_Oy} ${Shoulder_3_Oz}"/>
       <axis xyz="0 0 -1"/>
       <limit lower="-2.618" upper="2.618" effort="1770" velocity="6.5"/>
@@ -181,5 +164,5 @@
       <parent link="arm${arm_num}_3"/>
       <child link="arm${arm_num}_4"/>
-      <origin xyz="0.040 ${rot*0.05615} -0.074"/>
+      <origin xyz="${Elbow_1_Ox} ${rot*Elbow_1_Oy} ${Elbow_1_Oz}"/>
       <axis xyz="0 ${rot} 0"/>
       <xacro:unless value="${rot-1}" >
@@ -195,5 +178,5 @@
       <parent link="arm${arm_num}_4"/>
       <child link="arm${arm_num}_5"/>
-      <origin xyz="-0.015 ${-rot*0.05615} -0.061"/>
+      <origin xyz="${Wrist_1_Ox} ${-rot*Wrist_1_Oy} ${Wrist_1_Oz}"/>
       <axis xyz="0 0 -1"/>
       <limit lower="-2.618" upper="2.618" effort="950" velocity="6.5"/>
@@ -204,5 +187,5 @@
       <parent link="arm${arm_num}_5"/>
       <child link="arm${arm_num}_6"/>
-      <origin xyz="0 ${rot*0.049} -0.180"/>
+      <origin xyz="${Wrist_2_Ox} ${rot*Wrist_2_Oy} ${Wrist_2_Oz}"/>
       <axis xyz="0 ${rot} 0"/>
       <limit lower="-1.570" upper="1.570" effort="950" velocity="6.5"/>
@@ -213,5 +196,5 @@
       <parent link="arm${arm_num}_6"/>
       <child link="arm${arm_num}_7"/>
-      <origin xyz="0 ${-rot*0.049} -0.169"/>
+      <origin xyz="${Wrist_3_Ox} ${-rot*Wrist_3_Oy} ${Wrist_3_Oz}"/>
       <axis xyz="0 0 -1"/>
       <limit lower="-2.618" upper="2.618" effort="400" velocity="6.5"/>
@@ -240,4 +223,8 @@
   <xacro:include filename="$(find centauro)/centauro_urdf/urdf/centauro_no_end_effector.urdf.xacro" />
 </xacro:if>
+<!-- adds and additional box of a 10x10x10 cm size and mass "MASS" 5 cm towards x direction from the endeffector axis. It may be needed to stabilize a simulation -->
+<xacro:if value="${MASS > 0}" >
+  <xacro:include filename="$(find centauro)/centauro_urdf/urdf/centauro_mass.urdf.xacro" />
+</xacro:if>
 <!-- /end-effector -->
 </xacro:macro>

File: centauro/centauro_urdf/urdf/centauro_hand.urdf.xacro (robot description, xacro)
@@ -4,7 +4,7 @@
    <link name="arm${arm_num}_8">
       <inertial>
-         <origin xyz="0 0 0.10" rpy="0 0 0"/>
-         <mass value="0.3"/>
-         <inertia ixx="0.00024500"  ixy="0"  ixz="0" iyy="0.00024500" iyz="0" izz="0.00024500" />
+         <origin xyz="${Hand_x} ${Hand_y} ${Hand_z}" rpy="0 0 0"/>
+         <mass value="${Hand_mass}"/>
+         <inertia ixx="${Hand_xx}"  ixy="${Hand_xy}"  ixz="${Hand_xz}" iyy="${Hand_yy}" iyz="${Hand_yz}" izz="${Hand_zz}" />
       </inertial>
       <visual>
@@ -20,5 +20,5 @@
       <parent link="arm${arm_num}_7"/>
       <child link="arm${arm_num}_8"/>
-      <origin xyz="0 0 -0.0405" rpy="0 ${PI} ${-PI/2}"/>
+      <origin xyz="${End_effector_Ox} ${End_effector_Oy} ${End_effector_Oz}" rpy="${End_effector_roll} ${End_effector_pitch} ${End_effector_yaw}"/>
       <axis xyz="1 0 0" />
       <limit velocity="6.5" effort="400" lower="0.0" upper="1.57075" />

File: centauro/centauro_urdf/urdf/centauro_leg.urdf.xacro (robot description, xacro)
@@ -246,5 +246,5 @@
 	<parent link="pelvis"/>
 	<child link="hip1_${leg_num}"/>
-	<origin xyz="${origin_x*0.30} ${origin_y*0.15} 0" rpy="0 0 ${PI/2}"/>
+	<origin xyz="${origin_x*Leg_1_Ox} ${origin_y*Leg_1_Oy} ${Leg_1_Oz}" rpy="${Leg_1_roll} ${Leg_1_pitch} ${Leg_1_yaw}"/>
 	<axis xyz="0 0 ${-origin_y}"/>
         <limit lower="-2.09" upper="2.09" effort="1770" velocity="6.5"/> <!-- TODO -->
@@ -253,5 +253,5 @@
 	<parent link="hip1_${leg_num}"/>
 	<child link="hip2_${leg_num}"/>
-	<origin xyz="0 0 -0.2"/>
+	<origin xyz="${Leg_2_Ox} ${Leg_2_Oy} ${Leg_2_Oz}"/>
 	<axis xyz="0 ${-origin_y} 0"/>
         <limit lower="-3.14" upper="3.14" effort="3300" velocity="6.5"/> <!-- TODO -->
@@ -260,5 +260,5 @@
 	<parent link="hip2_${leg_num}"/>
 	<child link="knee_${leg_num}"/>
-	<origin xyz="0 0 -0.35"/>
+	<origin xyz="${Leg_3_Ox} ${Leg_3_Oy} ${Leg_3_Oz}"/>
 	<axis xyz="0 ${-origin_y} 0"/>
         <limit  lower="-3.14" upper="3.14" effort="3300" velocity="600.5"/> <!-- TODO -->

File: centauro/centauro_urdf/urdf/centauro_no_end_effector.urdf.xacro (robot description, xacro)
@@ -7,5 +7,5 @@
       <parent link="arm${arm_num}_7"/>
       <child link="arm${arm_num}_8"/>
-      <origin xyz="0 0 -0.0405" rpy="0 ${PI} ${-PI/2}"/>
+      <origin xyz="${End_effector_Ox} ${End_effector_Oy} ${End_effector_Oz}" rpy="${End_effector_roll} ${End_effector_pitch} ${End_effector_yaw}"/>
       <axis xyz="1 0 0" />
       <limit velocity="0" effort="0" lower="0.0" upper="0" />

File: centauro/centauro_urdf/urdf/centauro_stick.urdf.xacro (robot description, xacro)
@@ -4,8 +4,9 @@
    <link name="arm${arm_num}_8">
       <inertial>
-         <origin xyz="0 0 0.075" rpy="0 0 0"/>
-         <mass value="2"/>
-         <inertia ixx="0.00290117"  ixy="0"  ixz="0" iyy="0.00290117" iyz="0" izz="0.00016900" />
-      </inertial>
+         <origin xyz="${Stick_x} ${Stick_y} ${Stick_z}" rpy="0 0 0"/>
+         <mass value="${Stick_mass}"/>
+       <inertia ixx="${Stick_xx}"  ixy="${Stick_xy}"  ixz="${Stick_xz}" iyy="${Stick_yy}" iyz="${Stick_yz}" izz="${Stick_zz}" />
+<!--          <inertia ixx="0.003"  ixy="0"  ixz="0" iyy="0.0025" iyz="0" izz="0.00016900" /> -->
+     </inertial>
       <visual>
          <xacro:visual_model.stick />
@@ -21,5 +22,5 @@
       <parent link="arm${arm_num}_7"/>
       <child link="arm${arm_num}_8"/>
-      <origin xyz="0 0 -0.0405" rpy="0 ${PI} ${-PI/2}"/>
+      <origin xyz="${End_effector_Ox} ${End_effector_Oy} ${End_effector_Oz}" rpy="${End_effector_roll} ${End_effector_pitch} ${End_effector_yaw}"/>
       <axis xyz="1 0 0" />
       <limit velocity="0" effort="0" lower="0.0" upper="0" />

File: centauro/centauro_urdf/urdf/centauro_torso.urdf.xacro (robot description, xacro)
@@ -22,9 +22,9 @@
    <xacro:if value="${pelvis}">
       <parent link="pelvis"/>
-      <origin xyz="0.30 0 0.1"/>
+      <origin xyz="${Torso_2_Ox} ${Torso_2_Oy} ${Torso_2_Oz}"/>
    </xacro:if>
    <xacro:unless value="${pelvis}">
       <parent link="world"/>
-      <origin xyz="0.30 0 ${0.1 + 0.85}"/>
+      <origin xyz="${Torso_2_Ox + Pelvis_Ox} ${Torso_2_Oy + Pelvis_Oy} ${Torso_2_Oz + Pelvis_Oz}"/>
    </xacro:unless>
    <child link="torso_2"/>

File: centauro/centauro_urdf/urdf/config.xacro (robot description, xacro)
@@ -14,4 +14,6 @@
 <xacro:property name="ONE_ARM" value="$(arg ONE_ARM)"/>
 <xacro:property name="GAZEBO" value="$(arg GAZEBO)"/>
+<xacro:property name="INERTIA_PARAM" value="$(arg INERTIA_PARAM)"/>
+<xacro:property name="KINEMATIC_PARAM" value="$(arg KINEMATIC_PARAM)"/>
 <xacro:property name="TORSO_ACTUATORS" value="$(arg TORSO_ACTUATORS)"/>
 <xacro:property name="ARM_ACTUATORS" value="$(arg ARM_ACTUATORS)"/>
@@ -19,4 +21,5 @@
 <xacro:property name="WHEELS_ACTUATORS" value="$(arg WHEELS_ACTUATORS)"/>
 <xacro:property name="ARM_SENSORS" value="$(arg ARM_SENSORS)"/>
+<xacro:property name="MASS" value="$(arg MASS)"/>
 <!-- dependend arguments -->
 <xacro:property name="arms" value="${'true' if ('false' not in [TORSO, ARMS] and 'false' in [ONE_ARM]) else 'false'}"/>
@@ -34,3 +37,6 @@
 <xacro:property name="arm_sensors" value="${'true' if ('false' not in [ARM_SENSORS, arm]) else 'false'}"/>
 <xacro:property name="leg_sensors" value="${'true' if ('false' not in [legs]) else 'false'}"/>
+<xacro:property name="package" value="$(find centauro)"/>
+<xacro:property name="inertia_parameters_file" value="${package + '/centauro_urdf/inertia_parameters/' + INERTIA_PARAM + '.xacro'}"/>
+<xacro:property name="kinematic_parameters_file" value="${package + '/centauro_urdf/kinematic_parameters/' + KINEMATIC_PARAM + '.xacro'}"/>
 </robot>

Commit message: Head integration

File: centauro/centauro_urdf/inertia_parameters/original.xacro (robot description, xacro)
@@ -13,5 +13,5 @@
 <xacro:property name="Pelvis_x" value=" -0.0135413420 "/>
 <xacro:property name="Pelvis_y" value=" -0.0029098264 "/>
-<xacro:property name="Pelvis_z" value=" 0.1806072100 "/>
+<xacro:property name="Pelvis_z" value=" 0.01400721 "/>
 <!-- Inertia -->
 <xacro:property name="Pelvis_xx" value=" 0.2002111900 "/>
@@ -102,7 +102,7 @@
 <xacro:property name="Wheel_mass" value=" 1.7289003000 "/>
 <!-- Center of Mass -->
-<xacro:property name="Torso_2_x" value=" 0.0047281261 "/>
-<xacro:property name="Torso_2_y" value=" 0.00038307386 "/>
-<xacro:property name="Torso_2_z" value=" 0.14972892 "/>
+<xacro:property name="Torso_2_x" value=" 0.0064454169 "/>
+<xacro:property name="Torso_2_y" value=" 0.0021390093 "/>
+<xacro:property name="Torso_2_z" value=" 0.1430209500 "/>
 <!-- Inertia -->
 <xacro:property name="Torso_2_xx" value=" 0.063643392 "/>
@@ -113,5 +113,44 @@
 <xacro:property name="Torso_2_yz" value=" -0.00004657 "/>
 <!-- Mass -->
-<xacro:property name="Torso_2_mass" value=" 4.5494226000 "/>
+<xacro:property name="Torso_2_mass" value=" 6.1886404000 "/>
+<!-- Center of Mass -->
+<xacro:property name="Neck_1_x" value=" 0.0404796740 "/>
+<xacro:property name="Neck_1_y" value=" 0.0213775730 "/>
+<xacro:property name="Neck_1_z" value=" -0.0145951120 "/>
+<!-- Inertia -->
+<xacro:property name="Neck_1_xx" value=" 0.0003718568 "/>
+<xacro:property name="Neck_1_yy" value=" 0.0001886879 "/>
+<xacro:property name="Neck_1_zz" value=" 0.0005023443 "/>
+<xacro:property name="Neck_1_xy" value=" -0.0000942983 "/>
+<xacro:property name="Neck_1_xz" value=" -0.0000280644 "/>
+<xacro:property name="Neck_1_yz" value=" -0.0000154534 "/>
+<!-- Mass -->
+<xacro:property name="Neck_1_mass" value=" 0.3387868600 "/>
+<!-- Center of Mass -->
+<xacro:property name="Neck_2_x" value=" 0.0484669180 "/>
+<xacro:property name="Neck_2_y" value=" -0.0598523180 "/>
+<xacro:property name="Neck_2_z" value=" -0.0085314894 "/>
+<!-- Inertia -->
+<xacro:property name="Neck_2_xx" value=" 0.0004682345 "/>
+<xacro:property name="Neck_2_yy" value=" 0.0002635246 "/>
+<xacro:property name="Neck_2_zz" value=" 0.0003763351 "/>
+<xacro:property name="Neck_2_xy" value=" -0.0000105438 "/>
+<xacro:property name="Neck_2_xz" value=" 0.0000724398 "/>
+<xacro:property name="Neck_2_yz" value=" 0.0000016904 "/>
+<!-- Mass -->
+<xacro:property name="Neck_2_mass" value=" 0.7852694200 "/>
+<!-- Center of Mass -->
+<xacro:property name="Neck_3_x" value=" 0.0484669180 "/>
+<xacro:property name="Neck_3_y" value=" -0.0598523180 "/>
+<xacro:property name="Neck_3_z" value=" -0.0085314894 "/>
+<!-- Inertia -->
+<xacro:property name="Neck_3_xx" value=" 0.0004682345 "/>
+<xacro:property name="Neck_3_yy" value=" 0.0002635246 "/>
+<xacro:property name="Neck_3_zz" value=" 0.0003763351 "/>
+<xacro:property name="Neck_3_xy" value=" -0.0000105438 "/>
+<xacro:property name="Neck_3_xz" value=" 0.0000724398 "/>
+<xacro:property name="Neck_3_yz" value=" 0.0000016904 "/>
+<!-- Mass -->
+<xacro:property name="Neck_3_mass" value=" 0.7852694200 "/>
 <!-- Center of Mass -->
 <xacro:property name="Shoulder_1_x" value=" -0.0031005886 "/>

File: centauro/centauro_urdf/kinematic_parameters/original.xacro (robot description, xacro)
@@ -14,9 +14,21 @@
 <xacro:property name="Pelvis_Ox" value=" 0.0 "/>
 <xacro:property name="Pelvis_Oy" value=" 0.0 "/>
-<xacro:property name="Pelvis_Oz" value=" 0.759 "/>
+<xacro:property name="Pelvis_Oz" value=" 0.92560000 "/>
 <!-- Origin -->
-<xacro:property name="Leg_1_Ox" value=" 0.225 "/>
+<xacro:property name="Neck_1_Ox" value=" 0.0 "/>
+<xacro:property name="Neck_1_Oy" value=" 0.0 "/>
+<xacro:property name="Neck_1_Oz" value=" 0.2795 "/>
+<!-- Origin -->
+<xacro:property name="Neck_2_Ox" value=" 0.054 "/>
+<xacro:property name="Neck_2_Oy" value=" 0.0596 "/>
+<xacro:property name="Neck_2_Oz" value=" -0.0124975 "/>
+<!-- Origin -->
+<xacro:property name="Neck_3_Ox" value=" 0.055 "/>
+<xacro:property name="Neck_3_Oy" value=" 0.00 "/>
+<xacro:property name="Neck_3_Oz" value=" 0.473262 "/>
+<!-- Origin -->
+<xacro:property name="Leg_1_Ox" value=" 0.250 "/>
 <xacro:property name="Leg_1_Oy" value=" -0.125 "/>
-<xacro:property name="Leg_1_Oz" value=" 0.11 "/>
+<xacro:property name="Leg_1_Oz" value="-0.05660000 "/>
 <xacro:property name="Leg_1_roll" value=" 3.141592653589793 "/>
 <xacro:property name="Leg_1_pitch" value=" 0.0 "/>
@@ -55,11 +67,11 @@
 <xacro:property name="Wheel_yaw" value=" 0.0 "/>
 <!-- Origin -->
-<xacro:property name="Torso_2_Ox" value=" 0.175 "/>
+<xacro:property name="Torso_2_Ox" value=" 0.200 "/>
 <xacro:property name="Torso_2_Oy" value=" 0.0 "/>
-<xacro:property name="Torso_2_Oz" value=" 0.36 "/>
+<xacro:property name="Torso_2_Oz" value=" 0.256 "/>
 <!-- Origin -->
 <xacro:property name="Shoulder_1_Ox" value=" 0.04576 "/> <!-- for the other arm it was 0.0457475 -->
 <xacro:property name="Shoulder_1_Oy" value=" 0.169137 "/>
-<xacro:property name="Shoulder_1_Oz" value=" 0.190626 "/>
+<xacro:property name="Shoulder_1_Oz" value=" 0.11662600 "/>
 <xacro:property name="Shoulder_1_roll" value=" 0.0 "/>
 <xacro:property name="Shoulder_1_pitch" value=" 0.0 "/>

File: centauro/centauro_urdf/urdf/centauro.urdf.xacro (robot description, xacro)
@@ -60,6 +60,9 @@
 <!-- /reference  -->
 <!-- torso -->
-<xacro:if value="${torso}">
+<xacro:if value="${torso == 'true'}">
    <xacro:include filename="$(find centauro)/centauro_urdf/urdf/centauro_torso.urdf.xacro"/>
+</xacro:if>
+<xacro:if value="${head == 'true'}">
+   <xacro:include filename="$(find centauro)/centauro_urdf/urdf/centauro_head.urdf.xacro"/>
 </xacro:if>
 <!-- /torso -->

File: centauro/centauro_urdf/urdf/centauro_torso.urdf.xacro (robot description, xacro)
@@ -5,5 +5,5 @@
 	<inertial>
 		<origin xyz="${Torso_2_x} ${Torso_2_y} ${Torso_2_z}"/>
-		<mass value="${Torso_2_mass}"/> <!-- mass  7: torso_1 (2) + torso_2 (5), head un_modelled -->
+		<mass value="${Torso_2_mass}"/>
                 <inertia ixx="${Torso_2_xx}" ixy="${Torso_2_xy}" ixz="${Torso_2_xz}" iyy="${Torso_2_yy}" iyz="${Torso_2_yz}" izz="${Torso_2_zz}"/>
         </inertial>

File: centauro/centauro_urdf/urdf/config.xacro (robot description, xacro)
@@ -10,4 +10,5 @@
 <xacro:property name="LEGS" value="$(arg LEGS)"/>
 <xacro:property name="TORSO" value="$(arg TORSO)"/>
+<xacro:property name="HEAD" value="$(arg HEAD)"/>
 <xacro:property name="WHEELS" value="$(arg WHEELS)"/>
 <xacro:property name="STATIC" value="$(arg STATIC)"/>
@@ -21,4 +22,5 @@
 <xacro:property name="LEG_ACTUATORS" value="$(arg LEG_ACTUATORS)"/>
 <xacro:property name="WHEELS_ACTUATORS" value="$(arg WHEELS_ACTUATORS)"/>
+<xacro:property name="HEAD_ACTUATORS" value="$(arg HEAD_ACTUATORS)"/>
 <xacro:property name="ARM_SENSORS" value="$(arg ARM_SENSORS)"/>
 <xacro:property name="LEG_SENSORS" value="$(arg LEG_SENSORS)"/>
@@ -31,4 +33,5 @@
 <xacro:property name="legs" value="${'true' if ('false' not in [LEGS] and 'true' not in [ONE_ARM]) else 'false'}"/>
 <xacro:property name="torso" value="${'true' if ('false' in [ONE_ARM] and 'true' in [TORSO]) else 'false'}"/>
+<xacro:property name="head" value="${'true' if ('false' not in [torso, HEAD]) else 'false'}"/>
 <xacro:property name="arm" value= "${'true' if ('true' in [arms, ONE_ARM]) else 'false'}" />
 <xacro:property name="pelvis" value= "${'true' if ('true' in [legs]) else 'false'}" />
@@ -40,5 +43,6 @@
 <xacro:property name="arm_actuators" value="${'true' if ('false' not in [ARM_ACTUATORS, TORSO_ACTUATORS, arm]) else 'false'}"/>
 <xacro:property name="leg_actuators" value="${'true' if ('false' not in [LEG_ACTUATORS, legs]) else 'false'}"/>
-<xacro:property name="wheels_actuators" value="${'true' if ('false' not in [WHEELS_ACTUATORS, LEG_ACTUATORS, wheels]) else 'false'}"/>
+<xacro:property name="head_actuators" value="${'true' if ('false' not in [HEAD_ACTUATORS, head]) else 'false'}"/>
+<xacro:property name="torso_actuators" value="${'true' if ('false' not in [TORSO_ACTUATORS, TORSO]) else 'false'}"/>
 <!-- SENSORS -->
 <xacro:property name="arm_sensors" value="${'true' if ('false' not in [ARM_SENSORS, arm]) else 'false'}"/>

File: centauro/centauro_urdf/urdf/models/model_config.xacro (robot description, xacro)
@@ -15,4 +15,7 @@
       <xacro:load_model path="upper_body/end_effectors/${END_EFFECTOR}"  model="${model}"/>
    </xacro:if>
+   <xacro:if value="${head == 'true'}" >
+      <xacro:load_model path="upper_body/head"  model="${model}"/>
+   </xacro:if>
 </xacro:macro>
 </robot>

File: centauro/centauro_urdf/urdf/models/upper_body/primitive.xacro (robot description, xacro)
@@ -2,7 +2,7 @@
 <robot name="centauro" xmlns:xacro="http://www.ros.org/wiki/xacro">
 <xacro:macro name="torso">
-   <origin xyz="0.0 0 0.20"  rpy="0.0 0.0 0.0"/>
+   <origin xyz="0.0 0 0.25"  rpy="0.0 0.0 0.0"/>
    <geometry>
-      <box size="0.2 0.3 0.1"/>
+      <box size="0.1 0.2 0.3"/>
    </geometry>
 </xacro:macro>
