Commit message: adjust force-torque sensor orientation

File: centauro/centauro_urdf/inertia_parameters/original.xacro (robot description, xacro)
@@ -244,4 +244,18 @@
 <!-- Mass -->
 <xacro:property name="Wrist_3_mass" value=" 0.5598103600 "/>
+<!-- FT-SENSOR-->
+<!-- Center of Mass -->
+<xacro:property name="Ft_arm_x" value=" 0.0 "/>
+<xacro:property name="Ft_arm_y" value=" 0.0 "/>
+<xacro:property name="Ft_arm_z" value=" 0.0 "/>
+<!-- Inertia -->
+<xacro:property name="Ft_arm_xx" value=" 1e-6 "/>
+<xacro:property name="Ft_arm_yy" value=" 1e-6 "/>
+<xacro:property name="Ft_arm_zz" value=" 1e-6 "/>
+<xacro:property name="Ft_arm_xy" value=" 0.0 "/>
+<xacro:property name="Ft_arm_xz" value=" 0.0 "/>
+<xacro:property name="Ft_arm_yz" value=" 0.0 "/>
+<!-- Mass -->
+<xacro:property name="Ft_arm_mass" value=" 0.150 "/>
 <!-- END-EFFECTORS-->
 <!-- SOFT HAND-->
@@ -249,5 +263,5 @@
 <xacro:property name="Hand_x" value=" 0 "/>
 <xacro:property name="Hand_y" value=" 0 "/>
-<xacro:property name="Hand_z" value=" 0.10 "/>
+<xacro:property name="Hand_z" value=" -0.07 "/>
 <!-- Inertia -->
 <xacro:property name="Hand_xx" value=" 0.00024500 "/>

File: centauro/centauro_urdf/kinematic_parameters/original.xacro (robot description, xacro)
@@ -101,12 +101,50 @@
 <xacro:property name="Wrist_3_Oy" value=" 0.049 "/>
 <xacro:property name="Wrist_3_Oz" value=" -0.169 "/>
+<!-- FT_SENSORS_ARM-->
+<!-- Origin -->
+<xacro:property name="Ft_arm_Ox" value=" 0.0 "/>
+<xacro:property name="Ft_arm_Oy" value=" 0.0 "/>
+<xacro:property name="Ft_arm_Oz" value=" -0.0405 "/>
+<xacro:property name="Ft_arm_roll" value=" 0.0 "/>
+<xacro:property name="Ft_arm_pitch" value=" ${PI} "/>
+<xacro:property name="Ft_arm_yaw" value=" ${-PI} "/>
 <!-- END-EFFECTORS-->
 <!-- SOFT HAND/STICK/NO_EE-->
 <!-- Origin -->
-<xacro:property name="End_effector_Ox" value=" 0.0 "/>
-<xacro:property name="End_effector_Oy" value=" 0.0 "/>
-<xacro:property name="End_effector_Oz" value=" -0.0405 "/>
-<xacro:property name="End_effector_roll" value=" 0.0 "/>
-<xacro:property name="End_effector_pitch" value=" ${PI} "/>
-<xacro:property name="End_effector_yaw" value=" ${-PI/2} "/>
+<xacro:property name="No_end_ft_Ox" value=" 0.0 "/>
+<xacro:property name="No_end_ft_Oy" value=" 0.0 "/>
+<xacro:property name="No_end_ft_Oz" value=" -0.0405 "/>
+<xacro:property name="No_end_ft_roll" value=" ${PI} "/>
+<xacro:property name="No_end_ft_pitch" value=" 0.0 "/>
+<xacro:property name="No_end_ft_yaw" value=" 0.0 "/>
+<xacro:property name="No_end_Ox" value=" 0.0 "/>
+<xacro:property name="No_end_Oy" value=" 0.0 "/>
+<xacro:property name="No_end_Oz" value=" 0.0 "/>
+<xacro:property name="No_end_roll" value=" 0.0 "/>
+<xacro:property name="No_end_pitch" value=" 0.0 "/>
+<xacro:property name="No_end_yaw" value=" 0.0 "/>
+<xacro:property name="Stick_ft_Ox" value=" 0.0 "/>
+<xacro:property name="Stick_ft_Oy" value=" 0.0 "/>
+<xacro:property name="Stick_ft_Oz" value=" 0.0 "/>
+<xacro:property name="Stick_ft_roll" value=" 0.0 "/>
+<xacro:property name="Stick_ft_pitch" value=" 0.0 "/>
+<xacro:property name="Stick_ft_yaw" value=" ${-PI/2} "/>
+<xacro:property name="Stick_Ox" value=" 0.0 "/>
+<xacro:property name="Stick_Oy" value=" 0.0 "/>
+<xacro:property name="Stick_Oz" value=" -0.0405 "/>
+<xacro:property name="Stick_roll" value=" 0.0 "/>
+<xacro:property name="Stick_pitch" value=" ${PI} "/>
+<xacro:property name="Stick_yaw" value=" ${-PI/2} "/>
+<xacro:property name="Hand_ft_Ox" value=" 0.0 "/>
+<xacro:property name="Hand_ft_Oy" value=" 0.0 "/>
+<xacro:property name="Hand_ft_Oz" value=" -0.0405 "/>
+<xacro:property name="Hand_ft_roll" value=" ${PI} "/>
+<xacro:property name="Hand_ft_pitch" value=" 0.0 "/>
+<xacro:property name="Hand_ft_yaw" value=" 0.0 "/>
+<xacro:property name="Hand_Ox" value=" 0.0 "/>
+<xacro:property name="Hand_Oy" value=" 0.0 "/>
+<xacro:property name="Hand_Oz" value=" 0.0 "/>
+<xacro:property name="Hand_roll" value=" 0.0 "/>
+<xacro:property name="Hand_pitch" value=" 0.0 "/>
+<xacro:property name="Hand_yaw" value=" 0.0 "/>
 </robot>

File: centauro/centauro_urdf/urdf/centauro_arm.urdf.xacro (robot description, xacro)
@@ -204,4 +204,25 @@
 <!-- /actuators -->
 <!-- end-effector -->
+<xacro:if value="${ft_sensors == 'true'}" >
+<!-- wrist pitch-->
+   <joint name="j_ft_${arm_num}" type="revolute">
+      <parent link="arm${arm_num}_7"/>
+      <child link="ft_arm${arm_num}"/>
+      <origin xyz="${Ft_arm_Ox} ${Ft_arm_Oy} ${Ft_arm_Oz}" rpy="${Ft_arm_roll} ${Ft_arm_pitch} ${Ft_arm_yaw}" />
+      <axis xyz="0 0 1"/>
+      <limit lower="0.0" upper="0.0" effort="0" velocity="0"/>
+   </joint>
+<!-- wrist pitch-->
+   <link name="ft_arm${arm_num}">
+      <inertial>
+         <origin xyz="${Ft_arm_x} ${-rot*Ft_arm_y} ${Ft_arm_z}"/>
+         <mass value="${Ft_arm_mass}"/>
+         <inertia ixx="${Ft_arm_xx}" ixy="${-rot*Ft_arm_xy}" ixz="${Ft_arm_xz}" iyy="${Ft_arm_yy}" iyz="${-rot*Ft_arm_yz}" izz="${Ft_arm_zz}"/>
+      </inertial>
+   </link>
+   <xacro:if value="${arm_actuators}">
+      <xacro:position_actuator joint="j_ft_${arm_num}" />
+   </xacro:if>
+</xacro:if>
 <xacro:if value="${END_EFFECTOR == 'soft_hand'}" >
   <xacro:include filename="$(find centauro)/centauro_urdf/urdf/centauro_hand.urdf.xacro" />

File: centauro/centauro_urdf/urdf/centauro_hand.urdf.xacro (robot description, xacro)
@@ -18,8 +18,14 @@
 <!-- /links -->
    <joint name="j_arm${arm_num}_8" type="revolute">
-      <parent link="arm${arm_num}_7"/>
+      <xacro:if value="${ft_sensors == 'true'}" >
+         <parent link="ft_arm${arm_num}"/>
+         <origin xyz="${Hand_ft_Ox} ${Hand_ft_Oy} ${Hand_ft_Oz}" rpy="${Hand_ft_roll} ${Hand_ft_pitch} ${Hand_ft_yaw}"/>
+      </xacro:if>
+      <xacro:unless value="${ft_sensors == 'true'}" >
+         <parent link="arm${arm_num}_7"/>
+         <origin xyz="${Hand_Ox} ${Hand_Oy} ${Hand_Oz}" rpy="${Hand_roll} ${Hand_pitch} ${Hand_yaw}"/>
+      </xacro:unless>
       <child link="arm${arm_num}_8"/>
-      <origin xyz="${End_effector_Ox} ${End_effector_Oy} ${End_effector_Oz}" rpy="${End_effector_roll} ${End_effector_pitch} ${End_effector_yaw}"/>
-      <axis xyz="1 0 0" />
+      <axis xyz="0 1 0" />
       <limit velocity="20.3" effort="40" lower="0.0" upper="1.57075" />
    </joint> -->

File: centauro/centauro_urdf/urdf/centauro_no_end_effector.urdf.xacro (robot description, xacro)
@@ -5,7 +5,13 @@
 <!-- /links -->
    <joint name="j_arm${arm_num}_8" type="revolute">
-      <parent link="arm${arm_num}_7"/>
+      <xacro:if value="${ft_sensors == 'true'}" >
+         <parent link="ft_arm${arm_num}"/>
+         <origin xyz="${No_end_ft_Ox} ${No_end_ft_Oy} ${No_end_ft_Oz}" rpy="${No_end_ft_roll} ${No_end_ft_pitch} ${No_end_ft_yaw}"/>
+      </xacro:if>
+      <xacro:unless value="${ft_sensors == 'true'}" >
+         <parent link="arm${arm_num}_7"/>
+         <origin xyz="${No_end_Ox} ${No_end_Oy} ${No_end_Oz}" rpy="${No_end_roll} ${No_end_pitch} ${No_end_yaw}"/>
+      </xacro:unless>
       <child link="arm${arm_num}_8"/>
-      <origin xyz="${End_effector_Ox} ${End_effector_Oy} ${End_effector_Oz}" rpy="${End_effector_roll} ${End_effector_pitch} ${End_effector_yaw}"/>
       <axis xyz="1 0 0" />
       <limit velocity="0" effort="0" lower="0.0" upper="0" />

File: centauro/centauro_urdf/urdf/centauro_stick.urdf.xacro (robot description, xacro)
@@ -19,10 +19,15 @@
 <!-- /links -->
 <!-- joints -->
-   <joint name="j_arm${arm_num}_8" type="revolute">
-      <parent link="arm${arm_num}_7"/>
+   <joint name="j_arm${arm_num}_8" type="fixed">
+      <xacro:if value="${ft_sensors == 'true'}" >
+         <parent link="ft_arm${arm_num}"/>
+         <origin xyz="${Stick_ft_Ox} ${Stick_ft_Oy} ${Stick_ft_Oz}" rpy="${Stick_ft_roll} ${Stick_ft_pitch} ${Stick_ft_yaw}"/>
+      </xacro:if>
+      <xacro:unless value="${ft_sensors == 'true'}" >
+         <parent link="arm${arm_num}_7"/>
+         <origin xyz="${Stick_Ox} ${Stick_Oy} ${Stick_Oz}" rpy="${Stick_roll} ${Stick_pitch} ${Stick_yaw}"/>
+      </xacro:unless>
       <child link="arm${arm_num}_8"/>
-      <origin xyz="${End_effector_Ox} ${End_effector_Oy} ${End_effector_Oz}" rpy="${End_effector_roll} ${End_effector_pitch} ${End_effector_yaw}"/>
       <axis xyz="1 0 0" />
-      <limit velocity="0" effort="0" lower="0.0" upper="0" />
    </joint> -->
 <!-- /joints -->

File: centauro/centauro_urdf/urdf/models/upper_body/end_effectors/soft_hand/primitive.xacro (robot description, xacro)
@@ -2,5 +2,5 @@
 <robot name="centauro" xmlns:xacro="http://www.ros.org/wiki/xacro">
 <xacro:macro name="soft_hand" >
-   <origin xyz="0 0 0.0" rpy="0 0 0" />
+   <origin xyz="0 0 -0.07" rpy="0 0 0" />
    <geometry>
       <box size="0.07 0.07 0.07" />

File: centauro_gazebo/sensors/ros_control/ft_sensor/load/arms.xacro (robot description, xacro)
@@ -2,7 +2,7 @@
 <robot  xmlns:xacro="http://www.ros.org/wiki/xacro">
 <xacro:include filename="$(find centauro)/centauro_urdf/urdf/config.xacro"/>
-  <xacro:force-torque_sensor joint="j_arm1_8" robot="centauro"/>
+  <xacro:force-torque_sensor joint="j_ft_1" robot="centauro"/>
   <xacro:if value="${arms}">
-    <xacro:force-torque_sensor joint="j_arm2_8" robot="centauro"/>
+    <xacro:force-torque_sensor joint="j_ft_2" robot="centauro"/>
   </xacro:if>
 </robot>

File: centauro_gazebo/sensors/xbotcore/ft_sensor/load/arms.xacro (robot description, xacro)
@@ -2,7 +2,7 @@
 <robot  xmlns:xacro="http://www.ros.org/wiki/xacro">
 <xacro:include filename="$(find centauro)/centauro_urdf/urdf/config.xacro"/>
-  <xacro:force-torque_sensor joint="j_arm1_8" robot="centauro" ft_name="left_arm_ft" pose="0 0 0 0 0 0"/>
+  <xacro:force-torque_sensor joint="j_ft_1" robot="centauro" ft_name="left_arm_ft" pose="0 0 0 0 0 0"/>
   <xacro:if value="${arms}">
-    <xacro:force-torque_sensor joint="j_arm2_8" robot="centauro" ft_name="right_arm_ft" pose="0 0 0 0 0 0"/>
+    <xacro:force-torque_sensor joint="j_ft_2" robot="centauro" ft_name="right_arm_ft" pose="0 0 0 0 0 0"/>
   </xacro:if>
 </robot>

Commit message: sensor transformation frames

File: centauro/centauro_urdf/inertia_parameters/original.xacro (robot description, xacro)
@@ -287,3 +287,17 @@
 <!-- Mass -->
 <xacro:property name="Stick_mass" value=" 0.150 "/>
+<!-- DUMMY-->
+<!-- Center of Mass -->
+<xacro:property name="Dummy_x" value=" 0.0 "/>
+<xacro:property name="Dummy_y" value=" 0.0 "/>
+<xacro:property name="Dummy_z" value=" 0.0 "/>
+<!-- Inertia -->
+<xacro:property name="Dummy_xx" value=" 1e-6 "/>
+<xacro:property name="Dummy_yy" value=" 1e-6 "/>
+<xacro:property name="Dummy_zz" value=" 1e-6 "/>
+<xacro:property name="Dummy_xy" value=" 0.0 "/>
+<xacro:property name="Dummy_xz" value=" 0.0 "/>
+<xacro:property name="Dummy_yz" value=" 0.0 "/>
+<!-- Mass -->
+<xacro:property name="Dummy_mass" value=" 0.100 "/>
 </robot>

File: centauro/centauro_urdf/kinematic_parameters/original.xacro (robot description, xacro)
@@ -148,3 +148,33 @@
 <xacro:property name="Hand_pitch" value=" 0.0 "/>
 <xacro:property name="Hand_yaw" value=" 0.0 "/>
+<xacro:property name="Camera_central_Ox" value=" 0.0559593 "/>
+<xacro:property name="Camera_central_Oy" value=" 5e-12 "/>
+<xacro:property name="Camera_central_Oz" value=" 0.390626 "/>
+<xacro:property name="Camera_central_roll" value=" 0.0 "/>
+<xacro:property name="Camera_central_pitch" value=" 0.349065586018 "/>
+<xacro:property name="Camera_central_yaw" value=" 0.0 "/>
+<xacro:property name="Camera_left_Ox" value=" 0.0191392 "/>
+<xacro:property name="Camera_left_Oy" value=" 0.0525845 "/>
+<xacro:property name="Camera_left_Oz" value=" 0.390626 "/>
+<xacro:property name="Camera_left_roll" value=" 0.0 "/>
+<xacro:property name="Camera_left_pitch" value=" 0.349065586018 "/>
+<xacro:property name="Camera_left_yaw" value=" 1.2217302006 "/>
+<xacro:property name="Camera_right_Ox" value=" 0.0191392 "/>
+<xacro:property name="Camera_right_Oy" value=" -0.0525845 "/>
+<xacro:property name="Camera_right_Oz" value=" 0.390626 "/>
+<xacro:property name="Camera_right_roll" value=" 0.0 "/>
+<xacro:property name="Camera_right_pitch" value=" 0.349065586018 "/>
+<xacro:property name="Camera_right_yaw" value=" -1.2217302006 "/>
+<xacro:property name="Kinect_Ox" value=" 0.03 "/>
+<xacro:property name="Kinect_Oy" value=" -0.0596 "/>
+<xacro:property name="Kinect_Oz" value=" 0.045855 "/>
+<xacro:property name="Kinect_roll" value=" 0.0 "/>
+<xacro:property name="Kinect_pitch" value=" 0.0 "/>
+<xacro:property name="Kinect_yaw" value=" 0.0 "/>
+<xacro:property name="Velodyne_Ox" value=" 0.138 "/>
+<xacro:property name="Velodyne_Oy" value=" 0.0 "/>
+<xacro:property name="Velodyne_Oz" value=" -0.033 "/>
+<xacro:property name="Velodyne_roll" value=" 0.0 "/>
+<xacro:property name="Velodyne_pitch" value=" 0.0 "/>
+<xacro:property name="Velodyne_yaw" value=" -3.14159265359 "/>
 </robot>

File: centauro/centauro_urdf/urdf/centauro_head.urdf.xacro (robot description, xacro)
@@ -42,4 +42,41 @@
 </link>
 <!-- /head links -->
+<!-- sensors links -->
+<link name="camera_central">
+	<inertial>
+		<origin xyz="${Dummy_x} ${Dummy_y} ${Dummy_z}"/>
+		<mass value="${Dummy_mass}"/>
+                <inertia ixx="${Dummy_xx}" ixy="${Dummy_xy}" ixz="${Dummy_xz}" iyy="${Dummy_yy}" iyz="${Dummy_yz}" izz="${Dummy_zz}"/>
+        </inertial>
+</link>
+<link name="camera_left">
+	<inertial>
+		<origin xyz="${Dummy_x} ${Dummy_y} ${Dummy_z}"/>
+		<mass value="${Dummy_mass}"/>
+                <inertia ixx="${Dummy_xx}" ixy="${Dummy_xy}" ixz="${Dummy_xz}" iyy="${Dummy_yy}" iyz="${Dummy_yz}" izz="${Dummy_zz}"/>
+        </inertial>
+</link>
+<link name="camera_right">
+	<inertial>
+		<origin xyz="${Dummy_x} ${Dummy_y} ${Dummy_z}"/>
+		<mass value="${Dummy_mass}"/>
+                <inertia ixx="${Dummy_xx}" ixy="${Dummy_xy}" ixz="${Dummy_xz}" iyy="${Dummy_yy}" iyz="${Dummy_yz}" izz="${Dummy_zz}"/>
+        </inertial>
+</link>
+<link name="kinect">
+	<inertial>
+		<origin xyz="${Dummy_x} ${Dummy_y} ${Dummy_z}"/>
+		<mass value="${Dummy_mass}"/>
+                <inertia ixx="${Dummy_xx}" ixy="${Dummy_xy}" ixz="${Dummy_xz}" iyy="${Dummy_yy}" iyz="${Dummy_yz}" izz="${Dummy_zz}"/>
+        </inertial>
+</link>
+<link name="velodyne">
+	<inertial>
+		<origin xyz="${Dummy_x} ${Dummy_y} ${Dummy_z}"/>
+		<mass value="${Dummy_mass}"/>
+                <inertia ixx="${Dummy_xx}" ixy="${Dummy_xy}" ixz="${Dummy_xz}" iyy="${Dummy_yy}" iyz="${Dummy_yz}" izz="${Dummy_zz}"/>
+        </inertial>
+</link>
+<!-- /sensors links -->
 <!-- head joints -->
 <joint name="neck_yaw" type="revolute">
@@ -65,4 +102,31 @@
 </joint>
 <!-- /head joints -->
+<!-- sensors transformations -->
+<joint name="j_camera_central" type="fixed">
+   <parent link="torso_2"/>
+   <origin xyz="${Camera_central_Ox} ${Camera_central_Oy} ${Camera_central_Oz}" rpy="${Camera_central_roll} ${Camera_central_pitch} ${Camera_central_yaw}"/>
+   <child link="camera_central"/>
+</joint>
+<joint name="j_camera_left" type="fixed">
+   <parent link="torso_2"/>
+   <origin xyz="${Camera_left_Ox} ${Camera_left_Oy} ${Camera_left_Oz}" rpy="${Camera_left_roll} ${Camera_left_pitch} ${Camera_left_yaw}"/>
+   <child link="camera_left"/>
+</joint>
+<joint name="j_camera_right" type="fixed">
+   <parent link="torso_2"/>
+   <origin xyz="${Camera_right_Ox} ${Camera_right_Oy} ${Camera_right_Oz}" rpy="${Camera_right_roll} ${Camera_right_pitch} ${Camera_right_yaw}"/>
+   <child link="camera_right"/>
+</joint>
+<joint name="j_kinect" type="fixed">
+   <parent link="neck_2"/>
+   <origin xyz="${Kinect_Ox} ${Kinect_Oy} ${Kinect_Oz}" rpy="${Kinect_roll} ${Kinect_pitch} ${Kinect_yaw}"/>
+   <child link="kinect"/>
+</joint>
+<joint name="j_velodyne" type="fixed">
+   <parent link="neck_3"/>
+   <origin xyz="${Velodyne_Ox} ${Velodyne_Oy} ${Velodyne_Oz}" rpy="${Velodyne_roll} ${Velodyne_pitch} ${Velodyne_yaw}"/>
+   <child link="velodyne"/>
+</joint>
+<!-- /sensors transformations -->
 <xacro:if value="${head_actuators}">
 <!-- torso actuators -->

Commit message: centauro_urdf: inertia: tensor for ft sensors

File: centauro/centauro_urdf/inertia_parameters/original.xacro (robot description, xacro)
@@ -250,7 +250,7 @@
 <xacro:property name="Ft_arm_z" value=" 0.0 "/>
 <!-- Inertia -->
-<xacro:property name="Ft_arm_xx" value=" 1e-6 "/>
-<xacro:property name="Ft_arm_yy" value=" 1e-6 "/>
-<xacro:property name="Ft_arm_zz" value=" 1e-6 "/>
+<xacro:property name="Ft_arm_xx" value=" ${ 2.0/5.0 * 0.150 * 0.05*0.05 }"/>
+<xacro:property name="Ft_arm_yy" value=" ${ 2.0/5.0 * 0.150 * 0.05*0.05 } "/>
+<xacro:property name="Ft_arm_zz" value=" ${ 2.0/5.0 * 0.150 * 0.05*0.05 } "/>
 <xacro:property name="Ft_arm_xy" value=" 0.0 "/>
 <xacro:property name="Ft_arm_xz" value=" 0.0 "/>

Commit message: integrate static HERI hend

File: centauro/centauro_urdf/inertia_parameters/original.xacro (robot description, xacro)
@@ -287,4 +287,17 @@
 <!-- Mass -->
 <xacro:property name="Stick_mass" value=" 0.150 "/>
+<!-- Center of Mass -->
+<xacro:property name="Heri_x" value=" 0.00270235 "/>
+<xacro:property name="Heri_y" value=" -0.01411486 "/>
+<xacro:property name="Heri_z" value=" 0.05023455 "/>
+<!-- Inertia -->
+<xacro:property name="Heri_xx" value=" 0.0062253159 "/>
+<xacro:property name="Heri_yy" value=" 0.0046306594 "/>
+<xacro:property name="Heri_zz" value=" 0.0037732152 "/>
+<xacro:property name="Heri_xy" value=" 0.0003312435 "/>
+<xacro:property name="Heri_xz" value=" 0.0000517232 "/>
+<xacro:property name="Heri_yz" value=" 0.0001950252 "/>
+<!-- Mass -->
+<xacro:property name="Heri_mass" value=" 1.8366865000 "/>
 <!-- DUMMY-->
 <!-- Center of Mass -->

File: centauro/centauro_urdf/kinematic_parameters/original.xacro (robot description, xacro)
@@ -136,4 +136,16 @@
 <xacro:property name="Stick_pitch" value=" ${PI} "/>
 <xacro:property name="Stick_yaw" value=" ${-PI/2} "/>
+<xacro:property name="Heri_ft_Ox" value=" 0.0 "/>
+<xacro:property name="Heri_ft_Oy" value=" 0.0 "/>
+<xacro:property name="Heri_ft_Oz" value=" 0.0 "/>
+<xacro:property name="Heri_ft_roll" value=" 0.0 "/>
+<xacro:property name="Heri_ft_pitch" value=" 0.0 "/>
+<xacro:property name="Heri_ft_yaw" value=" 0.0 "/>
+<xacro:property name="Heri_Ox" value=" 0.0 "/>
+<xacro:property name="Heri_Oy" value=" 0.0 "/>
+<xacro:property name="Heri_Oz" value=" -0.0405 "/>
+<xacro:property name="Heri_roll" value=" 0.0 "/>
+<xacro:property name="Heri_pitch" value=" ${PI} "/>
+<xacro:property name="Heri_yaw" value=" ${PI} "/>
 <xacro:property name="Hand_ft_Ox" value=" 0.0 "/>
 <xacro:property name="Hand_ft_Oy" value=" 0.0 "/>

File: centauro/centauro_urdf/urdf/centauro_arm.urdf.xacro (robot description, xacro)
@@ -232,4 +232,7 @@
   <xacro:include filename="$(find centauro)/centauro_urdf/urdf/centauro_stick.urdf.xacro" />
 </xacro:if>
+<xacro:if value="${end_effector == 'heri'}" >
+  <xacro:include filename="$(find centauro)/centauro_urdf/urdf/centauro_heri.urdf.xacro" />
+</xacro:if>
 <xacro:if value="${end_effector == 'schunk_hand'}" >
 	 <!-- schunk hand -->
@@ -239,5 +242,5 @@
    </xacro:svh>
 </xacro:if>
-<xacro:if value="${end_effector != 'stick' and end_effector != 'soft_hand' and end_effector != 'schunk_hand'}" >
+<xacro:if value="${end_effector != 'stick' and end_effector != 'soft_hand' and end_effector != 'schunk_hand' and end_effector != 'heri'}" >
   <xacro:include filename="$(find centauro)/centauro_urdf/urdf/centauro_no_end_effector.urdf.xacro" />
 </xacro:if>

File: centauro/centauro_urdf/urdf/models/model_config.xacro (robot description, xacro)
@@ -12,8 +12,8 @@
    <xacro:load_model path="upper_body" model="${model}"/>
    <xacro:load_model path="lower_body" model="${model}"/>
-   <xacro:if value="${left_end_effector in ['soft_hand', 'stick']}" >
+   <xacro:if value="${left_end_effector in ['soft_hand', 'stick', 'heri']}" >
       <xacro:load_model path="upper_body/end_effectors/${left_end_effector}"  model="${model}"/>
    </xacro:if>
-   <xacro:if value="${right_end_effector in ['soft_hand', 'stick']}" >
+   <xacro:if value="${right_end_effector in ['soft_hand', 'stick', 'heri']}" >
       <xacro:load_model path="upper_body/end_effectors/${right_end_effector}"  model="${model}"/>
    </xacro:if>

Commit message: updated pelvis parameters

File: centauro/centauro_urdf/inertia_parameters/original.xacro (robot description, xacro)
@@ -11,16 +11,16 @@
 <xacro:property name="wheel_weight" value=" 2.000000 "/>
 <!-- Center of Mass -->
-<xacro:property name="Pelvis_x" value=" -0.0135413420 "/>
-<xacro:property name="Pelvis_y" value=" -0.0029098264 "/>
-<xacro:property name="Pelvis_z" value=" 0.01400721 "/>
-<!-- Inertia -->
-<xacro:property name="Pelvis_xx" value=" 0.2002111900 "/>
-<xacro:property name="Pelvis_yy" value=" 0.5113621400 "/>
-<xacro:property name="Pelvis_zz" value=" 0.5440141100 "/>
-<xacro:property name="Pelvis_xy" value=" -0.0038421093 "/>
-<xacro:property name="Pelvis_xz" value=" -0.0332988490 "/>
-<xacro:property name="Pelvis_yz" value=" 0.0044698470 "/>
-<!-- Mass -->
-<xacro:property name="Pelvis_mass" value=" 24.1909450000 "/>
+<xacro:property name="Pelvis_x" value=" 0.0013890071 "/>
+<xacro:property name="Pelvis_y" value=" -0.0015989148 "/>
+<xacro:property name="Pelvis_z" value=" 0.0631010120 "/>
+<!-- Inertia -->
+<xacro:property name="Pelvis_xx" value=" 0.2391262700 "/>
+<xacro:property name="Pelvis_yy" value=" 0.7143007800 "/>
+<xacro:property name="Pelvis_zz" value=" 0.8187044800 "/>
+<xacro:property name="Pelvis_xy" value=" -0.0050541269 "/>
+<xacro:property name="Pelvis_xz" value=" -0.0197460550 "/>
+<xacro:property name="Pelvis_yz" value=" 0.0002131204 "/>
+<!-- Mass -->
+<xacro:property name="Pelvis_mass" value=" 16.0975740000 "/>
 <!-- Center of Mass -->
 <xacro:property name="Leg_1_x" value=" 0.0102141990 "/>
