Commit message: update torso mass and CoM position and update URDF accordingly

File: centauro/centauro_urdf/inertia_parameters/original.xacro (robot description, xacro)
@@ -102,7 +102,7 @@
 <xacro:property name="Wheel_mass" value=" 1.7289003000 "/>
 <!-- Center of Mass -->
-<xacro:property name="Torso_2_x" value=" 0.0064454169 "/>
-<xacro:property name="Torso_2_y" value=" 0.0021390093 "/>
-<xacro:property name="Torso_2_z" value=" 0.1430209500 "/>
+<xacro:property name="Torso_2_x" value=" -0.0194977940 "/>
+<xacro:property name="Torso_2_y" value=" 0.0045317835 "/>
+<xacro:property name="Torso_2_z" value=" 0.1376828300 "/>
 <!-- Inertia -->
 <xacro:property name="Torso_2_xx" value=" 0.063643392 "/>
@@ -113,5 +113,5 @@
 <xacro:property name="Torso_2_yz" value=" -0.00004657 "/>
 <!-- Mass -->
-<xacro:property name="Torso_2_mass" value=" 6.1886404000 "/>
+<xacro:property name="Torso_2_mass" value=" 11.4926890000 "/>
 <!-- Center of Mass -->
 <xacro:property name="Neck_1_x" value=" 0.0404796740 "/>

File: centauro/centauro_urdf/urdf/centauro.urdf (robot description, URDF)
Before this commit: robot centauro, 89 links, 88 joints
Links:
- added link ft_arm1, mass 0.15
- added link ft_arm2, mass 0.15
- link arm1_8: mass 0.15 -> 1.8366865; geometry collision mesh filename=package://centauro/centauro_urdf/meshes/convex_hull/heri.stl scale=0.001 -0.001 -0.001; visual mesh filename=package://centauro/centauro_urdf/meshes/simplified/heri.stl scale=0.001 -0.001 -0.001
- link pelvis: mass 24.190945 -> 16.097574
- link torso_2: mass 6.1886404 -> 11.492689
Joints:
- added joint j_ft_1: type revolute, parent arm1_7, child ft_arm1, origin xyz=0.0 0.0 -0.0405 rpy=0.0 3.14159265359 -3.14159265359, axis 0 0 1, limit lower=0.0 upper=0.0 effort=0 velocity=0
- added joint j_ft_2: type revolute, parent arm2_7, child ft_arm2, origin xyz=0.0 0.0 -0.0405 rpy=0.0 3.14159265359 -3.14159265359, axis 0 0 1, limit lower=0.0 upper=0.0 effort=0 velocity=0
- joint ankle_pitch_1: limit lower=-2.61799388 upper=2.61799388 effort=147 velocity=8.1 -> lower=-2.4056 upper=2.3184 effort=147 velocity=8.1
- joint ankle_pitch_2: limit lower=-2.61799388 upper=2.61799388 effort=147 velocity=8.1 -> lower=-2.3266 upper=2.3914 effort=147 velocity=8.1
- joint ankle_pitch_3: limit lower=-2.61799388 upper=2.61799388 effort=147 velocity=8.1 -> lower=-2.4696 upper=2.4464 effort=147 velocity=8.1
- joint ankle_pitch_4: limit lower=-2.61799388 upper=2.61799388 effort=147 velocity=8.1 -> lower=-2.3426 upper=2.3934 effort=147 velocity=8.1
- joint ankle_yaw_1: limit lower=-2.58308729 upper=2.58308729 effort=35 velocity=20.0 -> lower=-2.5626 upper=2.5384 effort=35 velocity=20.0
- joint ankle_yaw_2: limit lower=-2.58308729 upper=2.58308729 effort=35 velocity=20.0 -> lower=-2.5546 upper=2.5484 effort=35 velocity=20.0
- joint ankle_yaw_3: limit lower=-2.58308729 upper=2.58308729 effort=35 velocity=20.0 -> lower=-2.5606 upper=2.5454 effort=35 velocity=20.0
- joint ankle_yaw_4: limit lower=-2.58308729 upper=2.58308729 effort=35 velocity=20.0 -> lower=-2.6046 upper=2.5514 effort=35 velocity=20.0
- joint hip_pitch_1: limit lower=-2.09439510 upper=2.09439510 effort=304 velocity=8.8 -> lower=-2.0226 upper=2.02748 effort=304 velocity=8.8
- joint hip_pitch_2: limit lower=-2.09439510 upper=2.09439510 effort=304 velocity=8.8 -> lower=-2.0156 upper=2.0354 effort=304 velocity=8.8
- joint hip_pitch_3: limit lower=-2.09439510 upper=2.09439510 effort=304 velocity=8.8 -> lower=-2.0126 upper=2.0384 effort=304 velocity=8.8
- joint hip_pitch_4: limit lower=-2.09439510 upper=2.09439510 effort=304 velocity=8.8 -> lower=-2.0326 upper=2.0524 effort=304 velocity=8.8
- joint hip_yaw_1: limit lower=-1.13446401 upper=2.70526034 effort=304 velocity=8.8 -> lower=-0.9432 upper=2.5138 effort=304 velocity=8.8
- joint hip_yaw_2: limit lower=-2.70526034 upper=1.13446401 effort=304 velocity=8.8 -> lower=-2.511 upper=0.943 effort=304 velocity=8.8
- joint hip_yaw_3: limit lower=-2.70526034 upper=1.13446401 effort=304 velocity=8.8 -> lower=-2.51 upper=0.943 effort=304 velocity=8.8
- joint hip_yaw_4: limit lower=-1.13446401 upper=2.70526034 effort=304 velocity=8.8 -> lower=-0.9412 upper=2.5138 effort=304 velocity=8.8
- joint j_arm1_1: limit lower=-3.403 upper=1.658 effort=147 velocity=5.7 -> lower=-3.348 upper=1.578 effort=147 velocity=5.7
- joint j_arm1_2: limit lower=-3.49 upper=0 effort=147 velocity=5.7 -> lower=-3.42 upper=-0.056 effort=147 velocity=5.7
- joint j_arm1_3: limit lower=-2.618 upper=2.618 effort=147 velocity=8.2 -> lower=-2.5556 upper=2.5424 effort=147 velocity=8.2
- joint j_arm1_4: limit lower=-2.530 upper=0.349 effort=147 velocity=8.2 -> lower=-2.4636 upper=0.2804 effort=147 velocity=8.2
- joint j_arm1_5: limit lower=-2.618 upper=2.618 effort=55 velocity=11.6 -> lower=-2.5406 upper=2.5534 effort=55 velocity=11.6
- joint j_arm1_6: limit lower=-1.570 upper=1.570 effort=55 velocity=11.6 -> lower=-1.5096 upper=1.5044 effort=55 velocity=11.6
- joint j_arm1_7: limit lower=-2.618 upper=2.618 effort=27 velocity=20.3 -> lower=-2.5376 upper=2.5554 effort=27 velocity=20.3
- joint j_arm1_8: origin xyz=0.0 0.0 -0.0405 rpy=0.0 3.14159265359 -1.5707963268 -> xyz=0.0 0.0 0.0 rpy=0.0 0.0 0.0; parent arm1_7 -> ft_arm1
- joint j_arm2_1: limit lower=-1.658 upper=3.403 effort=147 velocity=5.7 -> lower=-1.6102 upper=3.3138 effort=147 velocity=5.7
- joint j_arm2_2: limit lower=0 upper=3.49 effort=147 velocity=5.7 -> lower=0.0578 upper=3.4288 effort=147 velocity=5.7
- joint j_arm2_3: limit lower=-2.618 upper=2.618 effort=147 velocity=8.2 -> lower=-2.5426 upper=2.5524 effort=147 velocity=8.2
- joint j_arm2_4: limit lower=-0.349 upper=2.530 effort=147 velocity=8.2 -> lower=-0.2796 upper=2.4564 effort=147 velocity=8.2
- joint j_arm2_5: limit lower=-2.618 upper=2.618 effort=55 velocity=11.6 -> lower=-2.5626 upper=2.5464 effort=55 velocity=11.6
- joint j_arm2_6: limit lower=-1.570 upper=1.570 effort=55 velocity=11.6 -> lower=-1.4726 upper=1.5364 effort=55 velocity=11.6
- joint j_arm2_7: limit lower=-2.618 upper=2.618 effort=27 velocity=20.3 -> lower=-3.0908 upper=2.0114 effort=27 velocity=20.3
- joint knee_pitch_1: limit lower=-2.61799388 upper=2.61799388 effort=304 velocity=8.8 -> lower=-2.4056 upper=2.3994 effort=304 velocity=8.8
- joint knee_pitch_2: limit lower=-2.61799388 upper=2.61799388 effort=304 velocity=8.8 -> lower=-2.4006 upper=2.4034 effort=304 velocity=8.8
- joint knee_pitch_3: limit lower=-2.61799388 upper=2.61799388 effort=304 velocity=8.8 -> lower=-2.4056 upper=2.4064 effort=304 velocity=8.8
- joint knee_pitch_4: limit lower=-2.61799388 upper=2.61799388 effort=304 velocity=8.8 -> lower=-2.4176 upper=2.3884 effort=304 velocity=8.8

Commit message: correct the inertia parameter

File: centauro/centauro_urdf/inertia_parameters/original.xacro (robot description, xacro)
@@ -207,5 +207,5 @@
 <!-- Center of Mass -->
 <xacro:property name="Wrist_1_x" value=" -0.00011079615 "/>
-<xacro:property name="Wrist_1_y" value=" 0.01159080036 "/>
+<xacro:property name="Wrist_1_y" value=" 0.011590836 "/>
 <xacro:property name="Wrist_1_z" value=" -0.07816026 "/>
 <!-- Inertia -->
