Commit message: Implementing plain gazebo FT

File: centauro_gazebo/sensors/force_torque_plugin.urdf.xacro (robot description, xacro)
@@ -1,5 +1,5 @@
 <!--<?xml version="1.0"?>-->
 <robot xmlns:xacro="http://www.ros.org/wiki/xacro">
-<xacro:macro name="force-torque_sensor" params="joint robot">
+<xacro:macro name="force-torque_sensor" params="joint robot ft_name pose">
     <xacro:if value="${ros_control}">
         <gazebo reference="${joint}">
@@ -16,12 +16,14 @@
     <xacro:if value="${xbotcore}">
         <gazebo reference="${joint}">
-            <provideFeedback>true</provideFeedback>
-        </gazebo>
-        <gazebo>
-            <plugin name="${joint}_ft_sensor" filename="libgazebo_ros_ft_sensor.so">
-                <updateRate>100.0</updateRate>
-                <topicName>${robot}/${joint}_ft_sensor</topicName>
-                <jointName>${joint}</jointName>
-            </plugin>
+            <sensor type="force_torque" name="${ft_name}">
+                        <force_torque>
+                        <frame>parent</frame>
+                        <measure_direction>child_to_parent</measure_direction>
+                        </force_torque>
+                <always_on>true</always_on>
+                <visualize>true</visualize>
+                <update_rate>1000</update_rate>
+                <pose>${pose}</pose>
+            </sensor>
         </gazebo>
     </xacro:if>
