Commit message: remove unnecessary parameters from ROS force torque sensor plugin.

File: centauro_gazebo/sensors/ros_control/ft_sensor/plugin.xacro (robot description, xacro)
@@ -1,5 +1,5 @@
 <!--<?xml version="1.0"?>-->
 <robot xmlns:xacro="http://www.ros.org/wiki/xacro">
-<xacro:macro name="force-torque_sensor" params="joint robot ft_name pose">
+<xacro:macro name="force-torque_sensor" params="joint robot">
     <xacro:if value="${ros_control}">
         <gazebo reference="${joint}">
