Commit message: added schunk hand meshes

File: centauro/centauro_urdf/urdf/models/upper_body/end_effectors/schunk_hand/svh_gazebo.urdf.xacro (robot description, xacro)
@@ -80,5 +80,5 @@
                 <origin rpy="0 0 0" xyz="0 0 0" />
                 <geometry>
-                    <mesh filename="package://schunk_svh_driver/description/meshes/camera_link.STL" />
+                    <mesh filename="package://centauro/centauro_urdf/meshes/schunk_hand/camera_link.STL" />
                 </geometry>
             </visual>
@@ -86,5 +86,5 @@
                <origin rpy="0 0 0" xyz="0 0 0" />
                 <geometry>
-                    <mesh filename="package://schunk_svh_driver/description/meshes/camera_link.STL" />
+                    <mesh filename="package://centauro/centauro_urdf/meshes/schunk_hand/camera_link.STL" />
                 </geometry>
             </collision>
@@ -106,5 +106,5 @@
                 <origin xyz="0 0 -0.032" rpy="0 0 0" />
                 <geometry>
-                    <mesh filename="package://schunk_svh_driver/description/meshes/base10.dae" />
+                    <mesh filename="package://centauro/centauro_urdf/meshes/schunk_hand/base10.dae" />
                 </geometry>
             </visual>
@@ -112,5 +112,5 @@
                 <origin xyz="0 0 -0.032" rpy="0 0 0" />
                 <geometry>
-                    <mesh filename="package://schunk_svh_driver/description/meshes/base10.dae" />
+                    <mesh filename="package://centauro/centauro_urdf/meshes/schunk_hand/base10.dae" />
                 </geometry>
             </collision>
@@ -131,5 +131,5 @@
                 <origin rpy="0 0 0" xyz="0 0.01313 0" />
                 <geometry>
-                    <mesh scale="${side*(1)} 1 1" filename="package://schunk_svh_driver/description/meshes/h10.dae" />
+                    <mesh scale="${side*(1)} 1 1" filename="package://centauro/centauro_urdf/meshes/schunk_hand/h10.dae" />
                 </geometry>
             </visual>
@@ -139,5 +139,5 @@
                 <geometry>
 					<box size="0.055 0.025 0.12"/>
-                    <!--mesh scale="${side*(1)} 1 1" filename="package://schunk_svh_driver/description/meshes/h10.dae" /-->
+                    <!--mesh scale="${side*(1)} 1 1" filename="package://centauro/centauro_urdf/meshes/schunk_hand/h10.dae" /-->
                 </geometry>
             </collision>
@@ -150,5 +150,5 @@
                 <origin xyz="${side*(-0.0007)} 0 -0.01002" />
                 <geometry>
-                    <mesh scale="${side*(1)} 1 1" filename="package://schunk_svh_driver/description/meshes/h11.dae" />
+                    <mesh scale="${side*(1)} 1 1" filename="package://centauro/centauro_urdf/meshes/schunk_hand/h11.dae" />
                 </geometry>
             </visual>
@@ -156,5 +156,5 @@
                 <origin xyz="${side*(-0.0007)} 0 -0.01002" />
                 <geometry>
-                    <mesh scale="${side*(1)} 1 1" filename="package://schunk_svh_driver/description/meshes/h11.dae" />
+                    <mesh scale="${side*(1)} 1 1" filename="package://centauro/centauro_urdf/meshes/schunk_hand/h11.dae" />
                 </geometry>
             </collision>
@@ -203,5 +203,5 @@
                 <origin xyz="0 0 0.02442" />
                 <geometry>
-                    <mesh scale="1 ${side*(1)} 1" filename="package://schunk_svh_driver/description/meshes/d10.dae" />
+                    <mesh scale="1 ${side*(1)} 1" filename="package://centauro/centauro_urdf/meshes/schunk_hand/d10.dae" />
                 </geometry>
             </visual>
@@ -209,5 +209,5 @@
                 <origin xyz="0 0 0.02442" />
                 <geometry>
-                    <mesh scale="1 ${side*(1)} 1" filename="package://schunk_svh_driver/description/meshes/d10.dae" />
+                    <mesh scale="1 ${side*(1)} 1" filename="package://centauro/centauro_urdf/meshes/schunk_hand/d10.dae" />
                 </geometry>
             </collision-->
@@ -221,10 +221,10 @@
             <visual>
                 <geometry>
-                    <mesh scale="1 ${side*(1)} ${side*(1)}" filename="package://schunk_svh_driver/description/meshes/d11.dae" />
-                </geometry>
-            </visual>
-            <!--collision>
-                <geometry>
-                    <mesh scale="1 ${side*(1)} ${side*(1)}" filename="package://schunk_svh_driver/description/meshes/d11.dae" />
+                    <mesh scale="1 ${side*(1)} ${side*(1)}" filename="package://centauro/centauro_urdf/meshes/schunk_hand/d11.dae" />
+                </geometry>
+            </visual>
+            <!--collision>
+                <geometry>
+                    <mesh scale="1 ${side*(1)} ${side*(1)}" filename="package://centauro/centauro_urdf/meshes/schunk_hand/d11.dae" />
                 </geometry>
             </collision-->
@@ -235,10 +235,10 @@
             <visual>
                 <geometry>
-                    <mesh scale="1 ${side*(1)} ${side*(1)}" filename="package://schunk_svh_driver/description/meshes/d12.dae" />
-                </geometry>
-            </visual>
-            <!--collision>
-                <geometry>
-                    <mesh scale="1 ${side*(1)} ${side*(1)}" filename="package://schunk_svh_driver/description/meshes/d12.dae" />
+                    <mesh scale="1 ${side*(1)} ${side*(1)}" filename="package://centauro/centauro_urdf/meshes/schunk_hand/d12.dae" />
+                </geometry>
+            </visual>
+            <!--collision>
+                <geometry>
+                    <mesh scale="1 ${side*(1)} ${side*(1)}" filename="package://centauro/centauro_urdf/meshes/schunk_hand/d12.dae" />
                 </geometry>
             </collision-->
@@ -249,10 +249,10 @@
             <visual>
                 <geometry>
-                    <mesh scale="1 ${side*(1)} ${side*(1)}" filename="package://schunk_svh_driver/description/meshes/d13.dae" />
-                </geometry>
-            </visual>
-            <!--collision>
-                <geometry>
-                    <mesh scale="1 ${side*(1)} ${side*(1)}" filename="package://schunk_svh_driver/description/meshes/d13.dae" />
+                    <mesh scale="1 ${side*(1)} ${side*(1)}" filename="package://centauro/centauro_urdf/meshes/schunk_hand/d13.dae" />
+                </geometry>
+            </visual>
+            <!--collision>
+                <geometry>
+                    <mesh scale="1 ${side*(1)} ${side*(1)}" filename="package://centauro/centauro_urdf/meshes/schunk_hand/d13.dae" />
                 </geometry>
             </collision-->
@@ -267,5 +267,5 @@
                 <origin xyz="0 0 0.01321" />
                 <geometry>
-                    <mesh filename="package://schunk_svh_driver/description/meshes/f10.dae" />
+                    <mesh filename="package://centauro/centauro_urdf/meshes/schunk_hand/f10.dae" />
                 </geometry>
             </visual>
@@ -273,5 +273,5 @@
                 <origin xyz="0 0 0.01321" />
                 <geometry>
-                    <mesh filename="package://schunk_svh_driver/description/meshes/f10.dae" />
+                    <mesh filename="package://centauro/centauro_urdf/meshes/schunk_hand/f10.dae" />
                 </geometry>
             </collision-->
@@ -282,10 +282,10 @@
             <visual>
                 <geometry>
-                    <mesh filename="package://schunk_svh_driver/description/meshes/f11.dae" />
-                </geometry>
-            </visual>
-            <!--collision>
-                <geometry>
-                    <mesh filename="package://schunk_svh_driver/description/meshes/f11.dae" />
+                    <mesh filename="package://centauro/centauro_urdf/meshes/schunk_hand/f11.dae" />
+                </geometry>
+            </visual>
+            <!--collision>
+                <geometry>
+                    <mesh filename="package://centauro/centauro_urdf/meshes/schunk_hand/f11.dae" />
                 </geometry>
             </collision-->
@@ -298,5 +298,5 @@
             <visual>
                 <geometry>
-                    <mesh filename="package://schunk_svh_driver/description/meshes/f12.dae" />
+                    <mesh filename="package://centauro/centauro_urdf/meshes/schunk_hand/f12.dae" />
                 </geometry>
             </visual>
@@ -316,5 +316,5 @@
             <visual>
                 <geometry>
-                    <mesh filename="package://schunk_svh_driver/description/meshes/f13.dae" />
+                    <mesh filename="package://centauro/centauro_urdf/meshes/schunk_hand/f13.dae" />
                 </geometry>
             </visual>
@@ -335,5 +335,5 @@
                 <origin xyz="0 0 0.01321" />
                 <geometry>
-                    <mesh filename="package://schunk_svh_driver/description/meshes/f20.dae" />
+                    <mesh filename="package://centauro/centauro_urdf/meshes/schunk_hand/f20.dae" />
                 </geometry>
             </visual>
@@ -341,5 +341,5 @@
                 <origin xyz="0 0 0.01321" />
                 <geometry>
-                    <mesh filename="package://schunk_svh_driver/description/meshes/f20.dae" />
+                    <mesh filename="package://centauro/centauro_urdf/meshes/schunk_hand/f20.dae" />
                 </geometry>
             </collision-->
@@ -350,10 +350,10 @@
             <visual>
                 <geometry>
-                    <mesh filename="package://schunk_svh_driver/description/meshes/f21.dae" />
-                </geometry>
-            </visual>
-            <!--collision>
-                <geometry>
-                    <mesh filename="package://schunk_svh_driver/description/meshes/f21.dae" />
+                    <mesh filename="package://centauro/centauro_urdf/meshes/schunk_hand/f21.dae" />
+                </geometry>
+            </visual>
+            <!--collision>
+                <geometry>
+                    <mesh filename="package://centauro/centauro_urdf/meshes/schunk_hand/f21.dae" />
                 </geometry>
             </collision-->
@@ -367,5 +367,5 @@
             <visual>
                 <geometry>
-                    <mesh filename="package://schunk_svh_driver/description/meshes/f22.dae" />
+                    <mesh filename="package://centauro/centauro_urdf/meshes/schunk_hand/f22.dae" />
                 </geometry>
             </visual>
@@ -385,5 +385,5 @@
             <visual>
                 <geometry>
-                    <mesh filename="package://schunk_svh_driver/description/meshes/f23.dae" />
+                    <mesh filename="package://centauro/centauro_urdf/meshes/schunk_hand/f23.dae" />
                 </geometry>
             </visual>
@@ -404,5 +404,5 @@
                 <origin xyz="0 0 -0.01321" />
                 <geometry>
-                    <mesh filename="package://schunk_svh_driver/description/meshes/f30.dae" />
+                    <mesh filename="package://centauro/centauro_urdf/meshes/schunk_hand/f30.dae" />
                 </geometry>
             </visual>
@@ -410,5 +410,5 @@
                 <origin xyz="0 0 -0.01321" />
                 <geometry>
-                    <mesh filename="package://schunk_svh_driver/description/meshes/f30.dae" />
+                    <mesh filename="package://centauro/centauro_urdf/meshes/schunk_hand/f30.dae" />
                 </geometry>
             </collision-->
@@ -419,10 +419,10 @@
             <visual>
                 <geometry>
-                    <mesh filename="package://schunk_svh_driver/description/meshes/f31.dae" />
-                </geometry>
-            </visual>
-            <!--collision>
-                <geometry>
-                    <mesh filename="package://schunk_svh_driver/description/meshes/f31.dae" />
+                    <mesh filename="package://centauro/centauro_urdf/meshes/schunk_hand/f31.dae" />
+                </geometry>
+            </visual>
+            <!--collision>
+                <geometry>
+                    <mesh filename="package://centauro/centauro_urdf/meshes/schunk_hand/f31.dae" />
                 </geometry>
             </collision-->
@@ -436,5 +436,5 @@
             <visual>
                 <geometry>
-                    <mesh filename="package://schunk_svh_driver/description/meshes/f32.dae" />
+                    <mesh filename="package://centauro/centauro_urdf/meshes/schunk_hand/f32.dae" />
                 </geometry>
             </visual>
@@ -454,5 +454,5 @@
             <visual>
                 <geometry>
-                    <mesh filename="package://schunk_svh_driver/description/meshes/f33.dae" />
+                    <mesh filename="package://centauro/centauro_urdf/meshes/schunk_hand/f33.dae" />
                 </geometry>
             </visual>
@@ -473,5 +473,5 @@
                 <origin xyz="0 0 -0.01321" />
                 <geometry>
-                    <mesh filename="package://schunk_svh_driver/description/meshes/f40.dae" />
+                    <mesh filename="package://centauro/centauro_urdf/meshes/schunk_hand/f40.dae" />
                 </geometry>
             </visual>
@@ -479,5 +479,5 @@
                 <origin xyz="0 0 -0.01321" />
                 <geometry>
-                    <mesh filename="package://schunk_svh_driver/description/meshes/f40.dae" />
+                    <mesh filename="package://centauro/centauro_urdf/meshes/schunk_hand/f40.dae" />
                 </geometry>
             </collision-->
@@ -488,10 +488,10 @@
             <visual>
                 <geometry>
-                    <mesh filename="package://schunk_svh_driver/description/meshes/f41.dae" />
-                </geometry>
-            </visual>
-            <!--collision>
-                <geometry>
-                    <mesh filename="package://schunk_svh_driver/description/meshes/f41.dae" />
+                    <mesh filename="package://centauro/centauro_urdf/meshes/schunk_hand/f41.dae" />
+                </geometry>
+            </visual>
+            <!--collision>
+                <geometry>
+                    <mesh filename="package://centauro/centauro_urdf/meshes/schunk_hand/f41.dae" />
                 </geometry>
             </collision-->
@@ -505,5 +505,5 @@
             <visual>
                 <geometry>
-                    <mesh filename="package://schunk_svh_driver/description/meshes/f42.dae" />
+                    <mesh filename="package://centauro/centauro_urdf/meshes/schunk_hand/f42.dae" />
                 </geometry>
             </visual>
@@ -523,5 +523,5 @@
             <visual>
                 <geometry>
-                    <mesh filename="package://schunk_svh_driver/description/meshes/f43.dae" />
+                    <mesh filename="package://centauro/centauro_urdf/meshes/schunk_hand/f43.dae" />
                 </geometry>
             </visual>

Commit message: centauro_urdf: add simplified camera_link mesh

File: centauro/centauro_urdf/urdf/models/upper_body/end_effectors/schunk_hand/svh_gazebo.urdf.xacro (robot description, xacro)
@@ -99,5 +99,5 @@
                 <origin rpy="0 0 0" xyz="0 0 0" />
                 <geometry>
-                    <mesh filename="package://centauro/centauro_urdf/meshes/schunk_hand/camera_link.STL" />
+                    <mesh filename="package://centauro/centauro_urdf/meshes/schunk_hand/camera_link_simplified.stl" />
                 </geometry>
             </visual>
@@ -105,5 +105,5 @@
                <origin rpy="0 0 0" xyz="0 0 0" />
                 <geometry>
-					<mesh filename="package://centauro/centauro_urdf/meshes/schunk_hand/camera_link_convex.stl" /> <!-- FIXME: convex hull? -->
+					<mesh filename="package://centauro/centauro_urdf/meshes/schunk_hand/camera_link_convex.stl" />
                 </geometry>
             </collision>
