Commit message: modified orientation of soft_hand mesh file

File: centauro/centauro_urdf/urdf/models/upper_body/end_effectors/soft_hand/simplified.xacro (robot description, xacro)
@@ -4,5 +4,5 @@
    <origin xyz="0.0 0.0 -0.038"  rpy="0.0 0.0  ${PI/2+rot*PI/2}"/>
    <geometry>
-      <mesh filename="package://centauro/centauro_urdf/meshes/soft_hand_open.stl" scale="0.001 0.001 0.001" />
+      <mesh filename="package://centauro/centauro_urdf/meshes/soft_hand_open.stl" scale="${-rot*0.001} 0.001 0.001" />
    </geometry>
 </xacro:macro>
