Commit message: some local changes to centauro simulation models

File: centauro/centauro_urdf/urdf/models/upper_body/end_effectors/soft_hand/primitive.xacro (robot description, xacro)
@@ -4,5 +4,5 @@
    <origin xyz="0 0 0.0" rpy="0 0 0" />
    <geometry>
-      <box size="0.07 0.07 0.07" />
+      <box size="0.1 0.03 0.25" />
    </geometry>
 </xacro:macro>

Commit message: soft hand shape changed

File: centauro/centauro_urdf/urdf/models/upper_body/end_effectors/soft_hand/primitive.xacro (robot description, xacro)
@@ -4,5 +4,5 @@
    <origin xyz="0 0 0.0" rpy="0 0 0" />
    <geometry>
-      <box size="0.1 0.03 0.25" />
+      <box size="0.03 0.1 0.25" />
    </geometry>
 </xacro:macro>

Commit message: last commit before update framework

File: centauro/centauro_urdf/urdf/models/upper_body/end_effectors/soft_hand/primitive.xacro (robot description, xacro)
@@ -4,5 +4,5 @@
    <origin xyz="0 0 0.0" rpy="0 0 0" />
    <geometry>
-      <box size="0.03 0.1 0.25" />
+      <box size="0.03 0.08 0.12" />
    </geometry>
 </xacro:macro>
