Commit message: add gmapping

File: centauro/centauro_urdf/urdf/models/upper_body/head/primitive.xacro (robot description, xacro)
@@ -3,19 +3,19 @@
 <xacro:macro name="neck_yaw">
    <origin xyz="0.0 0 0.0"  rpy="0.0 0.0 0.0"/>
-<!--   <geometry>
+   <geometry>
       <box size="0.05 0.05 0.05"/>
-   </geometry> -->
+   </geometry>
 </xacro:macro>
 <xacro:macro name="neck_pitch">
    <origin xyz="0.0 0 0.0"  rpy="0.0 0.0 0.0"/>
-<!--   <geometry>
+   <geometry>
       <box size="0.05 0.05 0.05"/>
-   </geometry> -->
+   </geometry>
 </xacro:macro>
 <xacro:macro name="velodyne">
    <origin xyz="0.0 0 0.0"  rpy="0.0 0.0 0.0"/>
-<!--   <geometry>
+   <geometry>
       <box size="0.05 0.05 0.05"/>
-   </geometry> -->
+   </geometry>
 </xacro:macro>
 </robot>
