Commit message: Lower-body kinematic parameters and mesh files

File: centauro/centauro_urdf/kinematic_parameters/original.xacro (robot description, xacro)
@@ -7,24 +7,48 @@
 <xacro:property name="Pelvis_Ox" value=" 0.0 "/>
 <xacro:property name="Pelvis_Oy" value=" 0.0 "/>
-<xacro:property name="Pelvis_Oz" value=" 0.85 "/>
+<xacro:property name="Pelvis_Oz" value=" 0.759 "/>
 <!-- Origin -->
-<xacro:property name="Leg_1_Ox" value=" 0.30 "/>
-<xacro:property name="Leg_1_Oy" value=" 0.15 "/>
-<xacro:property name="Leg_1_Oz" value=" 0 "/>
-<xacro:property name="Leg_1_roll" value=" 0 "/>
-<xacro:property name="Leg_1_pitch" value=" 0 "/>
-<xacro:property name="Leg_1_yaw" value=" ${PI/2} "/>
+<xacro:property name="Leg_1_Ox" value=" 0.225 "/>
+<xacro:property name="Leg_1_Oy" value=" -0.125 "/>
+<xacro:property name="Leg_1_Oz" value=" 0.11 "/>
+<xacro:property name="Leg_1_roll" value=" 3.141592653589793 "/>
+<xacro:property name="Leg_1_pitch" value=" 0.0 "/>
+<xacro:property name="Leg_1_yaw" value=" -0.5070986986495499 "/>
 <!-- Origin -->
 <xacro:property name="Leg_2_Ox" value=" 0.000000 "/>
 <xacro:property name="Leg_2_Oy" value=" 0.000000 "/>
-<xacro:property name="Leg_2_Oz" value=" -0.2 "/>
+<xacro:property name="Leg_2_Oz" value=" 0.059 "/>
+<xacro:property name="Leg_2_roll" value=" 1.5707963267948966 "/>
+<xacro:property name="Leg_2_pitch" value=" 0.0 "/>
+<xacro:property name="Leg_2_yaw" value=" 2.6344939549402433 "/>
 <!-- Origin -->
 <xacro:property name="Leg_3_Ox" value=" 0.000000 "/>
-<xacro:property name="Leg_3_Oy" value=" 0.000000 "/>
-<xacro:property name="Leg_3_Oz" value=" -0.350000 "/>
+<xacro:property name="Leg_3_Oy" value=" 0.3 "/>
+<xacro:property name="Leg_3_Oz" value=" -0.0036 "/>
+<xacro:property name="Leg_3_roll" value=" 3.14159265358979 "/>
+<xacro:property name="Leg_3_pitch" value=" 0.0 "/>
+<xacro:property name="Leg_3_yaw" value=" 1.5707963267948966 "/>
+<xacro:property name="Ankle_1_Ox" value=" 0.2 "/>
+<xacro:property name="Ankle_1_Oy" value=" 0.0 "/>
+<xacro:property name="Ankle_1_Oz" value=" -0.10015 "/>
+<xacro:property name="Ankle_1_roll" value=" 3.141592653589793 "/>
+<xacro:property name="Ankle_1_pitch" value=" 0.0 "/>
+<xacro:property name="Ankle_1_yaw" value=" 0.0 "/>
+<xacro:property name="Ankle_2_Ox" value=" 0.0 "/>
+<xacro:property name="Ankle_2_Oy" value=" 0.0 "/>
+<xacro:property name="Ankle_2_Oz" value=" 0.0 "/>
+<xacro:property name="Ankle_2_roll" value=" 1.5707963267948966 "/>
+<xacro:property name="Ankle_2_pitch" value=" 0.0 "/>
+<xacro:property name="Ankle_2_yaw" value=" 1.5707963267948966 "/>
+<xacro:property name="Wheel_Ox" value=" 0.0 "/>
+<xacro:property name="Wheel_Oy" value=" 0.00085 "/>
+<xacro:property name="Wheel_Oz" value=" 0.235 "/>
+<xacro:property name="Wheel_roll" value=" 1.5707963267948966 "/>
+<xacro:property name="Wheel_pitch" value=" 0.0 "/>
+<xacro:property name="Wheel_yaw" value=" 0.0 "/>
 <!-- Origin -->
-<xacro:property name="Torso_2_Ox" value=" 0.3 "/>
+<xacro:property name="Torso_2_Ox" value=" 0.175 "/>
 <xacro:property name="Torso_2_Oy" value=" 0.0 "/>
-<xacro:property name="Torso_2_Oz" value=" 0.1 "/>
+<xacro:property name="Torso_2_Oz" value=" 0.36 "/>
 <!-- Origin -->
 <xacro:property name="Shoulder_1_Ox" value=" 0.04576 "/> <!-- for the other arm it was 0.0457475 -->

File: centauro/centauro_urdf/urdf/centauro.urdf.xacro (robot description, xacro)
@@ -33,9 +33,7 @@
       <visual>
          <xacro:visual_model.pelvis />
-         <material name="grey"/>
       </visual>
       <collision>
          <xacro:collision_model.pelvis />
-         <material name="grey"/>
       </collision>
    </link>
@@ -72,7 +70,7 @@
 <!-- legs -->
 <xacro:if value="${legs}">
-<xacro:centauro_leg leg_num="1" origin_x="1" origin_y="1">
+<xacro:centauro_leg leg_num="1" origin_x="1" origin_y="-1">
 </xacro:centauro_leg>
-<xacro:centauro_leg leg_num="2" origin_x="1" origin_y="-1">
+<xacro:centauro_leg leg_num="2" origin_x="1" origin_y="1">
 </xacro:centauro_leg>
 <xacro:centauro_leg leg_num="3" origin_x="-1" origin_y="-1">

File: centauro/centauro_urdf/urdf/centauro_arm.urdf.xacro (robot description, xacro)
@@ -13,9 +13,8 @@
       <visual>
          <xacro:visual_model.arm1 />
-         <material name="blue"/>
+         <material name="dark_grey"/>
       </visual>
       <collision>
          <xacro:collision_model.arm1 />
-         <material name="blue"/>
       </collision>
    </link>
@@ -30,9 +29,7 @@
       <visual>
          <xacro:visual_model.arm2 />
-         <material name="grey"/>
       </visual>
       <collision>
          <xacro:collision_model.arm2 />
-         <material name="grey"/>
       </collision>
    </link>
@@ -47,9 +44,8 @@
       <visual>
          <xacro:visual_model.arm3 />
-         <material name="blue"/>
+         <material name="dark_grey"/>
       </visual>
       <collision>
          <xacro:collision_model.arm3 />
-         <material name="blue"/>
       </collision>
    </link>
@@ -64,9 +60,7 @@
       <visual>
          <xacro:visual_model.arm4 />
-         <material name="grey"/>
       </visual>
       <collision>
          <xacro:collision_model.arm4 />
-         <material name="grey"/>
       </collision>
    </link>
@@ -81,9 +75,8 @@
       <visual>
          <xacro:visual_model.arm5 />
-         <material name="blue"/>
+         <material name="dark_grey"/>
       </visual>
       <collision>
          <xacro:collision_model.arm5 />
-         <material name="blue"/>
       </collision>
    </link>
@@ -98,9 +91,7 @@
       <visual>
          <xacro:visual_model.arm6 />
-         <material name="grey"/>
       </visual>
       <collision>
          <xacro:collision_model.arm6 />
-         <material name="grey"/>
       </collision>
    </link>
@@ -114,9 +105,8 @@
       <visual>
          <xacro:visual_model.arm7 />
-         <material name="blue"/>
+         <material name="dark_grey"/>
       </visual>
       <collision>
          <xacro:collision_model.arm7 />
-         <material name="blue"/>
       </collision>
    </link>

File: centauro/centauro_urdf/urdf/centauro_leg.urdf.xacro (robot description, xacro)
@@ -5,37 +5,16 @@
 <link name="hip1_${leg_num}">
 	<inertial>
-		<origin xyz="${Leg_1_x} ${Leg_1_y} ${Leg_1_z}"/> <!-- TODO -->
+		<origin xyz="${Leg_1_x} ${Leg_1_y} ${Leg_1_z}"/>
 		<mass value="${Leg_1_mass}"/> <!-- org: 2 -->
 		<inertia ixx="${Leg_1_xx}" ixy="${Leg_1_xy}" ixz="${Leg_1_xz}" iyy="${Leg_1_yy}" iyz="${Leg_1_yz}" izz="${Leg_1_zz}"/>
 		<!-- <inertia ixx="0.01" ixy="0.01" ixz="0.01" iyy="0.01" iyz="0.01" izz="0.01"/> -->
 	</inertial>
-	<visual>
-		<origin xyz="0 0 -0.1"/>
-		<geometry>
-			<box size="${link_visual} ${link_visual} 0.2"/> <!-- OK: from hip-yaw to pelvis (0.1) + from plevis to hip-pitch (0.1)-->
-		</geometry>
-		<material name="grey"/>
-	</visual>
-	<visual>
-		<origin xyz="0 0 0" rpy="0 0 0" />
-		<geometry>
-			<cylinder length="${motors_length}" radius="${motors_radius}"/>
-		</geometry>
-		<material name="grey"/>
-	</visual>
-	<collision>
-		<origin xyz="0 0 -0.1"/>
-		<geometry>
-			<box size="${link_visual} ${link_visual} ${0.2-collision}"/> <!-- OK: from hip-yaw to pelvis (0.1) + from plevis to hip-pitch (0.1)-->
-		</geometry>
-		<material name="grey"/>
-	</collision>
-	<!-- <collision>
-		<origin xyz="0 0 0" rpy="0 0 0" />
-		<geometry>
-			<cylinder length="${motors_length}" radius="${motors_radius}"/>
-		</geometry>
-		<material name="grey"/>
-	</collision> -->
+      <visual>
+         <xacro:visual_model.leg1 />
+         <material name="dark_grey"/>
+      </visual>
+      <collision>
+         <xacro:collision_model.leg1 />
+      </collision>
 </link>
 <link name="hip2_${leg_num}">
@@ -46,97 +25,68 @@
 		<!-- <inertia ixx="0.01" ixy="0.01" ixz="0.01" iyy="0.01" iyz="0.01" izz="0.01"/> -->
 	</inertial>
-	<visual>
-		<origin xyz="0 0 -${0.35/2}"/>
-		<geometry>
-			<box size="${link_visual} ${link_visual} 0.35"/> <!-- OK -->
-		</geometry>
-		<material name="blue"/>
-	</visual>
-	<visual>
-		<origin xyz="0 0 0" rpy="${PI/2} 0 0" />
-		<geometry>
-			<cylinder length="${motors_length}" radius="${motors_radius}"/>
-		</geometry>
-		<material name="blue"/>
-	</visual>
-	<collision>
-		<origin xyz="0 0 -${0.35/2}"/>
-		<geometry>
-			<box size="${link_visual} ${link_visual} ${0.35-collision}"/> <!-- OK -->
-		</geometry>
-		<material name="blue"/>
-	</collision>
-	<!-- <collision>
-		<origin xyz="0 0 0" rpy="${PI/2} 0 0" />
-		<geometry>
-			<cylinder length="${motors_length}" radius="${motors_radius}"/>
-		</geometry>
-		<material name="blue"/>
-	</collision> -->
+      <visual>
+         <xacro:visual_model.leg2 />
+      </visual>
+      <collision>
+         <xacro:collision_model.leg2 />
+      </collision>
 </link>
 <link name="knee_${leg_num}">
 	<inertial>
-		<origin xyz="${Leg_3_x} ${Leg_3_y} ${Leg_3_z}"/>	<!-- TODO -->
+		<origin xyz="${Leg_3_x} ${Leg_3_y} ${Leg_3_z}"/>
 		<mass value="${Leg_3_mass}"/>  <!-- org: 3.5, foot un modeled-->
 		<inertia ixx="${Leg_3_xx}" ixy="${Leg_3_xy}" ixz="${Leg_3_xz}" iyy="${Leg_3_yy}" iyz="${Leg_3_yz}" izz="${Leg_3_zz}"/>
 	<!--	<inertia ixx="0.01" ixy="0.01" ixz="0.01" iyy="0.01" iyz="0.01" izz="0.01"/>  -->
 	</inertial>
-	<visual>
-		<origin xyz="0 0 -${0.3/2-link_width/4}"/>
-		<geometry>
-			<box size="${link_visual} ${link_visual} ${0.3-link_width/2}"/> <!-- OK: foot un modeled-->
-		</geometry>
-		<material name="grey"/>
-	</visual>
-	<visual>
-		<origin xyz="0 0 0" rpy="${PI/2} 0 0" />
-		<geometry>
-			<cylinder length="${motors_length}" radius="${motors_radius}"/>
-		</geometry>
-		<material name="blue"/>
-	</visual>
-	<visual>
-		<origin xyz="0 0 -${0.3-link_width/2}" />
-		<geometry>
-			<sphere radius="${link_width/2}"/>
-		</geometry>
-		<material name="blue"/>
-	</visual>
-	<collision>
-		<origin xyz="0 0 -${0.3/2-link_width/4}"/>
-		<geometry>
-			<box size="${link_visual} ${link_visual} ${0.3-link_width/2-collision}"/> <!-- OK: foot un modeled-->
-		</geometry>
-		<material name="grey"/>
-	</collision>
-<!--	<collision>
-		<origin xyz="0 0 0" rpy="${PI/2} 0 0" />
-		<geometry>
-			<cylinder length="${motors_length}" radius="${motors_radius}"/>
-		</geometry>
-		<material name="blue"/>
-	</collision> -->
-	<collision>
-		<origin xyz="0 0 -${0.3-link_width/2}" />
-		<geometry>
-			<sphere radius="${link_width/2}"/>
-		</geometry>
-		<material name="blue"/>
-	</collision>
-</link>
-<!-- ftsensor -->
-<!--<link name="ft_foot_${leg_num}">
-  <inertial>
-    <mass value="0.001"/>
-    <origin xyz="0 0 0"/>
-    <inertia ixx="1.0E-6" ixy="0" ixz="0" iyy="1.0E-6" iyz="0" izz="1.0E-6"/>
-  </inertial>
-  <visual>
-      <origin rpy="0 0 0" xyz="0 0 0"/>
-      <geometry>
-        <box size="0.01 0.01 0.01"/>
-      </geometry>
-  </visual>
-</link>-->
+      <visual>
+         <xacro:visual_model.leg3 />
+         <material name="dark_grey"/>
+      </visual>
+      <collision>
+         <xacro:collision_model.leg3 />
+      </collision>
+</link>
+<link name="ankle1_${leg_num}">
+	<inertial>
+		<origin xyz="${Wrist_3_x} ${Wrist_3_y} ${Wrist_3_z}"/>
+		<mass value="${Wrist_3_mass}"/>  <!-- org: 3.5, foot un modeled-->
+		<inertia ixx="${Wrist_3_xx}" ixy="${Wrist_3_xy}" ixz="${Wrist_3_xz}" iyy="${Wrist_3_yy}" iyz="${Wrist_3_yz}" izz="${Wrist_3_zz}"/>
+	<!--	<inertia ixx="0.01" ixy="0.01" ixz="0.01" iyy="0.01" iyz="0.01" izz="0.01"/>  -->
+	</inertial>
+      <visual>
+         <xacro:visual_model.ankle1 />
+      </visual>
+      <collision>
+         <xacro:collision_model.ankle1 />
+      </collision>
+</link>
+<link name="ankle2_${leg_num}">
+	<inertial>
+		<origin xyz="${Wrist_3_x} ${Wrist_3_y} ${Wrist_3_z}"/>
+		<mass value="${Wrist_3_mass}"/>  <!-- org: 3.5, foot un modeled-->
+		<inertia ixx="${Wrist_3_xx}" ixy="${Wrist_3_xy}" ixz="${Wrist_3_xz}" iyy="${Wrist_3_yy}" iyz="${Wrist_3_yz}" izz="${Wrist_3_zz}"/>
+	</inertial>
+      <visual>
+         <xacro:visual_model.ankle2 />
+         <material name="dark_grey"/>
+      </visual>
+      <collision>
+         <xacro:collision_model.ankle2 />
+      </collision>
+</link>
+<link name="wheel_${leg_num}">
+	<inertial>
+		<origin xyz="${Wrist_3_x} ${Wrist_3_y} ${Wrist_3_z}"/>
+		<mass value="${Wrist_3_mass}"/>  <!-- org: 3.5, foot un modeled-->
+		<inertia ixx="${Wrist_3_xx}" ixy="${Wrist_3_xy}" ixz="${Wrist_3_xz}" iyy="${Wrist_3_yy}" iyz="${Wrist_3_yz}" izz="${Wrist_3_zz}"/>
+	</inertial>
+      <visual>
+         <xacro:visual_model.wheel />
+         <material name="black"/>
+      </visual>
+      <collision>
+         <xacro:collision_model.wheel />
+      </collision>
+</link>
 <!-- wheels -->
 <xacro:if	value="${wheels}">
@@ -153,5 +103,4 @@
 				<cylinder length="${wheel_length}" radius="${wheel_radius}"/>
 			</geometry>
-			<material name="grey"/>
 		</visual>
 		<collision>
@@ -173,5 +122,4 @@
 				<box size="${wheel_radius} 0.01 0.01"/>
 			</geometry>
-			<material name="blue"/>
 		</visual>
 	</link>
@@ -187,5 +135,4 @@
 				<cylinder length="${wheel_length}" radius="${wheel_radius}"/>
 			</geometry>
-			<material name="blue"/>
 		</visual>
 		<collision>
@@ -207,5 +154,4 @@
 				<box size="${wheel_radius} 0.01 0.01"/>
 			</geometry>
-			<material name="blue"/>
 		</visual>
 	</link>
@@ -246,21 +192,47 @@
 	<parent link="pelvis"/>
 	<child link="hip1_${leg_num}"/>
-	<origin xyz="${origin_x*Leg_1_Ox} ${origin_y*Leg_1_Oy} ${Leg_1_Oz}" rpy="${Leg_1_roll} ${Leg_1_pitch} ${Leg_1_yaw}"/>
-	<axis xyz="0 0 ${-origin_y}"/>
-        <limit lower="-2.09" upper="2.09" effort="147" velocity="6.5"/> <!-- TODO -->
+	<origin xyz="${origin_x*Leg_1_Ox} ${origin_y*Leg_1_Oy} ${Leg_1_Oz}" rpy="${Leg_1_roll} ${Leg_1_pitch} ${PI/2-origin_x*PI/2+origin_x*origin_y*Leg_1_yaw}"/>
+	<axis xyz="0 0 1"/>
+        <xacro:if value="${origin_y*origin_x == 1}">
+        <limit lower="-2.35619449" upper="0.78539816" effort="304" velocity="8.8"/>
+        </xacro:if>
+        <xacro:if value="${origin_y*origin_x == -1}">
+        <limit lower="-0.78539816" upper="2.35619449" effort="304" velocity="8.8"/>
+        </xacro:if>
 </joint>
 <joint name="hip_pitch_${leg_num}" type="revolute">
 	<parent link="hip1_${leg_num}"/>
 	<child link="hip2_${leg_num}"/>
-	<origin xyz="${Leg_2_Ox} ${Leg_2_Oy} ${Leg_2_Oz}"/>
-	<axis xyz="0 ${-origin_y} 0"/>
-        <limit lower="-3.14" upper="3.14" effort="330" velocity="6.5"/> <!-- TODO -->
+	<origin xyz="${Leg_2_Ox} ${Leg_2_Oy} ${Leg_2_Oz}" rpy="${Leg_2_roll} ${Leg_2_pitch} ${origin_x*origin_y*Leg_2_yaw-origin_x*origin_y*PI/2 + PI/2}"/>
+	<axis xyz="0 0 1"/>
+        <limit lower="-2.09439510" upper="2.09439510" effort="304" velocity="8.8"/>
 </joint>
 <joint name="knee_pitch_${leg_num}" type="revolute">
 	<parent link="hip2_${leg_num}"/>
 	<child link="knee_${leg_num}"/>
-	<origin xyz="${Leg_3_Ox} ${Leg_3_Oy} ${Leg_3_Oz}"/>
-	<axis xyz="0 ${-origin_y} 0"/>
-        <limit  lower="-3.14" upper="3.14" effort="330" velocity="6.5"/> <!-- TODO -->
+	<origin xyz="${Leg_3_Ox} ${Leg_3_Oy} ${Leg_3_Oz}" rpy="${Leg_3_roll} ${Leg_3_pitch} ${Leg_3_yaw}"/>
+	<axis xyz="0 0 1"/>
+        <limit  lower="-2.61799388" upper="2.61799388" effort="304" velocity="8.8"/>
+</joint>
+<joint name="ankle_pitch_${leg_num}" type="revolute">
+	<parent link="knee_${leg_num}"/>
+	<child link="ankle1_${leg_num}"/>
+	<origin xyz="${Ankle_1_Ox} ${Ankle_1_Oy} ${Ankle_1_Oz}" rpy="${Ankle_1_roll} ${Ankle_1_pitch} ${Ankle_1_yaw}"/>
+	<axis xyz="0 0 1"/>
+        <limit  lower="-2.61799388" upper="2.61799388" effort="147" velocity="8.1"/>
+</joint>
+<joint name="ankle_yaw_${leg_num}" type="revolute">
+	<parent link="ankle1_${leg_num}"/>
+	<child link="ankle2_${leg_num}"/>
+	<origin xyz="${Ankle_2_Ox} ${Ankle_2_Oy} ${Ankle_2_Oz}" rpy="${Ankle_2_roll} ${Ankle_2_pitch} ${Ankle_2_yaw}"/>
+	<axis xyz="0 0 1"/>
+        <limit  lower="-2.79252680" upper="2.79252680" effort="35" velocity="20.0"/>
+</joint>
+<joint name="j_wheel_${leg_num}" type="continuous">
+	<parent link="ankle2_${leg_num}"/>
+	<child link="wheel_${leg_num}"/>
+	<origin xyz="${Wheel_Ox} ${Wheel_Oy} ${Wheel_Oz}" rpy="${Wheel_roll} ${Wheel_pitch} ${Wheel_yaw}"/>
+	<axis xyz="0 0 1"/>
+        <limit  effort="35" velocity="20.0"/>
 </joint>
 <!--
@@ -276,4 +248,7 @@
 	<xacro:position_actuator joint="hip_pitch_${leg_num}" />
 	<xacro:position_actuator joint="knee_pitch_${leg_num}"  />
+	<xacro:position_actuator joint="ankle_pitch_${leg_num}"  />
+	<xacro:position_actuator joint="ankle_yaw_${leg_num}"  />
+	<xacro:position_actuator joint="j_wheel_${leg_num}"  />
 </xacro:if>
 <!-- /actuators -->

File: centauro/centauro_urdf/urdf/centauro_stick.urdf.xacro (robot description, xacro)
@@ -11,5 +11,5 @@
       <visual>
          <xacro:visual_model.stick />
-         <material name="grey"/>
+         <material name="dark_grey"/>
       </visual>
       <collision>

File: centauro/centauro_urdf/urdf/centauro_torso.urdf.xacro (robot description, xacro)
@@ -10,9 +10,7 @@
 	<visual>
                 <xacro:visual_model.torso />
-		<material name="grey"/>
 	</visual>
 	<collision>
                 <xacro:collision_model.torso />
-		<material name="grey"/>
 	</collision>
 </link>

File: centauro/centauro_urdf/urdf/models/model_config.xacro (robot description, xacro)
@@ -17,4 +17,5 @@
    </xacro:macro>
    <xacro:load_model path="upper_body" model="${model}"/>
+   <xacro:load_model path="lower_body" model="${model}"/>
    <xacro:if value="${END_EFFECTOR == 'soft_hand'}" >
       <xacro:load_model path="upper_body/end_effectors/soft_hand"  model="${model}"/>

File: centauro/centauro_urdf/urdf/models/upper_body/primitives.xacro (robot description, xacro)
@@ -1,10 +1,4 @@
 <?xml version="1.0" ?>
 <robot name="centauro" xmlns:xacro="http://www.ros.org/wiki/xacro">
-<xacro:macro name="pelvis" >
-   <origin xyz="0 0 0"  rpy="0.0 0.0 0.0"/>
-   <geometry>
-      <box size="0.70 0.40 0.20"/>
-   </geometry>
-</xacro:macro>
 <xacro:macro name="torso">
    <origin xyz="0.0 0 0.20"  rpy="0.0 0.0 0.0"/>

Commit message: Imu attached to pelvis. Works on xbotcore.

File: centauro/centauro_urdf/kinematic_parameters/original.xacro (robot description, xacro)
@@ -4,4 +4,11 @@
 <xacro:property name="cos_m10" value="0.984807753012208"/>
 <xacro:property name="sin_m10" value="-0.17364817766693033"/>
+<!-- Origin -->
+<xacro:property name="Imu_x" value=" 0.0 "/>
+<xacro:property name="Imu_y" value=" 0.0 "/>
+<xacro:property name="Imu_z" value=" 0.0 "/>
+<xacro:property name="Imu_r" value=" 0.0 "/>
+<xacro:property name="Imu_p" value=" 0.0 "/>
+<xacro:property name="Imu_yaw" value=" 0.0 "/>
 <!-- Origin -->
 <xacro:property name="Pelvis_Ox" value=" 0.0 "/>

File: centauro/centauro_urdf/urdf/centauro.urdf.xacro (robot description, xacro)
@@ -7,5 +7,5 @@
 <!-- other files -->
 <xacro:include filename="$(find centauro)/centauro_urdf/urdf/config.xacro"/>
- <xacro:if value="${GAZEBO}">
+<xacro:if value="${GAZEBO}">
   <xacro:include filename="$(find centauro_gazebo)/urdf/centauro.gazebo"/>
 </xacro:if>
@@ -38,4 +38,15 @@
       </collision>
    </link>
+    <link name="imu_link">
+        <inertial>
+            <mass value="0.0"/>
+            <inertia ixx="0.0" ixy="0.0" ixz="0.0" iyy="0.0" iyz="0.0" izz="0.0"/>
+        </inertial>
+    </link>
+    <joint name="imu_joint" type="fixed">
+        <parent link="pelvis"/>
+        <origin xyz="${Imu_x} ${Imu_y} ${Imu_z}" rpy="${Imu_r} ${Imu_p} ${Imu_yaw}"/>
+        <child link="imu_link"/>
+    </joint>
 </xacro:if>
 <xacro:unless value="${pelvis}">

Commit message: accepted changes

File: centauro/centauro_urdf/kinematic_parameters/original.xacro (robot description, xacro)
@@ -5,9 +5,9 @@
 <xacro:property name="sin_m10" value="-0.17364817766693033"/>
 <!-- Origin -->
-<xacro:property name="Imu_x" value=" 0.0 "/>
-<xacro:property name="Imu_y" value=" 0.0 "/>
-<xacro:property name="Imu_z" value=" 0.0 "/>
-<xacro:property name="Imu_r" value=" 0.0 "/>
-<xacro:property name="Imu_p" value=" 0.0 "/>
+<xacro:property name="Imu_Ox" value=" 0.0 "/>
+<xacro:property name="Imu_Oy" value=" 0.0 "/>
+<xacro:property name="Imu_Oz" value=" 0.0 "/>
+<xacro:property name="Imu_raw" value=" 0.0 "/>
+<xacro:property name="Imu_pitch" value=" 0.0 "/>
 <xacro:property name="Imu_yaw" value=" 0.0 "/>
 <!-- Origin -->

Commit message: accepted changes

File: centauro/centauro_urdf/kinematic_parameters/original.xacro (robot description, xacro)
@@ -4,4 +4,11 @@
 <xacro:property name="cos_m10" value="0.984807753012208"/>
 <xacro:property name="sin_m10" value="-0.17364817766693033"/>
+<!-- Origin -->
+<xacro:property name="Imu_Ox" value=" 0.0 "/>
+<xacro:property name="Imu_Oy" value=" 0.0 "/>
+<xacro:property name="Imu_Oz" value=" 0.0 "/>
+<xacro:property name="Imu_raw" value=" 0.0 "/>
+<xacro:property name="Imu_pitch" value=" 0.0 "/>
+<xacro:property name="Imu_yaw" value=" 0.0 "/>
 <!-- Origin -->
 <xacro:property name="Pelvis_Ox" value=" 0.0 "/>

File: centauro/centauro_urdf/urdf/centauro.urdf.xacro (robot description, xacro)
@@ -7,5 +7,5 @@
 <!-- other files -->
 <xacro:include filename="$(find centauro)/centauro_urdf/urdf/config.xacro"/>
- <xacro:if value="${GAZEBO}">
+<xacro:if value="${GAZEBO}">
   <xacro:include filename="$(find centauro_gazebo)/urdf/centauro.gazebo"/>
 </xacro:if>

File: centauro/centauro_urdf/urdf/config.xacro (robot description, xacro)
@@ -14,4 +14,5 @@
 <xacro:property name="ONE_ARM" value="$(arg ONE_ARM)"/>
 <xacro:property name="GAZEBO" value="$(arg GAZEBO)"/>
+<xacro:property name="CONTROLLER" value="$(arg CONTROLLER)"/>
 <xacro:property name="INERTIA_PARAM" value="$(arg INERTIA_PARAM)"/>
 <xacro:property name="KINEMATIC_PARAM" value="$(arg KINEMATIC_PARAM)"/>

Commit message: add Velodyne and laser rotator

File: centauro/centauro_urdf/kinematic_parameters/original.xacro (robot description, xacro)
@@ -172,5 +172,5 @@
 <xacro:property name="Kinect_pitch" value=" 0.0 "/>
 <xacro:property name="Kinect_yaw" value=" 0.0 "/>
-<xacro:property name="Velodyne_Ox" value=" 0.138 "/>
+<xacro:property name="Velodyne_Ox" value=" -0.138 "/>
 <xacro:property name="Velodyne_Oy" value=" 0.0 "/>
 <xacro:property name="Velodyne_Oz" value=" -0.033 "/>

File: centauro/centauro_urdf/urdf/centauro_head.urdf.xacro (robot description, xacro)
@@ -71,5 +71,5 @@
         </inertial>
 </link>
-<link name="velodyne">
+<link name="velodyne_mount">
 	<inertial>
 		<origin xyz="${Dummy_x} ${Dummy_y} ${Dummy_z}"/>
@@ -126,7 +126,11 @@
    <parent link="neck_3"/>
    <origin xyz="${Velodyne_Ox} ${Velodyne_Oy} ${Velodyne_Oz}" rpy="${Velodyne_roll} ${Velodyne_pitch} ${Velodyne_yaw}"/>
-   <child link="velodyne"/>
+   <child link="velodyne_mount"/>
 </joint>
 <!-- /sensors transformations -->
+<xacro:include filename="$(find velodyne_description)/urdf/VLP-16.urdf.xacro"/>
+<VLP-16 parent="velodyne_mount" name="velodyne" topic="/velodyne_points" hz="10" samples="440">
+	<origin xyz="0 0 0" rpy="-1.57079 0 -1.57079" />
+</VLP-16>
 <xacro:if value="${head_actuators}">
 <!-- torso actuators -->
