Commit message: correct ankle yaw orientation and update convex_hull and primitives for wheel

File: centauro/centauro_urdf/kinematic_parameters/original.xacro (robot description, xacro)
@@ -14,5 +14,5 @@
 <xacro:property name="Pelvis_Ox" value=" 0.0 "/>
 <xacro:property name="Pelvis_Oy" value=" 0.0 "/>
-<xacro:property name="Pelvis_Oz" value=" 0.92560000 "/>
+<xacro:property name="Pelvis_Oz" value=" 0.92795000 "/>
 <!-- Origin -->
 <xacro:property name="Neck_1_Ox" value=" 0.0 "/>
@@ -62,8 +62,8 @@
 <xacro:property name="Wheel_Ox" value=" 0.0 "/>
 <xacro:property name="Wheel_Oy" value=" 0.00085 "/>
-<xacro:property name="Wheel_Oz" value=" 0.235 "/>
+<xacro:property name="Wheel_Oz" value=" 0.237350 "/>
 <xacro:property name="Wheel_roll" value=" 1.5707963267948966 "/>
 <xacro:property name="Wheel_pitch" value=" 0.0 "/>
-<xacro:property name="Wheel_yaw" value=" 0.0 "/>
+<xacro:property name="Wheel_yaw" value=" 3.14159265359 "/>
 <!-- Origin -->
 <xacro:property name="Torso_2_Ox" value=" 0.200 "/>

File: centauro/centauro_urdf/urdf/models/lower_body/primitive.xacro (robot description, xacro)
@@ -40,5 +40,6 @@
 		<origin xyz="0 0 0" />
 		<geometry>
-			<cylinder radius="0.075" length="0.1"/>
+<!--			<cylinder radius="0.078" length="0.1"/> -->
+                        <sphere radius="0.078"/>
 		</geometry>
 </xacro:macro>

Commit message: update hip-yaw hip-pitch transformation and wheel radious

File: centauro/centauro_urdf/kinematic_parameters/original.xacro (robot description, xacro)
@@ -14,5 +14,5 @@
 <xacro:property name="Pelvis_Ox" value=" 0.0 "/>
 <xacro:property name="Pelvis_Oy" value=" 0.0 "/>
-<xacro:property name="Pelvis_Oz" value=" 0.92795000 "/>
+<xacro:property name="Pelvis_Oz" value=" 0.93445 "/>
 <!-- Origin -->
 <xacro:property name="Neck_1_Ox" value=" 0.0 "/>
@@ -33,12 +33,12 @@
 <xacro:property name="Leg_1_roll" value=" 3.141592653589793 "/>
 <xacro:property name="Leg_1_pitch" value=" 0.0 "/>
-<xacro:property name="Leg_1_yaw" value=" -0.5070986986495499 "/>
+<xacro:property name="Leg_1_yaw" value=" -0.461416123228 "/>
 <!-- Origin -->
 <xacro:property name="Leg_2_Ox" value=" 0.000000 "/>
 <xacro:property name="Leg_2_Oy" value=" 0.000000 "/>
-<xacro:property name="Leg_2_Oz" value=" 0.059 "/>
-<xacro:property name="Leg_2_roll" value=" 1.5707963267948966 "/>
+<xacro:property name="Leg_2_Oz" value=" 0.0625 "/>
+<xacro:property name="Leg_2_roll" value=" 1.57079632679 "/>
 <xacro:property name="Leg_2_pitch" value=" 0.0 "/>
-<xacro:property name="Leg_2_yaw" value=" 2.6344939549402433 "/>
+<xacro:property name="Leg_2_yaw" value=" 2.68017653036 "/>
 <!-- Origin -->
 <xacro:property name="Leg_3_Ox" value=" 0.000000 "/>

Commit message: update hip-yaw hip-pitch transformation and wheel radious

File: centauro/centauro_urdf/kinematic_parameters/original.xacro (robot description, xacro)
@@ -14,5 +14,5 @@
 <xacro:property name="Pelvis_Ox" value=" 0.0 "/>
 <xacro:property name="Pelvis_Oy" value=" 0.0 "/>
-<xacro:property name="Pelvis_Oz" value=" 0.92795000 "/>
+<xacro:property name="Pelvis_Oz" value=" 0.93445 "/>
 <!-- Origin -->
 <xacro:property name="Neck_1_Ox" value=" 0.0 "/>
@@ -33,12 +33,12 @@
 <xacro:property name="Leg_1_roll" value=" 3.141592653589793 "/>
 <xacro:property name="Leg_1_pitch" value=" 0.0 "/>
-<xacro:property name="Leg_1_yaw" value=" -0.5070986986495499 "/>
+<xacro:property name="Leg_1_yaw" value=" -0.461416123228 "/>
 <!-- Origin -->
 <xacro:property name="Leg_2_Ox" value=" 0.000000 "/>
 <xacro:property name="Leg_2_Oy" value=" 0.000000 "/>
-<xacro:property name="Leg_2_Oz" value=" 0.059 "/>
-<xacro:property name="Leg_2_roll" value=" 1.5707963267948966 "/>
+<xacro:property name="Leg_2_Oz" value=" 0.0625 "/>
+<xacro:property name="Leg_2_roll" value=" 1.57079632679 "/>
 <xacro:property name="Leg_2_pitch" value=" 0.0 "/>
-<xacro:property name="Leg_2_yaw" value=" 2.6344939549402433 "/>
+<xacro:property name="Leg_2_yaw" value=" 2.68017653036 "/>
 <!-- Origin -->
 <xacro:property name="Leg_3_Ox" value=" 0.000000 "/>

File: centauro/centauro_urdf/urdf/models/lower_body/primitive.xacro (robot description, xacro)
@@ -40,6 +40,5 @@
 		<origin xyz="0 0 0" />
 		<geometry>
-<!--			<cylinder radius="0.075" length="0.1"/> -->
-			<sphere radius="0.075"/>
+			<sphere radius="0.078"/>
 		</geometry>
 </xacro:macro>

Commit message: schunk hand and sensors calibration - merge with centauro branch
added:
	schunk hand end_effector
	schunk hand mesh files
	simplifed mesh files
	test_world
	velodyne and kinect kinematics

integrated with the centauro.xacro:
	centauro_torso_fixed.launch - add torso:=fixed argument
	centauro_right_arm.launch - add arms:=right and arms:=left options, remove one_arm argument

updated:
	README.md

not added:
	create_urdf - replicates create_urdf_srdf_sdf.sh script
	centauro_eef - is it necessary, or is it software dependend
	centauro.srdf - only collision merged
	controllers and ik config files - against our policy to keep a simulator software independent
	include velodyne - external package dependency

File: centauro/centauro_urdf/kinematic_parameters/original.xacro (robot description, xacro)
@@ -172,5 +172,5 @@
 <xacro:property name="Kinect_pitch" value=" 0.0 "/>
 <xacro:property name="Kinect_yaw" value=" 0.0 "/>
-<xacro:property name="Velodyne_Ox" value=" 0.138 "/>
+<xacro:property name="Velodyne_Ox" value=" -0.138 "/>
 <xacro:property name="Velodyne_Oy" value=" 0.0 "/>
 <xacro:property name="Velodyne_Oz" value=" -0.033 "/>

File: centauro/centauro_urdf/urdf/centauro_arm.urdf.xacro (robot description, xacro)
@@ -231,5 +231,12 @@
   <xacro:include filename="$(find centauro)/centauro_urdf/urdf/centauro_stick.urdf.xacro" />
 </xacro:if>
-<xacro:if value="${end_effector != 'stick' and end_effector != 'soft_hand' }" >
+<xacro:if value="${end_effector == 'schunk_hand'}" >
+	 <!-- schunk hand -->
+   <xacro:include filename="$(find centauro)/centauro_urdf/urdf/models/upper_body/end_effectors/schunk_hand/svh_gazebo.urdf.xacro" />
+   <xacro:svh parent="arm2_7" name="right_hand" side="1">
+        <origin xyz="0 0 -0.04"  rpy= "${PI} 0 ${PI/2}" />
+   </xacro:svh>
+</xacro:if>
+<xacro:if value="${end_effector != 'stick' and end_effector != 'soft_hand' and end_effector != 'schunk_hand'}" >
   <xacro:include filename="$(find centauro)/centauro_urdf/urdf/centauro_no_end_effector.urdf.xacro" />
 </xacro:if>

File: centauro/centauro_urdf/urdf/centauro_head.urdf.xacro (robot description, xacro)
@@ -71,5 +71,6 @@
         </inertial>
 </link>
-<link name="velodyne">
+<link name="kinect2_rgb_optical_frame" />
+<link name="velodyne_mount">
 	<inertial>
 		<origin xyz="${Dummy_x} ${Dummy_y} ${Dummy_z}"/>
@@ -123,8 +124,13 @@
    <child link="kinect"/>
 </joint>
+<joint name="j_kinect_optical_frame" type="fixed">
+	<parent link="kinect"/>
+	<child link="kinect2_rgb_optical_frame" />
+	<origin xyz="0.050 -0.110 -0.035" rpy=" -${PI/2} 0 -${PI/2}"/>
+</joint>
 <joint name="j_velodyne" type="fixed">
    <parent link="neck_3"/>
    <origin xyz="${Velodyne_Ox} ${Velodyne_Oy} ${Velodyne_Oz}" rpy="${Velodyne_roll} ${Velodyne_pitch} ${Velodyne_yaw}"/>
-   <child link="velodyne"/>
+   <child link="velodyne_mount"/>
 </joint>
 <!-- /sensors transformations -->

File: centauro/centauro_urdf/urdf/centauro_right_arm.urdf.xacro (robot description, xacro)
@@ -18,5 +18,5 @@
   <xacro:include filename="$(find centauro)/centauro_urdf/urdf/centauro_leg.urdf.xacro"/>
 </xacro:if>
-<xacro:if value="${arms}">
+<xacro:if value="${arm}">
   <xacro:include filename="$(find centauro)/centauro_urdf/urdf/centauro_arm.urdf.xacro"/>
 </xacro:if>
@@ -61,5 +61,5 @@
 <!-- torso -->
 <xacro:if value="${torso == 'true'}">
-   <xacro:include filename="$(find centauro)/centauro_urdf/urdf/centauro_torso.urdf.xacro"/>
+   <xacro:include filename="$(find centauro)/centauro_urdf/urdf/centauro_torso_fixed.urdf.xacro"/>
 </xacro:if>
 <xacro:if value="${head == 'true'}">
@@ -68,13 +68,13 @@
 <!-- /torso -->
 <!-- arms -->
-<xacro:if value="${left_arm == 'true'}">
-   <xacro:centauro_arm arm_num="1"  rot="1"  parent="torso_2" end_effector="${LEFT_END_EFFECTOR}">
-      <origin xyz="${Shoulder_1_Ox} ${Shoulder_1_Oy} ${Shoulder_1_Oz}" rpy="${Shoulder_1_roll} ${Shoulder_1_pitch} ${Shoulder_1_yaw}"/>
-   </xacro:centauro_arm>
-</xacro:if>
-<xacro:if value="${right_arm == 'true'}">
+<xacro:if value="${arms == 'true'}">
    <xacro:centauro_arm arm_num="2" rot="-1"  parent="torso_2" end_effector="${RIGHT_END_EFFECTOR}">
       <origin xyz="${Shoulder_1_Ox} ${-Shoulder_1_Oy} ${Shoulder_1_Oz}" rpy="${Shoulder_1_roll} ${Shoulder_1_pitch} ${-Shoulder_1_yaw}" />
    </xacro:centauro_arm>
+</xacro:if>
+<xacro:if value="${arm == 'true' and arms == 'false'}">
+        <xacro:centauro_arm arm_num="1"  rot="1" parent="world">
+           <origin xyz="${Shoulder_1_Ox + Pelvis_Ox + Torso_2_Ox} ${Shoulder_1_Oy + Pelvis_Oy + Torso_2_Oy} ${Shoulder_1_Oz + Pelvis_Oz + Torso_2_Oz}" rpy="${Shoulder_1_roll} ${Shoulder_1_pitch} ${Shoulder_1_yaw}"/>
+        </xacro:centauro_arm>
 </xacro:if>
 <!-- /arms -->

File: centauro/centauro_urdf/urdf/centauro_torso.urdf.xacro (robot description, xacro)
@@ -17,5 +17,5 @@
 <!-- /torso links -->
 <!-- torso joints -->
-<joint name="torso_yaw" type="revolute">
+<joint name="torso_yaw" type="${torso_joint}">
    <xacro:if value="${pelvis}">
       <parent link="pelvis"/>

File: centauro/centauro_urdf/urdf/config.xacro (robot description, xacro)
@@ -14,5 +14,4 @@
 <xacro:property name="WHEELS" value="$(arg WHEELS)"/>
 <xacro:property name="STATIC" value="$(arg STATIC)"/>
-<xacro:property name="ONE_ARM" value="$(arg ONE_ARM)"/>
 <xacro:property name="GAZEBO" value="$(arg GAZEBO)"/>
 <xacro:property name="MIDDLEWARE" value="$(arg MIDDLEWARE)"/>
@@ -32,21 +31,23 @@
 <xacro:property name="MASS" value="$(arg MASS)"/>
 <!-- dependend arguments -->
-<xacro:property name="arms" value="${'true' if ('false' not in [TORSO, ARMS] and 'false' in [ONE_ARM]) else 'false'}"/>
-<xacro:property name="legs" value="${'true' if ('false' not in [LEGS] and 'true' not in [ONE_ARM]) else 'false'}"/>
-<xacro:property name="torso" value="${'true' if ('false' in [ONE_ARM] and 'true' in [TORSO]) else 'false'}"/>
+<xacro:property name="torso" value="${'true' if ('true' in [TORSO] or 'fixed' in [TORSO]) else 'false'}"/>
 <xacro:property name="head" value="${'true' if ('false' not in [torso, HEAD]) else 'false'}"/>
-<xacro:property name="arm" value= "${'true' if ('true' in [arms, ONE_ARM]) else 'false'}" />
+<xacro:property name="arms" value="${'true' if ('false' not in [TORSO, ARMS]) else 'false'}"/>
+<xacro:property name="left_arm" value= "${'true' if ('true' in [arms] and ('true' in [ARMS] or 'left' in [ARMS])) else 'false'}" />
+<xacro:property name="right_arm" value= "${'true' if ('true' in [arms] and ('true' in [ARMS] or 'right' in [ARMS])) else 'false'}" />
+<xacro:property name="legs" value="${'true' if ('false' not in [LEGS]) else 'false'}"/>
 <xacro:property name="pelvis" value= "${'true' if ('true' in [legs]) else 'false'}" />
 <xacro:property name="wheels" value="${'true' if ('false' not in [WHEELS, legs]) else 'false'}"/>
-<xacro:property name="static" value="${'true' if ('true' in [STATIC, ONE_ARM] or 'false' in [legs, LEG_ACTUATORS]) else 'false'}"/>
+<xacro:property name="static" value="${'true' if ('true' in [STATIC] or 'false' in [legs, LEG_ACTUATORS]) else 'false'}"/>
 <xacro:property name="reference" value="${'fixed' if (static == 'true') else 'floating'}" />
+<xacro:property name="torso_joint" value="${'fixed' if ('fixed' in [TORSO]) else 'revolute'}"/>
 <!-- ACTUATION -->
 <xacro:property name="torso_actuators" value="${'true' if ('false' not in [TORSO_ACTUATORS, TORSO]) else 'false'}"/>
-<xacro:property name="arm_actuators" value="${'true' if ('false' not in [ARM_ACTUATORS, TORSO_ACTUATORS, arm]) else 'false'}"/>
+<xacro:property name="arm_actuators" value="${'true' if ('false' not in [ARM_ACTUATORS, TORSO_ACTUATORS, arms]) else 'false'}"/>
 <xacro:property name="leg_actuators" value="${'true' if ('false' not in [LEG_ACTUATORS, legs]) else 'false'}"/>
 <xacro:property name="head_actuators" value="${'true' if ('false' not in [HEAD_ACTUATORS, head]) else 'false'}"/>
 <xacro:property name="torso_actuators" value="${'true' if ('false' not in [TORSO_ACTUATORS, TORSO]) else 'false'}"/>
 <!-- SENSORS -->
-<xacro:property name="arm_sensors" value="${'true' if ('false' not in [ARM_SENSORS, arm]) else 'false'}"/>
+<xacro:property name="arm_sensors" value="${'true' if ('false' not in [ARM_SENSORS, arms]) else 'false'}"/>
 <xacro:property name="leg_sensors" value="${'true' if ('false' not in [LEG_SENSORS, legs]) else 'false'}"/>
 <xacro:property name="ft_sensors" value="${'true' if ('false' not in [FT_SENSORS]) else 'false'}"/>

Commit message: centauro_urdf: IMU transform

File: centauro/centauro_urdf/kinematic_parameters/original.xacro (robot description, xacro)
@@ -5,7 +5,7 @@
 <xacro:property name="sin_m10" value="-0.17364817766693033"/>
 <!-- Origin -->
-<xacro:property name="Imu_Ox" value=" 0.0 "/>
-<xacro:property name="Imu_Oy" value=" 0.0 "/>
-<xacro:property name="Imu_Oz" value=" 0.0 "/>
+<xacro:property name="Imu_Ox" value="${0.26 - (0.0254 * (1.08 - 0.62))}"/>
+<xacro:property name="Imu_Oy" value="0.0"/>
+<xacro:property name="Imu_Oz" value="0.015"/>
 <xacro:property name="Imu_raw" value=" 0.0 "/>
 <xacro:property name="Imu_pitch" value=" 0.0 "/>

Commit message: Add kinect and velodyne support

File: centauro/centauro_urdf/kinematic_parameters/original.xacro (robot description, xacro)
@@ -4,8 +4,8 @@
 <xacro:property name="cos_m10" value="0.984807753012208"/>
 <xacro:property name="sin_m10" value="-0.17364817766693033"/>
-<!-- Origin -->
-<xacro:property name="Imu_Ox" value=" 0.0 "/>
+<!-- Origin N-->
+<xacro:property name="Imu_Ox" value="${0.26 - (0.0254 * (1.08 - 0.62))}"/>
 <xacro:property name="Imu_Oy" value=" 0.0 "/>
-<xacro:property name="Imu_Oz" value=" 0.0 "/>
+<xacro:property name="Imu_Oz" value="0.015"/>
 <xacro:property name="Imu_raw" value=" 0.0 "/>
 <xacro:property name="Imu_pitch" value=" 0.0 "/>

File: centauro/centauro_urdf/urdf/centauro_head.urdf.xacro (robot description, xacro)
@@ -1,4 +1,5 @@
 <?xml version="1.0"?>
 <robot xmlns:xacro="http://www.ros.org/wiki/xacro">
+<!--<xacro:include filename="$(find centauro)/centauro_urdf/urdf/sensors/kinect2.urdf.xacro"/> -->
 <!-- head links -->
 <link name="neck_1">
@@ -71,5 +72,4 @@
         </inertial>
 </link>
-<link name="kinect2_rgb_optical_frame" />
 <link name="velodyne_mount">
 	<inertial>
@@ -87,4 +87,5 @@
    <axis xyz="0 0 1"/>
    <limit lower="-0.78539816" upper="0.78539816" effort="35" velocity="5.7"/> <!-- TODO -->
+   <dynamics friction="${friction}" />
 </joint>
 <joint name="neck_pitch" type="revolute">
@@ -94,4 +95,5 @@
    <axis xyz="0 1 0"/>
    <limit lower="-0.34906585" upper="0.78539816" effort="35" velocity="5.7"/> <!-- TODO -->
+   <dynamics friction="${friction}" />
 </joint>
 <joint name="neck_velodyne" type="continuous">
@@ -101,6 +103,14 @@
    <axis xyz="0 0 1"/>
    <limit effort="35" velocity="5.7"/> <!-- TODO -->
+   <dynamics friction="${friction}" damping="${damping_arms}" />
 </joint>
 <!-- /head joints -->
+<xacro:if value="${head_actuators}">
+   <!-- head actuators -->
+   <xacro:position_actuator joint="neck_yaw" />
+   <xacro:position_actuator joint="neck_pitch" />
+   <xacro:position_actuator joint="neck_velodyne" />
+   <!-- /head actuators -->
+</xacro:if>
 <!-- sensors transformations  -->
 <joint name="j_camera_central" type="fixed">
@@ -124,8 +134,15 @@
    <child link="kinect"/>
 </joint>
+<link name="kinect2_rgb_frame" />
+<joint name="j_kinect2_rgb_frame" type="fixed">
+	<parent link="kinect" />
+	<child link="kinect2_rgb_frame" />
+	<origin xyz="0.050 -0.110 -0.035" />
+</joint>
+<link name="kinect2_rgb_optical_frame" />
 <joint name="j_kinect_optical_frame" type="fixed">
-	<parent link="kinect"/>
+	<parent link="kinect2_rgb_frame"/>
 	<child link="kinect2_rgb_optical_frame" />
-	<origin xyz="0.050 -0.110 -0.035" rpy=" -${PI/2} 0 -${PI/2}"/>
+	<origin rpy=" -${PI/2} 0 -${PI/2}"/>
 </joint>
 <joint name="j_velodyne" type="fixed">
@@ -134,11 +151,11 @@
    <child link="velodyne_mount"/>
 </joint>
+<!-- Kinect simulation -->
 <!-- /sensors transformations -->
-<xacro:if value="${head_actuators}">
-<!-- torso actuators -->
-<xacro:position_actuator joint="neck_yaw" />
-<xacro:position_actuator joint="neck_pitch" />
-<xacro:position_actuator joint="neck_velodyne" />
-<!-- /torso actuators -->
-</xacro:if>
+<link name="velodyne_calib" />
+<joint name="velodyne_calib" type="fixed">
+   <parent link="neck_3"/>
+  <origin xyz="-0.175768 0 -0.034219" rpy="-1.57772 0.0128311 1.57073"/>
+   <child link="velodyne_calib"/>
+</joint>
 </robot>

File: centauro/centauro_urdf/urdf/config.xacro (robot description, xacro)
@@ -29,4 +29,6 @@
 <xacro:property name="BUMBERS" value="$(arg BUMBERS)"/>
 <xacro:property name="IMU" value="$(arg IMU)"/>
+<xacro:property name="KINECT" value="$(arg KINECT)"/>
+<xacro:property name="VELODYNE" value="$(arg VELODYNE)"/>
 <xacro:property name="MASS" value="$(arg MASS)"/>
 <!-- dependend arguments -->
@@ -58,4 +60,6 @@
 <xacro:property name="bumbers" value="${'true' if ('false' not in [BUMBERS]) else 'false'}"/>
 <xacro:property name="imu" value="${'true' if ('false' not in [IMU, pelvis]) else 'false'}"/>
+<xacro:property name="kinect" value="${'true' if ('false' not in [KINECT, head]) else 'false'}"/>
+<xacro:property name="velodyne" value="${'true' if ('false' not in [VELODYNE, head]) else 'false'}"/>
 <!-- LOAD PARAMETERS -->
 <xacro:property name="package" value="$(find centauro)"/>
@@ -64,3 +68,8 @@
 <xacro:property name="kinematic_parameters_file" value="${package + '/centauro_urdf/kinematic_parameters/' + KINEMATIC_PARAM + '.xacro'}"/>
 <xacro:property name="middleware" value="${MIDDLEWARE}"/>
+<xacro:property name="friction" value="10.0" />
+<xacro:property name="damping_legs" value="1.0" />
+<xacro:property name="damping_arms" value="0.2" />
+<xacro:property name="friction_schunk" value="2.0" />
+<xacro:property name="damping_schunk" value="0.0" />
 </robot>

File: centauro_gazebo/sensors/config.xacro (robot description, xacro)
@@ -2,5 +2,5 @@
 <robot  xmlns:xacro="http://www.ros.org/wiki/xacro">
 <xacro:include filename="$(find centauro)/centauro_urdf/urdf/config.xacro"/>
-   <xacro:macro name="load_model" params="middleware sensor arm_sensors leg_sensors">
+   <xacro:macro name="load_model" params="middleware sensor arm_sensors leg_sensors head_sensors">
       <xacro:include filename="$(find centauro_gazebo)/sensors/${middleware}/${sensor}/plugin.xacro"/>
       <xacro:if value="${arm_sensors}">
@@ -10,14 +10,23 @@
          <xacro:include filename="$(find centauro_gazebo)/sensors/${middleware}/${sensor}/load/legs.xacro"/>
       </xacro:if>
+      <xacro:if value="${head_sensors}" >
+         <xacro:include filename="$(find centauro_gazebo)/sensors/${middleware}/${sensor}/load/head.xacro"/>
+      </xacro:if>
    </xacro:macro>
 <!-- Load all controllers macros -->
 <xacro:if value="${ft_sensors}">
-        <xacro:load_model middleware="${middleware}" sensor="ft_sensor" arm_sensors="${arm_sensors}" leg_sensors="${leg_sensors}"/>
+        <xacro:load_model middleware="${middleware}" sensor="ft_sensor" arm_sensors="${arm_sensors}" leg_sensors="${leg_sensors}" head_sensors="false"/>
 </xacro:if>
 <xacro:if value="${bumbers}">
-        <xacro:load_model middleware="${middleware}" sensor="bumber" arm_sensors="${arm_sensors}" leg_sensors="${leg_sensors}"/>
+        <xacro:load_model middleware="${middleware}" sensor="bumber" arm_sensors="${arm_sensors}" leg_sensors="${leg_sensors}" head_sensors="false"/>
 </xacro:if>
 <xacro:if value="${imu}">
-        <xacro:load_model middleware="${middleware}" sensor="imu" arm_sensors="${arm_sensors}" leg_sensors="${leg_sensors}"/>
+        <xacro:load_model middleware="${middleware}" sensor="imu" arm_sensors="${arm_sensors}" leg_sensors="${leg_sensors}" head_sensors="false"/>
+</xacro:if>
+<xacro:if value="${kinect}">
+        <xacro:load_model middleware="${middleware}" sensor="kinect" arm_sensors="false" leg_sensors="false" head_sensors="${head}"/>
+</xacro:if>
+<xacro:if value="${velodyne}">
+        <xacro:load_model middleware="${middleware}" sensor="velodyne" arm_sensors="false" leg_sensors="false" head_sensors="${head}"/>
 </xacro:if>
 </robot>

File: centauro_gazebo/sensors/ros_control/bumber/plugin.xacro (robot description, xacro)
@@ -3,9 +3,9 @@
 <xacro:macro name="contact_sensor" params="link robot">
 <gazebo reference="${link}">
-  <sensor name="${link}_contact_sensor_1" type="contact">
+  <sensor name="${link}_contact_sensor" type="contact">
     <always_on>true</always_on>
     <update_rate>1000.0</update_rate>
     <contact>
-      <collision>${link}_collision_1</collision>
+      <collision>${link}_collision</collision>
     </contact>
     <plugin name="${link}_bumper" filename="libgazebo_ros_bumper.so">

Commit message: update lidar kinematics

File: centauro/centauro_urdf/kinematic_parameters/original.xacro (robot description, xacro)
@@ -187,9 +187,9 @@
 <xacro:property name="Kinect_pitch" value=" 0.0 "/>
 <xacro:property name="Kinect_yaw" value=" 0.0 "/>
-<xacro:property name="Velodyne_Ox" value=" -0.138 "/>
-<xacro:property name="Velodyne_Oy" value=" 0.0 "/>
-<xacro:property name="Velodyne_Oz" value=" -0.033 "/>
-<xacro:property name="Velodyne_roll" value=" 0.0 "/>
+<xacro:property name="Velodyne_Ox" value=" 0.0283656 "/>
+<xacro:property name="Velodyne_Oy" value=" -0.00976704 "/>
+<xacro:property name="Velodyne_Oz" value=" 0.047 "/>
+<xacro:property name="Velodyne_roll" value=" 1.57079632679 "/>
 <xacro:property name="Velodyne_pitch" value=" 0.0 "/>
-<xacro:property name="Velodyne_yaw" value=" -3.14159265359 "/>
+<xacro:property name="Velodyne_yaw" value=" -0.331612273666 "/>
 </robot>

File: centauro/centauro_urdf/urdf/models/upper_body/head/mesh.xacro (robot description, xacro)
@@ -16,5 +16,5 @@
   <origin xyz="0.0 0 0.0"  rpy="0.0 0.0 0.0"/>
   <geometry>
-    <mesh filename="package://centauro/centauro_urdf/meshes/velodyne.stl" scale="0.001 0.001 0.001" />
+    <mesh filename="package://centauro/centauro_urdf/meshes/simplified/mesh_lidar.stl" scale="0.001 0.001 0.001" />
   </geometry>
 </xacro:macro>

File: centauro/centauro_urdf/urdf/models/upper_body/head/simplified.xacro (robot description, xacro)
@@ -16,5 +16,5 @@
   <origin xyz="0.0 0 0.0"  rpy="0.0 0.0 0.0"/>
   <geometry>
-    <mesh filename="package://centauro/centauro_urdf/meshes/simplified/velodyne.stl" scale="0.001 0.001 0.001" />
+    <mesh filename="package://centauro/centauro_urdf/meshes/simplified/mesh_lidar.stl" scale="0.001 0.001 0.001" />
   </geometry>
 </xacro:macro>
