Commit message: Integrate new upper body  * kinematics  * dynamic parameters  * mesh files  * joint limits  * joint direction conventions

File: centauro/centauro_urdf/limits/default.xacro (robot description, xacro)
@@ -14,17 +14,31 @@
 <xacro:property name="torso_yaw_lower" value="-2.618"/>
 <xacro:property name="torso_yaw_upper" value="2.618"/>
-<xacro:property name="j_arm_1_lower" value="${[-3.3480, -1.6102]}"/>
-<xacro:property name="j_arm_2_lower" value="${[-3.4200,  0.0578]}"/>
-<xacro:property name="j_arm_3_lower" value="${[-2.5556, -2.5426]}"/>
-<xacro:property name="j_arm_4_lower" value="${[-2.4636, -0.2796]}"/>
-<xacro:property name="j_arm_5_lower" value="${[-2.5406, -2.5626]}"/>
-<xacro:property name="j_arm_6_lower" value="${[-1.5096, -1.4726]}"/>
-<xacro:property name="j_arm_7_lower" value="${[-2.5376, -3.0908]}"/>
-<xacro:property name="j_arm_1_upper" value="${[ 1.5780, 3.3138]}"/>
-<xacro:property name="j_arm_2_upper" value="${[-0.0560, 3.4288]}"/>
-<xacro:property name="j_arm_3_upper" value="${[ 2.5424, 2.5524]}"/>
-<xacro:property name="j_arm_4_upper" value="${[ 0.2804, 2.4564]}"/>
-<xacro:property name="j_arm_5_upper" value="${[ 2.5534, 2.5464]}"/>
-<xacro:property name="j_arm_6_upper" value="${[ 1.5044, 1.5364]}"/>
-<xacro:property name="j_arm_7_upper" value="${[ 2.5554, 2.0114]}"/>
+<xacro:property name="j_arm_1_lower" value="${[-3.312, -3.3458]}"/>
+<xacro:property name="j_arm_2_lower" value="${ [0.020, -3.4258]}"/>
+<xacro:property name="j_arm_3_lower" value="${[-2.552, -2.5614]}"/>
+<xacro:property name="j_arm_4_lower" value="${[-2.465, -2.4794]}"/>
+<xacro:property name="j_arm_5_lower" value="${[-2.569, -2.5394]}"/>
+<xacro:property name="j_arm_6_lower" value="${[-1.529, -1.5154]}"/>
+<xacro:property name="j_arm_7_lower" value="${[-2.565, -2.5554]}"/>
+<xacro:property name="j_arm_1_upper" value="${[1.615, 1.6012]}"/>
+<xacro:property name="j_arm_2_upper" value="${[3.431, -0.0138]}"/>
+<xacro:property name="j_arm_3_upper" value="${[2.566, 2.5606]}"/>
+<xacro:property name="j_arm_4_upper" value="${[0.280, 0.2886]}"/>
+<xacro:property name="j_arm_5_upper" value="${[2.562, 2.5546]}"/>
+<xacro:property name="j_arm_6_upper" value="${[1.509, 1.5156]}"/>
+<xacro:property name="j_arm_7_upper" value="${[2.569, 2.5686]}"/>
+<xacro:property name="j_arm_1_velocity" value="${[3.86, 3.86 ]}"/>
+<xacro:property name="j_arm_2_velocity" value="${[3.86, 3.86 ]}"/>
+<xacro:property name="j_arm_3_velocity" value="${[6.06, 6.06 ]}"/>
+<xacro:property name="j_arm_4_velocity" value="${[6.06, 6.06 ]}"/>
+<xacro:property name="j_arm_5_velocity" value="${[11.72, 11.72 ]}"/>
+<xacro:property name="j_arm_6_velocity" value="${[11.72, 11.72 ]}"/>
+<xacro:property name="j_arm_7_velocity" value="${[20.35, 20.35 ]}"/>
+<xacro:property name="j_arm_1_torque" value="${[147.00, 147.00 ]}"/>
+<xacro:property name="j_arm_2_torque" value="${[147.00, 147.00 ]}"/>
+<xacro:property name="j_arm_3_torque" value="${[147.00, 147.00 ]}"/>
+<xacro:property name="j_arm_4_torque" value="${[147.00, 147.00 ]}"/>
+<xacro:property name="j_arm_5_torque" value="${[55.00, 55.00 ]}"/>
+<xacro:property name="j_arm_6_torque" value="${[55.00, 55.00 ]}"/>
+<xacro:property name="j_arm_7_torque" value="${[28.32, 28.32 ]}"/>
 </robot>

File: centauro/centauro_urdf/urdf/models/upper_body/mesh.xacro (robot description, xacro)
@@ -10,11 +10,11 @@
    <origin xyz="0.0 0.0 0.0"  rpy="0.0 0.0 0.0"/>
    <geometry>
-      <mesh filename="package://centauro/centauro_urdf/meshes/link2.stl" scale="0.001 ${-rot*0.001} 0.001" />
+      <mesh filename="package://centauro/centauro_urdf/meshes/simplified/ShoulderPitch.STL" scale="0.001 ${-rot*0.001} 0.001" />
    </geometry>
-   </xacro:macro>
+</xacro:macro>
 <xacro:macro name="arm2">
    <origin xyz="0.0 0.0 0.0"  rpy="0.0 0.0 0.0"/>
    <geometry>
-      <mesh filename="package://centauro/centauro_urdf/meshes/link3.stl" scale="0.001 ${-rot*0.001} 0.001" />
+      <mesh filename="package://centauro/centauro_urdf/meshes/simplified/ShoulderRoll.STL" scale="0.001 ${-rot*0.001} 0.001" />
    </geometry>
 </xacro:macro>
@@ -22,5 +22,5 @@
    <origin xyz="0.0 0.0 0.0"  rpy="0.0 0.0 0.0"/>
    <geometry>
-      <mesh filename="package://centauro/centauro_urdf/meshes/link4.stl" scale="0.001 ${-rot*0.001} 0.001" />
+      <mesh filename="package://centauro/centauro_urdf/meshes/simplified/ShoulderYaw.STL" scale="0.001 ${-rot*0.001} 0.001" />
    </geometry>
 </xacro:macro>
@@ -28,5 +28,5 @@
    <origin xyz="0.0 0.0 0.0"  rpy="0.0 0.0 0.0"/>
    <geometry>
-      <mesh filename="package://centauro/centauro_urdf/meshes/link5.stl" scale="0.001 ${-rot*0.001} 0.001" />
+      <mesh filename="package://centauro/centauro_urdf/meshes/simplified/Elbow.STL" scale="0.001 ${-rot*0.001} 0.001" />
    </geometry>
 </xacro:macro>
@@ -34,5 +34,5 @@
    <origin xyz="0.0 0.0 0.0"  rpy="0.0 0.0 0.0"/>
    <geometry>
-      <mesh filename="package://centauro/centauro_urdf/meshes/link6.stl" scale="0.001 ${-rot*0.001} 0.001" />
+      <mesh filename="package://centauro/centauro_urdf/meshes/simplified/Forearm.STL" scale="0.001 ${-rot*0.001} 0.001" />
    </geometry>
 </xacro:macro>
@@ -40,5 +40,5 @@
    <origin xyz="0.0 0.0 0.0"  rpy="0.0 0.0 0.0"/>
    <geometry>
-      <mesh filename="package://centauro/centauro_urdf/meshes/link7.stl" scale="0.001 ${-rot*0.001} 0.001" />
+      <mesh filename="package://centauro/centauro_urdf/meshes/simplified/ForearmPitch.STL" scale="0.001 ${-rot*0.001} 0.001" />
    </geometry>
 </xacro:macro>
@@ -46,5 +46,11 @@
    <origin xyz="0.0 0.0 0.0"  rpy="0.0 0.0 0.0"/>
    <geometry>
-      <mesh filename="package://centauro/centauro_urdf/meshes/link8.stl" scale="0.001 ${-rot*0.001} 0.001" />
+      <mesh filename="package://centauro/centauro_urdf/meshes/simplified/ForearmYaw.STL" scale="0.001 ${-rot*0.001} 0.001" />
+   </geometry>
+</xacro:macro>
+<xacro:macro name="arm8">
+   <origin xyz="0.0 0.0 0.0"  rpy="${PI} 0.0 0.0"/>
+   <geometry>
+      <mesh filename="package://centauro/centauro_urdf/meshes/simplified/Wrist.STL" scale="0.001 ${-rot*0.001} 0.001" />
    </geometry>
 </xacro:macro>

File: centauro/centauro_urdf/urdf/models/upper_body/simplified.xacro (robot description, xacro)
@@ -10,5 +10,5 @@
    <origin xyz="0.0 0.0 0.0"  rpy="0.0 0.0 0.0"/>
    <geometry>
-      <mesh filename="package://centauro/centauro_urdf/meshes/simplified/link2.stl" scale="0.001 ${-rot*0.001} 0.001" />
+      <mesh filename="package://centauro/centauro_urdf/meshes/simplified/ShoulderPitch.STL" scale="0.001 ${-rot*0.001} 0.001" />
    </geometry>
 </xacro:macro>
@@ -16,5 +16,5 @@
    <origin xyz="0.0 0.0 0.0"  rpy="0.0 0.0 0.0"/>
    <geometry>
-      <mesh filename="package://centauro/centauro_urdf/meshes/simplified/link3.stl" scale="0.001 ${-rot*0.001} 0.001" />
+      <mesh filename="package://centauro/centauro_urdf/meshes/simplified/ShoulderRoll.STL" scale="0.001 ${-rot*0.001} 0.001" />
    </geometry>
 </xacro:macro>
@@ -22,5 +22,5 @@
    <origin xyz="0.0 0.0 0.0"  rpy="0.0 0.0 0.0"/>
    <geometry>
-      <mesh filename="package://centauro/centauro_urdf/meshes/simplified/link4.stl" scale="0.001 ${-rot*0.001} 0.001" />
+      <mesh filename="package://centauro/centauro_urdf/meshes/simplified/ShoulderYaw.STL" scale="0.001 ${-rot*0.001} 0.001" />
    </geometry>
 </xacro:macro>
@@ -28,5 +28,5 @@
    <origin xyz="0.0 0.0 0.0"  rpy="0.0 0.0 0.0"/>
    <geometry>
-      <mesh filename="package://centauro/centauro_urdf/meshes/simplified/link5.stl" scale="0.001 ${-rot*0.001} 0.001" />
+      <mesh filename="package://centauro/centauro_urdf/meshes/simplified/Elbow.STL" scale="0.001 ${-rot*0.001} 0.001" />
    </geometry>
 </xacro:macro>
@@ -34,5 +34,5 @@
    <origin xyz="0.0 0.0 0.0"  rpy="0.0 0.0 0.0"/>
    <geometry>
-      <mesh filename="package://centauro/centauro_urdf/meshes/simplified/link6.stl" scale="0.001 ${-rot*0.001} 0.001" />
+      <mesh filename="package://centauro/centauro_urdf/meshes/simplified/Forearm.STL" scale="0.001 ${-rot*0.001} 0.001" />
    </geometry>
 </xacro:macro>
@@ -40,5 +40,5 @@
    <origin xyz="0.0 0.0 0.0"  rpy="0.0 0.0 0.0"/>
    <geometry>
-      <mesh filename="package://centauro/centauro_urdf/meshes/simplified/link7.stl" scale="0.001 ${-rot*0.001} 0.001" />
+      <mesh filename="package://centauro/centauro_urdf/meshes/simplified/ForearmPitch.STL" scale="0.001 ${-rot*0.001} 0.001" />
    </geometry>
 </xacro:macro>
@@ -46,11 +46,11 @@
    <origin xyz="0.0 0.0 0.0"  rpy="0.0 0.0 0.0"/>
    <geometry>
-      <mesh filename="package://centauro/centauro_urdf/meshes/simplified/link8.stl" scale="0.001 ${-rot*0.001} 0.001" />
+      <mesh filename="package://centauro/centauro_urdf/meshes/simplified/ForearmYaw.STL" scale="0.001 ${-rot*0.001} 0.001" />
    </geometry>
 </xacro:macro>
 <xacro:macro name="arm8">
-   <origin xyz="0.0 0.0 0.0"  rpy="0.0 0.0 0.0"/>
+   <origin xyz="0.0 0.0 0.0"  rpy="${PI} 0.0 0.0"/>
    <geometry>
-      <mesh filename="package://centauro/centauro_urdf/meshes/simplified/link9.stl" scale="0.001 ${-rot*0.001} 0.001" />
+      <mesh filename="package://centauro/centauro_urdf/meshes/simplified/Wrist.STL" scale="0.001 ${-rot*0.001} 0.001" />
    </geometry>
 </xacro:macro>

Commit message: new hip yaw limits

File: centauro/centauro_urdf/limits/default.xacro (robot description, xacro)
@@ -2,6 +2,8 @@
 <robot  xmlns:xacro="http://www.ros.org/wiki/xacro">
 <!-- Origin -->
-<xacro:property name="hip_yaw_lower" value="${[-0.9432,-2.5110, -2.5100 ,-0.9412]}"/>
-<xacro:property name="hip_yaw_upper" value="${[ 2.5138, 0.9430,  0.9430 , 2.5138]}"/>
+<!-- <xacro:property name="hip_yaw_lower" value="${[-0.9432,-2.5110, -2.5100 ,-0.9412]}"/>
+<xacro:property name="hip_yaw_upper" value="${[ 2.5138, 0.9430,  0.9430 , 2.5138]}"/> -->
+<xacro:property name="hip_yaw_lower" value="${[-2.827,-2.583, -2.583 ,-2.827]}"/>
+<xacro:property name="hip_yaw_upper" value="${[ 2.583, 2.827,  2.827 , 2.583]}"/>
 <xacro:property name="hip_pitch_lower" value="${[-2.0226, -2.0156, -2.0126 , -2.0326]}"/>
 <xacro:property name="hip_pitch_upper" value="${[ 2.02748, 2.0354,  2.0384 ,  2.0524]}"/>
@@ -15,5 +17,5 @@
 <xacro:property name="torso_yaw_upper" value="2.618"/>
 <xacro:property name="j_arm_1_lower" value="${[-3.312, -3.3458]}"/>
-<xacro:property name="j_arm_2_lower" value="${ [0.020, -3.4258]}"/>
+<xacro:property name="j_arm_2_lower" value="${[ 0.020, -3.4258]}"/>
 <xacro:property name="j_arm_3_lower" value="${[-2.552, -2.5614]}"/>
 <xacro:property name="j_arm_4_lower" value="${[-2.465, -2.4794]}"/>

Commit message: hip yaw limits update based on firmware limits

File: centauro/centauro_urdf/limits/default.xacro (robot description, xacro)
@@ -2,8 +2,8 @@
 <robot  xmlns:xacro="http://www.ros.org/wiki/xacro">
 <!-- Origin -->
-<!-- <xacro:property name="hip_yaw_lower" value="${[-0.9432,-2.5110, -2.5100 ,-0.9412]}"/>
-<xacro:property name="hip_yaw_upper" value="${[ 2.5138, 0.9430,  0.9430 , 2.5138]}"/> -->
-<xacro:property name="hip_yaw_lower" value="${[-2.827,-2.583, -2.583 ,-2.827]}"/>
-<xacro:property name="hip_yaw_upper" value="${[ 2.583, 2.827,  2.827 , 2.583]}"/>
+<!-- <xacro:property name="hip_yaw_lower" value="${[-2.827,-2.583, -2.583 ,-2.827]}"/>
+<xacro:property name="hip_yaw_upper" value="${[ 2.583, 2.827,  2.827 , 2.583]}"/> -->
+<xacro:property name="hip_yaw_lower" value="${[-2.030,-2.510, -2.510 ,-2.030]}"/>
+<xacro:property name="hip_yaw_upper" value="${[ 2.510, 2.030,  2.030 , 2.510]}"/>
 <xacro:property name="hip_pitch_lower" value="${[-2.0226, -2.0156, -2.0126 , -2.0326]}"/>
 <xacro:property name="hip_pitch_upper" value="${[ 2.02748, 2.0354,  2.0384 ,  2.0524]}"/>

Commit message: read the velocity and torque limits from the external file

File: centauro/centauro_urdf/limits/default.xacro (robot description, xacro)
@@ -44,3 +44,9 @@
 <xacro:property name="j_arm_6_torque" value="${[55.00, 55.00 ]}"/>
 <xacro:property name="j_arm_7_torque" value="${[28.32, 28.32 ]}"/>
+<xacro:property name="motor_A_velocity" value="8.8"/>
+<xacro:property name="motor_B_velocity" value="8.1"/>
+<xacro:property name="motor_C_velocity" value="20.0"/>
+<xacro:property name="motor_A_effort" value="304"/>
+<xacro:property name="motor_B_effort" value="147"/>
+<xacro:property name="motor_C_effort" value="35"/>
 </robot>

File: centauro/centauro_urdf/urdf/centauro.urdf.xacro (robot description, xacro)
@@ -12,5 +12,5 @@
 <xacro:include filename="${inertia_parameters_file}"/>
 <xacro:include filename="${kinematic_parameters_file}"/>
-<xacro:include filename="$(find centauro)/centauro_urdf/limits/default.xacro"/>
+<xacro:include filename="$(find centauro)/centauro_urdf/limits/${limits}.xacro"/>
 <xacro:include filename="$(find centauro)/centauro_urdf/materials.xacro"/>
 <xacro:include filename="$(find centauro)/centauro_urdf/urdf/models/model.xacro"/>

File: centauro/centauro_urdf/urdf/centauro_arm.urdf.xacro (robot description, xacro)
@@ -126,5 +126,5 @@
       <parent link="arm${arm_num}_1"/>
       <child link="arm${arm_num}_2"/>
-      <origin xyz="${Shoulder_2_Ox} ${rot*Shoulder_2_Oy} ${Shoulder_2_Oz}" rpy="${Shoulder_2_roll} ${Shoulder_2_pitch} ${Shoulder_2_yaw}"/>
+      <origin xyz="${Shoulder_2_Ox} ${rot*Shoulder_2_Oy} ${Shoulder_2_Oz}" rpy="${rot*Shoulder_2_roll} ${Shoulder_2_pitch} ${Shoulder_2_yaw}"/>
       <axis xyz="1 0 0"/>
       <limit lower="${j_arm_2_lower[arm_num-1]}" upper="${j_arm_2_upper[arm_num-1]}" effort="${j_arm_2_torque[arm_num-1]}" velocity="${j_arm_2_velocity[arm_num-1]}"/>

File: centauro/centauro_urdf/urdf/centauro_leg.urdf.xacro (robot description, xacro)
@@ -94,5 +94,5 @@
 	<origin xyz="${origin_x*Leg_1_Ox} ${origin_y*Leg_1_Oy} ${Leg_1_Oz}" rpy="${Leg_1_roll} ${Leg_1_pitch} ${PI/2-origin_x*PI/2+origin_x*origin_y*Leg_1_yaw}"/>
 	<axis xyz="0 0 1"/>
-        <limit lower="${hip_yaw_lower[leg_num-1]}" upper="${hip_yaw_upper[leg_num-1]}" effort="304" velocity="8.8"/>
+        <limit lower="${hip_yaw_lower[leg_num-1]}" upper="${hip_yaw_upper[leg_num-1]}" effort="${motor_A_effort}" velocity="${motor_A_velocity}"/> <!-- 200 Nm, 1 rad/s-->
 </joint>
 <joint name="hip_pitch_${leg_num}" type="revolute">
@@ -101,5 +101,5 @@
 	<origin xyz="${Leg_2_Ox} ${Leg_2_Oy} ${Leg_2_Oz}" rpy="${Leg_2_roll} ${Leg_2_pitch} ${origin_x*origin_y*Leg_2_yaw-origin_x*origin_y*PI/2 + PI/2}"/>
 	<axis xyz="0 0 1"/>
-        <limit lower="${hip_pitch_lower[leg_num-1]}" upper="${hip_pitch_upper[leg_num-1]}" effort="304" velocity="8.8"/>
+        <limit lower="${hip_pitch_lower[leg_num-1]}" upper="${hip_pitch_upper[leg_num-1]}" effort="${motor_A_effort}" velocity="${motor_A_velocity}"/> <!-- 200 Nm, 1 rad/s-->
 </joint>
 <joint name="knee_pitch_${leg_num}" type="revolute">
@@ -108,5 +108,5 @@
 	<origin xyz="${Leg_3_Ox} ${Leg_3_Oy} ${Leg_3_Oz}" rpy="${Leg_3_roll} ${Leg_3_pitch} ${Leg_3_yaw}"/>
 	<axis xyz="0 0 1"/>
-        <limit lower="${knee_pitch_lower[leg_num-1]}" upper="${knee_pitch_upper[leg_num-1]}" effort="304" velocity="8.8"/>
+        <limit lower="${knee_pitch_lower[leg_num-1]}" upper="${knee_pitch_upper[leg_num-1]}" effort="${motor_A_effort}" velocity="${motor_A_velocity}"/> <!-- 200 Nm, 1 rad/s-->
 </joint>
 <joint name="ankle_pitch_${leg_num}" type="revolute">
@@ -115,5 +115,5 @@
 	<origin xyz="${Ankle_1_Ox} ${Ankle_1_Oy} ${Ankle_1_Oz}" rpy="${Ankle_1_roll} ${Ankle_1_pitch} ${Ankle_1_yaw}"/>
 	<axis xyz="0 0 1"/>
-        <limit lower="${ankle_pitch_lower[leg_num-1]}" upper="${ankle_pitch_upper[leg_num-1]}" effort="147" velocity="8.1"/>
+        <limit lower="${ankle_pitch_lower[leg_num-1]}" upper="${ankle_pitch_upper[leg_num-1]}" effort="${motor_B_effort}" velocity="${motor_B_velocity}"/> <!-- 98 Nm, 1 rad/s-->
 </joint>
 <joint name="ankle_yaw_${leg_num}" type="revolute">
@@ -122,5 +122,5 @@
 	<origin xyz="${Ankle_2_Ox} ${Ankle_2_Oy} ${Ankle_2_Oz}" rpy="${Ankle_2_roll} ${Ankle_2_pitch} ${Ankle_2_yaw}"/>
 	<axis xyz="0 0 1"/>
-        <limit lower="${ankle_yaw_lower[leg_num-1]}" upper="${ankle_yaw_upper[leg_num-1]}" effort="35" velocity="20.0"/>
+        <limit lower="${ankle_yaw_lower[leg_num-1]}" upper="${ankle_yaw_upper[leg_num-1]}" effort="${motor_C_effort}" velocity="${motor_C_velocity}"/>  <!-- 23 Nm, 1 rad/s-->
 </joint>
 <joint name="j_wheel_${leg_num}" type="continuous">
@@ -129,5 +129,5 @@
 	<origin xyz="${Wheel_Ox} ${Wheel_Oy} ${Wheel_Oz}" rpy="${Wheel_roll} ${Wheel_pitch} ${Wheel_yaw}"/>
 	<axis xyz="0 0 1"/>
-        <limit  effort="35" velocity="20.0"/>
+        <limit  effort="${motor_C_effort}" velocity="${motor_C_velocity}"/>  <!-- 23 Nm, 1 rad/s-->
 </joint>
 <!--

File: centauro/centauro_urdf/urdf/config.xacro (robot description, xacro)
@@ -19,4 +19,5 @@
 <xacro:property name="INERTIA_PARAM" value="$(arg INERTIA_PARAM)"/>
 <xacro:property name="KINEMATIC_PARAM" value="$(arg KINEMATIC_PARAM)"/>
+<xacro:property name="LIMITS" value="$(arg LIMITS)"/>
 <xacro:property name="TORSO_ACTUATORS" value="$(arg TORSO_ACTUATORS)"/>
 <xacro:property name="ARM_ACTUATORS" value="$(arg ARM_ACTUATORS)"/>
@@ -67,4 +68,5 @@
 <xacro:property name="inertia_parameters_file" value="${package + '/centauro_urdf/inertia_parameters/' + INERTIA_PARAM + '.xacro'}"/>
 <xacro:property name="kinematic_parameters_file" value="${package + '/centauro_urdf/kinematic_parameters/' + KINEMATIC_PARAM + '.xacro'}"/>
+<xacro:property name="limits" value="${LIMITS}"/>
 <xacro:property name="middleware" value="${MIDDLEWARE}"/>
 <xacro:property name="friction" value="10.0" />
